Commit message: Updated APIs since force/torque refactor.

File: common/xacro/api/valkyrie_sim_api.xacro (robot description, xacro)
@@ -2,4 +2,4 @@
 	<xacro:property name="SimApi" value="robot_hardware_interface/TurbodriverSimAPI" />
     <xacro:property name="ImuSensorSimApi" value="simulated_imu_sensor::SimulatedImuSensor" />
-    <xacro:property name="ForceTorqueSensorApi" value="ati_sensor_interface::ATISensorInterface" />
+    <xacro:property name="ForceTorqueSensorApi" value="sensor_interface::SimForceTorqueSensor" />
 </robot>
