Commit message: adding index finger as a turbodriver api

File: common/xacro/api/forearm_api.xacro (robot description, xacro)
@@ -2,5 +2,5 @@
     <xacro:property name="ForearmYawApi" value="robot_hardware_interface/TurbodriverAPI" />
     <xacro:property name="ThumbFingerApi" value="midas_finger_interface/MidasFingerAPI" />
-    <xacro:property name="IndexFingerApi" value="midas_finger_interface/MidasFingerAPI"/>
+    <xacro:property name="IndexFingerApi" value="robot_hardware_interface/TurbodriverAPI"/>
     <xacro:property name="MiddleFingerApi" value="midas_finger_interface/MidasFingerAPI"/>
     <xacro:property name="PinkyApi" value="midas_finger_interface/MidasFingerAPI"/>

File: common/xacro/nodes/valkyrie_nodes.xacro (robot description, xacro)
@@ -26,4 +26,5 @@
 	<xacro:property name="left_foot_ATI_node" value="/left_leg/ankle/left_actuator" />
 	<xacro:property name="right_foot_ATI_node" value="/right_leg/ankle/left_actuator" />
+	<xacro:property name="IndexFingerNode" value="/${prefix}_arm/hand/index"/>
 	<xacro:property name="IndexFingerPitch1Node" value="/${prefix}_arm/forearm_sensors/index/pitch_1"/>
 	<xacro:property name="IndexFingerPitch2Node" value="/${prefix}_arm/forearm_sensors/index/pitch_2"/>

File: model/robots/forearm_right.xacro (robot description, xacro)
@@ -17,9 +17,4 @@
     <xacro:make_pinky_finger prefix="${prefix}" reflect="${reflect}" pinky_finger_root_link="${prefix}Palm"/>
     <xacro:simple_position_transmission jointName="${ForearmYawActuatorName}" actuatorName="${ForearmYawActuatorName}" nodeName="${ForearmYawNode}" actuatorApi="${ForearmYawApi}"/>
-    <xacro:index_finger_transmissions_hw prefix="${prefix}" reflect="${reflect}"/>
-    <xacro:middle_finger_transmissions_hw prefix="${prefix}" reflect="${reflect}"/>
-    <xacro:pinky_finger_transmissions_hw prefix="${prefix}" reflect="${reflect}"/>
-    <xacro:thumb_transmissions_hw prefix="${prefix}" reflect="${reflect}"/>
-    <xacro:athena1_transmission prefix="${prefix}" transmissionName="${prefix}ArmAthena1Transmission" actuatorApi="${Athena1Api}" nodeName="${Athena1Node}"/>
-    <xacro:athena2_transmission prefix="${prefix}" transmissionName="${prefix}ArmAthena2Transmission" actuatorApi="${Athena2Api}" nodeName="${Athena2Node}"/>
+    <xacro:simple_position_transmission jointName="${IndexFingerPitch1ActuatorName}" actuatorName="${IndexFingerPitch1ActuatorName}" nodeName="${IndexFingerNode}" actuatorApi="${IndexFingerApi}"/>
 </robot>
