Commit message: Fixed ati sensor publishe rate after merge conflict.

File: common/xacro/api/valkyrie_A_api.xacro (robot description, xacro)
@@ -19,5 +19,5 @@
     <xacro:property name="WaistLeftActuatorApi" value="robot_hardware_interface/TurbodriverAPI_linear_futek" />
     <xacro:property name="WaistRightActuatorApi" value="robot_hardware_interface/TurbodriverAPI_linear_futek" />
-    <xacro:property name="AtiSensorApi" value="TurbodriverForceTorqueSensor" />
+    <xacro:property name="ForceTorqueSensorApi" value="ati_sensor_interface::ATISensorInterface" />
     <xacro:property name="ImuMicrostrainHardwareApi" value="imu_3dm_gx4_15_sensor::Imu3DmGx415Sensor" />
     <xacro:property name="ImuVectorNavHardwareApi" value="val_imu_vectornav_vn100_interface/ImuVecotNavInterface" />

File: common/xacro/api/valkyrie_B_api.xacro (robot description, xacro)
@@ -19,5 +19,5 @@
     <xacro:property name="WaistLeftActuatorApi" value="robot_hardware_interface/TurbodriverAPI_linear_Renishaw" />
     <xacro:property name="WaistRightActuatorApi" value="robot_hardware_interface/TurbodriverAPI_linear_Renishaw" />
-    <xacro:property name="AtiSensorApi" value="TurbodriverForceTorqueSensor" />
+    <xacro:property name="ForceTorqueSensorApi" value="ati_sensor_interface::ATISensorInterface" />
     <xacro:property name="ImuMicrostrainHardwareApi" value="imu_3dm_gx4_15_sensor::Imu3DmGx415Sensor" />
     <xacro:property name="ImuVectorNavHardwareApi" value="val_imu_vectornav_vn100_interface/ImuVecotNavInterface" />

File: common/xacro/api/valkyrie_C_api.xacro (robot description, xacro)
@@ -19,5 +19,5 @@
     <xacro:property name="WaistLeftActuatorApi" value="robot_hardware_interface/TurbodriverAPI_linear_Renishaw" />
     <xacro:property name="WaistRightActuatorApi" value="robot_hardware_interface/TurbodriverAPI_linear_Renishaw" />
-    <xacro:property name="AtiSensorApi" value="TurbodriverForceTorqueSensor" />
+    <xacro:property name="ForceTorqueSensorApi" value="ati_sensor_interface::ATISensorInterface" />
     <xacro:property name="ImuMicrostrainHardwareApi" value="imu_3dm_gx4_15_sensor::Imu3DmGx415Sensor" />
     <xacro:property name="ImuVectorNavHardwareApi" value="val_imu_vectornav_vn100_interface/ImuVecotNavInterface" />

File: common/xacro/api/valkyrie_sim_api.xacro (robot description, xacro)
@@ -2,4 +2,4 @@
 	<xacro:property name="SimApi" value="robot_hardware_interface/TurbodriverSimAPI" />
     <xacro:property name="ImuSensorSimApi" value="simulated_imu_sensor::SimulatedImuSensor" />
-    <xacro:property name="AtiSensorApi" value="TurbodriverForceTorqueSensor" />
+    <xacro:property name="ForceTorqueSensorApi" value="ati_sensor_interface::ATISensorInterface" />
 </robot>

File: model/robots/common/xacro/leg/leg.xacro (robot description, xacro)
@@ -159,5 +159,5 @@
                         sensor_number="${ATI_serial_number}"
                         sensor_node="${ATI_node}"
-                        sensor_api="${AtiSensorApi}" />
+                        sensor_api="${ForceTorqueSensorApi}" />
   </xacro:macro>
   <xacro:macro name="leg_transmissions_hw" params="prefix">

Commit message: Fixed actuator API.

File: common/xacro/api/valkyrie_A_api.xacro (robot description, xacro)
@@ -17,6 +17,6 @@
     <xacro:property name="UpperNeckPitchApi" value="robot_hardware_interface/TurbodriverAPI" />
     <xacro:property name="TrunkYawApi" value="robot_hardware_interface/TurbodriverAPI" />
-    <xacro:property name="WaistLeftActuatorApi" value="robot_hardware_interface/TurbodriverAPI_linear_futek" />
-    <xacro:property name="WaistRightActuatorApi" value="robot_hardware_interface/TurbodriverAPI_linear_futek" />
+    <xacro:property name="WaistLeftActuatorApi" value="robot_hardware_interface/TurbodriverAPI_linear_renishaw_output_velocity" />
+    <xacro:property name="WaistRightActuatorApi" value="robot_hardware_interface/TurbodriverAPI_linear_renishaw_output_velocity" />
     <xacro:property name="ForceTorqueSensorApi" value="ati_sensor_interface::ATISensorInterface" />
     <xacro:property name="ImuMicrostrainHardwareApi" value="imu_3dm_gx4_15_sensor::Imu3DmGx415Sensor" />

Commit message: Fixed typo in plugin name.

File: common/xacro/api/valkyrie_A_api.xacro (robot description, xacro)
@@ -17,6 +17,6 @@
     <xacro:property name="UpperNeckPitchApi" value="robot_hardware_interface/TurbodriverAPI" />
     <xacro:property name="TrunkYawApi" value="robot_hardware_interface/TurbodriverAPI" />
-    <xacro:property name="WaistLeftActuatorApi" value="robot_hardware_interface/TurbodriverAPI_linear_renishaw_output_velocity" />
-    <xacro:property name="WaistRightActuatorApi" value="robot_hardware_interface/TurbodriverAPI_linear_renishaw_output_velocity" />
+    <xacro:property name="WaistLeftActuatorApi" value="robot_hardware_interface::TurbodriverLinearRenishawOutputVelocity" />
+    <xacro:property name="WaistRightActuatorApi" value="robot_hardware_interface::TurbodriverLinearRenishawOutputVelocity" />
     <xacro:property name="ForceTorqueSensorApi" value="ati_sensor_interface::ATISensorInterface" />
     <xacro:property name="ImuMicrostrainHardwareApi" value="imu_3dm_gx4_15_sensor::Imu3DmGx415Sensor" />

Commit message: Set unit A torso transmission to be regular Pushrod transmission.

File: common/xacro/api/valkyrie_A_api.xacro (robot description, xacro)
@@ -17,6 +17,6 @@
     <xacro:property name="UpperNeckPitchApi" value="robot_hardware_interface/TurbodriverAPI" />
     <xacro:property name="TrunkYawApi" value="robot_hardware_interface/TurbodriverAPI" />
-    <xacro:property name="WaistLeftActuatorApi" value="robot_hardware_interface::TurbodriverLinearRenishawOutputVelocity" />
-    <xacro:property name="WaistRightActuatorApi" value="robot_hardware_interface::TurbodriverLinearRenishawOutputVelocity" />
+    <xacro:property name="WaistLeftActuatorApi" value="robot_hardware_interface:/TurbodriverAPI_linear_Renishaw" />
+    <xacro:property name="WaistRightActuatorApi" value="robot_hardware_interface/TurbodriverAPI_linear_Renishaw" />
     <xacro:property name="ForceTorqueSensorApi" value="ati_sensor_interface::ATISensorInterface" />
     <xacro:property name="ImuMicrostrainHardwareApi" value="imu_3dm_gx4_15_sensor::Imu3DmGx415Sensor" />

File: model/robots/common/xacro/config/valkyrie_A_transmissions.xacro (robot description, xacro)
@@ -1,5 +1,5 @@
 <?xml version="1.0" ?>
 <robot name="valkyrie_transmissions" xmlns:xacro="http://www.ros.org/wiki/xacro">
-	<xacro:property name="TorsoTransmissionType" value="robot_transmission_interface::TorsoPushrodTransmissionWithOutputVelocityLoader"/>
+	<xacro:property name="TorsoTransmissionType" value="robot_transmission_interface::TorsoPushrodTransmissionLoader"/>
 	<xacro:property name="AnkleTransmissionType" value="robot_transmission_interface::AnklePushrodTransmissionLoader"/>
 </robot>

Commit message: adding fingers to hardware

File: common/xacro/api/valkyrie_A_api.xacro (robot description, xacro)
@@ -30,3 +30,12 @@
     <xacro:property name="Athena1Api" value="athena_forearm_interface/AthenaForearmAPI" />
     <xacro:property name="Athena2Api" value="athena_finger_interface/AthenaFingerAPI" />
+    <xacro:property name="ForearmYawApi" value="robot_hardware_interface/TurbodriverAPI" />
+    <xacro:property name="IndexFingerApi" value="robot_hardware_interface/TurbodriverAPI"/>
+    <xacro:property name="MiddleFingerApi" value="robot_hardware_interface/TurbodriverAPI"/>
+    <xacro:property name="PinkyFingerApi" value="robot_hardware_interface/TurbodriverAPI"/>
+    <xacro:property name="ThumbRollFingerApi" value="robot_hardware_interface/TurbodriverAPI"/>
+    <xacro:property name="ThumbProximalFingerApi" value="robot_hardware_interface/TurbodriverAPI"/>
+    <xacro:property name="ThumbDistalFingerApi" value="robot_hardware_interface/TurbodriverAPI"/>
+    <xacro:property name="WristRightActuatorApi" value="robot_hardware_interface/TurbodriverAPI_linear_futek"/>
+    <xacro:property name="WristLeftActuatorApi" value="robot_hardware_interface/TurbodriverAPI_linear_futek"/>
 </robot>

File: common/xacro/api/valkyrie_B_api.xacro (robot description, xacro)
@@ -30,3 +30,12 @@
     <xacro:property name="Athena1Api" value="athena_forearm_interface/AthenaForearmAPI" />
     <xacro:property name="Athena2Api" value="athena_finger_interface/AthenaFingerAPI" />
+    <xacro:property name="ForearmYawApi" value="robot_hardware_interface/TurbodriverAPI" />
+    <xacro:property name="IndexFingerApi" value="robot_hardware_interface/TurbodriverAPI"/>
+    <xacro:property name="MiddleFingerApi" value="robot_hardware_interface/TurbodriverAPI"/>
+    <xacro:property name="PinkyFingerApi" value="robot_hardware_interface/TurbodriverAPI"/>
+    <xacro:property name="ThumbRollFingerApi" value="robot_hardware_interface/TurbodriverAPI"/>
+    <xacro:property name="ThumbProximalFingerApi" value="robot_hardware_interface/TurbodriverAPI"/>
+    <xacro:property name="ThumbDistalFingerApi" value="robot_hardware_interface/TurbodriverAPI"/>
+    <xacro:property name="WristRightActuatorApi" value="robot_hardware_interface/TurbodriverAPI_linear_futek"/>
+    <xacro:property name="WristLeftActuatorApi" value="robot_hardware_interface/TurbodriverAPI_linear_futek"/>
 </robot>

File: common/xacro/api/valkyrie_C_api.xacro (robot description, xacro)
@@ -30,3 +30,12 @@
     <xacro:property name="Athena1Api" value="athena_forearm_interface/AthenaForearmAPI" />
     <xacro:property name="Athena2Api" value="athena_finger_interface/AthenaFingerAPI" />
+    <xacro:property name="ForearmYawApi" value="robot_hardware_interface/TurbodriverAPI" />
+    <xacro:property name="IndexFingerApi" value="robot_hardware_interface/TurbodriverAPI"/>
+    <xacro:property name="MiddleFingerApi" value="robot_hardware_interface/TurbodriverAPI"/>
+    <xacro:property name="PinkyFingerApi" value="robot_hardware_interface/TurbodriverAPI"/>
+    <xacro:property name="ThumbRollFingerApi" value="robot_hardware_interface/TurbodriverAPI"/>
+    <xacro:property name="ThumbProximalFingerApi" value="robot_hardware_interface/TurbodriverAPI"/>
+    <xacro:property name="ThumbDistalFingerApi" value="robot_hardware_interface/TurbodriverAPI"/>
+    <xacro:property name="WristRightActuatorApi" value="robot_hardware_interface/TurbodriverAPI_linear_futek"/>
+    <xacro:property name="WristLeftActuatorApi" value="robot_hardware_interface/TurbodriverAPI_linear_futek"/>
 </robot>

File: common/xacro/api/valkyrie_D_api.xacro (robot description, xacro)
@@ -30,3 +30,12 @@
     <xacro:property name="Athena1Api" value="athena_forearm_interface/AthenaForearmAPI" />
     <xacro:property name="Athena2Api" value="athena_finger_interface/AthenaFingerAPI" />
+     <xacro:property name="ForearmYawApi" value="robot_hardware_interface/TurbodriverAPI" />
+    <xacro:property name="IndexFingerApi" value="robot_hardware_interface/TurbodriverAPI"/>
+    <xacro:property name="MiddleFingerApi" value="robot_hardware_interface/TurbodriverAPI"/>
+    <xacro:property name="PinkyFingerApi" value="robot_hardware_interface/TurbodriverAPI"/>
+    <xacro:property name="ThumbRollFingerApi" value="robot_hardware_interface/TurbodriverAPI"/>
+    <xacro:property name="ThumbProximalFingerApi" value="robot_hardware_interface/TurbodriverAPI"/>
+    <xacro:property name="ThumbDistalFingerApi" value="robot_hardware_interface/TurbodriverAPI"/>
+    <xacro:property name="WristRightActuatorApi" value="robot_hardware_interface/TurbodriverAPI_linear_futek"/>
+    <xacro:property name="WristLeftActuatorApi" value="robot_hardware_interface/TurbodriverAPI_linear_futek"/>
 </robot>

File: model/robots/common/xacro/arm/arm.xacro (robot description, xacro)
@@ -235,7 +235,12 @@
     <xacro:simple_transmission jointName="${ShoulderYawJointName}" actuatorName="${ShoulderYawActuatorName}" nodeName="${ShoulderYawNode}" actuatorApi="${ShoulderYawApi}"/>
     <xacro:simple_transmission jointName="${ElbowPitchJointName}" actuatorName="${ElbowPitchActuatorName}" nodeName="${ElbowPitchNode}" actuatorApi="${ElbowPitchApi}"/>
-    <xacro:simple_position_transmission jointName="${ForearmYawActuatorName}" actuatorName="${ForearmYawActuatorName}" nodeName="${ForearmYawNode}" actuatorApi="${ForearmYawApi}"/>
-    <xacro:athena1_transmission prefix="${prefix}" transmissionName="${prefix}ArmAthena1Transmission" actuatorApi="${Athena1Api}" nodeName="${Athena1Node}"/>
-    <xacro:athena2_transmission prefix="${prefix}" transmissionName="${prefix}ArmAthena2Transmission" actuatorApi="${Athena2Api}" nodeName="${Athena2Node}"/>
+    <xacro:simple_transmission jointName="${ForearmYawActuatorName}" actuatorName="${ForearmYawActuatorName}" nodeName="${ForearmYawNode}" actuatorApi="${ForearmYawApi}"/>
+    <xacro:pushrod_transmission transmissionName="${prefix}WristTransmission" transmissionType="${WristTransmissionType}" joint1Name="${WristPitchJointName}" joint2Name="${WristRollJointName}" joint1Role="pitch" joint2Role="roll" actuator1Name="${WristRightActuatorName}" actuator2Name="${WristLeftActuatorName}" actuator1Node="${WristRightActuatorNode}" actuator2Node="${WristLeftActuatorNode}" actuator1Api="${WristRightActuatorApi}" actuator2Api="${WristLeftActuatorApi}" actuator1Role="bottom" actuator2Role="top"/>
+    <xacro:simple_transmission jointName="${IndexFingerPitch1ActuatorName}" actuatorName="${IndexFingerPitch1ActuatorName}" nodeName="${IndexFingerNode}" actuatorApi="${IndexFingerApi}"/>
+    <xacro:simple_transmission jointName="${MiddleFingerPitch1ActuatorName}" actuatorName="${MiddleFingerPitch1ActuatorName}" nodeName="${MiddleFingerNode}" actuatorApi="${MiddleFingerApi}"/>
+    <xacro:simple_transmission jointName="${PinkyPitch1ActuatorName}" actuatorName="${PinkyPitch1ActuatorName}" nodeName="${PinkyFingerNode}" actuatorApi="${PinkyFingerApi}"/>
+    <xacro:simple_transmission jointName="${ThumbRollActuatorName}" actuatorName="${ThumbRollActuatorName}" nodeName="${ThumbRollNode}" actuatorApi="${ThumbRollFingerApi}"/>
+    <xacro:simple_transmission jointName="${ThumbPitch1ActuatorName}" actuatorName="${ThumbPitch1ActuatorName}" nodeName="${ThumbProximalNode}" actuatorApi="${ThumbProximalFingerApi}"/>
+    <xacro:simple_transmission jointName="${ThumbPitch2ActuatorName}" actuatorName="${ThumbPitch2ActuatorName}" nodeName="${ThumbDistalNode}" actuatorApi="${ThumbDistalFingerApi}"/>
   </xacro:macro>
   <xacro:macro name="arm_transmissions_no_hands" params="prefix">

File: model/robots/common/xacro/config/valkyrie_A_transmissions.xacro (robot description, xacro)
@@ -3,3 +3,4 @@
 	<xacro:property name="TorsoTransmissionType" value="robot_transmission_interface::TorsoPushrodTransmissionLoader"/>
 	<xacro:property name="AnkleTransmissionType" value="robot_transmission_interface::AnklePushrodTransmissionLoader"/>
+	<xacro:property name="WristTransmissionType" value="robot_transmission_interface/WristPushrodTransmission"/>
 </robot>

File: model/robots/common/xacro/config/valkyrie_B_transmissions.xacro (robot description, xacro)
@@ -3,3 +3,4 @@
 	<xacro:property name="TorsoTransmissionType" value="robot_transmission_interface::TorsoPushrodTransmissionLoader"/>
 	<xacro:property name="AnkleTransmissionType" value="robot_transmission_interface::AnklePushrodTransmissionLoader"/>
+	<xacro:property name="WristTransmissionType" value="robot_transmission_interface/WristPushrodTransmission"/>
 </robot>
