Commit message: adding finger sensors to urdf

File: common/xacro/api/valkyrie_A_api.xacro (robot description, xacro)
@@ -23,8 +23,4 @@
     <xacro:property name="ImuVectorNavHardwareApi" value="val_imu_vectornav_vn100_interface/ImuVecotNavInterface" />
     <xacro:property name="ImuSensorSimApi" value="val_imu_gazebo_interface/ImuGazeboInterface" />
-    <xacro:property name="ThumbFingerApi" value="midas_finger_interface/MidasFingerAPI" />
-    <xacro:property name="IndexFingerApi" value="midas_finger_interface/MidasFingerAPI"/>
-    <xacro:property name="MiddleFingerApi" value="midas_finger_interface/MidasFingerAPI"/>
-    <xacro:property name="PinkyApi" value="midas_finger_interface/MidasFingerAPI"/>
     <xacro:property name="SimApi" value="robot_hardware_interface/TurbodriverSimAPI" />
     <xacro:property name="Athena1Api" value="athena_forearm_interface/AthenaForearmAPI" />
@@ -37,4 +33,17 @@
     <xacro:property name="ThumbProximalFingerApi" value="robot_hardware_interface/TurbodriverAPI"/>
     <xacro:property name="ThumbDistalFingerApi" value="robot_hardware_interface/TurbodriverAPI"/>
+    <xacro:property name="IndexFingerProximalApi" value="robot_hardware_interface/TurbodriverFingerProx"/>
+    <xacro:property name="IndexFingerMedialApi" value="robot_hardware_interface/TurbodriverFingerMed"/>
+    <xacro:property name="IndexFingerDistalApi" value="robot_hardware_interface/TurbodriverFingerDis"/>
+    <xacro:property name="MiddleFingerProximalApi" value="robot_hardware_interface/TurbodriverFingerProx"/>
+    <xacro:property name="MiddleFingerMedialApi" value="robot_hardware_interface/TurbodriverFingerMed"/>
+    <xacro:property name="MiddleFingerDistalApi" value="robot_hardware_interface/TurbodriverFingerDis"/>
+    <xacro:property name="PinkyFingerProximalApi" value="robot_hardware_interface/TurbodriverFingerProx"/>
+    <xacro:property name="PinkyFingerMedialApi" value="robot_hardware_interface/TurbodriverFingerMed"/>
+    <xacro:property name="PinkyFingerDistalApi" value="robot_hardware_interface/TurbodriverFingerDis"/>
+    <xacro:property name="ThumbFingerProximalApi" value="robot_hardware_interface/TurbodriverFingerProx"/>
+    <xacro:property name="ThumbFingerMedialApi" value="robot_hardware_interface/TurbodriverFingerMed"/>
+    <xacro:property name="ThumbFingerDistalApi" value="robot_hardware_interface/TurbodriverFingerDis"/>
+    <xacro:property name="ThumbFingerRollApi" value="robot_hardware_interface/TurbodriverFingerRoll"/>
     <xacro:property name="WristRightActuatorApi" value="robot_hardware_interface/TurbodriverAPI_linear_futek"/>
     <xacro:property name="WristLeftActuatorApi" value="robot_hardware_interface/TurbodriverAPI_linear_futek"/>

File: common/xacro/api/valkyrie_B_api.xacro (robot description, xacro)
@@ -23,8 +23,4 @@
     <xacro:property name="ImuVectorNavHardwareApi" value="val_imu_vectornav_vn100_interface/ImuVecotNavInterface" />
     <xacro:property name="ImuSensorSimApi" value="val_imu_gazebo_interface/ImuGazeboInterface" />
-    <xacro:property name="ThumbFingerApi" value="midas_finger_interface/MidasFingerAPI" />
-    <xacro:property name="IndexFingerApi" value="midas_finger_interface/MidasFingerAPI"/>
-    <xacro:property name="MiddleFingerApi" value="midas_finger_interface/MidasFingerAPI"/>
-    <xacro:property name="PinkyApi" value="midas_finger_interface/MidasFingerAPI"/>
     <xacro:property name="SimApi" value="robot_hardware_interface/TurbodriverSimAPI" />
     <xacro:property name="Athena1Api" value="athena_forearm_interface/AthenaForearmAPI" />
@@ -37,4 +33,17 @@
     <xacro:property name="ThumbProximalFingerApi" value="robot_hardware_interface/TurbodriverAPI"/>
     <xacro:property name="ThumbDistalFingerApi" value="robot_hardware_interface/TurbodriverAPI"/>
+    <xacro:property name="IndexFingerProximalApi" value="robot_hardware_interface/TurbodriverFingerProx"/>
+    <xacro:property name="IndexFingerMedialApi" value="robot_hardware_interface/TurbodriverFingerMed"/>
+    <xacro:property name="IndexFingerDistalApi" value="robot_hardware_interface/TurbodriverFingerDis"/>
+    <xacro:property name="MiddleFingerProximalApi" value="robot_hardware_interface/TurbodriverFingerProx"/>
+    <xacro:property name="MiddleFingerMedialApi" value="robot_hardware_interface/TurbodriverFingerMed"/>
+    <xacro:property name="MiddleFingerDistalApi" value="robot_hardware_interface/TurbodriverFingerDis"/>
+    <xacro:property name="PinkyFingerProximalApi" value="robot_hardware_interface/TurbodriverFingerProx"/>
+    <xacro:property name="PinkyFingerMedialApi" value="robot_hardware_interface/TurbodriverFingerMed"/>
+    <xacro:property name="PinkyFingerDistalApi" value="robot_hardware_interface/TurbodriverFingerDis"/>
+    <xacro:property name="ThumbFingerProximalApi" value="robot_hardware_interface/TurbodriverFingerProx"/>
+    <xacro:property name="ThumbFingerMedialApi" value="robot_hardware_interface/TurbodriverFingerMed"/>
+    <xacro:property name="ThumbFingerDistalApi" value="robot_hardware_interface/TurbodriverFingerDis"/>
+    <xacro:property name="ThumbFingerRollApi" value="robot_hardware_interface/TurbodriverFingerRoll"/>
     <xacro:property name="WristRightActuatorApi" value="robot_hardware_interface/TurbodriverAPI_linear_futek"/>
     <xacro:property name="WristLeftActuatorApi" value="robot_hardware_interface/TurbodriverAPI_linear_futek"/>

File: common/xacro/api/valkyrie_C_api.xacro (robot description, xacro)
@@ -23,8 +23,4 @@
     <xacro:property name="ImuVectorNavHardwareApi" value="val_imu_vectornav_vn100_interface/ImuVecotNavInterface" />
     <xacro:property name="ImuSensorSimApi" value="val_imu_gazebo_interface/ImuGazeboInterface" />
-    <xacro:property name="ThumbFingerApi" value="midas_finger_interface/MidasFingerAPI" />
-    <xacro:property name="IndexFingerApi" value="midas_finger_interface/MidasFingerAPI"/>
-    <xacro:property name="MiddleFingerApi" value="midas_finger_interface/MidasFingerAPI"/>
-    <xacro:property name="PinkyApi" value="midas_finger_interface/MidasFingerAPI"/>
     <xacro:property name="SimApi" value="robot_hardware_interface/TurbodriverSimAPI" />
     <xacro:property name="Athena1Api" value="athena_forearm_interface/AthenaForearmAPI" />
@@ -37,4 +33,17 @@
     <xacro:property name="ThumbProximalFingerApi" value="robot_hardware_interface/TurbodriverAPI"/>
     <xacro:property name="ThumbDistalFingerApi" value="robot_hardware_interface/TurbodriverAPI"/>
+    <xacro:property name="IndexFingerProximalApi" value="robot_hardware_interface/TurbodriverFingerProx"/>
+    <xacro:property name="IndexFingerMedialApi" value="robot_hardware_interface/TurbodriverFingerMed"/>
+    <xacro:property name="IndexFingerDistalApi" value="robot_hardware_interface/TurbodriverFingerDis"/>
+    <xacro:property name="MiddleFingerProximalApi" value="robot_hardware_interface/TurbodriverFingerProx"/>
+    <xacro:property name="MiddleFingerMedialApi" value="robot_hardware_interface/TurbodriverFingerMed"/>
+    <xacro:property name="MiddleFingerDistalApi" value="robot_hardware_interface/TurbodriverFingerDis"/>
+    <xacro:property name="PinkyFingerProximalApi" value="robot_hardware_interface/TurbodriverFingerProx"/>
+    <xacro:property name="PinkyFingerMedialApi" value="robot_hardware_interface/TurbodriverFingerMed"/>
+    <xacro:property name="PinkyFingerDistalApi" value="robot_hardware_interface/TurbodriverFingerDis"/>
+    <xacro:property name="ThumbFingerProximalApi" value="robot_hardware_interface/TurbodriverFingerProx"/>
+    <xacro:property name="ThumbFingerMedialApi" value="robot_hardware_interface/TurbodriverFingerMed"/>
+    <xacro:property name="ThumbFingerDistalApi" value="robot_hardware_interface/TurbodriverFingerDis"/>
+    <xacro:property name="ThumbFingerRollApi" value="robot_hardware_interface/TurbodriverFingerRoll"/>
     <xacro:property name="WristRightActuatorApi" value="robot_hardware_interface/TurbodriverAPI_linear_futek"/>
     <xacro:property name="WristLeftActuatorApi" value="robot_hardware_interface/TurbodriverAPI_linear_futek"/>

File: common/xacro/api/valkyrie_D_api.xacro (robot description, xacro)
@@ -23,12 +23,8 @@
     <xacro:property name="ImuVectorNavHardwareApi" value="val_imu_vectornav_vn100_interface/ImuVecotNavInterface" />
     <xacro:property name="ImuSensorSimApi" value="val_imu_gazebo_interface/ImuGazeboInterface" />
-    <xacro:property name="ThumbFingerApi" value="midas_finger_interface/MidasFingerAPI" />
-    <xacro:property name="IndexFingerApi" value="midas_finger_interface/MidasFingerAPI"/>
-    <xacro:property name="MiddleFingerApi" value="midas_finger_interface/MidasFingerAPI"/>
-    <xacro:property name="PinkyApi" value="midas_finger_interface/MidasFingerAPI"/>
     <xacro:property name="SimApi" value="robot_hardware_interface/TurbodriverSimAPI" />
     <xacro:property name="Athena1Api" value="athena_forearm_interface/AthenaForearmAPI" />
     <xacro:property name="Athena2Api" value="athena_finger_interface/AthenaFingerAPI" />
-     <xacro:property name="ForearmYawApi" value="robot_hardware_interface/TurbodriverAPI" />
+    <xacro:property name="ForearmYawApi" value="robot_hardware_interface/TurbodriverAPI" />
     <xacro:property name="IndexFingerApi" value="robot_hardware_interface/TurbodriverAPI"/>
     <xacro:property name="MiddleFingerApi" value="robot_hardware_interface/TurbodriverAPI"/>
@@ -37,4 +33,17 @@
     <xacro:property name="ThumbProximalFingerApi" value="robot_hardware_interface/TurbodriverAPI"/>
     <xacro:property name="ThumbDistalFingerApi" value="robot_hardware_interface/TurbodriverAPI"/>
+    <xacro:property name="IndexFingerProximalApi" value="robot_hardware_interface/TurbodriverFingerProx"/>
+    <xacro:property name="IndexFingerMedialApi" value="robot_hardware_interface/TurbodriverFingerMed"/>
+    <xacro:property name="IndexFingerDistalApi" value="robot_hardware_interface/TurbodriverFingerDis"/>
+    <xacro:property name="MiddleFingerProximalApi" value="robot_hardware_interface/TurbodriverFingerProx"/>
+    <xacro:property name="MiddleFingerMedialApi" value="robot_hardware_interface/TurbodriverFingerMed"/>
+    <xacro:property name="MiddleFingerDistalApi" value="robot_hardware_interface/TurbodriverFingerDis"/>
+    <xacro:property name="PinkyFingerProximalApi" value="robot_hardware_interface/TurbodriverFingerProx"/>
+    <xacro:property name="PinkyFingerMedialApi" value="robot_hardware_interface/TurbodriverFingerMed"/>
+    <xacro:property name="PinkyFingerDistalApi" value="robot_hardware_interface/TurbodriverFingerDis"/>
+    <xacro:property name="ThumbFingerProximalApi" value="robot_hardware_interface/TurbodriverFingerProx"/>
+    <xacro:property name="ThumbFingerMedialApi" value="robot_hardware_interface/TurbodriverFingerMed"/>
+    <xacro:property name="ThumbFingerDistalApi" value="robot_hardware_interface/TurbodriverFingerDis"/>
+    <xacro:property name="ThumbFingerRollApi" value="robot_hardware_interface/TurbodriverFingerRoll"/>
     <xacro:property name="WristRightActuatorApi" value="robot_hardware_interface/TurbodriverAPI_linear_futek"/>
     <xacro:property name="WristLeftActuatorApi" value="robot_hardware_interface/TurbodriverAPI_linear_futek"/>

File: common/xacro/nodes/valkyrie_nodes.xacro (robot description, xacro)
@@ -37,21 +37,22 @@
 	<xacro:property name="right_foot_ATI_node" value="/right_leg/ankle/left_actuator" />
 	<xacro:property name="IndexFingerNode" value="/${prefix}_arm/hand/index"/>
-	<xacro:property name="IndexFingerPitch1Node" value="/${prefix}_arm/forearm_sensors/index/pitch_1"/>
-	<xacro:property name="IndexFingerPitch2Node" value="/${prefix}_arm/forearm_sensors/index/pitch_2"/>
-	<xacro:property name="IndexFingerPitch3Node" value="/${prefix}_arm/forearm_sensors/index/pitch_3"/>
+	<xacro:property name="IndexFingerPitch1Node" value="/${prefix}_arm/forearm_sensors/index"/>
+	<xacro:property name="IndexFingerPitch2Node" value="/${prefix}_arm/forearm_sensors/index"/>
+	<xacro:property name="IndexFingerPitch3Node" value="/${prefix}_arm/forearm_sensors/index"/>
 	<xacro:property name="MiddleFingerNode" value="/${prefix}_arm/hand/middle"/>
-	<xacro:property name="MiddleFingerPitch1Node" value="/${prefix}_arm/forearm_sensors/middle/pitch_1"/>
-	<xacro:property name="MiddleFingerPitch2Node" value="/${prefix}_arm/forearm_sensors/middle/pitch_2"/>
-	<xacro:property name="MiddleFingerPitch3Node" value="/${prefix}_arm/forearm_sensors/middle/pitch_3"/>
+	<xacro:property name="MiddleFingerPitch1Node" value="/${prefix}_arm/forearm_sensors/middle"/>
+	<xacro:property name="MiddleFingerPitch2Node" value="/${prefix}_arm/forearm_sensors/middle"/>
+	<xacro:property name="MiddleFingerPitch3Node" value="/${prefix}_arm/forearm_sensors/middle"/>
 	<xacro:property name="PinkyFingerNode" value="/${prefix}_arm/hand/pinky"/>
-	<xacro:property name="PinkyPitch1Node" value="/${prefix}_arm/forearm_sensors/pinky/pitch_1"/>
-	<xacro:property name="PinkyPitch2Node" value="/${prefix}_arm/forearm_sensors/pinky/pitch_2"/>
-	<xacro:property name="PinkyPitch3Node" value="/${prefix}_arm/forearm_sensors/pinky/pitch_3"/>
+	<xacro:property name="PinkyPitch1Node" value="/${prefix}_arm/forearm_sensors/pinky"/>
+	<xacro:property name="PinkyPitch2Node" value="/${prefix}_arm/forearm_sensors/pinky"/>
+	<xacro:property name="PinkyPitch3Node" value="/${prefix}_arm/forearm_sensors/pinky"/>
 	<xacro:property name="ThumbRollNode" value="/${prefix}_arm/hand/thumb_roll"/>
 	<xacro:property name="ThumbProximalNode" value="/${prefix}_arm/hand/thumb_proximal"/>
 	<xacro:property name="ThumbDistalNode" value="/${prefix}_arm/hand/thumb_distal"/>
-	<xacro:property name="ThumbPitch1Node" value="/${prefix}_arm/forearm_sensors/thumb/pitch_1"/>
-	<xacro:property name="ThumbPitch2Node" value="/${prefix}_arm/forearm_sensors/thumb/pitch_2"/>
-	<xacro:property name="ThumbPitch3Node" value="/${prefix}_arm/forearm_sensors/thumb/pitch_3"/>
+	<xacro:property name="ThumbRollSensNode" value="/${prefix}_arm/forearm_sensors/thumb"/>
+	<xacro:property name="ThumbPitch1Node" value="/${prefix}_arm/forearm_sensors/thumb"/>
+	<xacro:property name="ThumbPitch2Node" value="/${prefix}_arm/forearm_sensors/thumb"/>
+	<xacro:property name="ThumbPitch3Node" value="/${prefix}_arm/forearm_sensors/thumb"/>
 	<xacro:macro name="all_channels" >
 		<Channels>

File: model/robots/common/xacro/index_finger/index_finger.xacro (robot description, xacro)
@@ -78,7 +78,7 @@
   </xacro:macro>
   <xacro:macro name="index_finger_transmissions_hw" params="prefix reflect">
-    <xacro:simple_forearm_position_transmission jointName="${IndexFingerPitch1JointName}" actuatorName="${prefix}IndexPitch1Actuator" nodeName="${IndexFingerPitch1Node}" actuatorApi="${IndexFingerApi}" reflect="${reflect}"/>
-    <xacro:simple_forearm_position_transmission jointName="${IndexFingerPitch2JointName}" actuatorName="${prefix}IndexPitch2Actuator" nodeName="${IndexFingerPitch2Node}" actuatorApi="${IndexFingerApi}" reflect="${reflect}"/>
-    <xacro:simple_forearm_position_transmission jointName="${IndexFingerPitch3JointName}" actuatorName="${prefix}IndexPitch3Actuator" nodeName="${IndexFingerPitch3Node}" actuatorApi="${IndexFingerApi}" reflect="${reflect}"/>
+    <xacro:simple_forearm_position_transmission jointName="${IndexFingerPitch1JointName}" actuatorName="${prefix}IndexPitch1Actuator" nodeName="${IndexFingerPitch1Node}" actuatorApi="${IndexFingerProximalApi}" reflect="${reflect}"/>
+    <xacro:simple_forearm_position_transmission jointName="${IndexFingerPitch2JointName}" actuatorName="${prefix}IndexPitch2Actuator" nodeName="${IndexFingerPitch2Node}" actuatorApi="${IndexFingerMedialApi}" reflect="${reflect}"/>
+    <xacro:simple_forearm_position_transmission jointName="${IndexFingerPitch3JointName}" actuatorName="${prefix}IndexPitch3Actuator" nodeName="${IndexFingerPitch3Node}" actuatorApi="${IndexFingerDistalApi}" reflect="${reflect}"/>
   </xacro:macro>
   <xacro:macro name="index_finger_transmissions_sim" params="prefix">

File: model/robots/common/xacro/middle_finger/middle_finger.xacro (robot description, xacro)
@@ -78,7 +78,7 @@
   </xacro:macro>
   <xacro:macro name="middle_finger_transmissions_hw" params="prefix reflect">
-    <xacro:simple_forearm_position_transmission jointName="${MiddleFingerPitch1JointName}" actuatorName="${prefix}MiddlePitch1Actuator" nodeName="${MiddleFingerPitch1Node}" actuatorApi="${MiddleFingerApi}" reflect="${reflect}"/>
-    <xacro:simple_forearm_position_transmission jointName="${MiddleFingerPitch2JointName}" actuatorName="${prefix}MiddlePitch2Actuator" nodeName="${MiddleFingerPitch2Node}" actuatorApi="${MiddleFingerApi}" reflect="${reflect}"/>
-    <xacro:simple_forearm_position_transmission jointName="${MiddleFingerPitch3JointName}" actuatorName="${prefix}MiddlePitch3Actuator" nodeName="${MiddleFingerPitch3Node}" actuatorApi="${MiddleFingerApi}" reflect="${reflect}"/>
+    <xacro:simple_forearm_position_transmission jointName="${MiddleFingerPitch1JointName}" actuatorName="${prefix}MiddlePitch1Actuator" nodeName="${MiddleFingerPitch1Node}" actuatorApi="${MiddleFingerProximalApi}" reflect="${reflect}"/>
+    <xacro:simple_forearm_position_transmission jointName="${MiddleFingerPitch2JointName}" actuatorName="${prefix}MiddlePitch2Actuator" nodeName="${MiddleFingerPitch2Node}" actuatorApi="${MiddleFingerMedialApi}" reflect="${reflect}"/>
+    <xacro:simple_forearm_position_transmission jointName="${MiddleFingerPitch3JointName}" actuatorName="${prefix}MiddlePitch3Actuator" nodeName="${MiddleFingerPitch3Node}" actuatorApi="${MiddleFingerDistalApi}" reflect="${reflect}"/>
   </xacro:macro>
   <xacro:macro name="middle_finger_transmissions_sim" params="prefix">

File: model/robots/common/xacro/pinky_finger/pinky_finger.xacro (robot description, xacro)
@@ -78,7 +78,7 @@
   </xacro:macro>
   <xacro:macro name="pinky_finger_transmissions_hw" params="prefix reflect">
-    <xacro:simple_forearm_position_transmission jointName="${PinkyPitch1JointName}" actuatorName="${prefix}PinkyPitch1Actuator" nodeName="${PinkyPitch1Node}" actuatorApi="${PinkyApi}" reflect="${reflect}"/>
-    <xacro:simple_forearm_position_transmission jointName="${PinkyPitch2JointName}" actuatorName="${prefix}PinkyPitch2Actuator" nodeName="${PinkyPitch2Node}" actuatorApi="${PinkyApi}" reflect="${reflect}"/>
-    <xacro:simple_forearm_position_transmission jointName="${PinkyPitch3JointName}" actuatorName="${prefix}PinkyPitch3Actuator" nodeName="${PinkyPitch3Node}" actuatorApi="${PinkyApi}" reflect="${reflect}"/>
+    <xacro:simple_forearm_position_transmission jointName="${PinkyPitch1JointName}" actuatorName="${prefix}PinkyPitch1Actuator" nodeName="${PinkyPitch1Node}" actuatorApi="${PinkyFingerProximalApi}" reflect="${reflect}"/>
+    <xacro:simple_forearm_position_transmission jointName="${PinkyPitch2JointName}" actuatorName="${prefix}PinkyPitch2Actuator" nodeName="${PinkyPitch2Node}" actuatorApi="${PinkyFingerMedialApi}" reflect="${reflect}"/>
+    <xacro:simple_forearm_position_transmission jointName="${PinkyPitch3JointName}" actuatorName="${prefix}PinkyPitch3Actuator" nodeName="${PinkyPitch3Node}" actuatorApi="${PinkyFingerDistalApi}" reflect="${reflect}"/>
   </xacro:macro>
   <xacro:macro name="pinky_transmissions_sim" params="prefix">

File: model/robots/common/xacro/thumb/thumb.xacro (robot description, xacro)
@@ -96,8 +96,8 @@
   </xacro:macro>
   <xacro:macro name="thumb_transmissions_hw" params="prefix reflect">
-    <xacro:simple_position_transmission jointName="${ThumbRollJointName}" actuatorName="${prefix}ThumbRollActuator" nodeName="${ThumbRollNode}" actuatorApi="${ThumbFingerApi}"/>
-    <xacro:simple_forearm_position_transmission jointName="${ThumbPitch1JointName}" actuatorName="${prefix}ThumbPitch1Actuator" nodeName="${ThumbPitch1Node}" actuatorApi="${ThumbFingerApi}" reflect="${reflect}"/>
-    <xacro:simple_forearm_position_transmission jointName="${ThumbPitch2JointName}" actuatorName="${prefix}ThumbPitch2Actuator" nodeName="${ThumbPitch2Node}" actuatorApi="${ThumbFingerApi}" reflect="${reflect}"/>
-    <xacro:simple_forearm_position_transmission jointName="${ThumbPitch3JointName}" actuatorName="${prefix}ThumbPitch3Actuator" nodeName="${ThumbPitch3Node}" actuatorApi="${ThumbFingerApi}" reflect="${reflect}"/>
+    <xacro:simple_position_transmission jointName="${ThumbRollJointName}" actuatorName="${prefix}ThumbRollActuator" nodeName="${ThumbRollSensNode}" actuatorApi="${ThumbFingerRollApi}"/>
+    <xacro:simple_forearm_position_transmission jointName="${ThumbPitch1JointName}" actuatorName="${prefix}ThumbPitch1Actuator" nodeName="${ThumbPitch1Node}" actuatorApi="${ThumbFingerProximalApi}" reflect="${reflect}"/>
+    <xacro:simple_forearm_position_transmission jointName="${ThumbPitch2JointName}" actuatorName="${prefix}ThumbPitch2Actuator" nodeName="${ThumbPitch2Node}" actuatorApi="${ThumbFingerMedialApi}" reflect="${reflect}"/>
+    <xacro:simple_forearm_position_transmission jointName="${ThumbPitch3JointName}" actuatorName="${prefix}ThumbPitch3Actuator" nodeName="${ThumbPitch3Node}" actuatorApi="${ThumbFingerDistalApi}" reflect="${reflect}"/>
   </xacro:macro>
   <xacro:macro name="thumb_transmissions_sim" params="prefix">

File: model/robots/common/xacro/valkyrie_base_hw.xacro (robot description, xacro)
@@ -26,5 +26,5 @@
     <xacro:arm_transmissions_hw prefix="right" reflect="-1"/>
     <xacro:neck_transmissions_hw />
-<!--    <xacro:index_finger_transmissions_hw prefix="left" reflect="1" />
+    <xacro:index_finger_transmissions_hw prefix="left" reflect="1" />
     <xacro:middle_finger_transmissions_hw prefix="left" reflect="1"/>
     <xacro:pinky_finger_transmissions_hw prefix="left" reflect="1"/>
@@ -33,4 +33,4 @@
     <xacro:middle_finger_transmissions_hw prefix="right" reflect="-1"/>
     <xacro:pinky_finger_transmissions_hw prefix="right" reflect="-1"/>
-    <xacro:thumb_transmissions_hw prefix="right" reflect="-1"/> -->
+    <xacro:thumb_transmissions_hw prefix="right" reflect="-1"/>
 </robot>
