Commit message: committing for fulling checkout

File: common/xacro/api/valkyrie_B_api.xacro (robot description, xacro)
@@ -11,6 +11,6 @@
     <xacro:property name="ElbowPitchApi" value="robot_hardware_interface/TurbodriverAPI" />
     <xacro:property name="ForearmYawApi" value="robot_hardware_interface/TurbodriverAPI" />
-    <xacro:property name="WristTopActuatorApi" value="robot_hardware_interface/TurbodriverAPI_linear_futek" />
-    <xacro:property name="WristBottomActuatorApi" value="robot_hardware_interface/TurbodriverAPI_linear_futek" />
+    <xacro:property name="WristTopActuatorApi" value="robot_hardware_interface::TurbodriverLinearFutekJointVelocity" />
+    <xacro:property name="WristBottomActuatorApi" value="robot_hardware_interface::TurbodriverLinearFutekJointVelocity" />
     <xacro:property name="LowerNeckPitchApi" value="robot_hardware_interface/TurbodriverAPI" />
     <xacro:property name="NeckYawApi" value="robot_hardware_interface/TurbodriverAPI" />
@@ -46,5 +46,5 @@
     <xacro:property name="ThumbFingerDistalApi" value="robot_hardware_interface/TurbodriverFingerDis"/>
     <xacro:property name="ThumbFingerRollApi" value="robot_hardware_interface/TurbodriverFingerRoll"/>
-    <xacro:property name="WristRightActuatorApi" value="robot_hardware_interface/TurbodriverAPI_linear_futek"/>
-    <xacro:property name="WristLeftActuatorApi" value="robot_hardware_interface/TurbodriverAPI_linear_futek"/>
+    <xacro:property name="WristRightActuatorApi" value="robot_hardware_interface::TurbodriverLinearFutekJointVelocity"/>
+    <xacro:property name="WristLeftActuatorApi" value="robot_hardware_interface::TurbodriverLinearFutekJointVelocity"/>
 </robot>

File: common/xacro/serial_numbers/valkyrie_A_serials.xacro (robot description, xacro)
@@ -16,12 +16,12 @@
 	<xacro:property name="leftArmJ3SerialNumber" value="v_f_005" />
 	<xacro:property name="leftArmJ4SerialNumber" value="v_f_020" />
-        <xacro:property name="leftArmJ5SerialNumber" value="v_g_007" />
-        <xacro:property name="leftForearmSerialNumber" value="v_h_003"/>
+        <xacro:property name="leftArmJ5SerialNumber" value="v_g_018" />
+        <xacro:property name="leftForearmSerialNumber" value="v_h_007"/>
 	<xacro:property name="rightArmJ1SerialNumber" value="v_a_001" />
 	<xacro:property name="rightArmJ2SerialNumber" value="v_b_003" />
 	<xacro:property name="rightArmJ3SerialNumber" value="v_f_004" />
 	<xacro:property name="rightArmJ4SerialNumber" value="v_f_003" />
-        <xacro:property name="rightArmJ5SerialNumber" value="v_g_006" />
-        <xacro:property name="rightForearmSerialNumber" value="v_h_004"/>
+        <xacro:property name="rightArmJ5SerialNumber" value="v_g_017" />
+        <xacro:property name="rightForearmSerialNumber" value="v_h_008" />
 	<xacro:property name="neckJ1SerialNumber" value="v_g_006" />
 	<xacro:property name="neckJ2SerialNumber" value="v_g_007" />
@@ -30,6 +30,4 @@
 	<xacro:property name="waistRightActuatorSerialNumber" value="v_e_005" />
 	<xacro:property name="waistLeftActuatorSerialNumber" value="v_e_006" />
-	<xacro:property name="leftForearmSerialNumber" value="v_h_005"/>
-    <xacro:property name="rightForearmSerialNumber" value="v_h_008"/>
 	<xacro:property name="left_foot_ATI_serial" value="FT17218" />
 	<xacro:property name="right_foot_ATI_serial" value="FT14018" />

File: common/xacro/serial_numbers/valkyrie_B_serials.xacro (robot description, xacro)
@@ -16,12 +16,12 @@
 	<xacro:property name="leftArmJ3SerialNumber" value="v_f_007" />
 	<xacro:property name="leftArmJ4SerialNumber" value="v_f_008" />
-        <xacro:property name="leftArmJ5SerialNumber" value="v_g_018" />
-        <xacro:property name="leftForearmSerialNumber" value="v_h_007"/>
+        <xacro:property name="leftArmJ5SerialNumber" value="v_g_021" />
+        <xacro:property name="leftForearmSerialNumber" value="v_h_003"/>
 	<xacro:property name="rightArmJ1SerialNumber" value="v_a_010" />
 	<xacro:property name="rightArmJ2SerialNumber" value="v_b_008" />
 	<xacro:property name="rightArmJ3SerialNumber" value="v_f_009" />
 	<xacro:property name="rightArmJ4SerialNumber" value="v_f_010" />
-        <xacro:property name="rightArmJ5SerialNumber" value="v_g_017" />
-        <xacro:property name="rightForearmSerialNumber" value="v_h_008" />
+        <xacro:property name="rightArmJ5SerialNumber" value="v_g_020" />
+        <xacro:property name="rightForearmSerialNumber" value="v_h_004"/>
 	<xacro:property name="neckJ1SerialNumber" value="v_g_019" />
 	<xacro:property name="neckJ2SerialNumber" value="v_g_010" />
