Commit message: changed firmware layout in instance file

File: common/xacro/firmware/valkyrie_firmware.xacro (robot description, xacro)
@@ -44,6 +44,6 @@
     <!-- Arm Public -->
     <xacro:property name="ShoulderPitchPublicProcFirmware" value="${PublicTurboProcRotaryFirmwareExtension}" />
-    <xacro:property name="LeftShoulderPitchPublicFPGAFirmware" value="${PublicTurboFPGAFirmwareExtension01}" />
-    <xacro:property name="RightShoulderPitchPublicFPGAFirmware" value="${PublicTurboFPGAFirmwareExtension04}" />
+    <xacro:property name="leftShoulderPitchPublicFPGAFirmware" value="${PublicTurboFPGAFirmwareExtension01}" />
+    <xacro:property name="rightShoulderPitchPublicFPGAFirmware" value="${PublicTurboFPGAFirmwareExtension04}" />
     <xacro:property name="ShoulderRollPublicProcFirmware" value="${PublicTurboProcRotaryFirmwareExtension}" />
     <xacro:property name="ShoulderRollPublicFPGAFirmware" value="${PublicTurboFPGAFirmwareExtension02}" />
@@ -56,6 +56,6 @@
     <!-- Arm Private -->
     <xacro:property name="ShoulderPitchPrivateProcFirmware" value="${PrivateTurboProcRotaryFirmwareExtension}" />
-    <xacro:property name="LeftShoulderPitchPrivateFPGAFirmware" value="${PrivateTurboFPGAFirmwareExtension01}" />
-    <xacro:property name="RightShoulderPitchPrivateFPGAFirmware" value="${PrivateTurboFPGAFirmwareExtension04}" />
+    <xacro:property name="leftShoulderPitchPrivateFPGAFirmware" value="${PrivateTurboFPGAFirmwareExtension01}" />
+    <xacro:property name="rightShoulderPitchPrivateFPGAFirmware" value="${PrivateTurboFPGAFirmwareExtension04}" />
     <xacro:property name="ShoulderRollPrivateProcFirmware" value="${PrivateTurboProcRotaryFirmwareExtension}" />
     <xacro:property name="ShoulderRollPrivateFPGAFirmware" value="${PrivateTurboFPGAFirmwareExtension02}" />

File: instance/instances/robots/forearm_testbench_left.xacro (robot description, xacro)
@@ -11,5 +11,5 @@
 	<xacro:firmware_base_url/>
     <Mechanisms>
-    <xacro:simple_mechanism name="testbench_actuator" serial_number="${forearm_yaw_serial_number}" node="${testbench_node}" processor_firmware="" fpga_firmware=""/>
+    <xacro:simple_mechanism name="testbench_actuator" serial_number="${forearm_yaw_serial_number}" node="${testbench_node}" />
     <xacro:forearm mechanism_name="${prefix}Forearm" serial_number="${forearm_serial_number}" athena1_node="${Athena1Node}" athena2_node="${Athena2Node}" />
 	</Mechanisms>

File: instance/instances/robots/forearm_testbench_right.xacro (robot description, xacro)
@@ -11,5 +11,5 @@
 	<xacro:firmware_base_url/>
     <Mechanisms>
-    <xacro:simple_mechanism name="testbench_actuator" serial_number="${forearm_yaw_serial_number}" node="${testbench_node}" processor_firmware="" fpga_firmware=""/>
+    <xacro:simple_mechanism name="testbench_actuator" serial_number="${forearm_yaw_serial_number}" node="${testbench_node}" />
     <xacro:forearm mechanism_name="${prefix}Forearm" serial_number="${forearm_serial_number}" athena1_node="${Athena1Node}" athena2_node="${Athena2Node}" />
 	</Mechanisms>

File: instance/instances/robots/xacro/common/valkyrie_full_template.xacro (robot description, xacro)
@@ -7,7 +7,7 @@
 	<xacro:include filename="$(find val_description)/instance/instances/robots/xacro/sensors/imu.xacro" />
 	<xacro:include filename="$(find val_description)/instance/instances/robots/xacro/sensors/ati_force_torque.xacro" />
+	<xacro:include filename="$(find val_description)/instance/instances/robots/xacro/firmware/firmware.xacro" />
 	<RobotInstance id="${instance}" />
 	<xacro:all_channels/>
-	<xacro:firmware_base_url/>
 	<Mechanisms>
 		<xacro:leg prefix="left" j1_serial_number="${leftLegJ1SerialNumber}" j2_serial_number="${leftLegJ2SerialNumber}" j3_serial_number="${leftLegJ3SerialNumber}" j4_serial_number="${leftLegJ4SerialNumber}" ankle_left_actuator_serial="${leftAnkleLeftActuatorSerialNumber}" ankle_right_actuator_serial="${leftAnkleRightActuatorSerialNumber}"/>
@@ -22,3 +22,5 @@
 		<xacro:ati_force_torque name="right_foot_force_torque" serial_number="${right_foot_ATI_serial}" node="${right_foot_ATI_node}"/>
 	</Devices>
+	<xacro:firmware_base_url/>
+    <xacro:firmware />
 </robot>

File: instance/instances/robots/xacro/limbs/arm.xacro (robot description, xacro)
@@ -2,11 +2,10 @@
     <xacro:include filename="$(find val_description)/instance/instances/robots/xacro/mechanisms/mechanisms.xacro"/>
     <xacro:include filename="$(find val_description)/common/xacro/joint_names/valkyrie_joint_names.xacro"/>
-    <xacro:include filename="$(find val_description)/common/xacro/firmware/valkyrie_firmware.xacro"/>
     <xacro:macro name="arm" params="prefix j1_serial_number j2_serial_number j3_serial_number j4_serial_number j5_serial_number forearm_serial_number" >
-    	<xacro:simple_mechanism name="${ShoulderPitchJointName}" serial_number="${j1_serial_number}" node="${ShoulderPitchNode}" processor_firmware="${ShoulderPitchProcFirmware}" fpga_firmware="${ShoulderPitchFPGAFirmware}"/>
-    	<xacro:simple_mechanism name="${ShoulderRollJointName}" serial_number="${j2_serial_number}" node="${ShoulderRollNode}" processor_firmware="${ShoulderRollProcFirmware}" fpga_firmware="${ShoulderRollFPGAFirmware}"/>
-    	<xacro:simple_mechanism name="${ShoulderYawJointName}" serial_number="${j3_serial_number}" node="${ShoulderYawNode}" processor_firmware="${ShoulderYawProcFirmware}" fpga_firmware="${ShoulderYawFPGAFirmware}"/>
-    	<xacro:simple_mechanism name="${ElbowPitchJointName}" serial_number="${j4_serial_number}" node="${ElbowPitchNode}" processor_firmware="${ElbowPitchProcFirmware}" fpga_firmware="${ElbowPitchFPGAFirmware}"/>
-    	<xacro:simple_mechanism name="${ForearmYawJointName}" serial_number="${j5_serial_number}" node="${ForearmYawNode}" processor_firmware="${ForearmYawProcFirmware}" fpga_firmware="${ForearmYawFPGAFirmware}"/>
+    	<xacro:simple_mechanism name="${ShoulderPitchJointName}" serial_number="${j1_serial_number}" node="${ShoulderPitchNode}" />
+    	<xacro:simple_mechanism name="${ShoulderRollJointName}" serial_number="${j2_serial_number}" node="${ShoulderRollNode}" />
+    	<xacro:simple_mechanism name="${ShoulderYawJointName}" serial_number="${j3_serial_number}" node="${ShoulderYawNode}" />
+    	<xacro:simple_mechanism name="${ElbowPitchJointName}" serial_number="${j4_serial_number}" node="${ElbowPitchNode}" />
+    	<xacro:simple_mechanism name="${ForearmYawJointName}" serial_number="${j5_serial_number}" node="${ForearmYawNode}" />
         <xacro:forearm mechanism_name="${prefix}Forearm" serial_number="${forearm_serial_number}" athena1_node="${Athena1Node}" athena2_node="${Athena2Node}" />
     </xacro:macro>

File: instance/instances/robots/xacro/limbs/leg.xacro (robot description, xacro)
@@ -3,9 +3,9 @@
     <xacro:include filename="$(find val_description)/common/xacro/joint_names/valkyrie_joint_names.xacro"/>
     <xacro:macro name="leg" params="prefix j1_serial_number j2_serial_number j3_serial_number j4_serial_number ankle_left_actuator_serial ankle_right_actuator_serial" >
-    	<xacro:simple_mechanism name="${HipYawJointName}" serial_number="${j1_serial_number}" node="${HipYawNode}" processor_firmware="${HipYawProcFirmware}" fpga_firmware="${HipYawFPGAFirmware}"/>
-    	<xacro:simple_mechanism name="${HipRollJointName}" serial_number="${j2_serial_number}" node="${HipRollNode}" processor_firmware="${HipRollProcFirmware}" fpga_firmware="${HipRollFPGAFirmware}"/>
-    	<xacro:simple_mechanism name="${HipPitchJointName}" serial_number="${j3_serial_number}" node="${HipPitchNode}" processor_firmware="${HipPitchProcFirmware}" fpga_firmware="${HipPitchFPGAFirmware}"/>
-    	<xacro:simple_mechanism name="${KneePitchJointName}" serial_number="${j4_serial_number}" node="${KneePitchNode}" processor_firmware="${KneePitchProcFirmware}" fpga_firmware="${KneePitchFPGAFirmware}"/>
-    	<xacro:two_active_joint_mechanism mechanism_name="${prefix}Ankle" actuator0_name="${AnkleLeftActuatorName}" actuator1_name="${AnkleRightActuatorName}" joint0_name="${AnklePitchJointName}" joint1_name="${AnkleRollJointName}" actuator0_serial="${ankle_left_actuator_serial}" actuator1_serial="${ankle_right_actuator_serial}" actuator0_node="${AnkleLeftActuatorNode}" actuator1_node="${AnkleRightActuatorNode}" processor_firmware0="${AnkleLeftActuatorProcFirmware}" fpga_firmware0="${AnkleLeftActuatorFPGAFirmware}" processor_firmware1="${AnkleRightActuatorProcFirmware}" fpga_firmware1="${AnkleRightActuatorFPGAFirmware}"/>
+    	<xacro:simple_mechanism name="${HipYawJointName}" serial_number="${j1_serial_number}" node="${HipYawNode}" />
+    	<xacro:simple_mechanism name="${HipRollJointName}" serial_number="${j2_serial_number}" node="${HipRollNode}" />
+    	<xacro:simple_mechanism name="${HipPitchJointName}" serial_number="${j3_serial_number}" node="${HipPitchNode}" />
+    	<xacro:simple_mechanism name="${KneePitchJointName}" serial_number="${j4_serial_number}" node="${KneePitchNode}" />
+    	<xacro:two_active_joint_mechanism mechanism_name="${prefix}Ankle" actuator0_name="${AnkleLeftActuatorName}" actuator1_name="${AnkleRightActuatorName}" joint0_name="${AnklePitchJointName}" joint1_name="${AnkleRollJointName}" actuator0_serial="${ankle_left_actuator_serial}" actuator1_serial="${ankle_right_actuator_serial}" actuator0_node="${AnkleLeftActuatorNode}" actuator1_node="${AnkleRightActuatorNode}" />
     </xacro:macro>
 </robot>

File: instance/instances/robots/xacro/limbs/neck.xacro (robot description, xacro)
@@ -3,7 +3,7 @@
     <xacro:include filename="$(find val_description)/common/xacro/joint_names/valkyrie_joint_names.xacro"/>
     <xacro:macro name="neck" params="j1_serial_number j2_serial_number j3_serial_number" >
-    	<xacro:simple_mechanism name="${LowerNeckPitchJointName}" serial_number="${j1_serial_number}" node="${LowerNeckPitchNode}" processor_firmware="${LowerNeckPitchProcessorFirmware}" fpga_firmware="${LowerNeckPitchFPGAFirmware"/>
-    	<xacro:simple_mechanism name="${NeckYawJointName}" serial_number="${j2_serial_number}" node="${NeckYawNode}" processor_firmware="${NeckYawProcessorFirmware}" fpga_firmware="${NeckYawFPGAFirmware}"/>
-    	<xacro:simple_mechanism name="${UpperNeckPitchJointName}" serial_number="${j3_serial_number}" node="${UpperNeckPitchNode}" processor_firmware="${UpperNeckPitchProcessorFirmware}" fpga_firmware="${UpperNeckPitchFPGAFirmware}"/>
+    	<xacro:simple_mechanism name="${LowerNeckPitchJointName}" serial_number="${j1_serial_number}" node="${LowerNeckPitchNode}" />
+    	<xacro:simple_mechanism name="${NeckYawJointName}" serial_number="${j2_serial_number}" node="${NeckYawNode}" />
+    	<xacro:simple_mechanism name="${UpperNeckPitchJointName}" serial_number="${j3_serial_number}" node="${UpperNeckPitchNode}" />
     </xacro:macro>
 </robot>

File: instance/instances/robots/xacro/limbs/waist.xacro (robot description, xacro)
@@ -4,6 +4,6 @@
     <xacro:include filename="$(find val_description)/common/xacro/actuator_names/valkyrie_actuator_names.xacro"/>
     <xacro:macro name="waist" params="j1_serial_number waist_left_actuator_serial waist_right_actuator_serial" >
-    	<xacro:simple_mechanism name="${TorsoYawJointName}" serial_number="${j1_serial_number}" node="${TrunkYawNode}" processor_firmware="${TrunkYawProcessorFirmware}" fpga_firmware="${TrunkYawFPGAFirmware}"/>
-    	<xacro:two_active_joint_mechanism mechanism_name="waist" actuator0_name="${WaistLeftActuatorName}" actuator1_name="${WaistRightActuatorName}" joint0_name="${TorsoPitchJointName}" joint1_name="${TorsoRollJointName}" actuator0_serial="${waist_left_actuator_serial}" actuator1_serial="${waist_right_actuator_serial}" actuator0_node="${WaistLeftActuatorNode}" actuator1_node="${WaistRightActuatorNode}" processor_firmware0="${WaistLeftActuatorProcessorFirmware}" fpga_firmware0="${WaistLeftActuatorFPGAFirmware}" processor_firmware1="${WaistRightActuatorProcessorFirmware}" fpga_firmware1="${WaistRightActuatorFPGAFirmware}"/>/>
+    	<xacro:simple_mechanism name="${TorsoYawJointName}" serial_number="${j1_serial_number}" node="${TrunkYawNode}" />
+    	<xacro:two_active_joint_mechanism mechanism_name="waist" actuator0_name="${WaistLeftActuatorName}" actuator1_name="${WaistRightActuatorName}" joint0_name="${TorsoPitchJointName}" joint1_name="${TorsoRollJointName}" actuator0_serial="${waist_left_actuator_serial}" actuator1_serial="${waist_right_actuator_serial}" actuator0_node="${WaistLeftActuatorNode}" actuator1_node="${WaistRightActuatorNode}" />/>
     </xacro:macro>
 </robot>

File: instance/instances/robots/xacro/mechanisms/mechanisms.xacro (robot description, xacro)
@@ -1,9 +1,7 @@
 <robot xmlns:xacro="http://ros.org/wiki/xacro" name="actuators">
-  <xacro:macro name="simple_mechanism" params="name serial_number node processor_firmware fpga_firmware">
+  <xacro:macro name="simple_mechanism" params="name serial_number node ">
   	<Mechanism id="${name}" type="simple">
   		<SerialNumber id="${serial_number}" />
   		<Node id="${node}" />
-  		<Processor_Firmware id="${processor_firmware}" />
-  		<Fpga_Firmware id="${fpga_firmware}" />
 	</Mechanism>
 </xacro:macro>
@@ -12,18 +10,16 @@
 	</Joint>
 </xacro:macro>
-<xacro:macro name="actuator" params="name serial_number node processor_firmware fpga_firmware" >
+<xacro:macro name="actuator" params="name serial_number node " >
 	<Actuator id="${name}">
 		<SerialNumber id="${serial_number}" />
 		<Node id="${node}" />
-		<Processor_Firmware id="${processor_firmware}" />
-		<Fpga_Firmware id="${fpga_firmware}" />
 	</Actuator>
 </xacro:macro>
-<xacro:macro name="two_active_joint_mechanism" params="mechanism_name actuator0_name actuator1_name joint0_name joint1_name actuator0_serial actuator0_node actuator1_serial actuator1_node processor_firmware0 fpga_firmware0 processor_firmware1 fpga_firmware1" >
+<xacro:macro name="two_active_joint_mechanism" params="mechanism_name actuator0_name actuator1_name joint0_name joint1_name actuator0_serial actuator0_node actuator1_serial actuator1_node " >
 	<Mechanism id="${mechanism_name}" type="complex">
 		<xacro:joint name="${joint0_name}" type="active"/>
 		<xacro:joint name="${joint1_name}" type="active"/>
-		<xacro:actuator name="${actuator0_name}" serial_number="${actuator0_serial}" node="${actuator0_node}" processor_firmware="${processor_firmware0}" fpga_firmware="${fpga_firmware0}"/>
-		<xacro:actuator name="${actuator1_name}" serial_number="${actuator1_serial}" node="${actuator1_node}" processor_firmware="${processor_firmware1}" fpga_firmware="${fpga_firmware1}"/>
+		<xacro:actuator name="${actuator0_name}" serial_number="${actuator0_serial}" node="${actuator0_node}" />
+		<xacro:actuator name="${actuator1_name}" serial_number="${actuator1_serial}" node="${actuator1_node}" />
 	</Mechanism>
 </xacro:macro>

Commit message: fixed typo in bintray url

File: common/xacro/firmware/valkyrie_firmware.xacro (robot description, xacro)
@@ -2,6 +2,6 @@
 <robot name="valkyrie_firmware_locations" xmlns:xacro="http://www.ros.org/wiki/xacro">
     <!-- Public Base URL -->
-    <xacro:property name="PublicProcFirmwareBaseURL" value="http://nasa-jsc-robotics/bintray.com/val-firmware/"/>
-    <xacro:property name="PublicFPGAFirmwareBaseURL" value="http://nasa-jsc-robotics/bintray.com/val-firmware/"/>
+    <xacro:property name="PublicProcFirmwareBaseURL" value="http://nasa-jsc-robotics.bintray.com/val-firmware/"/>
+    <xacro:property name="PublicFPGAFirmwareBaseURL" value="http://nasa-jsc-robotics.bintray.com/val-firmware/"/>
     <!-- Private Base URL -->
     <xacro:property name="PrivateProcFirmwareBaseURL" value="http://flexo.jsc.nasa.gov/bamboo/browse/EMB-SEAP/latest/artifact/shared/"/>
