Commit message: Adding calibration angle to instance file.

File: instance/instances/robots/xacro/common/valkyrie_full_template.xacro (robot description, xacro)
@@ -1,18 +1,19 @@
 <robot xmlns:xacro="http://ros.org/wiki/xacro" name="valkyrie_template">
 	<xacro:include filename="$(find val_description)/common/xacro/nodes/valkyrie_nodes.xacro" />
-	<xacro:include filename="$(find val_description)/instance/instances/robots/xacro/limbs/leg.xacro" />
-	<xacro:include filename="$(find val_description)/instance/instances/robots/xacro/limbs/arm.xacro" />
-	<xacro:include filename="$(find val_description)/instance/instances/robots/xacro/limbs/neck.xacro" />
-	<xacro:include filename="$(find val_description)/instance/instances/robots/xacro/limbs/waist.xacro" />
+	<xacro:include filename="$(find val_description)/instance/instances/robots/xacro/limbs/leg/leg.xacro" />
+	<xacro:include filename="$(find val_description)/instance/instances/robots/xacro/limbs/arm/arm.xacro" />
+	<xacro:include filename="$(find val_description)/instance/instances/robots/xacro/limbs/neck/neck.xacro" />
+	<xacro:include filename="$(find val_description)/instance/instances/robots/xacro/limbs/waist/waist.xacro" />
 	<xacro:include filename="$(find val_description)/instance/instances/robots/xacro/sensors/imu.xacro" />
 	<xacro:include filename="$(find val_description)/instance/instances/robots/xacro/sensors/ati_force_torque.xacro" />
+	<xacro:include filename="$(find val_description)/instance/instances/robots/xacro/common/joint_calibration_angles.xacro" />
 	<RobotInstance id="${instance}" />
 	<xacro:all_channels/>
 	<xacro:firmware_base_url/>
 	<Mechanisms>
-		<xacro:leg prefix="left" j1_serial_number="${leftLegJ1SerialNumber}" j2_serial_number="${leftLegJ2SerialNumber}" j3_serial_number="${leftLegJ3SerialNumber}" j4_serial_number="${leftLegJ4SerialNumber}" ankle_left_actuator_serial="${leftAnkleLeftActuatorSerialNumber}" ankle_right_actuator_serial="${leftAnkleRightActuatorSerialNumber}"/>
-		<xacro:leg prefix="right" j1_serial_number="${rightLegJ1SerialNumber}" j2_serial_number="${rightLegJ2SerialNumber}" j3_serial_number="${rightLegJ3SerialNumber}" j4_serial_number="${rightLegJ4SerialNumber}" ankle_left_actuator_serial="${rightAnkleLeftActuatorSerialNumber}" ankle_right_actuator_serial="${rightAnkleRightActuatorSerialNumber}" />
-		<xacro:arm prefix="left" j1_serial_number="${leftArmJ1SerialNumber}" j2_serial_number="${leftArmJ2SerialNumber}" j3_serial_number="${leftArmJ3SerialNumber}" j4_serial_number="${leftArmJ4SerialNumber}" j5_serial_number="${leftArmJ5SerialNumber}" forearm_serial_number="${leftForearmSerialNumber}" />
-		<xacro:arm prefix="right" j1_serial_number="${rightArmJ1SerialNumber}" j2_serial_number="${rightArmJ2SerialNumber}" j3_serial_number="${rightArmJ3SerialNumber}" j4_serial_number="${rightArmJ4SerialNumber}" j5_serial_number="${rightArmJ5SerialNumber}" forearm_serial_number="${rightForearmSerialNumber}" />
+		<xacro:leg prefix="left" reflect="1" j1_serial_number="${leftLegJ1SerialNumber}" j2_serial_number="${leftLegJ2SerialNumber}" j3_serial_number="${leftLegJ3SerialNumber}" j4_serial_number="${leftLegJ4SerialNumber}" ankle_left_actuator_serial="${leftAnkleLeftActuatorSerialNumber}" ankle_right_actuator_serial="${leftAnkleRightActuatorSerialNumber}"/>
+		<xacro:leg prefix="right" reflect="-1" j1_serial_number="${rightLegJ1SerialNumber}" j2_serial_number="${rightLegJ2SerialNumber}" j3_serial_number="${rightLegJ3SerialNumber}" j4_serial_number="${rightLegJ4SerialNumber}" ankle_left_actuator_serial="${rightAnkleLeftActuatorSerialNumber}" ankle_right_actuator_serial="${rightAnkleRightActuatorSerialNumber}" />
+		<xacro:arm prefix="left" reflect="1" j1_serial_number="${leftArmJ1SerialNumber}" j2_serial_number="${leftArmJ2SerialNumber}" j3_serial_number="${leftArmJ3SerialNumber}" j4_serial_number="${leftArmJ4SerialNumber}" j5_serial_number="${leftArmJ5SerialNumber}" forearm_serial_number="${leftForearmSerialNumber}" />
+		<xacro:arm prefix="right" reflect="-1" j1_serial_number="${rightArmJ1SerialNumber}" j2_serial_number="${rightArmJ2SerialNumber}" j3_serial_number="${rightArmJ3SerialNumber}" j4_serial_number="${rightArmJ4SerialNumber}" j5_serial_number="${rightArmJ5SerialNumber}" forearm_serial_number="${rightForearmSerialNumber}" />
 		<xacro:neck j1_serial_number="${neckJ1SerialNumber}" j2_serial_number="${neckJ2SerialNumber}" j3_serial_number="${neckJ3SerialNumber}" />
 		<xacro:waist j1_serial_number="${trunkSerialNumber}" waist_left_actuator_serial="${waistLeftActuatorSerialNumber}" waist_right_actuator_serial="${waistRightActuatorSerialNumber}"/>

File: instance/instances/robots/xacro/mechanisms/mechanisms.xacro (robot description, xacro)
@@ -1,4 +1,4 @@
 <robot xmlns:xacro="http://ros.org/wiki/xacro" name="actuators">
-  <xacro:macro name="simple_mechanism" params="name serial_number node processor_firmware fpga_firmware">
+  <xacro:macro name="simple_mechanism" params="name serial_number node processor_firmware fpga_firmware calibration_angle:=0.0">
   	<Mechanism id="${name}" type="simple">
   		<SerialNumber id="${serial_number}" />
@@ -6,8 +6,10 @@
   		<Processor_Firmware id="${processor_firmware}" />
   		<Fpga_Firmware id="${fpga_firmware}" />
+  		<CalibrationAngle value="${calibration_angle}"/>
 	</Mechanism>
 </xacro:macro>
-<xacro:macro name="joint" params="name type">
+<xacro:macro name="joint" params="name type calibration_angle:=0.0">
 	<Joint id="${name}" type="${type}">
+		<CalibrationAngle value="${calibration_angle}"/>
 	</Joint>
 </xacro:macro>
@@ -20,8 +22,8 @@
 	</Actuator>
 </xacro:macro>
-<xacro:macro name="two_active_joint_mechanism" params="mechanism_name actuator0_name actuator1_name joint0_name joint1_name actuator0_serial actuator0_node actuator1_serial actuator1_node processor_firmware0 fpga_firmware0 processor_firmware1 fpga_firmware1" >
+<xacro:macro name="two_active_joint_mechanism" params="mechanism_name actuator0_name actuator1_name joint0_name joint1_name  actuator0_serial actuator0_node actuator1_serial actuator1_node processor_firmware0 fpga_firmware0 processor_firmware1 fpga_firmware1 joint0_cal_angle:=0.0 joint1_cal_angle:=0.0" >
 	<Mechanism id="${mechanism_name}" type="complex">
-		<xacro:joint name="${joint0_name}" type="active"/>
-		<xacro:joint name="${joint1_name}" type="active"/>
+		<xacro:joint name="${joint0_name}" type="active" calibration_angle="${joint0_cal_angle}"/>
+		<xacro:joint name="${joint1_name}" type="active" calibration_angle="${joint1_cal_angle}"/>
 		<xacro:actuator name="${actuator0_name}" serial_number="${actuator0_serial}" node="${actuator0_node}" processor_firmware="${processor_firmware0}" fpga_firmware="${fpga_firmware0}"/>
 		<xacro:actuator name="${actuator1_name}" serial_number="${actuator1_serial}" node="${actuator1_node}" processor_firmware="${processor_firmware1}" fpga_firmware="${fpga_firmware1}"/>
