Commit message: Added actuator type and calibration angle to the mechanisms in the instance file.

File: instance/instances/robots/xacro/limbs/leg/leg.xacro (robot description, xacro)
@@ -7,5 +7,5 @@
     	<xacro:simple_mechanism name="${HipPitchJointName}" serial_number="${j3_serial_number}" node="${HipPitchNode}" processor_firmware="${HipPitchProcFirmware}" fpga_firmware="${HipPitchFPGAFirmware}" calibration_angle="${HipPitchCalibrationAngle}"/>
     	<xacro:simple_mechanism name="${KneePitchJointName}" serial_number="${j4_serial_number}" node="${KneePitchNode}" processor_firmware="${KneePitchProcFirmware}" fpga_firmware="${KneePitchFPGAFirmware}" calibration_angle="${KneePitchCalibrationAngle}"/>
-    	<xacro:two_active_joint_mechanism mechanism_name="${prefix}Ankle" actuator0_name="${AnkleLeftActuatorName}" actuator1_name="${AnkleRightActuatorName}" joint0_name="${AnklePitchJointName}" joint0_cal_angle="${AnklePitchCalibrationAngle}" joint1_cal_angle="${AnkleRollCalibrationAngle}" joint1_name="${AnkleRollJointName}" actuator0_serial="${ankle_left_actuator_serial}" actuator1_serial="${ankle_right_actuator_serial}" actuator0_node="${AnkleLeftActuatorNode}" actuator1_node="${AnkleRightActuatorNode}" processor_firmware0="${AnkleLeftActuatorProcFirmware}" fpga_firmware0="${AnkleLeftActuatorFPGAFirmware}" processor_firmware1="${AnkleRightActuatorProcFirmware}" fpga_firmware1="${AnkleRightActuatorFPGAFirmware}"/>
+    	<xacro:pushrod_mechanism mechanism_name="${prefix}Ankle" actuator0_name="${AnkleLeftActuatorName}" actuator1_name="${AnkleRightActuatorName}" joint0_name="${AnklePitchJointName}" joint0_cal_angle="${AnklePitchCalibrationAngle}" joint1_cal_angle="${AnkleRollCalibrationAngle}" joint1_name="${AnkleRollJointName}" actuator0_serial="${ankle_left_actuator_serial}" actuator1_serial="${ankle_right_actuator_serial}" actuator0_node="${AnkleLeftActuatorNode}" actuator1_node="${AnkleRightActuatorNode}" processor_firmware0="${AnkleLeftActuatorProcFirmware}" fpga_firmware0="${AnkleLeftActuatorFPGAFirmware}" processor_firmware1="${AnkleRightActuatorProcFirmware}" fpga_firmware1="${AnkleRightActuatorFPGAFirmware}" joint0_node="${AnkleRightActuatorNode}" joint1_node="${AnkleLeftActuatorNode}"/>
     </xacro:macro>
 </robot>

File: instance/instances/robots/xacro/limbs/waist/waist.xacro (robot description, xacro)
@@ -5,5 +5,5 @@
     <xacro:macro name="waist" params="j1_serial_number waist_left_actuator_serial waist_right_actuator_serial" >
     	<xacro:simple_mechanism name="${TorsoYawJointName}" serial_number="${j1_serial_number}" node="${TrunkYawNode}" processor_firmware="${TrunkYawProcessorFirmware}" fpga_firmware="${TrunkYawFPGAFirmware}" calibration_angle="${TorsoYawCalibrationAngle}"/>
-    	<xacro:two_active_joint_mechanism mechanism_name="waist" actuator0_name="${WaistLeftActuatorName}" actuator1_name="${WaistRightActuatorName}" joint0_name="${TorsoPitchJointName}" joint0_cal_angle="${WaistPitchCalibrationAngle}" joint1_name="${TorsoRollJointName}" joint1_cal_angle="${WaistPitchCalibrationAngle}"  actuator0_serial="${waist_left_actuator_serial}" actuator1_serial="${waist_right_actuator_serial}" actuator0_node="${WaistLeftActuatorNode}" actuator1_node="${WaistRightActuatorNode}" processor_firmware0="${WaistLeftActuatorProcessorFirmware}" fpga_firmware0="${WaistLeftActuatorFPGAFirmware}" processor_firmware1="${WaistRightActuatorProcessorFirmware}" fpga_firmware1="${WaistRightActuatorFPGAFirmware}"/>
+    	<xacro:pushrod mechanism_name="waist" actuator0_name="${WaistLeftActuatorName}" actuator1_name="${WaistRightActuatorName}" joint0_name="${TorsoPitchJointName}" joint0_cal_angle="${WaistPitchCalibrationAngle}" joint1_name="${TorsoRollJointName}" joint1_cal_angle="${WaistPitchCalibrationAngle}"  actuator0_serial="${waist_left_actuator_serial}" actuator1_serial="${waist_right_actuator_serial}" actuator0_node="${WaistLeftActuatorNode}" actuator1_node="${WaistRightActuatorNode}" processor_firmware0="${WaistLeftActuatorProcessorFirmware}" fpga_firmware0="${WaistLeftActuatorFPGAFirmware}" processor_firmware1="${WaistRightActuatorProcessorFirmware}" fpga_firmware1="${WaistRightActuatorFPGAFirmware}" joint0_node="${WaistRightActuatorNode}" joint1_node="${WaistLeftActuatorNode}"/>
     </xacro:macro>
 </robot>

File: instance/instances/robots/xacro/mechanisms/mechanisms.xacro (robot description, xacro)
@@ -9,11 +9,12 @@
 	</Mechanism>
 </xacro:macro>
-<xacro:macro name="joint" params="name type calibration_angle:=0.0">
+<xacro:macro name="joint" params="name type node calibration_angle:=0.0">
 	<Joint id="${name}" type="${type}">
 		<CalibrationAngle value="${calibration_angle}"/>
+		<Node id="${node}"/>
 	</Joint>
 </xacro:macro>
-<xacro:macro name="actuator" params="name serial_number node processor_firmware fpga_firmware" >
-	<Actuator id="${name}">
+<xacro:macro name="actuator" params="name type serial_number node processor_firmware fpga_firmware" >
+	<Actuator id="${name}" type="${type}">
 		<SerialNumber id="${serial_number}" />
 		<Node id="${node}" />
@@ -22,11 +23,14 @@
 	</Actuator>
 </xacro:macro>
-<xacro:macro name="two_active_joint_mechanism" params="mechanism_name actuator0_name actuator1_name joint0_name joint1_name  actuator0_serial actuator0_node actuator1_serial actuator1_node processor_firmware0 fpga_firmware0 processor_firmware1 fpga_firmware1 joint0_cal_angle:=0.0 joint1_cal_angle:=0.0" >
+<xacro:macro name="two_active_joint_mechanism" params="mechanism_name actuator0_name actuator1_name actuator0_type actuator1_type joint0_name joint1_name actuator0_serial actuator0_node actuator1_serial actuator1_node processor_firmware0 fpga_firmware0 processor_firmware1 fpga_firmware1 joint0_node:=${actuator0_node} joint1_node:=${actuator1_node} joint0_cal_angle:=0.0 joint1_cal_angle:=0.0" >
 	<Mechanism id="${mechanism_name}" type="complex">
-		<xacro:joint name="${joint0_name}" type="active" calibration_angle="${joint0_cal_angle}"/>
-		<xacro:joint name="${joint1_name}" type="active" calibration_angle="${joint1_cal_angle}"/>
-		<xacro:actuator name="${actuator0_name}" serial_number="${actuator0_serial}" node="${actuator0_node}" processor_firmware="${processor_firmware0}" fpga_firmware="${fpga_firmware0}"/>
-		<xacro:actuator name="${actuator1_name}" serial_number="${actuator1_serial}" node="${actuator1_node}" processor_firmware="${processor_firmware1}" fpga_firmware="${fpga_firmware1}"/>
+		<xacro:joint name="${joint0_name}" type="active" node="${joint0_node}" calibration_angle="${joint0_cal_angle}"/>
+		<xacro:joint name="${joint1_name}" type="active" node="${joint1_node}" calibration_angle="${joint1_cal_angle}"/>
+		<xacro:actuator name="${actuator0_name}" type="${actuator0_type}" serial_number="${actuator0_serial}" node="${actuator0_node}" processor_firmware="${processor_firmware0}" fpga_firmware="${fpga_firmware0}"/>
+		<xacro:actuator name="${actuator1_name}" type="${actuator1_type}" serial_number="${actuator1_serial}" node="${actuator1_node}" processor_firmware="${processor_firmware1}" fpga_firmware="${fpga_firmware1}"/>
 	</Mechanism>
+</xacro:macro>
+<xacro:macro name="pushrod_mechanism" params="mechanism_name actuator0_name actuator1_name joint0_name joint1_name actuator0_serial actuator0_node actuator1_serial actuator1_node processor_firmware0 fpga_firmware0 processor_firmware1 fpga_firmware1 joint0_node:=${actuator0_node} joint1_node:=${actuator1_node} joint0_cal_angle:=0.0 joint1_cal_angle:=0.0" >
+	<xacro:two_active_joint_mechanism  mechanism_name="${mechanism_name}" actuator0_name="${actuator0_name}" actuator1_name="${actuator1_name}" actuator0_type="linear" actuator1_type="linear" joint0_name="${joint0_name}" joint1_name="${joint1_name}" actuator0_serial="${actuator0_serial}" actuator0_node="${actuator0_node}" actuator1_serial="${actuator1_serial}" actuator1_node="${actuator1_node}" processor_firmware0="${processor_firmware0}" fpga_firmware0="${fpga_firmware0}" processor_firmware1="${processor_firmware1}" fpga_firmware1="${fpga_firmware1}" joint0_node="${joint0_node}" joint1_node="${joint1_node}" joint0_cal_angle="${joint0_cal_angle}" joint1_cal_angle="${joint1_cal_angle}"/>
 </xacro:macro>
 <xacro:macro name="forearm" params="mechanism_name serial_number athena1_node athena2_node">
