Commit message: Updated ankle ROM based on hardware.

File: model/robots/common/xacro/leg/joint_limits.xacro (robot description, xacro)
@@ -11,12 +11,12 @@
   <xacro:property name="HipPitchPositionLimit_Lower" value="-2.42" />
   <xacro:property name="KneePitchPositionLimit_Lower" value="-0.083" />
-  <xacro:property name="AnklePitchPositionLimit_Lower" value="-0.8644" />
-  <xacro:property name="AnkleRollPositionLimit_Lower" value="-0.349" />
+  <xacro:property name="AnklePitchPositionLimit_Lower" value="-0.93" />
+  <xacro:property name="AnkleRollPositionLimit_Lower" value="-0.4" />
   <xacro:property name="HipYawPositionLimit_Upper" value="0.4141" />
   <xacro:property name="HipRollPositionLimit_Upper" value="0.467" />
   <xacro:property name="HipPitchPositionLimit_Upper" value="1.619" />
   <xacro:property name="KneePitchPositionLimit_Upper" value="2.057" />
-  <xacro:property name="AnklePitchPositionLimit_Upper" value="0.875" />
-  <xacro:property name="AnkleRollPositionLimit_Upper" value="0.348" />
+  <xacro:property name="AnklePitchPositionLimit_Upper" value="0.65" />
+  <xacro:property name="AnkleRollPositionLimit_Upper" value="0.4" />
   <xacro:property name="HipYawVelocityLimit" value="5.89" />
   <xacro:property name="HipRollVelocityLimit" value="7" />
