Commit message: Still working on leg meshes.

File: model/robots/common/xacro/leg/leg.xacro (robot description, xacro)
@@ -9,12 +9,4 @@
                     visual_mesh="${leg_mesh_dir}/lj1_${prefix}.dae"
                     collision_mesh="${leg_mesh_dir}/lj1_${prefix}.dae"/>
-    <!-- <xacro:standard_link name="${HipRollLinkName}"
-                    mass="${HipRollLinkMass}"
-                    origin_xyz="${HipRollLinkComPosition}"
-                    ixx="${HipRollLinkInertia_IXX}" ixy="${HipRollLinkInertia_IXY}" ixz="${HipRollLinkInertia_IXZ}"
-                    iyy="${HipRollLinkInertia_IYY}" iyz="${HipRollLinkInertia_IYZ}" izz="${HipRollLinkInertia_IZZ}"
-                    origin_rpy="0 0 0"
-                    visual_mesh="${leg_mesh_dir}/lj2_${prefix}.dae"
-                    collision_mesh="${leg_mesh_dir}/lj2_${prefix}.dae"/> -->
     <xacro:link_no_mesh_no_collision name="${HipRollLinkName}"
                     mass="${HipRollLinkMass}"

File: model/robots/common/xacro/waist/waist_angled_j1s_includes.xacro (robot description, xacro)
@@ -1,21 +1,14 @@
 <?xml version="1.0" ?>
 <robot xmlns:xacro="http://www.ros.org/wiki/xacro" name="waist_angled_j1s_frame_parameters">
-  <xacro:property name="TorsoYawFrameOrigin_X" value="0.0"/>
-  <xacro:property name="TorsoYawFrameOrigin_Y" value="0.0"/>
-  <xacro:property name="TorsoYawFrameOrigin_Z" value="0.0"/>
-  <xacro:property name="TorsoYawFrameOrientation_Roll" value="0.0"/>
-  <xacro:property name="TorsoYawFrameOrientation_Pitch" value="0.0"/>
-  <xacro:property name="TorsoYawFrameOrientation_Yaw" value="0.0"/>
-  <xacro:property name="TorsoPitchFrameOrigin_X" value="0.04191"/>
-  <xacro:property name="TorsoPitchFrameOrigin_Y" value="0.0"/>
-  <xacro:property name="TorsoPitchFrameOrigin_Z" value="0.04502658"/>
-  <xacro:property name="TorsoPitchFrameOrientation_Roll" value="0.0"/>
-  <xacro:property name="TorsoPitchFrameOrientation_Pitch" value="0.0"/>
-  <xacro:property name="TorsoPitchFrameOrientation_Yaw" value="0.0"/>
-  <xacro:property name="TorsoRollFrameOrigin_X" value="0.0"/>
-  <xacro:property name="TorsoRollFrameOrigin_Y" value="0.0"/>
-  <xacro:property name="TorsoRollFrameOrigin_Z" value="0.0203"/>
-  <xacro:property name="TorsoRollFrameOrientation_Roll" value="0.0"/>
-  <xacro:property name="TorsoRollFrameOrientation_Pitch" value="0.0"/>
-  <xacro:property name="TorsoRollFrameOrientation_Yaw" value="0.0"/>
+  <xacro:include filename="$(find val_description)/model/robots/common/xacro/waist/joint_axes.xacro"/>
+  <xacro:include filename="$(find val_description)/model/robots/common/xacro/waist/joint_axes.xacro"/>
+  <xacro:include filename="$(find val_description)/model/robots/common/xacro/waist/link_names.xacro"/>
+  <xacro:include filename="$(find val_description)/model/robots/common/xacro/waist/joint_limits.xacro"/>
+  <xacro:include filename="$(find val_description)/model/robots/common/xacro/waist/frame_parameters.xacro"/>
+  <xacro:include filename="$(find val_description)/model/robots/common/xacro/waist/mass_parameters.xacro"/>
+  <xacro:include filename="$(find val_description)/common/xacro/joint_names/valkyrie_joint_names.xacro"/>
+  <xacro:include filename="$(find val_description)/common/xacro/actuator_names/valkyrie_actuator_names.xacro"/>
+  <xacro:include filename="$(find val_description)/model/robots/common/xacro/sensors/microstrain.xacro"/>
+  <xacro:include filename="$(find val_description)/model/robots/common/xacro/sensors/flea.xacro"/>
+  <xacro:include filename="$(find val_description)/model/robots/common/xacro/waist/waist.xacro"/>
 </robot>
