Commit message: Have leg meshes and COM's updated for new angled j1 valkyrie.

File: model/robots/common/xacro/leg/angled_j1s_includes.xacro (robot description, xacro)
@@ -4,5 +4,5 @@
 	<xacro:include filename="$(find val_description)/model/robots/common/xacro/leg/joint_limits.xacro"/>
 	<xacro:include filename="$(find val_description)/model/robots/common/xacro/leg/angled_j1s_frame_parameters.xacro"/>
-	<xacro:include filename="$(find val_description)/model/robots/common/xacro/leg/mass_parameters.xacro"/>
+	<xacro:include filename="$(find val_description)/model/robots/common/xacro/leg/angled_j1s_mass_parameters.xacro"/>
 	<xacro:include filename="$(find val_description)/common/xacro/joint_names/valkyrie_joint_names.xacro"/>
 	<xacro:include filename="$(find val_description)/common/xacro/actuator_names/valkyrie_actuator_names.xacro"/>

File: model/robots/common/xacro/leg/angled_j1s_mass_parameters.xacro (robot description, xacro)
@@ -2,5 +2,5 @@
 <robot xmlns:xacro="http://www.ros.org/wiki/xacro" name="leg_mass_parameters">
   <xacro:property name="HipYawLinkMass" value="2.39" />
-  <xacro:property name="HipYawLinkComPosition" value="0.02176 ${reflect*-0.00131} 0.03867" />
+  <xacro:property name="HipYawLinkComPosition" value="0.02176 ${reflect*-0.001310013} -0.070448123" />
   <xacro:property name="HipYawLinkInertia_IXX" value="0.017260978" />
   <xacro:property name="HipYawLinkInertia_IXY" value="0.000000000" />
@@ -10,5 +10,5 @@
   <xacro:property name="HipYawLinkInertia_IZZ" value="0.011238178" />
   <xacro:property name="HipRollLinkMass" value="3.665000" />
-  <xacro:property name="HipRollLinkComPosition" value="0.012959 ${reflect*0.007550} -0.015950" />
+  <xacro:property name="HipRollLinkComPosition" value="0.0129592 ${reflect*0.000101876} -0.017646398" />
   <xacro:property name="HipRollLinkInertia_IXX" value="0.005978962" />
   <xacro:property name="HipRollLinkInertia_IXY" value="${reflect*-0.000234823}" />
@@ -18,5 +18,5 @@
   <xacro:property name="HipRollLinkInertia_IZZ" value="0.008193117" />
   <xacro:property name="HipPitchLinkMass" value="10.20" />
-  <xacro:property name="HipPitchLinkComPosition" value="0.016691 ${reflect*0.091397} -0.207875" />
+  <xacro:property name="HipPitchLinkComPosition" value="0.0166917 ${reflect*0.0914112} -0.207876" />
   <xacro:property name="HipPitchLinkInertia_IXX" value="0.240834130" />
   <xacro:property name="HipPitchLinkInertia_IXY" value="${reflect*0.000035915}" />
@@ -26,5 +26,5 @@
   <xacro:property name="HipPitchLinkInertia_IZZ" value="0.023276352" />
   <xacro:property name="KneePitchLinkMass" value="6.200000" />
-  <xacro:property name="KneePitchLinkComPosition" value="-0.022183  0.001703  -0.189418" />
+  <xacro:property name="KneePitchLinkComPosition" value="-0.02214819  ${reflect*0.034433936}  -0.189418765" />
   <xacro:property name="KneePitchLinkInertia_IXX" value="0.086935683" />
   <xacro:property name="KneePitchLinkInertia_IXY" value="0.000099290" />

File: model/robots/common/xacro/waist/angled_j1s_includes.xacro (robot description, xacro)
@@ -5,6 +5,6 @@
   <xacro:include filename="$(find val_description)/model/robots/common/xacro/waist/link_names.xacro"/>
   <xacro:include filename="$(find val_description)/model/robots/common/xacro/waist/joint_limits.xacro"/>
-  <xacro:include filename="$(find val_description)/model/robots/common/xacro/waist/frame_parameters.xacro"/>
-  <xacro:include filename="$(find val_description)/model/robots/common/xacro/waist/mass_parameters.xacro"/>
+  <xacro:include filename="$(find val_description)/model/robots/common/xacro/waist/angled_j1s_frame_parameters.xacro"/>
+  <xacro:include filename="$(find val_description)/model/robots/common/xacro/waist/angled_j1s_mass_parameters.xacro"/>
   <xacro:include filename="$(find val_description)/common/xacro/joint_names/valkyrie_joint_names.xacro"/>
   <xacro:include filename="$(find val_description)/common/xacro/actuator_names/valkyrie_actuator_names.xacro"/>

File: model/robots/valkyrie_sim_angled_legj1s.xacro (robot description, xacro)
@@ -8,5 +8,5 @@
     <xacro:property name="leg_mesh_dir" value="package://val_description/model/meshes/legs_angled_j1s"/>
     <xacro:property name="arm_mesh_dir" value="package://val_description/model/meshes/arms"/>
-    <xacro:property name="waist_mesh_dir" value="package://val_description/model/meshes/torso"/>
+    <xacro:property name="waist_mesh_dir" value="package://val_description/model/meshes/torso_angled_j1s"/>
     <xacro:property name="head_mesh_dir" value="package://val_description/model/meshes/head"/>
     <xacro:property name="pelvis_mesh_dir" value="package://val_description/model/meshes/pelvis_angled_j1s"/>
@@ -30,5 +30,5 @@
     <xacro:include filename="$(find val_description)/model/robots/common/xacro/arm/arm_includes.xacro"/>
     <!-- Waist include -->
-    <xacro:include filename="$(find val_description)/model/robots/common/xacro/waist/waist_includes.xacro"/>
+    <xacro:include filename="$(find val_description)/model/robots/common/xacro/waist/angled_j1s_includes.xacro"/>
     <!-- Base xacro file that calls macros from included files above -->
     <xacro:include filename="$(find val_description)/model/robots/common/xacro/valkyrie_base_sim.xacro"/>
