Commit message: Adding new transmissions xacro so different robots can have different transmissions. Also moved a bunch of xacro includes to prevent a bunch of duplicate stuff.

File: model/robots/common/xacro/valkyrie_arm_mass_sims_base_hw.xacro (robot description, xacro)
@@ -1,3 +1,6 @@
 <robot xmlns:xacro="http://ros.org/wiki/xacro" name="valkyrie">
+    <xacro:property name="mesh_root" value="package://val_description/model/meshes"/>
+    <xacro:include filename="$(find val_description)/model/robots/common/xacro/generic_models.xacro" />
+    <xacro:include filename="$(find val_description)/model/robots/common/xacro/common_bodies.xacro" />
     <xacro:make_pelvis />
     <xacro:make_waist waist_root_link="${Pelvis_Link_Name}" />

File: model/robots/common/xacro/valkyrie_arm_mass_sims_base_sim.xacro (robot description, xacro)
@@ -1,3 +1,6 @@
 <robot xmlns:xacro="http://ros.org/wiki/xacro" name="valkyrie">
+    <xacro:property name="mesh_root" value="package://val_description/model/meshes"/>
+    <xacro:include filename="$(find val_description)/model/robots/common/xacro/generic_models.xacro" />
+    <xacro:include filename="$(find val_description)/model/robots/common/xacro/common_bodies.xacro" />
     <xacro:make_pelvis />
     <xacro:make_waist waist_root_link="${Pelvis_Link_Name}" />

File: model/robots/common/xacro/valkyrie_base_hw.xacro (robot description, xacro)
@@ -1,3 +1,6 @@
 <robot xmlns:xacro="http://ros.org/wiki/xacro" name="valkyrie">
+    <xacro:property name="mesh_root" value="package://val_description/model/meshes"/>
+    <xacro:include filename="$(find val_description)/model/robots/common/xacro/generic_models.xacro" />
+    <xacro:include filename="$(find val_description)/model/robots/common/xacro/common_bodies.xacro" />
     <xacro:make_pelvis />
     <xacro:make_waist waist_root_link="${Pelvis_Link_Name}" />

File: model/robots/common/xacro/valkyrie_base_sim.xacro (robot description, xacro)
@@ -1,3 +1,6 @@
 <robot xmlns:xacro="http://ros.org/wiki/xacro" name="valkyrie">
+    <xacro:property name="mesh_root" value="package://val_description/model/meshes"/>
+    <xacro:include filename="$(find val_description)/model/robots/common/xacro/generic_models.xacro" />
+    <xacro:include filename="$(find val_description)/model/robots/common/xacro/common_bodies.xacro" />
     <xacro:make_pelvis />
     <xacro:make_waist waist_root_link="${Pelvis_Link_Name}" />

File: model/robots/common/xacro/waist/waist.xacro (robot description, xacro)
@@ -108,5 +108,5 @@
    <xacro:macro name="waist_transmissions_hw">
     <xacro:simple_transmission jointName="${TorsoYawJointName}" actuatorName="${TorsoYawActuatorName}" nodeName="${TrunkYawNode}" actuatorApi="${TrunkYawApi}"/>
-    <xacro:pushrod_transmission transmissionName="waistTransmission" transmissionType="TorsoPushrodTransmission" joint1Name="${TorsoPitchJointName}" joint2Name="${TorsoRollJointName}" joint1Role="pitch" joint2Role="roll" actuator1Name="${WaistRightActuatorName}" actuator2Name="${WaistLeftActuatorName}" actuator1Node="${WaistRightActuatorNode}" actuator2Node="${WaistLeftActuatorNode}" actuator1Api="${WaistRightActuatorApi}" actuator2Api="${WaistLeftActuatorApi}" actuator1Role="right" actuator2Role="left"/>
+    <xacro:pushrod_transmission transmissionName="waistTransmission" transmissionType="${TorsoTransmissionType}" joint1Name="${TorsoPitchJointName}" joint2Name="${TorsoRollJointName}" joint1Role="pitch" joint2Role="roll" actuator1Name="${WaistRightActuatorName}" actuator2Name="${WaistLeftActuatorName}" actuator1Node="${WaistRightActuatorNode}" actuator2Node="${WaistLeftActuatorNode}" actuator1Api="${WaistRightActuatorApi}" actuator2Api="${WaistLeftActuatorApi}" actuator1Role="right" actuator2Role="left"/>
    </xacro:macro>
    <xacro:macro name="waist_transmissions_sim">

File: model/robots/valkyrie_A.xacro (robot description, xacro)
@@ -1,6 +1,4 @@
 <robot xmlns:xacro="http://ros.org/wiki/xacro" name="valkyrie">
-    <xacro:property name="mesh_root" value="package://val_description/model/meshes"/>
-    <xacro:include filename="$(find val_description)/model/robots/common/xacro/generic_models.xacro" />
-    <xacro:include filename="$(find val_description)/model/robots/common/xacro/common_bodies.xacro" />
+    <xacro:include filename="$(find val_description)/model/robots/valkyrie_A_transmissions.xacro" />
     <xacro:include filename="$(find val_description)/model/robots/common/xacro/valkyrie_base_hw.xacro"/>
     <xacro:include filename="$(find val_description)/common/xacro/serial_numbers/valkyrie_A_serials.xacro"/>

File: model/robots/valkyrie_A_arm_mass_sims.xacro (robot description, xacro)
@@ -1,6 +1,4 @@
 <robot xmlns:xacro="http://ros.org/wiki/xacro" name="valkyrie">
-    <xacro:property name="mesh_root" value="package://val_description/model/meshes"/>
-    <xacro:include filename="$(find val_description)/model/robots/common/xacro/generic_models.xacro" />
-    <xacro:include filename="$(find val_description)/model/robots/common/xacro/common_bodies.xacro" />
+    <xacro:include filename="$(find val_description)/model/robots/valkyrie_A_transmissions.xacro" />
     <xacro:include filename="$(find val_description)/model/robots/common/xacro/valkyrie_arm_mass_sims_base_hw.xacro"/>
     <xacro:include filename="$(find val_description)/common/xacro/serial_numbers/valkyrie_A_serials.xacro"/>

File: model/robots/valkyrie_B.xacro (robot description, xacro)
@@ -1,6 +1,4 @@
 <robot xmlns:xacro="http://ros.org/wiki/xacro" name="valkyrie">
-    <xacro:property name="mesh_root" value="package://val_description/model/meshes"/>
-    <xacro:include filename="$(find val_description)/model/robots/common/xacro/generic_models.xacro" />
-    <xacro:include filename="$(find val_description)/model/robots/common/xacro/common_bodies.xacro" />
+    <xacro:include filename="$(find val_description)/model/robots/valkyrie_B_transmissions.xacro" />
     <xacro:include filename="$(find val_description)/model/robots/common/xacro/valkyrie_base_hw.xacro"/>
     <xacro:include filename="$(find val_description)/common/xacro/serial_numbers/valkyrie_B_serials.xacro"/>

File: model/robots/valkyrie_B_arm_mass_sims.xacro (robot description, xacro)
@@ -1,6 +1,4 @@
 <robot xmlns:xacro="http://ros.org/wiki/xacro" name="valkyrie">
-    <xacro:property name="mesh_root" value="package://val_description/model/meshes"/>
-    <xacro:include filename="$(find val_description)/model/robots/common/xacro/generic_models.xacro" />
-    <xacro:include filename="$(find val_description)/model/robots/common/xacro/common_bodies.xacro" />
+    <xacro:include filename="$(find val_description)/model/robots/valkyrie_B_transmissions.xacro" />
     <xacro:include filename="$(find val_description)/model/robots/common/xacro/valkyrie_arm_mass_sims_base_hw.xacro"/>
     <xacro:include filename="$(find val_description)/common/xacro/serial_numbers/valkyrie_B_serials.xacro"/>

File: model/robots/valkyrie_C.xacro (robot description, xacro)
@@ -1,6 +1,4 @@
 <robot xmlns:xacro="http://ros.org/wiki/xacro" name="valkyrie">
-    <xacro:property name="mesh_root" value="package://val_description/model/meshes"/>
-    <xacro:include filename="$(find val_description)/model/robots/common/xacro/generic_models.xacro" />
-    <xacro:include filename="$(find val_description)/model/robots/common/xacro/common_bodies.xacro" />
+    <xacro:include filename="$(find val_description)/model/robots/valkyrie_C_transmissions.xacro" />
     <xacro:include filename="$(find val_description)/model/robots/common/xacro/valkyrie_base_hw.xacro"/>
     <xacro:include filename="$(find val_description)/common/xacro/serial_numbers/valkyrie_C_serials.xacro"/>

File: model/robots/valkyrie_C_arm_mass_sims.xacro (robot description, xacro)
@@ -1,6 +1,4 @@
 <robot xmlns:xacro="http://ros.org/wiki/xacro" name="valkyrie">
-    <xacro:property name="mesh_root" value="package://val_description/model/meshes"/>
-    <xacro:include filename="$(find val_description)/model/robots/common/xacro/generic_models.xacro" />
-    <xacro:include filename="$(find val_description)/model/robots/common/xacro/common_bodies.xacro" />
+    <xacro:include filename="$(find val_description)/model/robots/valkyrie_C_transmissions.xacro" />
     <xacro:include filename="$(find val_description)/model/robots/common/xacro/valkyrie_arm_mass_sims_base_hw.xacro"/>
     <xacro:include filename="$(find val_description)/common/xacro/serial_numbers/valkyrie_C_serials.xacro"/>

File: model/robots/valkyrie_D.xacro (robot description, xacro)
@@ -1,6 +1,4 @@
 <robot xmlns:xacro="http://ros.org/wiki/xacro" name="valkyrie">
-    <xacro:property name="mesh_root" value="package://val_description/model/meshes"/>
-    <xacro:include filename="$(find val_description)/model/robots/common/xacro/generic_models.xacro" />
-    <xacro:include filename="$(find val_description)/model/robots/common/xacro/common_bodies.xacro" />
+    <xacro:include filename="$(find val_description)/model/robots/valkyrie_D_transmissions.xacro" />
     <xacro:include filename="$(find val_description)/model/robots/common/xacro/valkyrie_base_hw.xacro"/>
     <xacro:include filename="$(find val_description)/common/xacro/serial_numbers/valkyrie_D_serials.xacro"/>

File: model/robots/valkyrie_D_arm_mass_sims.xacro (robot description, xacro)
@@ -1,6 +1,4 @@
 <robot xmlns:xacro="http://ros.org/wiki/xacro" name="valkyrie">
-    <xacro:property name="mesh_root" value="package://val_description/model/meshes"/>
-    <xacro:include filename="$(find val_description)/model/robots/common/xacro/generic_models.xacro" />
-    <xacro:include filename="$(find val_description)/model/robots/common/xacro/common_bodies.xacro" />
+    <xacro:include filename="$(find val_description)/model/robots/valkyrie_D_transmissions.xacro" />
     <xacro:include filename="$(find val_description)/model/robots/common/xacro/valkyrie_arm_mass_sims_base_hw.xacro"/>
     <xacro:include filename="$(find val_description)/common/xacro/serial_numbers/valkyrie_D_serials.xacro"/>

File: model/robots/valkyrie_sim.xacro (robot description, xacro)
@@ -5,8 +5,5 @@
       </plugin>
     </gazebo>
-    <xacro:property name="mesh_root" value="package://val_description/model/meshes"/>
     <xacro:include filename="$(find val_description)/common/xacro/api/valkyrie_sim_api.xacro"/>
-    <xacro:include filename="$(find val_description)/model/robots/common/xacro/generic_models.xacro" />
-    <xacro:include filename="$(find val_description)/model/robots/common/xacro/common_bodies.xacro" />
     <xacro:include filename="$(find val_description)/model/urdf/multisense_sl.urdf" />
     <xacro:include filename="$(find val_description)/common/xacro/serial_numbers/valkyrie_A_serials.xacro"/>

File: model/robots/valkyrie_sim_arm_mass_sims.xacro (robot description, xacro)
@@ -5,8 +5,5 @@
       </plugin>
     </gazebo>
-    <xacro:property name="mesh_root" value="package://val_description/model/meshes"/>
     <xacro:include filename="$(find val_description)/common/xacro/api/valkyrie_sim_api.xacro"/>
-    <xacro:include filename="$(find val_description)/model/robots/common/xacro/generic_models.xacro" />
-    <xacro:include filename="$(find val_description)/model/robots/common/xacro/common_bodies.xacro" />
     <xacro:include filename="$(find val_description)/model/urdf/multisense_sl.urdf" />
     <xacro:include filename="$(find val_description)/common/xacro/serial_numbers/valkyrie_A_serials.xacro"/>

File: model/robots/valkyrie_sim_gazebo_sync.xacro (robot description, xacro)
@@ -6,8 +6,5 @@
       </plugin>
     </gazebo>
-    <xacro:property name="mesh_root" value="package://val_description/model/meshes"/>
     <xacro:include filename="$(find val_description)/common/xacro/api/valkyrie_sim_api.xacro"/>
-    <xacro:include filename="$(find val_description)/model/robots/common/xacro/generic_models.xacro" />
-    <xacro:include filename="$(find val_description)/model/robots/common/xacro/common_bodies.xacro" />
     <xacro:include filename="$(find val_description)/model/urdf/multisense_sl.urdf" />
     <xacro:include filename="$(find val_description)/common/xacro/serial_numbers/valkyrie_A_serials.xacro"/>
