Commit message: Abstracted out the sensor transforms so different robots can have different oriented sensors.

File: model/robots/common/xacro/gazebo_self_collide.xacro (robot description, xacro)
@@ -8,8 +8,8 @@
       <self_collide>false</self_collide>
     </gazebo>
-    <gazebo reference="leftHipRollLink">
+    <gazebo reference="leftHipYawLink">
       <self_collide>false</self_collide>
     </gazebo>
-    <gazebo reference="rightHipRollLink">
+    <gazebo reference="rightHipYawLink">
       <self_collide>false</self_collide>
     </gazebo>

File: model/robots/common/xacro/leg/leg.xacro (robot description, xacro)
@@ -49,5 +49,5 @@
                     height="0.16"
                     depth="0.064"
-                    box_xyz="0.066 0.0 -0.056"
+                    box_xyz="0.045 0.0 -0.056"
                     box_rpy="0.0 0.0 0.0" />
     <!-- foot contact parameters copied from atlas_description in drcsim -->

File: model/robots/common/xacro/pelvis/pelvis.xacro (robot description, xacro)
@@ -11,23 +11,13 @@
                         collision_mesh="${pelvis_mesh_dir}/pelvis.dae"/>
     </xacro:macro>
-    <xacro:macro name="v1_pelvis_sensors">
-        <xacro:microstrain_sensor sensorName="pelvisRearImu"
-                                  parentLink="${Pelvis_Link_Name}"
-                                  origin_xyz="-0.075844901 0.0 -0.111056426"
-                                  origin_rpy="-3.14159 0.476467 -3.14159" />
-        <xacro:microstrain_sensor sensorName="pelvisMiddleImu"
-                                  parentLink="${Pelvis_Link_Name}"
-                                  origin_xyz="0.150 0.0 0.08"
-                                  origin_rpy="0.0 0.0 0.7854" />
-    </xacro:macro>
     <xacro:macro name="v1_pelvis_middle_sensors_usb" params="sensor_node_tag sensor_api_tag sensor_port_tag">
         <xacro:microstrain_sensor sensorName="pelvisRearImu"
                                   parentLink="${Pelvis_Link_Name}"
-                                  origin_xyz="-0.075844901 0.0 -0.111056426"
-                                  origin_rpy="-3.14159 0.476467 -3.14159" />
+                                  origin_xyz="${PelvisRearImuFrameOrigin_XYZ}"
+                                  origin_rpy="${PelvisRearImuFrameOrientation_RPY}" />
         <xacro:usb_microstrain_sensor sensorName="pelvisMiddleImu"
                                   parentLink="${Pelvis_Link_Name}"
-                                  origin_xyz="0.0 0.0 -0.10819638"
-                                  origin_rpy="3.14159 0.0 0.0"
+                                  origin_xyz="${PelvisMiddleImuFrameOrigin_XYZ}"
+                                  origin_rpy="${PelvisMiddleImuFrameOrientation_RPY}"
                                   sensor_node="${sensor_node_tag}"
                                   sensor_api="${sensor_api_tag}"
@@ -37,6 +27,6 @@
         <xacro:usb_microstrain_sensor sensorName="pelvisRearImu"
                                   parentLink="${Pelvis_Link_Name}"
-                                  origin_xyz="-0.075844901 0.0 -0.111056426"
-                                  origin_rpy="-3.14159 0.476467 -3.14159"
+                                  origin_xyz="${PelvisRearImuFrameOrigin_XYZ}"
+                                  origin_rpy="${PelvisRearImuFrameOrientation_RPY}"
                         				  sensor_node="${sensor_node_tag}"
                         				  sensor_api="${sensor_api_tag}"
@@ -44,22 +34,6 @@
         <xacro:microstrain_sensor sensorName="pelvisMiddleImu"
                                   parentLink="${Pelvis_Link_Name}"
-                                  origin_xyz="0.0 0.0 -0.10819638"
-                                  origin_rpy="3.14159 0.0 0.0" />
-    </xacro:macro>
-    <xacro:macro name="v1_pelvis_sensors_usb" params="middle_sensor_node_tag middle_sensor_api_tag middle_sensor_port_tag rear_sensor_node_tag rear_sensor_api_tag rear_sensor_port_tag">
-        <xacro:usb_microstrain_sensor sensorName="pelvisRearImu"
-                                  parentLink="${Pelvis_Link_Name}"
-                                  origin_xyz="-0.075844901 0.0 -0.111056426"
-                                  origin_rpy="-3.14159 0.476467 -3.14159"
-                                  sensor_node="${rear_sensor_node_tag}"
-                                  sensor_api="${rear_sensor_api_tag}"
-                                  sensor_port="${rear_sensor_port_tag}" />
-        <xacro:usb_microstrain_sensor sensorName="pelvisMiddleImu"
-                                  parentLink="${Pelvis_Link_Name}"
-                                  origin_xyz="0.0 0.0 -0.10819638"
-                                  origin_rpy="3.14159 0.0 0.0"
-                                  sensor_node="${middle_sensor_node_tag}"
-                                  sensor_api="${middle_sensor_api_tag}"
-                                  sensor_port="${middle_sensor_port_tag}" />
+                                  origin_xyz="${PelvisMiddleImuFrameOrigin_XYZ}"
+                                  origin_rpy="${PelvisMiddleImuFrameOrientation_RPY}" />
     </xacro:macro>
 </robot>

File: model/robots/common/xacro/waist/waist.xacro (robot description, xacro)
@@ -56,27 +56,9 @@
     <xacro:make_waist_common waist_root_link="${waist_root_link}"/>
   </xacro:macro>
-  <xacro:macro name="v1_trunk_sensors">
-    <xacro:microstrain_sensor sensorName="leftTorsoImu"
-                              parentLink="${TorsoRollLinkName}"
-                              origin_xyz="-0.0627634 0.134239 0.3630676"
-                              origin_rpy="-1.5707 0.0 0.0" />
-    <xacro:flea3_camera sensorName="rightHazardCamera"
-                        parentLink="${TorsoRollLinkName}"
-                        origin_xyz="0.0345 -0.0406 0.1135"
-                        origin_rpy="1.57 0.0 1.57"
-                        imageFormat="R8G8B8"
-                        frameRate="60"/>
-    <xacro:flea3_camera sensorName="leftHazardCamera"
-                        parentLink="${TorsoRollLinkName}"
-                        origin_xyz="0.0345 0.0406 0.1135"
-                        origin_rpy="1.57 0.0 1.57"
-                        imageFormat="R8G8B8"
-                        frameRate="60"/>
-   </xacro:macro>
   <xacro:macro name="v1_trunk_sensors_usb" params="sensor_node_tag sensor_api_tag sensor_port_tag">
     <xacro:usb_microstrain_sensor sensorName="leftTorsoImu"
                               parentLink="${TorsoRollLinkName}"
-                              origin_xyz="-0.0627634 0.134239 0.3630676"
-                              origin_rpy="-1.5707 0.0 0.0"
+                              origin_xyz="${TorsoImuFrameOrigin_XYZ}"
+                              origin_rpy="${TorsoImuFrameOrientation_RPY}"
                               sensor_node="${sensor_node_tag}"
                               sensor_api="${sensor_api_tag}"

File: model/robots/valkyrie_A.xacro (robot description, xacro)
@@ -8,4 +8,5 @@
 	<xacro:include filename="$(find val_description)/model/robots/common/xacro/generic_models.xacro" />
     <xacro:include filename="$(find val_description)/common/xacro/nodes/valkyrie_nodes.xacro"/>
+    <xacro:include filename="$(find val_description)/model/robots/common/xacro/sensors/sensor_transforms.xacro"/>
     <xacro:include filename="$(find val_description)/model/robots/common/xacro/config/valkyrie_A_transmissions.xacro" />
 	<xacro:include filename="$(find val_description)/common/xacro/serial_numbers/valkyrie_A_serials.xacro"/>

File: model/robots/valkyrie_A_arm_mass_sims.xacro (robot description, xacro)
@@ -8,4 +8,5 @@
     <xacro:include filename="$(find val_description)/model/robots/common/xacro/generic_models.xacro" />
     <xacro:include filename="$(find val_description)/common/xacro/nodes/valkyrie_nodes.xacro"/>
+    <xacro:include filename="$(find val_description)/model/robots/common/xacro/sensors/sensor_transforms.xacro"/>
     <xacro:include filename="$(find val_description)/model/robots/common/xacro/config/valkyrie_A_transmissions.xacro" />
     <xacro:include filename="$(find val_description)/common/xacro/serial_numbers/valkyrie_A_serials.xacro"/>

File: model/robots/valkyrie_B.xacro (robot description, xacro)
@@ -8,4 +8,5 @@
 	<xacro:include filename="$(find val_description)/model/robots/common/xacro/generic_models.xacro" />
     <xacro:include filename="$(find val_description)/common/xacro/nodes/valkyrie_nodes.xacro"/>
+    <xacro:include filename="$(find val_description)/model/robots/common/xacro/sensors/sensor_transforms.xacro"/>
     <xacro:include filename="$(find val_description)/model/robots/common/xacro/config/valkyrie_B_transmissions.xacro" />
 	<xacro:include filename="$(find val_description)/common/xacro/serial_numbers/valkyrie_B_serials.xacro"/>

File: model/robots/valkyrie_B_arm_mass_sims.xacro (robot description, xacro)
@@ -8,4 +8,5 @@
     <xacro:include filename="$(find val_description)/model/robots/common/xacro/generic_models.xacro" />
     <xacro:include filename="$(find val_description)/common/xacro/nodes/valkyrie_nodes.xacro"/>
+    <xacro:include filename="$(find val_description)/model/robots/common/xacro/sensors/sensor_transforms.xacro"/>
     <xacro:include filename="$(find val_description)/model/robots/common/xacro/config/valkyrie_B_transmissions.xacro"/>
     <xacro:include filename="$(find val_description)/common/xacro/serial_numbers/valkyrie_B_serials.xacro"/>

File: model/robots/valkyrie_C.xacro (robot description, xacro)
@@ -8,4 +8,5 @@
 	<xacro:include filename="$(find val_description)/model/robots/common/xacro/generic_models.xacro" />
     <xacro:include filename="$(find val_description)/common/xacro/nodes/valkyrie_nodes.xacro"/>
+    <xacro:include filename="$(find val_description)/model/robots/common/xacro/sensors/sensor_transforms.xacro"/>
     <xacro:include filename="$(find val_description)/model/robots/common/xacro/config/valkyrie_C_transmissions.xacro" />
     <xacro:include filename="$(find val_description)/common/xacro/serial_numbers/valkyrie_C_serials.xacro"/>

File: model/robots/valkyrie_C_arm_mass_sims.xacro (robot description, xacro)
@@ -8,4 +8,5 @@
     <xacro:include filename="$(find val_description)/model/robots/common/xacro/generic_models.xacro" />
     <xacro:include filename="$(find val_description)/common/xacro/nodes/valkyrie_nodes.xacro"/>
+    <xacro:include filename="$(find val_description)/model/robots/common/xacro/sensors/sensor_transforms.xacro"/>
     <xacro:include filename="$(find val_description)/model/robots/common/xacro/config/valkyrie_C_transmissions.xacro" />
     <xacro:include filename="$(find val_description)/common/xacro/serial_numbers/valkyrie_C_serials.xacro"/>

File: model/robots/valkyrie_D.xacro (robot description, xacro)
@@ -8,4 +8,5 @@
 	<xacro:include filename="$(find val_description)/model/robots/common/xacro/generic_models.xacro" />
     <xacro:include filename="$(find val_description)/common/xacro/nodes/valkyrie_nodes.xacro"/>
+    <xacro:include filename="$(find val_description)/model/robots/common/xacro/sensors/sensor_transforms.xacro"/>
     <xacro:include filename="$(find val_description)/model/robots/common/xacro/config/valkyrie_D_transmissions.xacro" />
     <xacro:include filename="$(find val_description)/common/xacro/serial_numbers/valkyrie_D_serials.xacro"/>

File: model/robots/valkyrie_D_arm_mass_sims.xacro (robot description, xacro)
@@ -8,4 +8,5 @@
     <xacro:include filename="$(find val_description)/model/robots/common/xacro/generic_models.xacro" />
     <xacro:include filename="$(find val_description)/common/xacro/nodes/valkyrie_nodes.xacro"/>
+    <xacro:include filename="$(find val_description)/model/robots/common/xacro/sensors/sensor_transforms.xacro"/>
     <xacro:include filename="$(find val_description)/model/robots/common/xacro/config/valkyrie_D_transmissions.xacro" />
     <xacro:include filename="$(find val_description)/common/xacro/serial_numbers/valkyrie_D_serials.xacro"/>

File: model/robots/valkyrie_sim.xacro (robot description, xacro)
@@ -14,4 +14,5 @@
     <xacro:include filename="$(find val_description)/model/robots/common/xacro/generic_models.xacro" />
     <xacro:include filename="$(find val_description)/common/xacro/nodes/valkyrie_sim_nodes.xacro"/>
+    <xacro:include filename="$(find val_description)/model/robots/common/xacro/sensors/sensor_transforms.xacro"/>
     <xacro:include filename="$(find val_description)/common/xacro/api/valkyrie_sim_api.xacro"/>
     <xacro:include filename="$(find val_description)/model/urdf/multisense_sl.urdf" />

File: model/robots/valkyrie_sim_angled_legj1s.xacro (robot description, xacro)
@@ -14,4 +14,5 @@
     <xacro:include filename="$(find val_description)/model/robots/common/xacro/generic_models.xacro" />
     <xacro:include filename="$(find val_description)/common/xacro/nodes/valkyrie_sim_nodes.xacro"/>
+    <xacro:include filename="$(find val_description)/model/robots/common/xacro/sensors/angled_lj1s_sensor_transforms.xacro"/>
     <xacro:include filename="$(find val_description)/common/xacro/api/valkyrie_sim_api.xacro"/>
     <xacro:include filename="$(find val_description)/model/urdf/multisense_sl.urdf" />
@@ -34,4 +35,12 @@
     <xacro:include filename="$(find val_description)/model/robots/common/xacro/valkyrie_base_sim.xacro"/>
     <xacro:add_self_collide />
+    <!-- Until the pumpkin shells are replaced, this needs to be here or there will be lots of
+    unecessary contacts between the hip pitch link and the hip yaw link. -->
+    <gazebo reference="leftHipPitchLink">
+      <self_collide>false</self_collide>
+    </gazebo>
+    <gazebo reference="rightHipPitchLink">
+      <self_collide>false</self_collide>
+    </gazebo>
     <xacro:add_sim_harness harnessed_link="${TorsoRollLinkName}" />
 </robot>

File: model/robots/valkyrie_sim_arm_mass_sims.xacro (robot description, xacro)
@@ -12,4 +12,5 @@
     <xacro:include filename="$(find val_description)/model/robots/common/xacro/generic_models.xacro" />
     <xacro:include filename="$(find val_description)/common/xacro/nodes/valkyrie_sim_nodes.xacro"/>
+    <xacro:include filename="$(find val_description)/model/robots/common/xacro/sensors/sensor_transforms.xacro"/>
     <xacro:include filename="$(find val_description)/common/xacro/api/valkyrie_sim_api.xacro"/>
     <xacro:include filename="$(find val_description)/model/urdf/multisense_sl.urdf" />

File: model/robots/valkyrie_sim_gazebo_sync.xacro (robot description, xacro)
@@ -15,4 +15,5 @@
     <xacro:include filename="$(find val_description)/model/robots/common/xacro/generic_models.xacro" />
     <xacro:include filename="$(find val_description)/common/xacro/nodes/valkyrie_sim_nodes.xacro"/>
+    <xacro:include filename="$(find val_description)/model/robots/common/xacro/sensors/sensor_transforms.xacro"/>
     <xacro:include filename="$(find val_description)/common/xacro/api/valkyrie_sim_api.xacro"/>
     <xacro:include filename="$(find val_description)/model/urdf/multisense_sl.urdf" />
