Commit message: Lowered position control gains.

File: model/robots/common/xacro/gains.xacro (robot description, xacro)
@@ -1,20 +1,20 @@
 <robot xmlns:xacro="http://ros.org/wiki/xacro" name="valkyrie_nodes">
-    <xacro:property name="ForearmYawKp" value="20000" />
-    <xacro:property name="ForearmYawKd" value="400" />
+    <xacro:property name="ForearmYawKp" value="2000" />
+    <xacro:property name="ForearmYawKd" value="30" />
     <xacro:property name="ForearmYawKi" value="0.0" />
-    <xacro:property name="WristPitchKp" value="20000" />
-    <xacro:property name="WristPitchKd" value="400" />
+    <xacro:property name="WristPitchKp" value="2000" />
+    <xacro:property name="WristPitchKd" value="30" />
     <xacro:property name="WristPitchKi" value="0.0" />
-    <xacro:property name="WristRollKp" value="20000" />
-    <xacro:property name="WristRollKd" value="400" />
+    <xacro:property name="WristRollKp" value="2000" />
+    <xacro:property name="WristRollKd" value="30" />
     <xacro:property name="WristRollKi" value="0.0" />
-    <xacro:property name="LowerNeckPitchKp" value="20000" />
-    <xacro:property name="LowerNeckPitchKd" value="400" />
+    <xacro:property name="LowerNeckPitchKp" value="2000" />
+    <xacro:property name="LowerNeckPitchKd" value="30" />
     <xacro:property name="LowerNeckPitchKi" value="0.0" />
-    <xacro:property name="NeckYawKp" value="20000" />
-    <xacro:property name="NeckYawKd" value="400" />
+    <xacro:property name="NeckYawKp" value="2000" />
+    <xacro:property name="NeckYawKd" value="30" />
     <xacro:property name="NeckYawKi" value="0.0" />
-    <xacro:property name="UpperNeckPitchKp" value="20000" />
-    <xacro:property name="UpperNeckPitchKd" value="400" />
+    <xacro:property name="UpperNeckPitchKp" value="2000" />
+    <xacro:property name="UpperNeckPitchKd" value="30" />
     <xacro:property name="UpperNeckPitchKi" value="0.0" />
 </robot>

Commit message: Modified position control gains from John Hsu's suggested values.

File: model/robots/common/xacro/gains.xacro (robot description, xacro)
@@ -1,20 +1,20 @@
 <robot xmlns:xacro="http://ros.org/wiki/xacro" name="valkyrie_nodes">
-    <xacro:property name="ForearmYawKp" value="2000" />
-    <xacro:property name="ForearmYawKd" value="30" />
+    <xacro:property name="ForearmYawKp" value="1000" />
+    <xacro:property name="ForearmYawKd" value="0.0" />
     <xacro:property name="ForearmYawKi" value="0.0" />
-    <xacro:property name="WristPitchKp" value="2000" />
-    <xacro:property name="WristPitchKd" value="30" />
+    <xacro:property name="WristPitchKp" value="500" />
+    <xacro:property name="WristPitchKd" value="0" />
     <xacro:property name="WristPitchKi" value="0.0" />
-    <xacro:property name="WristRollKp" value="2000" />
-    <xacro:property name="WristRollKd" value="30" />
+    <xacro:property name="WristRollKp" value="500" />
+    <xacro:property name="WristRollKd" value="0" />
     <xacro:property name="WristRollKi" value="0.0" />
-    <xacro:property name="LowerNeckPitchKp" value="2000" />
-    <xacro:property name="LowerNeckPitchKd" value="30" />
+    <xacro:property name="LowerNeckPitchKp" value="200" />
+    <xacro:property name="LowerNeckPitchKd" value="0" />
     <xacro:property name="LowerNeckPitchKi" value="0.0" />
-    <xacro:property name="NeckYawKp" value="2000" />
-    <xacro:property name="NeckYawKd" value="30" />
+    <xacro:property name="NeckYawKp" value="50" />
+    <xacro:property name="NeckYawKd" value="0" />
     <xacro:property name="NeckYawKi" value="0.0" />
-    <xacro:property name="UpperNeckPitchKp" value="2000" />
-    <xacro:property name="UpperNeckPitchKd" value="30" />
+    <xacro:property name="UpperNeckPitchKp" value="200" />
+    <xacro:property name="UpperNeckPitchKd" value="0" />
     <xacro:property name="UpperNeckPitchKi" value="0.0" />
 </robot>

Commit message: increase neck Kd gains to improve damping

File: model/robots/common/xacro/gains.xacro (robot description, xacro)
@@ -9,12 +9,12 @@
     <xacro:property name="WristRollKd" value="0" />
     <xacro:property name="WristRollKi" value="0.0" />
-    <xacro:property name="LowerNeckPitchKp" value="200" />
-    <xacro:property name="LowerNeckPitchKd" value="0" />
+    <xacro:property name="LowerNeckPitchKp" value="50" />
+    <xacro:property name="LowerNeckPitchKd" value="3" />
     <xacro:property name="LowerNeckPitchKi" value="0.0" />
     <xacro:property name="NeckYawKp" value="50" />
-    <xacro:property name="NeckYawKd" value="0" />
+    <xacro:property name="NeckYawKd" value="3" />
     <xacro:property name="NeckYawKi" value="0.0" />
-    <xacro:property name="UpperNeckPitchKp" value="200" />
-    <xacro:property name="UpperNeckPitchKd" value="0" />
+    <xacro:property name="UpperNeckPitchKp" value="50" />
+    <xacro:property name="UpperNeckPitchKd" value="3" />
     <xacro:property name="UpperNeckPitchKi" value="0.0" />
     <xacro:property name="ThumbRollKp" value="5.0" />

Commit message: updating neck gains to prevent neck droop

File: model/robots/common/xacro/gains.xacro (robot description, xacro)
@@ -11,5 +11,5 @@
     <xacro:property name="LowerNeckPitchKp" value="50" />
     <xacro:property name="LowerNeckPitchKd" value="3" />
-    <xacro:property name="LowerNeckPitchKi" value="0.0" />
+    <xacro:property name="LowerNeckPitchKi" value="3" />
     <xacro:property name="NeckYawKp" value="50" />
     <xacro:property name="NeckYawKd" value="3" />
