Commit message: Reconfigured how the transmission types get into the URDF.

File: model/robots/common/xacro/generic_models.xacro (robot description, xacro)
@@ -240,5 +240,5 @@
   <xacro:macro name="pushrod_transmission" params="transmissionName transmissionType joint1Name joint2Name joint1Role joint2Role actuator1Name actuator2Name actuator1Node actuator2Node actuator1Api actuator2Api actuator1Role actuator2Role">
     <transmission name="${transmissionName}">
-      <type>robot_transmission_interface/${transmissionType}</type>
+      <type>${transmissionType}</type>
       <joint name="${joint1Name}">
         <role>${joint1Role}</role>

File: model/robots/common/xacro/leg/leg.xacro (robot description, xacro)
@@ -166,5 +166,5 @@
     <xacro:simple_transmission jointName="${HipPitchJointName}" actuatorName="${HipPitchActuatorName}" nodeName="${HipPitchNode}" actuatorApi="${HipPitchApi}"/>
     <xacro:simple_transmission jointName="${KneePitchJointName}" actuatorName="${KneePitchActuatorName}" nodeName="${KneePitchNode}" actuatorApi="${KneePitchApi}"/>
-    <xacro:pushrod_transmission transmissionName="${prefix}AnkleTransmission" transmissionType="AnklePushrodTransmission" joint1Name="${AnklePitchJointName}" joint2Name="${AnkleRollJointName}" joint1Role="pitch" joint2Role="roll" actuator1Name="${AnkleRightActuatorName}" actuator2Name="${AnkleLeftActuatorName}" actuator1Node="${AnkleRightActuatorNode}" actuator2Node="${AnkleLeftActuatorNode}" actuator1Api="${AnkleRightActuatorApi}" actuator2Api="${AnkleLeftActuatorApi}" actuator1Role="right" actuator2Role="left"/>
+    <xacro:pushrod_transmission transmissionName="${prefix}AnkleTransmission" transmissionType="${AnkleTransmissionType}" joint1Name="${AnklePitchJointName}" joint2Name="${AnkleRollJointName}" joint1Role="pitch" joint2Role="roll" actuator1Name="${AnkleRightActuatorName}" actuator2Name="${AnkleLeftActuatorName}" actuator1Node="${AnkleRightActuatorNode}" actuator2Node="${AnkleLeftActuatorNode}" actuator1Api="${AnkleRightActuatorApi}" actuator2Api="${AnkleLeftActuatorApi}" actuator1Role="right" actuator2Role="left"/>
   </xacro:macro>
   <xacro:macro name="leg_transmissions_sim" params="prefix">

File: model/robots/valkyrie_A_transmissions.xacro (robot description, xacro)
@@ -1,6 +1,5 @@
 <?xml version="1.0" ?>
 <robot name="valkyrie_transmissions" xmlns:xacro="http://www.ros.org/wiki/xacro">
-	<xacro:property name="TorsoTransmissionType" value="TorsoPushrodTransmissionWithOutputVelocity"/>
-	<xacro:property name="leftAnkleTransmissionType" value="AnklePushrodTransmission"/>
-	<xacro:property name="rightAnkleTransmissionType" value="AnklePushrodTransmission"/>
+	<xacro:property name="TorsoTransmissionType" value="robot_transmission_interface::TorsoPushrodTransmissionWithOutputVelocityLoader"/>
+	<xacro:property name="AnkleTransmissionType" value="robot_transmission_interface::AnklePushrodTransmissionLoader"/>
 </robot>

File: model/robots/valkyrie_B_transmissions.xacro (robot description, xacro)
@@ -1,6 +1,5 @@
 <?xml version="1.0" ?>
 <robot name="valkyrie_transmissions" xmlns:xacro="http://www.ros.org/wiki/xacro">
-	<xacro:property name="TorsoTransmissionType" value="TorsoPushrodTransmission"/>
-	<xacro:property name="leftAnkleTransmissionType" value="AnklePushrodTransmission"/>
-	<xacro:property name="rightAnkleTransmissionType" value="AnklePushrodTransmission"/>
+	<xacro:property name="TorsoTransmissionType" value="robot_transmission_interface::TorsoPushrodTransmissionLoader"/>
+	<xacro:property name="AnkleTransmissionType" value="robot_transmission_interface::AnklePushrodTransmissionLoader"/>
 </robot>

Commit message: Adding stuff for thumb transmissions to work in sim.

File: model/robots/common/xacro/generic_models.xacro (robot description, xacro)
@@ -225,4 +225,29 @@
     </transmission>
   </xacro:macro>
+  <xacro:macro name="finger_transmission" params="joint1Name actuatorName node1Name actuatorApi joint2Name joint3Name ratio1 ratio2 node2Name node3Name">
+    <transmission name="${joint1Name}Transmission">
+      <type>transmission_interface/SimpleTransmission</type>
+      <joint name="${joint1Name}">
+        <hardwareInterface>PositionJointInterface</hardwareInterface>
+      </joint>
+      <actuator name="${actuatorName}">
+        <node name="${nodeName}"/>
+        <mechanicalReduction>1</mechanicalReduction>
+        <api name="${actuatorApi}" />
+      </actuator>
+      <children>
+        <joint name="${joint2Name}" ratio="${ratio1}" parent="${joint1Name}" childNode="${node2Name}"/>
+        <joint name="${joint3Name}" ratio="${ratio2}" parent="${joint1Name}" childNode="${node3Name}"/>
+      </children>
+    </transmission>
+  </xacro:macro>
+  <xacro:macro name="simple_passive_transmission" params="jointName nodeName">
+    <transmission name="${jointName}PassiveTransmission">
+      <type>transmission_interface/SimpleTransmission</type>
+      <joint name="${jointName}">
+      </joint>
+      <node>${nodeName}</node>
+    </transmission>
+  </xacro:macro>
   <xacro:macro name="simple_forearm_position_transmission" params="jointName actuatorName nodeName actuatorApi reflect">
     <transmission name="${jointName}Transmission">

File: model/robots/common/xacro/thumb/thumb.xacro (robot description, xacro)
@@ -7,4 +7,5 @@
   <xacro:include filename="$(find val_description)/model/robots/common/xacro/thumb/frame_parameters.xacro"/>
   <xacro:include filename="$(find val_description)/model/robots/common/xacro/thumb/mass_parameters.xacro"/>
+  <xacro:include filename="$(find val_description)/model/robots/common/xacro/thumb/mechanical_info.xacro"/>
   <xacro:macro name="make_thumb" params="prefix reflect thumb_root_link">
     <xacro:standard_link name="${ThumbRollLinkName}"
@@ -90,3 +91,9 @@
     <xacro:simple_forearm_position_transmission jointName="${ThumbPitch3JointName}" actuatorName="${prefix}ThumbPitch3Actuator" nodeName="${ThumbPitch3Node}" actuatorApi="${ThumbFingerApi}" reflect="${reflect}"/>
   </xacro:macro>
+  <xacro:macro name="thumb_transmissions_sim" params="prefix">
+    <xacro:simple_position_transmission jointName="${ThumbRollJointName}" actuatorName="${prefix}ThumbRollActuator" nodeName="${ThumbRollNode}" actuatorApi="${ThumbFingerApi}"/>
+    <xacro:finger_transmission joint1Name="${ThumbPitch1JointName}" actuatorName="${prefix}ThumbPitch1Actuator" node1Name="${ThumbPitch1Node}" actuatorApi="${ThumbFingerApi}" joint2Name="${ThumbPitch2JointName}" joint3Name="${ThumbPitch3JointName}" ratio1="${Pulley2Ratio}" ratio2="${Pulley3Ratio}" node2Name="${ThumbPitch2Node}" node3Name="${ThumbPitch3Node}" />
+    <xacro:simple_passive_transmission jointName="${ThumbPitch2JointName}" nodeName="${ThumbPitch2Node}"/>
+    <xacro:simple_passive_transmission jointName="${ThumbPitch3JointName}" nodeName="${ThumbPitch3Node}"/>
+  </xacro:macro>
 </robot>

File: model/robots/common/xacro/valkyrie_base_sim.xacro (robot description, xacro)
@@ -26,3 +26,5 @@
     <xacro:arm_transmissions_sim prefix="right"/>
     <xacro:neck_transmissions_sim />
+    <xacro:thumb_transmissions_sim prefix="left"/>
+    <xacro:thumb_transmissions_sim prefix="right"/>
 </robot>

Commit message: Have fingers working in sim.

File: model/robots/common/xacro/generic_models.xacro (robot description, xacro)
@@ -225,5 +225,5 @@
     </transmission>
   </xacro:macro>
-  <xacro:macro name="simple_transmission_with_child_joints" params="jointName actuatorName nodeName actuatorApi child1JointName child1Ratio child2JointName child2Ratio">
+  <xacro:macro name="simple_transmission_with_two_child_joints" params="jointName actuatorName nodeName actuatorApi child1JointName child1Ratio child2JointName child2Ratio">
     <transmission name="${jointName}Transmission">
       <type>transmission_interface/SimpleTransmission</type>

File: model/robots/common/xacro/index_finger/index_finger.xacro (robot description, xacro)
@@ -79,5 +79,5 @@
   </xacro:macro>
   <xacro:macro name="index_finger_transmissions_sim" params="prefix">
-    <xacro:simple_transmission_with_child_joints jointName="${IndexFingerPitch1JointName}" actuatorName="${prefix}IndexFingerPitch1Actuator" nodeName="${IndexFingerPitch1Node}" actuatorApi="${SimApi}" child1JointName="${IndexFingerPitch2JointName}" child1Ratio="${Pulley2Ratio}" child2JointName="${IndexFingerPitch3JointName}" child2Ratio="${Pulley3Ratio}"/>
+    <xacro:simple_transmission_with_two_child_joints jointName="${IndexFingerPitch1JointName}" actuatorName="${prefix}IndexFingerPitch1Actuator" nodeName="${IndexFingerPitch1Node}" actuatorApi="${SimApi}" child1JointName="${IndexFingerPitch2JointName}" child1Ratio="${Pulley2Ratio}" child2JointName="${IndexFingerPitch3JointName}" child2Ratio="${Pulley3Ratio}"/>
     <xacro:simple_passive_transmission jointName="${IndexFingerPitch2JointName}" nodeName="${IndexFingerPitch2Node}" apiName="${SimApi}"/>
     <xacro:simple_passive_transmission jointName="${IndexFingerPitch3JointName}" nodeName="${IndexFingerPitch3Node}" apiName="${SimApi}"/>

File: model/robots/common/xacro/middle_finger/mechanical_info.xacro (robot description, xacro)
@@ -5,4 +5,4 @@
   <!-- Pulley-3 diameter = 0.01016 -->
   <xacro:property name="Pulley2Ratio" value="1.344" />
-  <xacro:property name="Pulley3Ratio" value="1.25" />
+  <xacro:property name="Pulley3Ratio" value="1.68" />
 </robot>

File: model/robots/common/xacro/middle_finger/middle_finger.xacro (robot description, xacro)
@@ -79,5 +79,5 @@
   </xacro:macro>
   <xacro:macro name="middle_finger_transmissions_sim" params="prefix">
-    <xacro:simple_transmission_with_child_joints jointName="${MiddleFingerPitch1JointName}" actuatorName="${prefix}MiddleFingerPitch1Actuator" nodeName="${MiddleFingerPitch1Node}" actuatorApi="${SimApi}" child1JointName="${MiddleFingerPitch2JointName}" child1Ratio="${Pulley2Ratio}" child2JointName="${MiddleFingerPitch3JointName}" child2Ratio="${Pulley3Ratio}"/>
+    <xacro:simple_transmission_with_two_child_joints jointName="${MiddleFingerPitch1JointName}" actuatorName="${prefix}MiddleFingerPitch1Actuator" nodeName="${MiddleFingerPitch1Node}" actuatorApi="${SimApi}" child1JointName="${MiddleFingerPitch2JointName}" child1Ratio="${Pulley2Ratio}" child2JointName="${MiddleFingerPitch3JointName}" child2Ratio="${Pulley3Ratio}"/>
     <xacro:simple_passive_transmission jointName="${MiddleFingerPitch2JointName}" nodeName="${MiddleFingerPitch2Node}" apiName="${SimApi}"/>
     <xacro:simple_passive_transmission jointName="${MiddleFingerPitch3JointName}" nodeName="${MiddleFingerPitch3Node}" apiName="${SimApi}"/>

File: model/robots/common/xacro/pinky_finger/mechanical_info.xacro (robot description, xacro)
@@ -5,4 +5,4 @@
   <!-- Pulley-3 diameter = 0.01016 -->
   <xacro:property name="Pulley2Ratio" value="1.344" />
-  <xacro:property name="Pulley3Ratio" value="1.25" />
+  <xacro:property name="Pulley3Ratio" value="1.68" />
 </robot>

File: model/robots/common/xacro/pinky_finger/pinky_finger.xacro (robot description, xacro)
@@ -79,5 +79,5 @@
   </xacro:macro>
   <xacro:macro name="pinky_transmissions_sim" params="prefix">
-    <xacro:simple_transmission_with_child_joints jointName="${PinkyPitch1JointName}" actuatorName="${prefix}PinkyPitch1Actuator" nodeName="${PinkyPitch1Node}" actuatorApi="${SimApi}" child1JointName="${PinkyPitch2JointName}" child1Ratio="${Pulley2Ratio}" child2JointName="${PinkyPitch3JointName}" child2Ratio="${Pulley3Ratio}"/>
+    <xacro:simple_transmission_with_two_child_joints jointName="${PinkyPitch1JointName}" actuatorName="${prefix}PinkyPitch1Actuator" nodeName="${PinkyPitch1Node}" actuatorApi="${SimApi}" child1JointName="${PinkyPitch2JointName}" child1Ratio="${Pulley2Ratio}" child2JointName="${PinkyPitch3JointName}" child2Ratio="${Pulley3Ratio}"/>
     <xacro:simple_passive_transmission jointName="${PinkyPitch2JointName}" nodeName="${PinkyPitch2Node}" apiName="${SimApi}"/>
     <xacro:simple_passive_transmission jointName="${PinkyPitch3JointName}" nodeName="${PinkyPitch3Node}" apiName="${SimApi}"/>

File: model/robots/common/xacro/thumb/mechanical_info.xacro (robot description, xacro)
@@ -5,4 +5,4 @@
   <!-- Pulley-3 diameter = 0.01016 -->
   <xacro:property name="Pulley2Ratio" value="1.344" />
-  <xacro:property name="Pulley3Ratio" value="1.25" />
+  <xacro:property name="Pulley3Ratio" value="1.68" />
 </robot>

File: model/robots/common/xacro/thumb/thumb.xacro (robot description, xacro)
@@ -98,5 +98,5 @@
   <xacro:macro name="thumb_transmissions_sim" params="prefix">
     <xacro:simple_position_transmission jointName="${ThumbRollJointName}" actuatorName="${prefix}ThumbRollActuator" nodeName="${ThumbRollNode}" actuatorApi="${SimApi}"/>
-    <xacro:simple_transmission_with_child_joints jointName="${ThumbPitch1JointName}" actuatorName="${prefix}ThumbPitch1Actuator" nodeName="${ThumbPitch1Node}" actuatorApi="${SimApi}" child1JointName="${ThumbPitch2JointName}" child1Ratio="${Pulley2Ratio}" child2JointName="${ThumbPitch3JointName}" child2Ratio="${Pulley3Ratio}"/>
+    <xacro:simple_transmission_with_two_child_joints jointName="${ThumbPitch1JointName}" actuatorName="${prefix}ThumbPitch1Actuator" nodeName="${ThumbPitch1Node}" actuatorApi="${SimApi}" child1JointName="${ThumbPitch2JointName}" child1Ratio="${Pulley2Ratio}" child2JointName="${ThumbPitch3JointName}" child2Ratio="${Pulley3Ratio}"/>
     <xacro:simple_passive_transmission jointName="${ThumbPitch2JointName}" nodeName="${ThumbPitch2Node}" apiName="${SimApi}"/>
     <xacro:simple_passive_transmission jointName="${ThumbPitch3JointName}" nodeName="${ThumbPitch3Node}" apiName="${SimApi}"/>

File: model/robots/common/xacro/valkyrie_base_sim.xacro (robot description, xacro)
@@ -28,3 +28,10 @@
     <xacro:neck_transmissions_sim />
     <xacro:thumb_transmissions_sim prefix="left"/>
+    <xacro:thumb_transmissions_sim prefix="right"/>
+    <xacro:index_finger_transmissions_sim prefix="left"/>
+    <xacro:index_finger_transmissions_sim prefix="right"/>
+    <xacro:middle_finger_transmissions_sim prefix="left"/>
+    <xacro:middle_finger_transmissions_sim prefix="right"/>
+    <xacro:pinky_transmissions_sim prefix="left"/>
+    <xacro:pinky_transmissions_sim prefix="right"/>
 </robot>

File: model/robots/forearm_sim.xacro (robot description, xacro)
@@ -38,11 +38,10 @@
     </link>
     <xacro:make_thumb prefix="left" reflect="1" thumb_root_link="leftPalm"/>
-    <xacro:make_index_finger prefix="left" reflect="1" index_finger_root_link="leftPalm"/>
+    <!-- <xacro:make_index_finger prefix="left" reflect="1" index_finger_root_link="leftPalm"/>
     <xacro:make_middle_finger prefix="left" reflect="1" middle_finger_root_link="leftPalm"/>
-    <xacro:make_pinky_finger prefix="left" reflect="1" pinky_finger_root_link="leftPalm"/>
+    <xacro:make_pinky_finger prefix="left" reflect="1" pinky_finger_root_link="leftPalm"/> -->
     <xacro:thumb_transmissions_sim prefix="left"/>
-    <xacro:index_finger_transmissions_sim prefix="left"/>
+    <!-- <xacro:index_finger_transmissions_sim prefix="left"/>
     <xacro:middle_finger_transmissions_sim prefix="left"/>
-    <xacro:pinky_transmissions_sim prefix="left"/>
-    <xacro:add_sim_harness harnessed_link="leftPalm" />
+    <xacro:pinky_transmissions_sim prefix="left"/> -->
 </robot>

File: model/robots/tmp/valkyrie_sim.xacro (robot description, xacro)
@@ -5,4 +5,5 @@
       </plugin>
     </gazebo>
+    <schedule_topic_creator_file package="val_gazebo" relative_file_path="/configuration/valkyrie_sim_shm_topics.yaml"/>
     <xacro:property name="mesh_root" value="package://val_description/model/meshes"/>
     <xacro:include filename="$(find val_description)/common/xacro/api/valkyrie_sim_api.xacro"/>

File: model/robots/tmp/valkyrie_sim_gazebo_sync.xacro (robot description, xacro)
@@ -6,4 +6,5 @@
       </plugin>
     </gazebo>
+    <schedule_topic_creator_file package="val_gazebo" relative_file_path="/configuration/valkyrie_sim_shm_topics.yaml"/>
     <xacro:property name="mesh_root" value="package://val_description/model/meshes"/>
     <xacro:include filename="$(find val_description)/common/xacro/api/valkyrie_sim_api.xacro"/>

Commit message: Working on j1/j2 meshes.

File: model/robots/common/xacro/generic_models.xacro (robot description, xacro)
@@ -24,4 +24,15 @@
     </link>
   </xacro:macro>
+  <xacro:macro name="link_no_mesh_no_collision" params="name mass origin_rpy origin_xyz ixx ixy ixz iyy iyz izz">
+    <link name="${name}">
+      <inertial>
+        <mass value="${mass}"/>
+        <origin rpy="${origin_rpy}" xyz="${origin_xyz}"/>
+        <inertia ixx="${ixx}" ixy="${ixy}" ixz="${ixz}"
+                 iyy="${iyy}" iyz="${iyz}"
+                 izz="${izz}" />
+        </inertial>
+    </link>
+  </xacro:macro>
   <xacro:macro name="link_no_mesh" params="name width height depth mass origin_xyz origin_rpy ixx ixy ixz iyy iyz izz">
     <link name="${name}">

File: model/robots/common/xacro/leg/leg.xacro (robot description, xacro)
@@ -9,5 +9,5 @@
                     visual_mesh="${leg_mesh_dir}/lj1_${prefix}.dae"
                     collision_mesh="${leg_mesh_dir}/lj1_${prefix}.dae"/>
-    <xacro:standard_link name="${HipRollLinkName}"
+    <!-- <xacro:standard_link name="${HipRollLinkName}"
                     mass="${HipRollLinkMass}"
                     origin_xyz="${HipRollLinkComPosition}"
@@ -16,5 +16,11 @@
                     origin_rpy="0 0 0"
                     visual_mesh="${leg_mesh_dir}/lj2_${prefix}.dae"
-                    collision_mesh="${leg_mesh_dir}/lj2_${prefix}.dae"/>
+                    collision_mesh="${leg_mesh_dir}/lj2_${prefix}.dae"/> -->
+    <xacro:link_no_mesh_no_collision name="${HipRollLinkName}"
+                    mass="${HipRollLinkMass}"
+                    origin_xyz="${HipRollLinkComPosition}"
+                    ixx="${HipRollLinkInertia_IXX}" ixy="${HipRollLinkInertia_IXY}" ixz="${HipRollLinkInertia_IXZ}"
+                    iyy="${HipRollLinkInertia_IYY}" iyz="${HipRollLinkInertia_IYZ}" izz="${HipRollLinkInertia_IZZ}"
+                    origin_rpy="0 0 0"/>
     <xacro:standard_link name="${HipPitchLinkName}"
                     mass="${HipPitchLinkMass}"

Commit message: screw it, disconnecting that pulley and exposing empty interface until I figure out what to do with it

File: model/robots/common/xacro/generic_models.xacro (robot description, xacro)
@@ -312,9 +312,10 @@
     </transmission>
   </xacro:macro>
-  <xacro:macro name="simple_effort_transmission_two_actuator" params="jointName actuatorName nodeName actuatorApi childActuator">
-    <transmission name="${jointName}Transmission">
-      <type>transmission_interface/SimpleTransmission</type>
-      <joint name="${jointName}">
-        <hardwareInterface>EffortJointInterface</hardwareInterface>
+  <xacro:macro name="simple_effort_transmission_two_actuator" params="jointName actuatorName nodeName actuatorApi childActuator child1JointName child1Ratio">
+    <transmission name="${jointName}Transmission">
+      <type>transmission_interface/SimpleTransmission</type>
+      <joint name="${jointName}">
+        <hardwareInterface>EffortJointInterface</hardwareInterface>
+        <child name="${child1JointName}" ratio="${child1Ratio}"/>
       </joint>
       <actuator name="${actuatorName}">
@@ -326,5 +327,5 @@
     </transmission>
   </xacro:macro>
-  <xacro:macro name="simple_effort_transmission_two_actuator_three_joint" params="jointName actuatorName nodeName actuatorApi child1JointName child1Ratio child2JointName child2Ratio">
+  <xacro:macro name="simple_effort_transmission_two_actuator_three_joint" params="jointName actuatorName nodeName actuatorApi childActuator child1JointName child1Ratio child2JointName child2Ratio child3JointName child3Ratio">
     <transmission name="${jointName}Transmission">
       <type>transmission_interface/SimpleTransmission</type>
@@ -333,4 +334,5 @@
         <child name="${child1JointName}" ratio="${child1Ratio}"/>
         <child name="${child2JointName}" ratio="${child2Ratio}"/>
+        <child name="${child3JointName}" ratio="${child3Ratio}"/>
       </joint>
       <actuator name="${actuatorName}">

File: model/robots/common/xacro/thumb/thumb.xacro (robot description, xacro)
@@ -104,4 +104,5 @@
   <xacro:macro name="thumb_transmissions_sim" params="prefix">
     <xacro:simple_effort_transmission_with_one_child_joint jointName="${prefix}${ThumbRollActuatorName}" actuatorName="${prefix}${ThumbRollActuatorName}" nodeName="/${prefix}${ThumbRollNode}" actuatorApi="${SimApi}" child1JointName="${prefix}${ThumbRollJointName}" child1Ratio="1"/>
+    <xacro:simple_transmission jointName="${prefix}${ThumbPitch1ActuatorName}" actuatorName="${prefix}${ThumbPitch1ActuatorName}" nodeName="/${prefix}${ThumbProximalNode}" actuatorApi="${SimApi}" />
     <xacro:simple_effort_transmission_with_three_child_joints jointName="${prefix}${ThumbPitch2ActuatorName}" actuatorName="${prefix}${ThumbPitch2ActuatorName}" nodeName="/${prefix}${ThumbDistalNode}" actuatorApi="${SimApi}" child1JointName="${prefix}${ThumbPitch1JointName}" child1Ratio="${Pulley1Ratio}" child2JointName="${prefix}${ThumbPitch2JointName}" child2Ratio="${Pulley2Ratio}" child3JointName="${prefix}${ThumbPitch3JointName}" child3Ratio="${Pulley3Ratio}"/>
     <xacro:simple_passive_transmission jointName="${prefix}${ThumbRollJointName}" nodeName="/${prefix}${ThumbRollSenseNode}" apiName="${SimApi}" reflect="1"/>
