Commit message: cleaning up some unused transmission models

File: model/robots/common/xacro/generic_models.xacro (robot description, xacro)
@@ -312,36 +312,4 @@
     </transmission>
   </xacro:macro>
-  <xacro:macro name="simple_effort_transmission_two_actuator" params="jointName actuatorName nodeName actuatorApi childActuator child1JointName child1Ratio">
-    <transmission name="${jointName}Transmission">
-      <type>transmission_interface/SimpleTransmission</type>
-      <joint name="${jointName}">
-        <hardwareInterface>EffortJointInterface</hardwareInterface>
-        <child name="${child1JointName}" ratio="${child1Ratio}"/>
-      </joint>
-      <actuator name="${actuatorName}">
-        <node name="${nodeName}"/>
-        <mechanicalReduction>1</mechanicalReduction>
-        <api name="${actuatorApi}" />
-        <child name="${childActuator}" />
-      </actuator>
-    </transmission>
-  </xacro:macro>
-  <xacro:macro name="simple_effort_transmission_two_actuator_three_joint" params="jointName actuatorName nodeName actuatorApi childActuator child1JointName child1Ratio child2JointName child2Ratio child3JointName child3Ratio">
-    <transmission name="${jointName}Transmission">
-      <type>transmission_interface/SimpleTransmission</type>
-      <joint name="${jointName}">
-        <hardwareInterface>EffortJointInterface</hardwareInterface>
-        <child name="${child1JointName}" ratio="${child1Ratio}"/>
-        <child name="${child2JointName}" ratio="${child2Ratio}"/>
-        <child name="${child3JointName}" ratio="${child3Ratio}"/>
-      </joint>
-      <actuator name="${actuatorName}">
-        <node name="${nodeName}"/>
-        <mechanicalReduction>1</mechanicalReduction>
-        <api name="${actuatorApi}" />
-        <child name="${childActuator}" />
-      </actuator>
-    </transmission>
-  </xacro:macro>
   <xacro:macro name="simple_passive_transmission" params="jointName nodeName apiName reflect">
     <transmission name="${jointName}PassiveTransmission">
@@ -420,59 +388,3 @@
     </transmission>
   </xacro:macro>
-  <xacro:macro name="athena1_transmission" params="prefix transmissionName actuatorApi nodeName">
-    <transmission name="${transmissionName}">
-      <type>robot_transmission_interface/AthenaForearmTransmission</type>
-      <joint name="${prefix}WristPitch">
-        <role>wristPitch</role>
-        <hardwareInterface>PositionJointInterface</hardwareInterface>
-      </joint>
-      <joint name="${prefix}WristRoll">
-        <role>wristRoll</role>
-        <hardwareInterface>PositionJointInterface</hardwareInterface>
-      </joint>
-      <joint name="${prefix}ThumbMotorRoll">
-        <role>thumbRoll</role>
-        <hardwareInterface>PositionJointInterface</hardwareInterface>
-      </joint>
-      <joint name="${prefix}ThumbMotorPitch1">
-        <role>thumbPitch1</role>
-        <hardwareInterface>PositionJointInterface</hardwareInterface>
-      </joint>
-      <actuator name="${prefix}Athena1Actuator">
-        <role>athena1Actuator</role>
-        <node name="${nodeName}"/>
-        <mechanicalReduction>1</mechanicalReduction>
-        <hardwareInterface>PositionJointInterface</hardwareInterface>
-        <api name="${actuatorApi}"/>
-      </actuator>
-    </transmission>
-  </xacro:macro>
-  <xacro:macro name="athena2_transmission" params="prefix transmissionName actuatorApi nodeName">
-    <transmission name="${transmissionName}">
-      <type>robot_transmission_interface/AthenaFingerTransmission</type>
-      <joint name="${prefix}ThumbMotorPitch2">
-        <role>thumbPitch2</role>
-        <hardwareInterface>PositionJointInterface</hardwareInterface>
-      </joint>
-      <joint name="${prefix}IndexFingerMotorPitch1">
-        <role>indexFingerPitch1</role>
-        <hardwareInterface>PositionJointInterface</hardwareInterface>
-      </joint>
-      <joint name="${prefix}MiddleFingerMotorPitch1">
-        <role>middleFingerPitch1</role>
-        <hardwareInterface>PositionJointInterface</hardwareInterface>
-      </joint>
-      <joint name="${prefix}PinkyMotorPitch1">
-        <role>pinkyPitch1</role>
-        <hardwareInterface>PositionJointInterface</hardwareInterface>
-      </joint>
-      <actuator name="${prefix}Athena2Actuator">
-        <role>athena2Actuator</role>
-        <node name="${nodeName}"/>
-        <mechanicalReduction>1</mechanicalReduction>
-        <hardwareInterface>PositionJointInterface</hardwareInterface>
-        <api name="${actuatorApi}"/>
-      </actuator>
-    </transmission>
-  </xacro:macro>
 </robot>

Commit message: removing unused transmission definitions to prevent confusion

File: model/robots/common/xacro/generic_models.xacro (robot description, xacro)
@@ -266,34 +266,4 @@
     </transmission>
   </xacro:macro>
-  <xacro:macro name="simple_transmission_with_two_child_joints" params="jointName actuatorName nodeName actuatorApi child1JointName child1Ratio child2JointName child2Ratio">
-    <transmission name="${jointName}Transmission">
-      <type>transmission_interface/SimpleTransmission</type>
-      <joint name="${jointName}">
-        <hardwareInterface>PositionJointInterface</hardwareInterface>
-        <child name="${child1JointName}" ratio="${child1Ratio}"/>
-        <child name="${child2JointName}" ratio="${child2Ratio}"/>
-      </joint>
-      <actuator name="${actuatorName}">
-        <node name="${nodeName}"/>
-        <mechanicalReduction>1</mechanicalReduction>
-        <api name="${actuatorApi}" />
-      </actuator>
-    </transmission>
-  </xacro:macro>
-  <xacro:macro name="simple_position_transmission_with_three_child_joints" params="jointName actuatorName nodeName actuatorApi child1JointName child1Ratio child2JointName child2Ratio">
-    <transmission name="${jointName}Transmission">
-      <type>transmission_interface/SimpleTransmission</type>
-      <joint name="${jointName}">
-        <hardwareInterface>PositionJointInterface</hardwareInterface>
-        <child name="${child1JointName}" ratio="${child1Ratio}"/>
-        <child name="${child2JointName}" ratio="${child2Ratio}"/>
-      </joint>
-      <actuator name="${actuatorName}">
-        <node name="${nodeName}"/>
-        <mechanicalReduction>1</mechanicalReduction>
-        <api name="${actuatorApi}" />
-      </actuator>
-    </transmission>
-  </xacro:macro>
   <xacro:macro name="simple_effort_transmission_with_three_child_joints" params="jointName actuatorName nodeName actuatorApi child1JointName child1Ratio child2JointName child2Ratio child3JointName child3Ratio">
     <transmission name="${jointName}Transmission">

Commit message: use massless link for virtual frame leftFootCenter and Corners

File: model/robots/common/xacro/generic_models.xacro (robot description, xacro)
@@ -278,4 +278,13 @@
                        origin_xyz="${origin_xyz}"/>
   </xacro:macro>
+  <xacro:macro name="massless_virtual_fixed_frame_offset" params="name parentLink origin_xyz origin_rpy">
+    <xacro:massless_virtual_link name="${name}_Frame"
+                    origin_rpy="0 0 0"
+                    origin_xyz="0 0 0"/>
+    <xacro:fixed_joint jointName="${name}_Offset"
+                       parent="${parentLink}" child="${name}_Frame"
+                       origin_rpy="${origin_rpy}"
+                       origin_xyz="${origin_xyz}"/>
+  </xacro:macro>
   <xacro:macro name="simple_transmission" params="jointName actuatorName nodeName actuatorApi">
     <transmission name="${jointName}Transmission">

File: model/robots/common/xacro/leg/leg.xacro (robot description, xacro)
@@ -137,25 +137,25 @@
   </xacro:macro>
   <xacro:macro name="v1_leg_sensors" params="prefix reflect ATI_serial_number ATI_node">
-    <xacro:virtual_fixed_frame_offset name="${prefix}COP"
+    <xacro:massless_virtual_fixed_frame_offset name="${prefix}COP"
                        parentLink="${prefix}Foot"
                        origin_xyz="0.0189 0.0 -0.0783"
                        origin_rpy="0.0 0.0 0.0"/>
-    <xacro:virtual_fixed_frame_offset name="${prefix}FootCenter"
+    <xacro:massless_virtual_fixed_frame_offset name="${prefix}FootCenter"
                        parentLink="${prefix}Foot"
                        origin_xyz="0.045 0.0 -0.088"
                        origin_rpy="0.0 0.0 0.0"/>
-    <xacro:virtual_fixed_frame_offset name="${prefix}FootCorner1"
+    <xacro:massless_virtual_fixed_frame_offset name="${prefix}FootCorner1"
                        parentLink="${prefix}Foot"
                        origin_xyz="0.17 0.07 -0.088"
                        origin_rpy="0.0 0.0 0.0"/>
-    <xacro:virtual_fixed_frame_offset name="${prefix}FootCorner2"
+    <xacro:massless_virtual_fixed_frame_offset name="${prefix}FootCorner2"
                        parentLink="${prefix}Foot"
                        origin_xyz="0.17 -0.07 -0.088"
                        origin_rpy="0.0 0.0 0.0"/>
-    <xacro:virtual_fixed_frame_offset name="${prefix}FootCorner3"
+    <xacro:massless_virtual_fixed_frame_offset name="${prefix}FootCorner3"
                        parentLink="${prefix}Foot"
                        origin_xyz="-0.08 -0.07 -0.088"
                        origin_rpy="0.0 0.0 0.0"/>
-    <xacro:virtual_fixed_frame_offset name="${prefix}FootCorner4"
+    <xacro:massless_virtual_fixed_frame_offset name="${prefix}FootCorner4"
                        parentLink="${prefix}Foot"
                        origin_xyz="-0.08 0.07 -0.088"

Commit message: Remove collision in simulation for hip yaw meshes

File: model/robots/common/xacro/generic_models.xacro (robot description, xacro)
@@ -22,4 +22,21 @@
         <origin rpy="0 0 0" xyz="0 0 0"/>
       </collision>
+    </link>
+  </xacro:macro>
+  <xacro:macro name="standard_link_no_collision" params="name mass origin_rpy origin_xyz ixx ixy ixz iyy iyz izz visual_mesh">
+    <link name="${name}">
+      <inertial>
+        <mass value="${mass}"/>
+        <origin rpy="${origin_rpy}" xyz="${origin_xyz}"/>
+        <inertia ixx="${ixx}" ixy="${ixy}" ixz="${ixz}"
+                 iyy="${iyy}" iyz="${iyz}"
+                 izz="${izz}" />
+        </inertial>
+        <visual>
+          <geometry>
+            <mesh filename="${visual_mesh}"/>
+          </geometry>
+          <origin rpy="0.0 0.0 0.0" xyz="0.0 0.0 0.0"/>
+        </visual>
     </link>
   </xacro:macro>

File: model/robots/common/xacro/leg/leg.xacro (robot description, xacro)
@@ -2,11 +2,10 @@
 <robot xmlns:xacro="http://www.ros.org/wiki/xacro" name="leg">
   <xacro:macro name="make_leg_links" params="prefix reflect leg_root_link">
-    <xacro:standard_link name="${prefix}HipYawLink"
+    <xacro:standard_link_no_collision name="${prefix}HipYawLink"
                     mass="${HipYawLinkMass}"
                     origin_xyz="0.02176 ${reflect*-0.00131} 0.03867" origin_rpy="0 0 0"
                     ixx="${HipYawLinkInertia_IXX}" ixy="${HipYawLinkInertia_IXY}" ixz="${HipYawLinkInertia_IXZ}"
                     iyy="${HipYawLinkInertia_IYY}" iyz="${HipYawLinkInertia_IYZ}" izz="${HipYawLinkInertia_IZZ}"
-                    visual_mesh="${leg_mesh_dir}/lj1_${prefix}.dae"
-                    collision_mesh="${leg_mesh_dir}/lj1_${prefix}.dae"/>
+                    visual_mesh="${leg_mesh_dir}/lj1_${prefix}.dae"/>
     <xacro:link_no_mesh_no_collision name="${prefix}HipRollLink"
                     mass="${HipRollLinkMass}"
