Commit message: New lj1_right dae file is good. Still kinda dark though.

File: model/robots/valkyrie_sim_angled_legj1s.xacro (robot description, xacro)
@@ -6,5 +6,5 @@
     </gazebo>
     <schedule_topic_creator_file package="val_gazebo" relative_file_path="/configuration/valkyrie_sim_shm_topics.yaml"/>
-    <xacro:property name="leg_mesh_dir" value="package://val_description/model/meshes/legs"/>
+    <xacro:property name="leg_mesh_dir" value="package://val_description/model/meshes/legs_angled_j1s"/>
     <xacro:property name="arm_mesh_dir" value="package://val_description/model/meshes/arms"/>
     <xacro:property name="waist_mesh_dir" value="package://val_description/model/meshes/torso"/>
