Commit message: Add rudimentary wall to arm-only setup

File: model/robots/valkyrie_arm_sim.xacro (robot description, xacro)
@@ -1,5 +1,21 @@
 <robot xmlns:xacro="http://ros.org/wiki/xacro" name="valkyrie_arm">
-    <link name="/world">
+    <link name="/world"/>
+    <material name="brick">
+        <color rgba="0.5 0.125 0.13 1"/>
+    </material>
+    <link name="wall">
+        <visual>
+            <origin rpy="0 0 0" xyz="0 -0.08 0.5"/>
+            <geometry>
+                <box size="1 0.16 1"/>
+            </geometry>
+            <material name="brick"/>
+        </visual>
     </link>
+    <joint name="wall_joint" type="fixed">
+        <parent link="/world"/>
+        <child link="wall"/>
+        <origin rpy="0.0 0.0 1.57" xyz="0.0 0.0 0.0"/>
+    </joint>
     <xacro:property name="arm_mesh_dir" value="package://val_description/model/meshes/arms"/>
     <xacro:property name="fingers_mesh_dir" value="package://val_description/model/meshes/fingers"/>
@@ -9,5 +25,5 @@
     <xacro:include filename="$(find val_description)/model/robots/common/xacro/common_bodies.xacro" />
     <xacro:include filename="$(find val_description)/model/robots/common/xacro/arm/arm_includes.xacro"/>
-    <xacro:make_arm prefix="right" reflect="-1" arm_root_link="/world" />
+    <xacro:make_arm prefix="right" reflect="-1" arm_root_link="wall" />
     <xacro:make_thumb prefix="right" reflect="-1" thumb_root_link="rightPalm"/>
     <xacro:make_index_finger prefix="right" reflect="-1" index_finger_root_link="rightPalm"/>

Commit message: Add Valkyrie arm sim xacro

File: model/robots/valkyrie_arm_sim.xacro (robot description, xacro)
@@ -12,5 +12,21 @@
             <material name="brick"/>
         </visual>
+        <inertial>
+            <mass value="1000000"/>
+            <origin rpy="0 0 0" xyz="0 -0.08 0.5"/>
+            <inertia ixx="85466" ixy="0" ixz="0" iyy="85466" iyz="0" izz="166666"/>
+        </inertial>
+        <collision>
+            <origin rpy="0 0 0" xyz="0 -0.08 0.5"/>
+            <geometry>
+                <box size="1 0.16 1"/>
+            </geometry>
+        </collision>
     </link>
+    <gazebo reference="wall">
+        <material>
+            Gazebo/Bricks
+        </material>
+    </gazebo>
     <joint name="wall_joint" type="fixed">
         <parent link="/world"/>
@@ -18,8 +34,9 @@
         <origin rpy="0.0 0.0 1.57" xyz="0.0 0.0 0.0"/>
     </joint>
+    <schedule_topic_creator_file package="val_gazebo" relative_file_path="/configuration/valkyrie_sim_shm_topics.yaml"/>
     <xacro:property name="arm_mesh_dir" value="package://val_description/model/meshes/arms"/>
     <xacro:property name="fingers_mesh_dir" value="package://val_description/model/meshes/fingers"/>
     <xacro:include filename="$(find val_description)/model/robots/common/xacro/generic_models.xacro" />
-    <xacro:include filename="$(find val_description)/common/xacro/nodes/valkyrie_sim_nodes.xacro"/>
+    <xacro:include filename="$(find val_description)/common/xacro/nodes/valkyrie_arm_sim_nodes.xacro"/>
     <xacro:include filename="$(find val_description)/common/xacro/api/valkyrie_sim_api.xacro"/>
     <xacro:include filename="$(find val_description)/model/robots/common/xacro/common_bodies.xacro" />
@@ -30,5 +47,4 @@
     <xacro:make_middle_finger prefix="right" reflect="-1" middle_finger_root_link="rightPalm"/>
     <xacro:make_pinky_finger prefix="right" reflect="-1" pinky_finger_root_link="rightPalm"/>
-    <xacro:include_multisense_sim />
     <xacro:arm_transmissions_sim prefix="right"/>
     <xacro:thumb_transmissions_sim prefix="right"/>
