Commit message: Add torso model

File: model/robots/single_arm_testbed.xacro (robot description, xacro)
@@ -1,45 +1,14 @@
 <robot xmlns:xacro="http://ros.org/wiki/xacro" name="valkyrie_arm">
     <link name="/world"/>
-    <material name="brick">
-        <color rgba="0.5 0.125 0.13 1"/>
-    </material>
-    <link name="wall">
-        <visual>
-            <origin rpy="0 0 0" xyz="0 -0.08 0.5"/>
-            <geometry>
-                <box size="1 0.16 1"/>
-            </geometry>
-            <material name="brick"/>
-        </visual>
-        <inertial>
-            <mass value="1000000"/>
-            <origin rpy="0 0 0" xyz="0 -0.08 0.5"/>
-            <inertia ixx="85466" ixy="0" ixz="0" iyy="85466" iyz="0" izz="166666"/>
-        </inertial>
-        <collision>
-            <origin rpy="0 0 0" xyz="0 -0.08 0.5"/>
-            <geometry>
-                <box size="1 0.16 1"/>
-            </geometry>
-        </collision>
-    </link>
-    <gazebo reference="wall">
-        <material>
-            Gazebo/Bricks
-        </material>
-    </gazebo>
-    <joint name="wall_joint" type="fixed">
-        <parent link="/world"/>
-        <child link="wall"/>
-        <origin rpy="0.0 0.0 1.57" xyz="0.0 0.0 0.0"/>
-    </joint>
     <gazebo>
-      <plugin filename="libval_gazebo.so" name="SharedMemorySimInterfacePlugin">
-        <robotNamespace>/val</robotNamespace>
-      </plugin>
+        <plugin filename="libval_gazebo.so" name="SharedMemorySimInterfacePlugin">
+            <robotNamespace>/val</robotNamespace>
+        </plugin>
     </gazebo>
     <schedule_topic_creator_file package="val_gazebo" relative_file_path="/configuration/valkyrie_sim_shm_topics.yaml"/>
     <xacro:property name="arm_mesh_dir" value="package://val_description/model/meshes/arms"/>
+    <xacro:property name="waist_mesh_dir" value="package://val_description/model/meshes/torso"/>
     <xacro:property name="fingers_mesh_dir" value="package://val_description/model/meshes/fingers"/>
+    <xacro:include filename="$(find val_description)/model/robots/support.xacro"/>
     <xacro:include filename="$(find val_description)/model/robots/common/xacro/generic_models.xacro" />
     <xacro:include filename="$(find val_description)/common/xacro/nodes/valkyrie_arm_sim_nodes.xacro"/>
@@ -47,5 +16,8 @@
     <xacro:include filename="$(find val_description)/model/robots/common/xacro/common_bodies.xacro" />
     <xacro:include filename="$(find val_description)/model/robots/common/xacro/arm/arm_includes.xacro"/>
-    <xacro:make_arm prefix="right" reflect="-1" arm_root_link="wall" />
+    <xacro:include filename="$(find val_description)/model/robots/common/xacro/waist/fixed_torso_includes.xacro"/>
+    <xacro:make_torso torso_root_link="wall" />
+    <xacro:make_support parent_link="/world" link_name="wall" />
+    <xacro:make_arm prefix="right" reflect="-1" arm_root_link="torso" />
     <xacro:make_thumb prefix="right" reflect="-1" thumb_root_link="rightPalm"/>
     <xacro:make_index_finger prefix="right" reflect="-1" index_finger_root_link="rightPalm"/>
