Commit message: More bandit renaming, and addition of mimic joints

File: model/robots/bandit.xacro (robot description, xacro)
@@ -1,3 +1,3 @@
-<robot xmlns:xacro="http://ros.org/wiki/xacro" name="valkyrie_arm">
+<robot xmlns:xacro="http://ros.org/wiki/xacro" name="bandit">
     <link name="/world"/>
     <gazebo>
@@ -12,5 +12,5 @@
     <xacro:include filename="$(find val_description)/model/robots/common/xacro/support.xacro"/>
     <xacro:include filename="$(find val_description)/model/robots/common/xacro/generic_models.xacro" />
-    <xacro:include filename="$(find val_description)/common/xacro/nodes/valkyrie_arm_sim_nodes.xacro"/>
+    <xacro:include filename="$(find val_description)/common/xacro/nodes/bandit_sim_nodes.xacro"/>
     <xacro:include filename="$(find val_description)/common/xacro/api/valkyrie_sim_api.xacro"/>
     <xacro:include filename="$(find val_description)/model/robots/common/xacro/common_bodies.xacro" />

File: model/robots/common/xacro/generic_models.xacro (robot description, xacro)
@@ -179,4 +179,20 @@
     </gazebo>
   </xacro:macro>
+  <xacro:macro name="revolute_joint_ex_mimic" params="jointName parent child origin_xyz origin_rpy axis damping friction *limits *controller_gains *mimic">
+    <joint name="${jointName}" type="revolute">
+      <origin rpy="${origin_rpy}" xyz="${origin_xyz}"/>
+      <axis xyz="${axis}"/>
+      <parent link="${parent}"/>
+      <child link="${child}"/>
+      <xacro:insert_block name="limits" />
+      <xacro:insert_block name="controller_gains" />
+      <xacro:insert_block name="mimic" />
+      <dynamics damping="${damping}" friction="${friction}"/>
+    </joint>
+    <gazebo reference="${jointName}">
+      <provideFeedback>1</provideFeedback>
+      <implicitSpringDamper>1</implicitSpringDamper>
+    </gazebo>
+  </xacro:macro>
   <xacro:macro name="floating_joint" params="jointName parent child origin_xyz origin_rpy">
     <joint name="${jointName}" type="floating">

File: model/robots/common/xacro/index_finger/index_finger.xacro (robot description, xacro)
@@ -49,5 +49,5 @@
         <controller_gains Kp="${IndexFingerPitch1Kp}" Kd="${IndexFingerPitch1Kd}" Ki="${IndexFingerPitch1Ki}"/>
     </xacro:revolute_joint_ex>
-    <xacro:revolute_joint_ex jointName="${prefix}${IndexFingerPitch2JointName}"
+    <xacro:revolute_joint_ex_mimic jointName="${prefix}${IndexFingerPitch2JointName}"
                           parent="${prefix}IndexFingerPitch1Link" child="${prefix}IndexFingerPitch2Link"
                           origin_xyz="${IndexFingerPitch2FrameOrigin_X} ${reflect * 0.0381} ${IndexFingerPitch2FrameOrigin_Z}"
@@ -61,6 +61,7 @@
         </xacro:if>
         <controller_gains Kp="${IndexFingerPitch1Kp}" Kd="${IndexFingerPitch1Kd}" Ki="${IndexFingerPitch1Ki}"/>
-    </xacro:revolute_joint_ex>
-    <xacro:revolute_joint_ex jointName="${prefix}${IndexFingerPitch3JointName}"
+        <mimic joint="${prefix}${IndexFingerPitch1JointName}" multiplier="${Pulley2Ratio}" offset="0"/>
+    </xacro:revolute_joint_ex_mimic>
+    <xacro:revolute_joint_ex_mimic jointName="${prefix}${IndexFingerPitch3JointName}"
                           parent="${prefix}IndexFingerPitch2Link" child="${prefix}IndexFingerPitch3Link"
                           origin_xyz="${IndexFingerPitch3FrameOrigin_X} ${reflect * 0.0229} ${IndexFingerPitch3FrameOrigin_Z}"
@@ -74,5 +75,6 @@
         </xacro:if>
         <controller_gains Kp="${IndexFingerPitch1Kp}" Kd="${IndexFingerPitch1Kd}" Ki="${IndexFingerPitch1Ki}"/>
-    </xacro:revolute_joint_ex>
+        <mimic joint="${prefix}${IndexFingerPitch1JointName}" multiplier="${Pulley3Ratio}" offset="0"/>
+    </xacro:revolute_joint_ex_mimic>
   </xacro:macro>
   <xacro:macro name="index_finger_transmissions_hw" params="prefix reflect">

File: model/robots/common/xacro/middle_finger/middle_finger.xacro (robot description, xacro)
@@ -49,5 +49,5 @@
         <controller_gains Kp="${MiddleFingerPitch1Kp}" Kd="${MiddleFingerPitch1Kd}" Ki="${MiddleFingerPitch1Ki}"/>
     </xacro:revolute_joint_ex>
-    <xacro:revolute_joint_ex jointName="${prefix}${MiddleFingerPitch2JointName}"
+    <xacro:revolute_joint_ex_mimic jointName="${prefix}${MiddleFingerPitch2JointName}"
                           parent="${prefix}MiddleFingerPitch1Link" child="${prefix}MiddleFingerPitch2Link"
                           origin_xyz="${MiddleFingerPitch2FrameOrigin_X} ${reflect * 0.0381} ${MiddleFingerPitch2FrameOrigin_Z}"
@@ -61,6 +61,7 @@
         </xacro:if>
         <controller_gains Kp="${MiddleFingerPitch1Kp}" Kd="${MiddleFingerPitch1Kd}" Ki="${MiddleFingerPitch1Ki}"/>
-    </xacro:revolute_joint_ex>
-    <xacro:revolute_joint_ex jointName="${prefix}${MiddleFingerPitch3JointName}"
+        <mimic joint="${prefix}${MiddleFingerPitch1JointName}" multiplier="${Pulley2Ratio}" offset="0"/>
+    </xacro:revolute_joint_ex_mimic>
+    <xacro:revolute_joint_ex_mimic jointName="${prefix}${MiddleFingerPitch3JointName}"
                           parent="${prefix}MiddleFingerPitch2Link" child="${prefix}MiddleFingerPitch3Link"
                           origin_xyz="${MiddleFingerPitch3FrameOrigin_X} ${reflect * 0.0229} ${MiddleFingerPitch3FrameOrigin_Z}"
@@ -74,5 +75,6 @@
         </xacro:if>
         <controller_gains Kp="${MiddleFingerPitch1Kp}" Kd="${MiddleFingerPitch1Kd}" Ki="${MiddleFingerPitch1Ki}"/>
-    </xacro:revolute_joint_ex>
+        <mimic joint="${prefix}${MiddleFingerPitch1JointName}" multiplier="${Pulley3Ratio}" offset="0"/>
+    </xacro:revolute_joint_ex_mimic>
   </xacro:macro>
   <xacro:macro name="middle_finger_transmissions_hw" params="prefix reflect">

File: model/robots/common/xacro/pinky_finger/pinky_finger.xacro (robot description, xacro)
@@ -49,5 +49,5 @@
         <controller_gains Kp="${PinkyPitch1Kp}" Kd="${PinkyPitch1Kd}" Ki="${PinkyPitch1Ki}"/>
     </xacro:revolute_joint_ex>
-    <xacro:revolute_joint_ex jointName="${prefix}${PinkyPitch2JointName}"
+    <xacro:revolute_joint_ex_mimic jointName="${prefix}${PinkyPitch2JointName}"
                           parent="${prefix}PinkyPitch1Link" child="${prefix}PinkyPitch2Link"
                           origin_xyz="${PinkyPitch2FrameOrigin_X} ${reflect * 0.0381} ${PinkyPitch2FrameOrigin_Z}"
@@ -61,6 +61,7 @@
         </xacro:if>
         <controller_gains Kp="${PinkyPitch1Kp}" Kd="${PinkyPitch1Kd}" Ki="${PinkyPitch1Ki}"/>
-    </xacro:revolute_joint_ex>
-    <xacro:revolute_joint_ex jointName="${prefix}${PinkyPitch3JointName}"
+        <mimic joint="${prefix}${PinkyPitch1JointName}" multiplier="${Pulley2Ratio}" offset="0"/>
+    </xacro:revolute_joint_ex_mimic>
+    <xacro:revolute_joint_ex_mimic jointName="${prefix}${PinkyPitch3JointName}"
                           parent="${prefix}PinkyPitch2Link" child="${prefix}PinkyPitch3Link"
                           origin_xyz="${PinkyPitch3FrameOrigin_X} ${reflect * 0.0229} ${PinkyPitch3FrameOrigin_Z}"
@@ -74,5 +75,6 @@
         </xacro:if>
         <controller_gains Kp="${PinkyPitch1Kp}" Kd="${PinkyPitch1Kd}" Ki="${PinkyPitch1Ki}"/>
-    </xacro:revolute_joint_ex>
+        <mimic joint="${prefix}${PinkyPitch1JointName}" multiplier="${Pulley3Ratio}" offset="0"/>
+    </xacro:revolute_joint_ex_mimic>
   </xacro:macro>
   <xacro:macro name="pinky_finger_transmissions_hw" params="prefix reflect">

File: model/robots/common/xacro/support.xacro (robot description, xacro)
@@ -1,3 +1,3 @@
-<robot xmlns:xacro="http://ros.org/wiki/xacro" name="valkyrie_arm">
+<robot xmlns:xacro="http://ros.org/wiki/xacro" name="bandit">
     <material name="brick">
         <color rgba="0.5 0.125 0.13 1"/>

File: model/robots/common/xacro/thumb/thumb.xacro (robot description, xacro)
@@ -67,5 +67,5 @@
         <controller_gains Kp="${ThumbPitch1Kp}" Kd="${ThumbPitch1Kd}" Ki="${ThumbPitch1Ki}"/>
     </xacro:revolute_joint_ex>
-    <xacro:revolute_joint_ex jointName="${prefix}${ThumbPitch2JointName}"
+    <xacro:revolute_joint_ex_mimic jointName="${prefix}${ThumbPitch2JointName}"
                           parent="${prefix}ThumbPitch1Link" child="${prefix}ThumbPitch2Link"
                           origin_xyz="${ThumbPitch2FrameOrigin_X} ${reflect * 0.0066} ${ThumbPitch2FrameOrigin_Z}"
@@ -79,6 +79,7 @@
         </xacro:if>
         <controller_gains Kp="${ThumbPitch2Kp}" Kd="${ThumbPitch2Kd}" Ki="${ThumbPitch2Ki}"/>
-    </xacro:revolute_joint_ex>
-    <xacro:revolute_joint_ex jointName="${prefix}${ThumbPitch3JointName}"
+        <mimic joint="${prefix}${ThumbPitch1JointName}" multiplier="${Pulley2Ratio}" offset="0"/>
+    </xacro:revolute_joint_ex_mimic>
+    <xacro:revolute_joint_ex_mimic jointName="${prefix}${ThumbPitch3JointName}"
                           parent="${prefix}ThumbPitch2Link" child="${prefix}ThumbPitch3Link"
                           origin_xyz="${ThumbPitch3FrameOrigin_X} ${reflect * 0.0049} ${ThumbPitch3FrameOrigin_Z}"
@@ -92,5 +93,6 @@
         </xacro:if>
         <controller_gains Kp="${ThumbPitch3Kp}" Kd="${ThumbPitch3Kd}" Ki="${ThumbPitch3Ki}"/>
-    </xacro:revolute_joint_ex>
+        <mimic joint="${prefix}${ThumbPitch1JointName}" multiplier="${Pulley3Ratio}" offset="0"/>
+    </xacro:revolute_joint_ex_mimic>
   </xacro:macro>
   <xacro:macro name="thumb_transmissions_hw" params="prefix reflect">
