Commit message: Removed sim_pinned xacro since the unpinned is harnessed until you lower it so it's basically the same thing. Also added a gazebo sync'd urdf that runs the gazebo plugin it a specific rate.

File: model/robots/valkyrie_sim.xacro (robot description, xacro)
@@ -3,5 +3,4 @@
       <plugin filename="libval_gazebo.so" name="SharedMemorySimInterfacePlugin">
           <robotNamespace>/val</robotNamespace>
-          <updateRateHz>500.0</updateRateHz>
       </plugin>
     </gazebo>

File: model/robots/valkyrie_sim_arm_mass_sims.xacro (robot description, xacro)
@@ -3,5 +3,4 @@
       <plugin filename="libval_gazebo.so" name="SharedMemorySimInterfacePlugin">
           <robotNamespace>/val</robotNamespace>
-          <updateRateHz>500.0</updateRateHz>
       </plugin>
     </gazebo>

File: model/robots/valkyrie_sim_gazebo_sync.xacro (robot description, xacro)
@@ -7,25 +7,12 @@
     </gazebo>
     <xacro:property name="mesh_root" value="package://val_description/model/meshes"/>
+    <xacro:include filename="$(find val_description)/common/xacro/api/valkyrie_sim_api.xacro"/>
     <xacro:include filename="$(find val_description)/model/robots/common/xacro/generic_models.xacro" />
-    <xacro:include filename="$(find val_description)/model/materials/materials.xacro" />
     <xacro:include filename="$(find val_description)/model/robots/common/xacro/common_bodies.xacro" />
-    <xacro:include filename="$(find val_description)/model/robots/common/xacro/valkyrie_base_sim.xacro"/>
     <xacro:include filename="$(find val_description)/model/urdf/multisense_sl.urdf" />
     <xacro:include filename="$(find val_description)/common/xacro/serial_numbers/valkyrie_A_serials.xacro"/>
     <xacro:include filename="$(find val_description)/common/xacro/dev_ports/valkyrie_gazebo_ports.xacro"/>
-    <xacro:include filename="$(find val_description)/common/xacro/api/valkyrie_sim_api.xacro"/>
-    <gazebo>
-      <joint name="fixed" type="revolute">
-        <parent>world</parent>
-        <child>${TorsoRollLinkName}</child>
-        <axis>
-          <xyz>0 0 1</xyz>
-          <use_parent_model_frame>true</use_parent_model_frame>
-          <limit>
-            <upper>0</upper>
-            <lower>0</lower>
-          </limit>
-        </axis>
-      </joint>
-    </gazebo>
+    <xacro:include filename="$(find val_description)/model/robots/common/xacro/valkyrie_base_sim.xacro"/>
+    <xacro:include filename="$(find val_description)/model/robots/common/xacro/gazebo_harness.xacro"/>
+    <xacro:add_sim_harness harnessed_link="${TorsoRollLinkName}" />
 </robot>

Commit message: sim models use model path for visuals rather than package path

File: model/robots/valkyrie_sim.xacro (robot description, xacro)
@@ -6,10 +6,10 @@
     </gazebo>
     <schedule_topic_creator_file package="val_gazebo" relative_file_path="/configuration/valkyrie_sim_shm_topics.yaml"/>
-    <xacro:property name="leg_mesh_dir" value="package://val_description/model/meshes/legs"/>
-    <xacro:property name="arm_mesh_dir" value="package://val_description/model/meshes/arms"/>
-    <xacro:property name="waist_mesh_dir" value="package://val_description/model/meshes/torso"/>
-    <xacro:property name="head_mesh_dir" value="package://val_description/model/meshes/head"/>
-    <xacro:property name="pelvis_mesh_dir" value="package://val_description/model/meshes/pelvis"/>
-    <xacro:property name="fingers_mesh_dir" value="package://val_description/model/meshes/fingers"/>
+    <xacro:property name="leg_mesh_dir" value="model://val_description/model/meshes/legs"/>
+    <xacro:property name="arm_mesh_dir" value="model://val_description/model/meshes/arms"/>
+    <xacro:property name="waist_mesh_dir" value="model://val_description/model/meshes/torso"/>
+    <xacro:property name="head_mesh_dir" value="model://val_description/model/meshes/head"/>
+    <xacro:property name="pelvis_mesh_dir" value="model://val_description/model/meshes/pelvis"/>
+    <xacro:property name="fingers_mesh_dir" value="model://val_description/model/meshes/fingers"/>
     <xacro:include filename="$(find val_description)/model/robots/common/xacro/generic_models.xacro" />
     <xacro:include filename="$(find val_description)/common/xacro/nodes/valkyrie_sim_nodes.xacro"/>

File: model/robots/valkyrie_sim_angled_legj1s.xacro (robot description, xacro)
@@ -6,10 +6,10 @@
     </gazebo>
     <schedule_topic_creator_file package="val_gazebo" relative_file_path="/configuration/valkyrie_sim_shm_topics.yaml"/>
-    <xacro:property name="leg_mesh_dir" value="package://val_description/model/meshes/legs_angled_j1s"/>
-    <xacro:property name="arm_mesh_dir" value="package://val_description/model/meshes/arms"/>
-    <xacro:property name="waist_mesh_dir" value="package://val_description/model/meshes/torso_angled_j1s"/>
-    <xacro:property name="head_mesh_dir" value="package://val_description/model/meshes/head"/>
-    <xacro:property name="pelvis_mesh_dir" value="package://val_description/model/meshes/pelvis_angled_j1s"/>
-    <xacro:property name="fingers_mesh_dir" value="package://val_description/model/meshes/fingers"/>
+    <xacro:property name="leg_mesh_dir" value="model://val_description/model/meshes/legs_angled_j1s"/>
+    <xacro:property name="arm_mesh_dir" value="model://val_description/model/meshes/arms"/>
+    <xacro:property name="waist_mesh_dir" value="model://val_description/model/meshes/torso_angled_j1s"/>
+    <xacro:property name="head_mesh_dir" value="model://val_description/model/meshes/head"/>
+    <xacro:property name="pelvis_mesh_dir" value="model://val_description/model/meshes/pelvis_angled_j1s"/>
+    <xacro:property name="fingers_mesh_dir" value="model://val_description/model/meshes/fingers"/>
     <xacro:include filename="$(find val_description)/model/robots/common/xacro/generic_models.xacro" />
     <xacro:include filename="$(find val_description)/common/xacro/nodes/valkyrie_sim_nodes.xacro"/>

File: model/robots/valkyrie_sim_arm_mass_sims.xacro (robot description, xacro)
@@ -5,9 +5,9 @@
       </plugin>
     </gazebo>
-    <xacro:property name="leg_mesh_dir" value="package://val_description/model/meshes/legs"/>
-    <xacro:property name="arm_mesh_dir" value="package://val_description/model/meshes/arms"/>
-    <xacro:property name="waist_mesh_dir" value="package://val_description/model/meshes/torso"/>
-    <xacro:property name="head_mesh_dir" value="package://val_description/model/meshes/head"/>
-    <xacro:property name="pelvis_mesh_dir" value="package://val_description/model/meshes/pelvis"/>
+    <xacro:property name="leg_mesh_dir" value="model://val_description/model/meshes/legs"/>
+    <xacro:property name="arm_mesh_dir" value="model://val_description/model/meshes/arms"/>
+    <xacro:property name="waist_mesh_dir" value="model://val_description/model/meshes/torso"/>
+    <xacro:property name="head_mesh_dir" value="model://val_description/model/meshes/head"/>
+    <xacro:property name="pelvis_mesh_dir" value="model://val_description/model/meshes/pelvis"/>
     <xacro:include filename="$(find val_description)/model/robots/common/xacro/generic_models.xacro" />
     <xacro:include filename="$(find val_description)/common/xacro/nodes/valkyrie_sim_nodes.xacro"/>

File: model/robots/valkyrie_sim_gazebo_sync.xacro (robot description, xacro)
@@ -7,10 +7,10 @@
     </gazebo>
     <schedule_topic_creator_file package="val_gazebo" relative_file_path="/configuration/valkyrie_sim_shm_topics.yaml"/>
-    <xacro:property name="leg_mesh_dir" value="package://val_description/model/meshes/legs"/>
-    <xacro:property name="arm_mesh_dir" value="package://val_description/model/meshes/arms"/>
-    <xacro:property name="waist_mesh_dir" value="package://val_description/model/meshes/torso"/>
-    <xacro:property name="head_mesh_dir" value="package://val_description/model/meshes/head"/>
-    <xacro:property name="pelvis_mesh_dir" value="package://val_description/model/meshes/pelvis"/>
-    <xacro:property name="fingers_mesh_dir" value="package://val_description/model/meshes/fingers"/>
+    <xacro:property name="leg_mesh_dir" value="model://val_description/model/meshes/legs"/>
+    <xacro:property name="arm_mesh_dir" value="model://val_description/model/meshes/arms"/>
+    <xacro:property name="waist_mesh_dir" value="model://val_description/model/meshes/torso"/>
+    <xacro:property name="head_mesh_dir" value="model://val_description/model/meshes/head"/>
+    <xacro:property name="pelvis_mesh_dir" value="model://val_description/model/meshes/pelvis"/>
+    <xacro:property name="fingers_mesh_dir" value="model://val_description/model/meshes/fingers"/>
     <xacro:include filename="$(find val_description)/model/robots/common/xacro/generic_models.xacro" />
     <xacro:include filename="$(find val_description)/common/xacro/nodes/valkyrie_sim_nodes.xacro"/>
