Commit message: [val_description] Fixed sim mesh paths

File: model/robots/valkyrie_D.xacro (robot description, xacro)
@@ -1,4 +1,4 @@
 <robot xmlns:xacro="http://www.ros.org/wiki/xacro" name="ValkyrieD">
-	<xacro:property name="leg_mesh_dir" value="package://val_description/model/meshes/legs"/>
+    <xacro:property name="leg_mesh_dir" value="package://val_description/model/meshes/legs"/>
     <xacro:property name="arm_mesh_dir" value="package://val_description/model/meshes/arms"/>
     <xacro:property name="waist_mesh_dir" value="package://val_description/model/meshes/torso"/>
@@ -6,5 +6,5 @@
     <xacro:property name="pelvis_mesh_dir" value="package://val_description/model/meshes/pelvis"/>
     <xacro:property name="fingers_mesh_dir" value="package://val_description/model/meshes/fingers"/>
-	<xacro:include filename="$(find val_description)/model/robots/common/xacro/generic_models.xacro" />
+    <xacro:include filename="$(find val_description)/model/robots/common/xacro/generic_models.xacro" />
     <xacro:include filename="$(find val_description)/common/xacro/nodes/valkyrie_nodes.xacro"/>
     <xacro:include filename="$(find val_description)/model/robots/common/xacro/sensors/sensor_transforms.xacro"/>

File: model/robots/valkyrie_D_arm_mass_sims.xacro (robot description, xacro)
@@ -1,4 +1,4 @@
 <robot xmlns:xacro="http://www.ros.org/wiki/xacro" name="valkyrie">
-	<xacro:property name="leg_mesh_dir" value="package://val_description/model/meshes/legs"/>
+    <xacro:property name="leg_mesh_dir" value="package://val_description/model/meshes/legs"/>
     <xacro:property name="arm_mesh_dir" value="package://val_description/model/meshes/arms"/>
     <xacro:property name="waist_mesh_dir" value="package://val_description/model/meshes/torso"/>

File: model/robots/valkyrie_sim.xacro (robot description, xacro)
@@ -6,10 +6,10 @@
     </gazebo>
     <schedule_topic_creator_file package="val_gazebo" relative_file_path="/configuration/valkyrie_sim_shm_topics.yaml"/>
-    <xacro:property name="leg_mesh_dir" value="model://val_description/model/meshes/legs"/>
-    <xacro:property name="arm_mesh_dir" value="model://val_description/model/meshes/arms"/>
-    <xacro:property name="waist_mesh_dir" value="model://val_description/model/meshes/torso"/>
-    <xacro:property name="head_mesh_dir" value="model://val_description/model/meshes/head"/>
-    <xacro:property name="pelvis_mesh_dir" value="model://val_description/model/meshes/pelvis"/>
-    <xacro:property name="fingers_mesh_dir" value="model://val_description/model/meshes/fingers"/>
+    <xacro:property name="leg_mesh_dir" value="package://val_description/model/meshes/legs"/>
+    <xacro:property name="arm_mesh_dir" value="package://val_description/model/meshes/arms"/>
+    <xacro:property name="waist_mesh_dir" value="package://val_description/model/meshes/torso"/>
+    <xacro:property name="head_mesh_dir" value="package://val_description/model/meshes/head"/>
+    <xacro:property name="pelvis_mesh_dir" value="package://val_description/model/meshes/pelvis"/>
+    <xacro:property name="fingers_mesh_dir" value="package://val_description/model/meshes/fingers"/>
     <xacro:include filename="$(find val_description)/model/robots/common/xacro/generic_models.xacro" />
     <xacro:include filename="$(find val_description)/common/xacro/nodes/valkyrie_sim_nodes.xacro"/>

File: model/robots/valkyrie_sim_arm_mass_sims.xacro (robot description, xacro)
@@ -7,9 +7,10 @@
     </gazebo>
     <schedule_topic_creator_file package="val_gazebo" relative_file_path="/configuration/valkyrie_sim_shm_topics.yaml"/>
-    <xacro:property name="leg_mesh_dir" value="model://val_description/model/meshes/legs"/>
-    <xacro:property name="arm_mesh_dir" value="model://val_description/model/meshes/arms"/>
-    <xacro:property name="waist_mesh_dir" value="model://val_description/model/meshes/torso"/>
-    <xacro:property name="head_mesh_dir" value="model://val_description/model/meshes/head"/>
-    <xacro:property name="pelvis_mesh_dir" value="model://val_description/model/meshes/pelvis"/>
+    <xacro:property name="leg_mesh_dir" value="package://val_description/model/meshes/legs"/>
+    <xacro:property name="arm_mesh_dir" value="package://val_description/model/meshes/arms"/>
+    <xacro:property name="waist_mesh_dir" value="package://val_description/model/meshes/torso"/>
+    <xacro:property name="head_mesh_dir" value="package://val_description/model/meshes/head"/>
+    <xacro:property name="pelvis_mesh_dir" value="package://val_description/model/meshes/pelvis"/>
+    <xacro:property name="fingers_mesh_dir" value="package://val_description/model/meshes/fingers"/>
     <xacro:include filename="$(find val_description)/model/robots/common/xacro/generic_models.xacro" />
     <xacro:include filename="$(find val_description)/common/xacro/nodes/valkyrie_sim_nodes.xacro"/>

File: model/robots/valkyrie_sim_arm_mass_sims_hd.xacro (robot description, xacro)
@@ -7,9 +7,9 @@
     </gazebo>
     <schedule_topic_creator_file package="val_gazebo" relative_file_path="/configuration/valkyrie_sim_shm_topics.yaml"/>
-    <xacro:property name="leg_mesh_dir" value="model://val_description/model/meshesHD"/>
-    <xacro:property name="arm_mesh_dir" value="model://val_description/model/meshesHD"/>
-    <xacro:property name="waist_mesh_dir" value="model://val_description/model/meshesHD"/>
-    <xacro:property name="head_mesh_dir" value="model://val_description/model/meshesHD"/>
-    <xacro:property name="pelvis_mesh_dir" value="model://val_description/model/meshesHD"/>
+    <xacro:property name="leg_mesh_dir" value="package://val_description/model/meshesHD"/>
+    <xacro:property name="arm_mesh_dir" value="package://val_description/model/meshesHD"/>
+    <xacro:property name="waist_mesh_dir" value="package://val_description/model/meshesHD"/>
+    <xacro:property name="head_mesh_dir" value="package://val_description/model/meshesHD"/>
+    <xacro:property name="pelvis_mesh_dir" value="package://val_description/model/meshesHD"/>
     <xacro:include filename="$(find val_description)/model/robots/common/xacro/generic_models.xacro" />
     <xacro:include filename="$(find val_description)/common/xacro/nodes/valkyrie_sim_nodes.xacro"/>
