Commit message: calibrating fingers for neu left forearm

File: common/xacro/serial_numbers/forearm_left_testbench_serials.xacro (robot description, xacro)
@@ -1,4 +1,4 @@
 <robot xmlns:xacro="http://ros.org/wiki/xacro" name="forearm_testbench">
-	<xacro:property name="forearm_serial_number" value="v_h_007" />
-	<xacro:property name="forearm_yaw_serial_number" value="v_g_016" />
+	<xacro:property name="forearm_serial_number" value="v_h_001" />
+	<xacro:property name="forearm_yaw_serial_number" value="v_g_005" />
 </robot>

File: common/xacro/serial_numbers/forearm_testbench_serials.xacro (robot description, xacro)
@@ -1,4 +1,4 @@
 <robot xmlns:xacro="http://ros.org/wiki/xacro" name="forearm_testbench">
-	<xacro:property name="forearm_yaw_serial_number" value="v_g_017" />
-	<xacro:property name="forearm_serial_number" value="v_h_008" />
+	<xacro:property name="forearm_yaw_serial_number" value="v_g_005" />
+	<xacro:property name="forearm_serial_number" value="v_h_001" />
 </robot>

Commit message: correcting calibration fo right forearm vh008

File: common/xacro/serial_numbers/forearm_left_testbench_serials.xacro (robot description, xacro)
@@ -1,4 +1,4 @@
 <robot xmlns:xacro="http://ros.org/wiki/xacro" name="forearm_testbench">
-	<xacro:property name="forearm_serial_number" value="v_h_001" />
-	<xacro:property name="forearm_yaw_serial_number" value="v_g_005" />
+	<xacro:property name="forearm_serial_number" value="v_h_005" />
+	<xacro:property name="forearm_yaw_serial_number" value="v_g_016" />
 </robot>
