Commit message: calibrating unit A right forearm

File: common/xacro/serial_numbers/forearm_right_testbench_serials.xacro (robot description, xacro)
@@ -1,4 +1,4 @@
 <robot xmlns:xacro="http://ros.org/wiki/xacro" name="forearm_testbench">
-	<xacro:property name="forearm_serial_number" value="v_h_006" />
-	<xacro:property name="forearm_yaw_serial_number" value="v_g_012" />
+	<xacro:property name="forearm_serial_number" value="v_h_008" />
+	<xacro:property name="forearm_yaw_serial_number" value="v_g_017" />
 </robot>

File: common/xacro/serial_numbers/forearm_testbench_serials.xacro (robot description, xacro)
@@ -1,4 +1,4 @@
 <robot xmlns:xacro="http://ros.org/wiki/xacro" name="forearm_testbench">
-	<xacro:property name="forearm_yaw_serial_number" value="v_g_016" />
-	<xacro:property name="forearm_serial_number" value="v_h_003" />
+	<xacro:property name="forearm_yaw_serial_number" value="v_g_017" />
+	<xacro:property name="forearm_serial_number" value="v_h_008" />
 </robot>

Commit message: updating calibration of right arm fingers

File: common/xacro/serial_numbers/forearm_right_testbench_serials.xacro (robot description, xacro)
@@ -1,4 +1,4 @@
 <robot xmlns:xacro="http://ros.org/wiki/xacro" name="forearm_testbench">
-	<xacro:property name="forearm_serial_number" value="v_h_008" />
-	<xacro:property name="forearm_yaw_serial_number" value="v_g_017" />
+	<xacro:property name="forearm_serial_number" value="v_h_002" />
+	<xacro:property name="forearm_yaw_serial_number" value="v_g_003" />
 </robot>

File: common/xacro/serial_numbers/forearm_testbench_serials.xacro (robot description, xacro)
@@ -1,4 +1,4 @@
 <robot xmlns:xacro="http://ros.org/wiki/xacro" name="forearm_testbench">
-	<xacro:property name="forearm_yaw_serial_number" value="v_g_016" />
-	<xacro:property name="forearm_serial_number" value="v_h_005" />
+	<xacro:property name="forearm_yaw_serial_number" value="v_g_003" />
+	<xacro:property name="forearm_serial_number" value="v_h_002" />
 </robot>
