Commit message: updating forearm tests

File: common/xacro/serial_numbers/forearm_testbench_serials.xacro (robot description, xacro)
@@ -1,4 +1,4 @@
 <robot xmlns:xacro="http://ros.org/wiki/xacro" name="forearm_testbench">
-	<xacro:property name="forearm_yaw_serial_number" value="v_g_005" />
-	<xacro:property name="forearm_serial_number" value="v_h_001" />
+	<xacro:property name="forearm_yaw_serial_number" value="v_g_017" />
+	<xacro:property name="forearm_serial_number" value="v_h_008" />
 </robot>

File: instance/instances/robots/forearm_testbench_left.xacro (robot description, xacro)
@@ -2,4 +2,6 @@
 	<xacro:property name="instance" value="forearm_testbench_left" />
 	<xacro:property name="prefix" value="left" />
+        <xacro:include filename="$(find val_description)/instance/instances/robots/xacro/firmware/firmware.xacro" />
+        <xacro:include filename="$(find val_description)/instance/instances/robots/xacro/firmware/forearm_firmware.xacro" />
 	<xacro:include filename="$(find val_description)/common/xacro/nodes/forearm_testbench_nodes_left.xacro" />
 	<xacro:include filename="$(find val_description)/common/xacro/serial_numbers/forearm_testbench_serials.xacro" />
@@ -9,5 +11,6 @@
     <Channels>
     </Channels>
-	<xacro:firmware_base_url/>
+        <xacro:firmware_base_url/>
+    <xacro:firmware />
     <Mechanisms>
     <xacro:simple_mechanism name="testbench_actuator" serial_number="${forearm_yaw_serial_number}" node="${testbench_node}" />

File: instance/instances/robots/forearm_testbench_right.xacro (robot description, xacro)
@@ -2,4 +2,6 @@
 	<xacro:property name="instance" value="forearm_testbench_right" />
 	<xacro:property name="prefix" value="right" />
+        <xacro:include filename="$(find val_description)/instance/instances/robots/xacro/firmware/firmware.xacro" />
+        <xacro:include filename="$(find val_description)/instance/instances/robots/xacro/firmware/forearm_firmware.xacro" />
 	<xacro:include filename="$(find val_description)/common/xacro/nodes/forearm_testbench_nodes_right.xacro" />
 	<xacro:include filename="$(find val_description)/common/xacro/serial_numbers/forearm_testbench_serials.xacro" />
@@ -9,5 +11,6 @@
     <Channels>
     </Channels>
-	<xacro:firmware_base_url/>
+        <xacro:firmware_base_url/>
+    <xacro:firmware />
     <Mechanisms>
     <xacro:simple_mechanism name="testbench_actuator" serial_number="${forearm_yaw_serial_number}" node="${testbench_node}" />

Commit message: updating

File: common/xacro/serial_numbers/forearm_testbench_serials.xacro (robot description, xacro)
@@ -1,4 +1,4 @@
 <robot xmlns:xacro="http://ros.org/wiki/xacro" name="forearm_testbench">
-	<xacro:property name="forearm_yaw_serial_number" value="v_g_017" />
-	<xacro:property name="forearm_serial_number" value="v_h_008" />
+	<xacro:property name="forearm_yaw_serial_number" value="v_g_016" />
+	<xacro:property name="forearm_serial_number" value="v_h_005" />
 </robot>

Commit message: updating forearm wrist calibration

File: common/xacro/serial_numbers/forearm_testbench_serials.xacro (robot description, xacro)
@@ -1,4 +1,4 @@
 <robot xmlns:xacro="http://ros.org/wiki/xacro" name="forearm_testbench">
-	<xacro:property name="forearm_yaw_serial_number" value="v_g_003" />
-	<xacro:property name="forearm_serial_number" value="v_h_002" />
+	<xacro:property name="forearm_yaw_serial_number" value="v_g_016" />
+	<xacro:property name="forearm_serial_number" value="v_h_005" />
 </robot>
