Commit message: pushing for of robot work

File: common/xacro/serial_numbers/valkyrie_B_serials.xacro (robot description, xacro)
@@ -16,12 +16,12 @@
 	<xacro:property name="leftArmJ3SerialNumber" value="v_f_007" />
 	<xacro:property name="leftArmJ4SerialNumber" value="v_f_008" />
-        <xacro:property name="leftArmJ5SerialNumber" value="v_g_021" />
-        <xacro:property name="leftForearmSerialNumber" value="v_h_003"/>
+        <xacro:property name="leftArmJ5SerialNumber" value="v_g_016" />
+        <xacro:property name="leftForearmSerialNumber" value="v_h_005"/>
 	<xacro:property name="rightArmJ1SerialNumber" value="v_a_010" />
 	<xacro:property name="rightArmJ2SerialNumber" value="v_b_008" />
 	<xacro:property name="rightArmJ3SerialNumber" value="v_f_009" />
 	<xacro:property name="rightArmJ4SerialNumber" value="v_f_010" />
-        <xacro:property name="rightArmJ5SerialNumber" value="v_g_020" />
-        <xacro:property name="rightForearmSerialNumber" value="v_h_004"/>
+        <xacro:property name="rightArmJ5SerialNumber" value="v_g_012" />
+        <xacro:property name="rightForearmSerialNumber" value="v_h_006"/>
 	<xacro:property name="neckJ1SerialNumber" value="v_g_019" />
 	<xacro:property name="neckJ2SerialNumber" value="v_g_010" />

Commit message: swaping legs

File: common/xacro/serial_numbers/valkyrie_B_serials.xacro (robot description, xacro)
@@ -1,15 +1,15 @@
 <robot xmlns:xacro="http://ros.org/wiki/xacro" name="valkyrie_B_serials">
 	<xacro:property name="leftLegJ1SerialNumber" value="v_a_009" />
-        <xacro:property name="leftLegJ2SerialNumber" value="v_b_006" />
-        <xacro:property name="leftLegJ3SerialNumber" value="v_c_004" />
-        <xacro:property name="leftLegJ4SerialNumber" value="v_d_003" />
-        <xacro:property name="leftAnkleLeftActuatorSerialNumber" value="v_e_019" />
-       <xacro:property name="leftAnkleRightActuatorSerialNumber" value="v_e_020" />
+        <xacro:property name="leftLegJ2SerialNumber" value="v_b_011" />
+    <xacro:property name="leftLegJ3SerialNumber" value="v_c_007" />
+    <xacro:property name="leftLegJ4SerialNumber" value="v_d_007" />
+    <xacro:property name="leftAnkleLeftActuatorSerialNumber" value="v_e_009" />
+    <xacro:property name="leftAnkleRightActuatorSerialNumber" value="v_e_010" />
 	<xacro:property name="rightLegJ1SerialNumber" value="v_a_007" />
-    <xacro:property name="rightLegJ2SerialNumber" value="v_b_001" />
-    <xacro:property name="rightLegJ3SerialNumber" value="v_c_001" />
-    <xacro:property name="rightLegJ4SerialNumber" value="v_d_004" />
-    <xacro:property name="rightAnkleLeftActuatorSerialNumber" value="v_e_003" />
-    <xacro:property name="rightAnkleRightActuatorSerialNumber" value="v_e_004" />
+       <xacro:property name="rightLegJ2SerialNumber" value="v_b_010" />
+    <xacro:property name="rightLegJ3SerialNumber" value="v_c_006" />
+    <xacro:property name="rightLegJ4SerialNumber" value="v_d_006" />
+    <xacro:property name="rightAnkleRightActuatorSerialNumber" value="v_e_008" />
+    <xacro:property name="rightAnkleLeftActuatorSerialNumber" value="v_e_007" />
 	<xacro:property name="leftArmJ1SerialNumber" value="v_a_002" />
 	<xacro:property name="leftArmJ2SerialNumber" value="v_b_005" />

File: common/xacro/serial_numbers/valkyrie_D_serials.xacro (robot description, xacro)
@@ -1,15 +1,15 @@
 <robot xmlns:xacro="http://ros.org/wiki/xacro" name="valkyrie_D_serials">
     <xacro:property name="leftLegJ1SerialNumber" value="v_a_017" />
-    <xacro:property name="leftLegJ2SerialNumber" value="v_b_011" />
-    <xacro:property name="leftLegJ3SerialNumber" value="v_c_007" />
-    <xacro:property name="leftLegJ4SerialNumber" value="v_d_007" />
-    <xacro:property name="leftAnkleLeftActuatorSerialNumber" value="v_e_009" />
-    <xacro:property name="leftAnkleRightActuatorSerialNumber" value="v_e_010" />
+    <xacro:property name="leftLegJ2SerialNumber" value="v_b_006" />
+        <xacro:property name="leftLegJ3SerialNumber" value="v_c_004" />
+        <xacro:property name="leftLegJ4SerialNumber" value="v_d_003" />
+        <xacro:property name="leftAnkleLeftActuatorSerialNumber" value="v_e_019" />
+       <xacro:property name="leftAnkleRightActuatorSerialNumber" value="v_e_020" />
     <xacro:property name="rightLegJ1SerialNumber" value="v_a_018" />
-   <xacro:property name="rightLegJ2SerialNumber" value="v_b_010" />
-    <xacro:property name="rightLegJ3SerialNumber" value="v_c_006" />
-    <xacro:property name="rightLegJ4SerialNumber" value="v_d_006" />
-    <xacro:property name="rightAnkleRightActuatorSerialNumber" value="v_e_008" />
-    <xacro:property name="rightAnkleLeftActuatorSerialNumber" value="v_e_007" />
+    <xacro:property name="rightLegJ2SerialNumber" value="v_b_001" />
+    <xacro:property name="rightLegJ3SerialNumber" value="v_c_001" />
+    <xacro:property name="rightLegJ4SerialNumber" value="v_d_004" />
+    <xacro:property name="rightAnkleLeftActuatorSerialNumber" value="v_e_003" />
+    <xacro:property name="rightAnkleRightActuatorSerialNumber" value="v_e_004" />
     <xacro:property name="leftArmJ1SerialNumber" value="v_a_019" />
     <xacro:property name="leftArmJ2SerialNumber" value="v_b_014" />

Commit message: switch b and d legs

File: common/xacro/serial_numbers/valkyrie_B_serials.xacro (robot description, xacro)
@@ -1,15 +1,15 @@
 <robot xmlns:xacro="http://www.ros.org/wiki/xacro" name="valkyrie_B_serials">
 	<xacro:property name="leftLegJ1SerialNumber" value="v_a_009" />
-        <xacro:property name="leftLegJ2SerialNumber" value="v_b_011" />
-    <xacro:property name="leftLegJ3SerialNumber" value="v_c_007" />
-    <xacro:property name="leftLegJ4SerialNumber" value="v_d_007" />
-    <xacro:property name="leftAnkleLeftActuatorSerialNumber" value="v_e_009" />
-    <xacro:property name="leftAnkleRightActuatorSerialNumber" value="v_e_010" />
+    <xacro:property name="leftLegJ2SerialNumber" value="v_b_006" />
+        <xacro:property name="leftLegJ3SerialNumber" value="v_c_004" />
+        <xacro:property name="leftLegJ4SerialNumber" value="v_d_003" />
+        <xacro:property name="leftAnkleLeftActuatorSerialNumber" value="v_e_019" />
+       <xacro:property name="leftAnkleRightActuatorSerialNumber" value="v_e_020" />
 	<xacro:property name="rightLegJ1SerialNumber" value="v_a_007" />
-       <xacro:property name="rightLegJ2SerialNumber" value="v_b_010" />
-    <xacro:property name="rightLegJ3SerialNumber" value="v_c_006" />
-    <xacro:property name="rightLegJ4SerialNumber" value="v_d_006" />
-    <xacro:property name="rightAnkleRightActuatorSerialNumber" value="v_e_008" />
-    <xacro:property name="rightAnkleLeftActuatorSerialNumber" value="v_e_007" />
+    <xacro:property name="rightLegJ2SerialNumber" value="v_b_001" />
+    <xacro:property name="rightLegJ3SerialNumber" value="v_c_001" />
+    <xacro:property name="rightLegJ4SerialNumber" value="v_d_004" />
+    <xacro:property name="rightAnkleLeftActuatorSerialNumber" value="v_e_003" />
+    <xacro:property name="rightAnkleRightActuatorSerialNumber" value="v_e_004" />
 	<xacro:property name="leftArmJ1SerialNumber" value="v_a_002" />
 	<xacro:property name="leftArmJ2SerialNumber" value="v_b_005" />

File: common/xacro/serial_numbers/valkyrie_D_serials.xacro (robot description, xacro)
@@ -1,15 +1,15 @@
 <robot xmlns:xacro="http://www.ros.org/wiki/xacro" name="valkyrie_D_serials">
     <xacro:property name="leftLegJ1SerialNumber" value="v_a_017" />
-    <xacro:property name="leftLegJ2SerialNumber" value="v_b_006" />
-        <xacro:property name="leftLegJ3SerialNumber" value="v_c_004" />
-        <xacro:property name="leftLegJ4SerialNumber" value="v_d_003" />
-        <xacro:property name="leftAnkleLeftActuatorSerialNumber" value="v_e_019" />
-       <xacro:property name="leftAnkleRightActuatorSerialNumber" value="v_e_020" />
+        <xacro:property name="leftLegJ2SerialNumber" value="v_b_011" />
+    <xacro:property name="leftLegJ3SerialNumber" value="v_c_007" />
+    <xacro:property name="leftLegJ4SerialNumber" value="v_d_007" />
+    <xacro:property name="leftAnkleLeftActuatorSerialNumber" value="v_e_009" />
+    <xacro:property name="leftAnkleRightActuatorSerialNumber" value="v_e_010" />
     <xacro:property name="rightLegJ1SerialNumber" value="v_a_018" />
-    <xacro:property name="rightLegJ2SerialNumber" value="v_b_001" />
-    <xacro:property name="rightLegJ3SerialNumber" value="v_c_001" />
-    <xacro:property name="rightLegJ4SerialNumber" value="v_d_004" />
-    <xacro:property name="rightAnkleLeftActuatorSerialNumber" value="v_e_003" />
-    <xacro:property name="rightAnkleRightActuatorSerialNumber" value="v_e_004" />
+       <xacro:property name="rightLegJ2SerialNumber" value="v_b_010" />
+    <xacro:property name="rightLegJ3SerialNumber" value="v_c_006" />
+    <xacro:property name="rightLegJ4SerialNumber" value="v_d_006" />
+    <xacro:property name="rightAnkleRightActuatorSerialNumber" value="v_e_008" />
+    <xacro:property name="rightAnkleLeftActuatorSerialNumber" value="v_e_007" />
     <xacro:property name="leftArmJ1SerialNumber" value="v_a_019" />
     <xacro:property name="leftArmJ2SerialNumber" value="v_b_014" />
