Commit message: Changed rear IMU so updated port. Recalibrated left forearm yaw and updated the serial number since we put a new forearm on unit D.

File: common/xacro/serial_numbers/valkyrie_D_serials.xacro (robot description, xacro)
@@ -16,5 +16,5 @@
     <xacro:property name="leftArmJ3SerialNumber" value="v_f_017" />
     <xacro:property name="leftArmJ4SerialNumber" value="v_f_016" />
-    <xacro:property name="leftArmJ5SerialNumber" value="v_g_016" />
+    <xacro:property name="leftArmJ5SerialNumber" value="v_g_018" />
     <xacro:property name="rightArmJ1SerialNumber" value="v_a_016" />
     <xacro:property name="rightArmJ2SerialNumber" value="v_b_013" />
@@ -28,5 +28,5 @@
     <xacro:property name="waistRightActuatorSerialNumber" value="v_e_023" />
     <xacro:property name="waistLeftActuatorSerialNumber" value="v_e_024" />
-    <xacro:property name="leftForearmSerialNumber" value="v_h_005"/>
+    <xacro:property name="leftForearmSerialNumber" value="v_h_007"/>
     <xacro:property name="rightForearmSerialNumber" value="v_h_006"/>
     <xacro:property name="left_foot_ATI_serial" value="FT17212" />

Commit message: updated D to have the correct forearms

File: common/xacro/serial_numbers/valkyrie_D_serials.xacro (robot description, xacro)
@@ -16,12 +16,12 @@
     <xacro:property name="leftArmJ3SerialNumber" value="v_f_017" />
     <xacro:property name="leftArmJ4SerialNumber" value="v_f_016" />
-    <xacro:property name="leftArmJ5SerialNumber" value="v_g_016" />
-    <xacro:property name="leftForearmSerialNumber" value="v_h_005" />
+    <xacro:property name="leftArmJ5SerialNumber" value="v_g_021" />
+    <xacro:property name="leftForearmSerialNumber" value="v_h_003" />
     <xacro:property name="rightArmJ1SerialNumber" value="v_a_016" />
     <xacro:property name="rightArmJ2SerialNumber" value="v_b_013" />
     <xacro:property name="rightArmJ3SerialNumber" value="v_f_018" />
     <xacro:property name="rightArmJ4SerialNumber" value="v_f_015" />
-    <xacro:property name="rightArmJ5SerialNumber" value="v_g_012" />
-    <xacro:property name="rightForearmSerialNumber" value="v_h_006"/>
+    <xacro:property name="rightArmJ5SerialNumber" value="v_g_020" />
+    <xacro:property name="rightForearmSerialNumber" value="v_h_004"/>
     <xacro:property name="neckJ1SerialNumber" value="v_g_014" />
     <xacro:property name="neckJ2SerialNumber" value="v_g_013" />
