Commit message: updated serial numbers for delivery of new legs to MIT

File: common/xacro/serial_numbers/valkyrie_A_serials.xacro (robot description, xacro)
@@ -1,15 +1,15 @@
 <robot xmlns:xacro="http://ros.org/wiki/xacro" name="valkyrie_A_serials">
 	<xacro:property name="leftLegJ1SerialNumber" value="v_a_006" />
-	<xacro:property name="leftLegJ2SerialNumber" value="v_b_006" />
-    <xacro:property name="leftLegJ3SerialNumber" value="v_c_004" />
-    <xacro:property name="leftLegJ4SerialNumber" value="v_d_003" />
+	<xacro:property name="leftLegJ2SerialNumber" value="v_b_016" />
+    <xacro:property name="leftLegJ3SerialNumber" value="v_c_008" />
+    <xacro:property name="leftLegJ4SerialNumber" value="v_d_008" />
     <xacro:property name="leftAnkleLeftActuatorSerialNumber" value="v_e_016" />
 	<xacro:property name="leftAnkleRightActuatorSerialNumber" value="v_e_015" />
 	<xacro:property name="rightLegJ1SerialNumber" value="v_a_003" />
-	<xacro:property name="rightLegJ2SerialNumber" value="v_b_001" />
-	<xacro:property name="rightLegJ3SerialNumber" value="v_c_001" />
-	<xacro:property name="rightLegJ4SerialNumber" value="v_d_004" />
-	<xacro:property name="rightAnkleLeftActuatorSerialNumber" value="v_e_003" />
-	<xacro:property name="rightAnkleRightActuatorSerialNumber" value="v_e_004" />
+	<xacro:property name="rightLegJ2SerialNumber" value="v_b_015" />
+	<xacro:property name="rightLegJ3SerialNumber" value="v_c_009" />
+	<xacro:property name="rightLegJ4SerialNumber" value="v_d_009" />
+	<xacro:property name="rightAnkleLeftActuatorSerialNumber" value="v_e_021" />
+	<xacro:property name="rightAnkleRightActuatorSerialNumber" value="v_e_022" />
 	<xacro:property name="leftArmJ1SerialNumber" value="v_a_005" />
 	<xacro:property name="leftArmJ2SerialNumber" value="v_b_004" />

File: common/xacro/serial_numbers/valkyrie_B_serials.xacro (robot description, xacro)
@@ -1,15 +1,15 @@
 <robot xmlns:xacro="http://ros.org/wiki/xacro" name="valkyrie_B_serials">
 	<xacro:property name="leftLegJ1SerialNumber" value="v_a_009" />
-    <xacro:property name="leftLegJ2SerialNumber" value="v_b_016" />
-	<xacro:property name="leftLegJ3SerialNumber" value="v_c_008" />
-	<xacro:property name="leftLegJ4SerialNumber" value="v_d_008" />
+    <xacro:property name="leftLegJ2SerialNumber" value="v_b_006" />
+	<xacro:property name="leftLegJ3SerialNumber" value="v_c_004" />
+	<xacro:property name="leftLegJ4SerialNumber" value="v_d_003" />
 	<xacro:property name="leftAnkleLeftActuatorSerialNumber" value="v_e_019" />
     <xacro:property name="leftAnkleRightActuatorSerialNumber" value="v_e_020" />
 	<xacro:property name="rightLegJ1SerialNumber" value="v_a_007" />
-	<xacro:property name="rightLegJ2SerialNumber" value="v_b_015" />
-    <xacro:property name="rightLegJ3SerialNumber" value="v_c_009" />
-    <xacro:property name="rightLegJ4SerialNumber" value="v_d_009" />
-    <xacro:property name="rightAnkleLeftActuatorSerialNumber" value="v_e_021" />
-    <xacro:property name="rightAnkleRightActuatorSerialNumber" value="v_e_022" />
+	<xacro:property name="rightLegJ2SerialNumber" value="v_b_001" />
+    <xacro:property name="rightLegJ3SerialNumber" value="v_c_001" />
+    <xacro:property name="rightLegJ4SerialNumber" value="v_d_004" />
+    <xacro:property name="rightAnkleLeftActuatorSerialNumber" value="v_e_003" />
+    <xacro:property name="rightAnkleRightActuatorSerialNumber" value="v_e_004" />
 	<xacro:property name="leftArmJ1SerialNumber" value="v_a_002" />
 	<xacro:property name="leftArmJ2SerialNumber" value="v_b_005" />

Commit message: swapped ATI for right leg

File: common/xacro/serial_numbers/valkyrie_A_serials.xacro (robot description, xacro)
@@ -31,5 +31,5 @@
     <xacro:property name="rightForearmSerialNumber" value="v_h_008"/>
 	<xacro:property name="left_foot_ATI_serial" value="FT17218" />
-	<xacro:property name="right_foot_ATI_serial" value="FT16592" />
+	<xacro:property name="right_foot_ATI_serial" value="FT14018" />
 	<xacro:property name="sim_ATI_serial" value="FT001SIM" />
 </robot>

File: common/xacro/serial_numbers/valkyrie_B_serials.xacro (robot description, xacro)
@@ -31,5 +31,5 @@
     <xacro:property name="rightForearmSerialNumber" value="v_h_004"/>
 	<xacro:property name="left_foot_ATI_serial" value="FT16594" />
-	<xacro:property name="right_foot_ATI_serial" value="FT14018" />
+	<xacro:property name="right_foot_ATI_serial" value="FT16592" />
     <xacro:property name="sim_ATI_serial" value="FT001SIM" />
 </robot>

Commit message: updated serial number for left arm j4

File: common/xacro/serial_numbers/valkyrie_A_serials.xacro (robot description, xacro)
@@ -15,5 +15,5 @@
 	<xacro:property name="leftArmJ2SerialNumber" value="v_b_004" />
 	<xacro:property name="leftArmJ3SerialNumber" value="v_f_005" />
-	<xacro:property name="leftArmJ4SerialNumber" value="v_f_002" />
+	<xacro:property name="leftArmJ4SerialNumber" value="v_f_020" />
 	<xacro:property name="leftArmJ5SerialNumber" value="v_g_018" />
 	<xacro:property name="rightArmJ1SerialNumber" value="v_a_001" />

Commit message: updating

File: common/xacro/serial_numbers/valkyrie_A_serials.xacro (robot description, xacro)
@@ -16,5 +16,6 @@
 	<xacro:property name="leftArmJ3SerialNumber" value="v_f_005" />
 	<xacro:property name="leftArmJ4SerialNumber" value="v_f_020" />
-	<xacro:property name="leftArmJ5SerialNumber" value="v_g_018" />
+	<xacro:property name="leftArmJ5SerialNumber" value="v_g_005" />
+	<!-- <xacro:property name="leftArmJ5SerialNumber" value="v_g_018" /> -->
 	<xacro:property name="rightArmJ1SerialNumber" value="v_a_001" />
 	<xacro:property name="rightArmJ2SerialNumber" value="v_b_003" />
@@ -28,6 +29,7 @@
 	<xacro:property name="waistRightActuatorSerialNumber" value="v_e_005" />
 	<xacro:property name="waistLeftActuatorSerialNumber" value="v_e_006" />
-	<xacro:property name="leftForearmSerialNumber" value="v_h_007"/>
-    <xacro:property name="rightForearmSerialNumber" value="v_h_008"/>
+	<xacro:property name="leftForearmSerialNumber" value="v_h_001"/>
+	<!-- <xacro:property name="leftForearmSerialNumber" value="v_h_007"/> -->
+    	<xacro:property name="rightForearmSerialNumber" value="v_h_008"/>
 	<xacro:property name="left_foot_ATI_serial" value="FT17218" />
 	<xacro:property name="right_foot_ATI_serial" value="FT14018" />

Commit message: updating serials and removing gear ratio form actuator files

File: common/xacro/serial_numbers/valkyrie_A_serials.xacro (robot description, xacro)
@@ -16,6 +16,5 @@
 	<xacro:property name="leftArmJ3SerialNumber" value="v_f_005" />
 	<xacro:property name="leftArmJ4SerialNumber" value="v_f_020" />
-	<xacro:property name="leftArmJ5SerialNumber" value="v_g_005" />
-	<!-- <xacro:property name="leftArmJ5SerialNumber" value="v_g_018" /> -->
+	<xacro:property name="leftArmJ5SerialNumber" value="v_g_016" />
 	<xacro:property name="rightArmJ1SerialNumber" value="v_a_001" />
 	<xacro:property name="rightArmJ2SerialNumber" value="v_b_003" />
@@ -29,6 +28,5 @@
 	<xacro:property name="waistRightActuatorSerialNumber" value="v_e_005" />
 	<xacro:property name="waistLeftActuatorSerialNumber" value="v_e_006" />
-	<xacro:property name="leftForearmSerialNumber" value="v_h_001"/>
-	<!-- <xacro:property name="leftForearmSerialNumber" value="v_h_007"/> -->
+	<xacro:property name="leftForearmSerialNumber" value="v_h_005"/>
     	<xacro:property name="rightForearmSerialNumber" value="v_h_008"/>
 	<xacro:property name="left_foot_ATI_serial" value="FT17218" />

Commit message: swapped legs for unit A and unit D to support UOE

File: common/xacro/serial_numbers/valkyrie_A_serials.xacro (robot description, xacro)
@@ -1,15 +1,15 @@
 <robot xmlns:xacro="http://ros.org/wiki/xacro" name="valkyrie_A_serials">
-	<xacro:property name="leftLegJ1SerialNumber" value="v_a_006" />
-	<xacro:property name="leftLegJ2SerialNumber" value="v_b_016" />
-    <xacro:property name="leftLegJ3SerialNumber" value="v_c_008" />
-    <xacro:property name="leftLegJ4SerialNumber" value="v_d_008" />
-    <xacro:property name="leftAnkleLeftActuatorSerialNumber" value="v_e_016" />
-	<xacro:property name="leftAnkleRightActuatorSerialNumber" value="v_e_015" />
-	<xacro:property name="rightLegJ1SerialNumber" value="v_a_003" />
-	<xacro:property name="rightLegJ2SerialNumber" value="v_b_015" />
-	<xacro:property name="rightLegJ3SerialNumber" value="v_c_009" />
-	<xacro:property name="rightLegJ4SerialNumber" value="v_d_009" />
-	<xacro:property name="rightAnkleLeftActuatorSerialNumber" value="v_e_021" />
-	<xacro:property name="rightAnkleRightActuatorSerialNumber" value="v_e_022" />
+    <xacro:property name="leftLegJ1SerialNumber" value="v_a_017" />
+    <xacro:property name="leftLegJ2SerialNumber" value="v_b_011" />
+    <xacro:property name="leftLegJ3SerialNumber" value="v_c_007" />
+    <xacro:property name="leftLegJ4SerialNumber" value="v_d_007" />
+    <xacro:property name="leftAnkleLeftActuatorSerialNumber" value="v_e_009" />
+    <xacro:property name="leftAnkleRightActuatorSerialNumber" value="v_e_010" />
+    <xacro:property name="rightLegJ1SerialNumber" value="v_a_018" />
+    <xacro:property name="rightLegJ2SerialNumber" value="v_b_010" />
+    <xacro:property name="rightLegJ3SerialNumber" value="v_c_006" />
+    <xacro:property name="rightLegJ4SerialNumber" value="v_d_006" />
+    <xacro:property name="rightAnkleRightActuatorSerialNumber" value="v_e_008" />
+    <xacro:property name="rightAnkleLeftActuatorSerialNumber" value="v_e_007" />
 	<xacro:property name="leftArmJ1SerialNumber" value="v_a_005" />
 	<xacro:property name="leftArmJ2SerialNumber" value="v_b_004" />

File: common/xacro/serial_numbers/valkyrie_D_serials.xacro (robot description, xacro)
@@ -1,15 +1,15 @@
 <robot xmlns:xacro="http://ros.org/wiki/xacro" name="valkyrie_D_serials">
-    <xacro:property name="leftLegJ1SerialNumber" value="v_a_017" />
-    <xacro:property name="leftLegJ2SerialNumber" value="v_b_011" />
-    <xacro:property name="leftLegJ3SerialNumber" value="v_c_007" />
-    <xacro:property name="leftLegJ4SerialNumber" value="v_d_007" />
-    <xacro:property name="leftAnkleLeftActuatorSerialNumber" value="v_e_009" />
-    <xacro:property name="leftAnkleRightActuatorSerialNumber" value="v_e_010" />
-    <xacro:property name="rightLegJ1SerialNumber" value="v_a_018" />
-    <xacro:property name="rightLegJ2SerialNumber" value="v_b_010" />
-    <xacro:property name="rightLegJ3SerialNumber" value="v_c_006" />
-    <xacro:property name="rightLegJ4SerialNumber" value="v_d_006" />
-    <xacro:property name="rightAnkleRightActuatorSerialNumber" value="v_e_008" />
-    <xacro:property name="rightAnkleLeftActuatorSerialNumber" value="v_e_007" />
+	<xacro:property name="leftLegJ1SerialNumber" value="v_a_006" />
+	<xacro:property name="leftLegJ2SerialNumber" value="v_b_016" />
+    <xacro:property name="leftLegJ3SerialNumber" value="v_c_008" />
+    <xacro:property name="leftLegJ4SerialNumber" value="v_d_008" />
+    <xacro:property name="leftAnkleLeftActuatorSerialNumber" value="v_e_016" />
+	<xacro:property name="leftAnkleRightActuatorSerialNumber" value="v_e_015" />
+	<xacro:property name="rightLegJ1SerialNumber" value="v_a_003" />
+	<xacro:property name="rightLegJ2SerialNumber" value="v_b_015" />
+	<xacro:property name="rightLegJ3SerialNumber" value="v_c_009" />
+	<xacro:property name="rightLegJ4SerialNumber" value="v_d_009" />
+	<xacro:property name="rightAnkleLeftActuatorSerialNumber" value="v_e_021" />
+	<xacro:property name="rightAnkleRightActuatorSerialNumber" value="v_e_022" />
     <xacro:property name="leftArmJ1SerialNumber" value="v_a_019" />
     <xacro:property name="leftArmJ2SerialNumber" value="v_b_014" />

Commit message: swapped back j1s since they don't go with the legs

File: common/xacro/serial_numbers/valkyrie_A_serials.xacro (robot description, xacro)
@@ -1,4 +1,4 @@
 <robot xmlns:xacro="http://ros.org/wiki/xacro" name="valkyrie_A_serials">
-    <xacro:property name="leftLegJ1SerialNumber" value="v_a_017" />
+	<xacro:property name="leftLegJ1SerialNumber" value="v_a_006" />
     <xacro:property name="leftLegJ2SerialNumber" value="v_b_011" />
     <xacro:property name="leftLegJ3SerialNumber" value="v_c_007" />
@@ -6,5 +6,5 @@
     <xacro:property name="leftAnkleLeftActuatorSerialNumber" value="v_e_009" />
     <xacro:property name="leftAnkleRightActuatorSerialNumber" value="v_e_010" />
-    <xacro:property name="rightLegJ1SerialNumber" value="v_a_018" />
+	<xacro:property name="rightLegJ1SerialNumber" value="v_a_003" />
     <xacro:property name="rightLegJ2SerialNumber" value="v_b_010" />
     <xacro:property name="rightLegJ3SerialNumber" value="v_c_006" />

File: common/xacro/serial_numbers/valkyrie_D_serials.xacro (robot description, xacro)
@@ -1,4 +1,4 @@
 <robot xmlns:xacro="http://ros.org/wiki/xacro" name="valkyrie_D_serials">
-	<xacro:property name="leftLegJ1SerialNumber" value="v_a_006" />
+    <xacro:property name="leftLegJ1SerialNumber" value="v_a_017" />
 	<xacro:property name="leftLegJ2SerialNumber" value="v_b_016" />
     <xacro:property name="leftLegJ3SerialNumber" value="v_c_008" />
@@ -6,5 +6,5 @@
     <xacro:property name="leftAnkleLeftActuatorSerialNumber" value="v_e_016" />
 	<xacro:property name="leftAnkleRightActuatorSerialNumber" value="v_e_015" />
-	<xacro:property name="rightLegJ1SerialNumber" value="v_a_003" />
+    <xacro:property name="rightLegJ1SerialNumber" value="v_a_018" />
 	<xacro:property name="rightLegJ2SerialNumber" value="v_b_015" />
 	<xacro:property name="rightLegJ3SerialNumber" value="v_c_009" />

Commit message: calibration and part swap for robots

File: common/xacro/serial_numbers/valkyrie_A_serials.xacro (robot description, xacro)
@@ -16,12 +16,12 @@
 	<xacro:property name="leftArmJ3SerialNumber" value="v_f_005" />
 	<xacro:property name="leftArmJ4SerialNumber" value="v_f_020" />
-	<xacro:property name="leftArmJ5SerialNumber" value="v_g_016" />
-	<xacro:property name="left_hand_serial_number" value="v_h_005" />
+        <xacro:property name="leftArmJ5SerialNumber" value="v_g_007" />
+        <xacro:property name="leftForearmSerialNumber" value="v_h_003"/>
 	<xacro:property name="rightArmJ1SerialNumber" value="v_a_001" />
 	<xacro:property name="rightArmJ2SerialNumber" value="v_b_003" />
 	<xacro:property name="rightArmJ3SerialNumber" value="v_f_004" />
 	<xacro:property name="rightArmJ4SerialNumber" value="v_f_003" />
-	<xacro:property name="rightArmJ5SerialNumber" value="v_g_017" />
-	<xacro:property name="right_hand_serial_number" value="v_h_008" />
+        <xacro:property name="rightArmJ5SerialNumber" value="v_g_006" />
+        <xacro:property name="rightForearmSerialNumber" value="v_h_004"/>
 	<xacro:property name="neckJ1SerialNumber" value="v_g_006" />
 	<xacro:property name="neckJ2SerialNumber" value="v_g_007" />

File: common/xacro/serial_numbers/valkyrie_B_serials.xacro (robot description, xacro)
@@ -1,11 +1,11 @@
 <robot xmlns:xacro="http://ros.org/wiki/xacro" name="valkyrie_B_serials">
 	<xacro:property name="leftLegJ1SerialNumber" value="v_a_009" />
-    <xacro:property name="leftLegJ2SerialNumber" value="v_b_006" />
-	<xacro:property name="leftLegJ3SerialNumber" value="v_c_004" />
-	<xacro:property name="leftLegJ4SerialNumber" value="v_d_003" />
-	<xacro:property name="leftAnkleLeftActuatorSerialNumber" value="v_e_019" />
-    <xacro:property name="leftAnkleRightActuatorSerialNumber" value="v_e_020" />
+        <xacro:property name="leftLegJ2SerialNumber" value="v_b_006" />
+        <xacro:property name="leftLegJ3SerialNumber" value="v_c_004" />
+        <xacro:property name="leftLegJ4SerialNumber" value="v_d_003" />
+        <xacro:property name="leftAnkleLeftActuatorSerialNumber" value="v_e_019" />
+       <xacro:property name="leftAnkleRightActuatorSerialNumber" value="v_e_020" />
 	<xacro:property name="rightLegJ1SerialNumber" value="v_a_007" />
-	<xacro:property name="rightLegJ2SerialNumber" value="v_b_001" />
+    <xacro:property name="rightLegJ2SerialNumber" value="v_b_001" />
     <xacro:property name="rightLegJ3SerialNumber" value="v_c_001" />
     <xacro:property name="rightLegJ4SerialNumber" value="v_d_004" />
@@ -16,10 +16,12 @@
 	<xacro:property name="leftArmJ3SerialNumber" value="v_f_007" />
 	<xacro:property name="leftArmJ4SerialNumber" value="v_f_008" />
-	<xacro:property name="leftArmJ5SerialNumber" value="v_g_007" />
+        <xacro:property name="leftArmJ5SerialNumber" value="v_g_018" />
+        <xacro:property name="leftForearmSerialNumber" value="v_h_007"/>
 	<xacro:property name="rightArmJ1SerialNumber" value="v_a_010" />
 	<xacro:property name="rightArmJ2SerialNumber" value="v_b_008" />
 	<xacro:property name="rightArmJ3SerialNumber" value="v_f_009" />
 	<xacro:property name="rightArmJ4SerialNumber" value="v_f_010" />
-	<xacro:property name="rightArmJ5SerialNumber" value="v_g_006" />
+        <xacro:property name="rightArmJ5SerialNumber" value="v_g_017" />
+        <xacro:property name="rightForearmSerialNumber" value="v_h_008" />
 	<xacro:property name="neckJ1SerialNumber" value="v_g_019" />
 	<xacro:property name="neckJ2SerialNumber" value="v_g_010" />
@@ -28,6 +30,4 @@
 	<xacro:property name="waistRightActuatorSerialNumber" value="v_e_011" />
 	<xacro:property name="waistLeftActuatorSerialNumber" value="v_e_012" />
-	<xacro:property name="leftForearmSerialNumber" value="v_h_003"/>
-    <xacro:property name="rightForearmSerialNumber" value="v_h_004"/>
 	<xacro:property name="left_foot_ATI_serial" value="FT16594" />
 	<xacro:property name="right_foot_ATI_serial" value="FT16592" />

File: common/xacro/serial_numbers/valkyrie_D_serials.xacro (robot description, xacro)
@@ -16,5 +16,6 @@
     <xacro:property name="leftArmJ3SerialNumber" value="v_f_017" />
     <xacro:property name="leftArmJ4SerialNumber" value="v_f_016" />
-    <xacro:property name="leftArmJ5SerialNumber" value="v_g_018" />
+    <xacro:property name="leftArmJ5SerialNumber" value="v_g_016" />
+    <xacro:property name="leftForearmSerialNumber" value="v_h_005" />
     <xacro:property name="rightArmJ1SerialNumber" value="v_a_016" />
     <xacro:property name="rightArmJ2SerialNumber" value="v_b_013" />
@@ -22,4 +23,5 @@
     <xacro:property name="rightArmJ4SerialNumber" value="v_f_015" />
     <xacro:property name="rightArmJ5SerialNumber" value="v_g_012" />
+    <xacro:property name="rightForearmSerialNumber" value="v_h_006"/>
     <xacro:property name="neckJ1SerialNumber" value="v_g_014" />
     <xacro:property name="neckJ2SerialNumber" value="v_g_013" />
@@ -28,6 +30,4 @@
     <xacro:property name="waistRightActuatorSerialNumber" value="v_e_023" />
     <xacro:property name="waistLeftActuatorSerialNumber" value="v_e_024" />
-    <xacro:property name="leftForearmSerialNumber" value="v_h_007"/>
-    <xacro:property name="rightForearmSerialNumber" value="v_h_006"/>
     <xacro:property name="left_foot_ATI_serial" value="FT17212" />
     <xacro:property name="right_foot_ATI_serial" value="FT16590" />

Commit message: inital unit D setup

File: common/xacro/serial_numbers/valkyrie_A_serials.xacro (robot description, xacro)
@@ -1,15 +1,15 @@
 <robot xmlns:xacro="http://ros.org/wiki/xacro" name="valkyrie_A_serials">
 	<xacro:property name="leftLegJ1SerialNumber" value="v_a_006" />
-    <xacro:property name="leftLegJ2SerialNumber" value="v_b_011" />
-    <xacro:property name="leftLegJ3SerialNumber" value="v_c_007" />
-    <xacro:property name="leftLegJ4SerialNumber" value="v_d_007" />
-    <xacro:property name="leftAnkleLeftActuatorSerialNumber" value="v_e_009" />
-    <xacro:property name="leftAnkleRightActuatorSerialNumber" value="v_e_010" />
+        <xacro:property name="leftLegJ2SerialNumber" value="v_b_016" />
+    <xacro:property name="leftLegJ3SerialNumber" value="v_c_008" />
+    <xacro:property name="leftLegJ4SerialNumber" value="v_d_008" />
+    <xacro:property name="leftAnkleLeftActuatorSerialNumber" value="v_e_016" />
+        <xacro:property name="leftAnkleRightActuatorSerialNumber" value="v_e_015" />
 	<xacro:property name="rightLegJ1SerialNumber" value="v_a_003" />
-    <xacro:property name="rightLegJ2SerialNumber" value="v_b_010" />
-    <xacro:property name="rightLegJ3SerialNumber" value="v_c_006" />
-    <xacro:property name="rightLegJ4SerialNumber" value="v_d_006" />
-    <xacro:property name="rightAnkleRightActuatorSerialNumber" value="v_e_008" />
-    <xacro:property name="rightAnkleLeftActuatorSerialNumber" value="v_e_007" />
+       <xacro:property name="rightLegJ2SerialNumber" value="v_b_015" />
+        <xacro:property name="rightLegJ3SerialNumber" value="v_c_009" />
+        <xacro:property name="rightLegJ4SerialNumber" value="v_d_009" />
+        <xacro:property name="rightAnkleLeftActuatorSerialNumber" value="v_e_021" />
+        <xacro:property name="rightAnkleRightActuatorSerialNumber" value="v_e_022" />
 	<xacro:property name="leftArmJ1SerialNumber" value="v_a_005" />
 	<xacro:property name="leftArmJ2SerialNumber" value="v_b_004" />

File: common/xacro/serial_numbers/valkyrie_D_serials.xacro (robot description, xacro)
@@ -1,15 +1,15 @@
 <robot xmlns:xacro="http://ros.org/wiki/xacro" name="valkyrie_D_serials">
     <xacro:property name="leftLegJ1SerialNumber" value="v_a_017" />
-	<xacro:property name="leftLegJ2SerialNumber" value="v_b_016" />
-    <xacro:property name="leftLegJ3SerialNumber" value="v_c_008" />
-    <xacro:property name="leftLegJ4SerialNumber" value="v_d_008" />
-    <xacro:property name="leftAnkleLeftActuatorSerialNumber" value="v_e_016" />
-	<xacro:property name="leftAnkleRightActuatorSerialNumber" value="v_e_015" />
+    <xacro:property name="leftLegJ2SerialNumber" value="v_b_011" />
+    <xacro:property name="leftLegJ3SerialNumber" value="v_c_007" />
+    <xacro:property name="leftLegJ4SerialNumber" value="v_d_007" />
+    <xacro:property name="leftAnkleLeftActuatorSerialNumber" value="v_e_009" />
+    <xacro:property name="leftAnkleRightActuatorSerialNumber" value="v_e_010" />
     <xacro:property name="rightLegJ1SerialNumber" value="v_a_018" />
-	<xacro:property name="rightLegJ2SerialNumber" value="v_b_015" />
-	<xacro:property name="rightLegJ3SerialNumber" value="v_c_009" />
-	<xacro:property name="rightLegJ4SerialNumber" value="v_d_009" />
-	<xacro:property name="rightAnkleLeftActuatorSerialNumber" value="v_e_021" />
-	<xacro:property name="rightAnkleRightActuatorSerialNumber" value="v_e_022" />
+   <xacro:property name="rightLegJ2SerialNumber" value="v_b_010" />
+    <xacro:property name="rightLegJ3SerialNumber" value="v_c_006" />
+    <xacro:property name="rightLegJ4SerialNumber" value="v_d_006" />
+    <xacro:property name="rightAnkleRightActuatorSerialNumber" value="v_e_008" />
+    <xacro:property name="rightAnkleLeftActuatorSerialNumber" value="v_e_007" />
     <xacro:property name="leftArmJ1SerialNumber" value="v_a_019" />
     <xacro:property name="leftArmJ2SerialNumber" value="v_b_014" />
