Commit message: correct actuator for unit a right leg

File: common/xacro/serial_numbers/valkyrie_A_serials.xacro (robot description, xacro)
@@ -7,5 +7,5 @@
         <xacro:property name="leftAnkleRightActuatorSerialNumber" value="v_e_015" />
 	<xacro:property name="rightLegJ1SerialNumber" value="v_a_003" />
-       <xacro:property name="rightLegJ2SerialNumber" value="v_b_015" />
+       <xacro:property name="rightLegJ2SerialNumber" value="v_b_017" />
         <xacro:property name="rightLegJ3SerialNumber" value="v_c_009" />
         <xacro:property name="rightLegJ4SerialNumber" value="v_d_009" />
