Commit message: Revived the ol' test bench xacro

File: common/xacro/nodes/actuator_testbench_nodes.xacro (robot description, xacro)
@@ -1,3 +1,3 @@
 <robot xmlns:xacro="http://ros.org/wiki/xacro" name="test_bench_nodes">
-	<xacro:property name="testbenchNode" value="/right_arm/j2" />
+	<xacro:property name="testbench_node" value="/right_leg/j4" />
 </robot>

File: common/xacro/serial_numbers/test_bench_serials.xacro (robot description, xacro)
@@ -1,3 +1,3 @@
 <robot xmlns:xacro="http://ros.org/wiki/xacro" name="test_bench_serials">
-	<xacro:property name="testbench_serial_number" value="v_g_016" />
+	<xacro:property name="testbench_serial_number" value="v_c_010" />
 </robot>

File: instance/instances/robots/xacro/common/test_bench_template.xacro (robot description, xacro)
@@ -1,11 +1,14 @@
 <robot xmlns:xacro="http://ros.org/wiki/xacro" name="test_bench_template">
 	<xacro:include filename="$(find val_description)/common/xacro/serial_numbers/test_bench_serials.xacro" />
-	<xacro:include filename="$(find val_description)/common/xacro/nodes/test_bench_nodes.xacro" />
+	<xacro:include filename="$(find val_description)/common/xacro/nodes/actuator_testbench_nodes.xacro" />
 	<xacro:include filename="$(find val_description)/instance/instances/robots/xacro/mechanisms/mechanisms.xacro"/>
+	<xacro:include filename="$(find val_description)/common/xacro/firmware/valkyrie_firmware.xacro"/>
 	<RobotInstance id="testbench" />
 	<Channels>
 	</Channels>
+	<xacro:all_channels/>
+        <xacro:firmware_base_url/>
 	<Mechanisms>
-		<xacro:simple_mechanism name="testbench_actuator" serial_number="${testbench_serial_number}" node="${testbench_node}"/>
+		<xacro:simple_mechanism name="testbench_actuator" serial_number="${testbench_serial_number}" node="${testbench_node}" processor_firmware="" fpga_firmware=""/>
 	</Mechanisms>
 	<Devices>

File: model/robots/test_bench.xacro (robot description, xacro)
@@ -8,5 +8,5 @@
       </joint>
       <actuator name="testbenchActuator">
-        <node name="${testbenchNode}"/>
+        <node name="${testbench_node}"/>
         <mechanicalReduction>1</mechanicalReduction>
         <api name="${testbenchApi}" />

Commit message: New batch of Unit E actuators

File: common/xacro/nodes/actuator_testbench_nodes.xacro (robot description, xacro)
@@ -1,3 +1,3 @@
 <robot xmlns:xacro="http://ros.org/wiki/xacro" name="test_bench_nodes">
-	<xacro:property name="testbench_node" value="/right_leg/j4" />
+	<xacro:property name="testbench_node" value="/right_leg/j3" />
 </robot>

File: common/xacro/serial_numbers/test_bench_serials.xacro (robot description, xacro)
@@ -1,3 +1,3 @@
 <robot xmlns:xacro="http://ros.org/wiki/xacro" name="test_bench_serials">
-	<xacro:property name="testbench_serial_number" value="v_c_010" />
+	<xacro:property name="testbench_serial_number" value="v_g_022" />
 </robot>
