Commit message: added hand mechanism

File: common/xacro/nodes/forearm_testbench_nodes.xacro (robot description, xacro)
@@ -1,5 +1,11 @@
 <robot xmlns:xacro="http://ros.org/wiki/xacro" name="test_bench_nodes">
-	<xacro:property name="testbench_node" value="/left_arm/j5" />
-	<xacro:property name="Athena1Node" value="/left_arm/athena1" />
-	<xacro:property name="Athena2Node" value="/left_arm/athena2" />
+    <xacro:property name="testbench_node" value="/right_arm/j5" />
+    <xacro:property name="IndexNode" value="/right_arm/hand/index" />
+    <xacro:property name="MiddleNode" value="/right_arm/hand/middle" />
+    <xacro:property name="PinkyNode" value="/right_arm/hand/pinky" />
+    <xacro:property name="ThumbProxNode" value="/right_arm/hand/thumb_proximal" />
+    <xacro:property name="ThumbDistNode" value="/right_arm/hand/thumb_distal" />
+    <xacro:property name="ThumbRollNode" value="/right_arm/hand/thumb_roll" />
+    <xacro:property name="WristLeftNode" value="/right_arm/wrist/left_actuator" />
+    <xacro:property name="WristRightNode" value="/right_arm/wrist/right_actuator" />
 </robot>

File: common/xacro/serial_numbers/forearm_right_testbench_serials.xacro (robot description, xacro)
@@ -1,4 +1,4 @@
 <robot xmlns:xacro="http://ros.org/wiki/xacro" name="forearm_testbench">
-	<xacro:property name="forearm_serial_number" value="v_h_002" />
-	<xacro:property name="forearm_yaw_serial_number" value="v_g_003" />
+    <xacro:property name="forearm_serial_number" value="v_h_002" />
+    <xacro:property name="forearm_yaw_serial_number" value="v_g_017" />
 </robot>

File: common/xacro/serial_numbers/forearm_testbench_serials.xacro (robot description, xacro)
@@ -1,4 +1,4 @@
 <robot xmlns:xacro="http://ros.org/wiki/xacro" name="forearm_testbench">
-	<xacro:property name="forearm_yaw_serial_number" value="v_g_016" />
-	<xacro:property name="forearm_serial_number" value="v_h_005" />
+	<xacro:property name="forearm_yaw_serial_number" value="v_g_017" />
+	<xacro:property name="hand_serial_number" value="v_h_008" />
 </robot>

File: instance/instances/robots/forearm_testbench_left.xacro (robot description, xacro)
@@ -15,5 +15,4 @@
     <Mechanisms>
     <xacro:simple_mechanism name="testbench_actuator" serial_number="${forearm_yaw_serial_number}" node="${testbench_node}" />
-    <xacro:forearm mechanism_name="${prefix}Forearm" serial_number="${forearm_serial_number}" athena1_node="${Athena1Node}" athena2_node="${Athena2Node}" />
 	</Mechanisms>
 	<Devices>

File: instance/instances/robots/forearm_testbench_right.xacro (robot description, xacro)
@@ -1,9 +1,9 @@
 <robot xmlns:xacro="http://ros.org/wiki/xacro" name="forearm_testbench_right">
-	<xacro:property name="instance" value="forearm_testbench_right" />
-	<xacro:property name="prefix" value="right" />
-        <xacro:include filename="$(find val_description)/instance/instances/robots/xacro/firmware/firmware.xacro" />
-        <xacro:include filename="$(find val_description)/instance/instances/robots/xacro/firmware/forearm_firmware.xacro" />
-	<xacro:include filename="$(find val_description)/common/xacro/nodes/forearm_testbench_nodes_right.xacro" />
-	<xacro:include filename="$(find val_description)/common/xacro/serial_numbers/forearm_testbench_serials.xacro" />
+    <xacro:property name="instance" value="forearm_testbench_right" />
+    <xacro:property name="prefix" value="right" />
+    <xacro:include filename="$(find val_description)/instance/instances/robots/xacro/firmware/firmware.xacro" />
+    <xacro:include filename="$(find val_description)/instance/instances/robots/xacro/firmware/forearm_firmware.xacro" />
+    <xacro:include filename="$(find val_description)/common/xacro/nodes/forearm_testbench_nodes.xacro" />
+    <xacro:include filename="$(find val_description)/common/xacro/serial_numbers/forearm_testbench_serials.xacro" />
     <xacro:include filename="$(find val_description)/instance/instances/robots/xacro/mechanisms/mechanisms.xacro"/>
     <xacro:include filename="$(find val_description)/common/xacro/joint_names/valkyrie_joint_names.xacro"/>
@@ -11,11 +11,11 @@
     <Channels>
     </Channels>
-        <xacro:firmware_base_url/>
+    <xacro:firmware_base_url/>
     <xacro:firmware />
     <Mechanisms>
     <xacro:simple_mechanism name="testbench_actuator" serial_number="${forearm_yaw_serial_number}" node="${testbench_node}" />
-    <xacro:forearm mechanism_name="${prefix}Forearm" serial_number="${forearm_serial_number}" athena1_node="${Athena1Node}" athena2_node="${Athena2Node}" />
-	</Mechanisms>
-	<Devices>
-	</Devices>
+    <xacro:hand_mechanism mechanism_name="${prefix}Hand" serial_number="${hand_serial_number}" index_node="${IndexNode}" middle_node="${MiddleNode}" pinky_node="${PinkyNode}" thumb_prox_node="${ThumbProxNode}" thumb_dist_node="${ThumbDistNode}" thumb_roll_node="${ThumbRollNode}" wrist_left_node="${WristLeftNode}" wrist_right_node="${WristRightNode}" />
+    </Mechanisms>
+    <Devices>
+    </Devices>
 </robot>

File: instance/instances/robots/xacro/mechanisms/mechanisms.xacro (robot description, xacro)
@@ -39,3 +39,18 @@
     </Mechanism>
 </xacro:macro>
+<xacro:macro name="hand_mechanism" params="mechanism_name serial_number index_node middle_node pinky_node thumb_prox_node thumb_dist_node thumb_roll_node wrist_left_node wrist_right_node" >
+    <Mechanism id="${mechanism_name}" type="hand">
+            <SerialNumber id="${serial_number}"/>
+            <Nodes>
+                <Index id="${index_node}"/>
+                <Middle id="${middle_node}"/>
+                <Pinky id="${pinky_node}"/>
+                <ThumbProx id="${thumb_prox_node}"/>
+                <ThumbDist id="${thumb_dist_node}"/>
+                <ThumbRoll id="${thumb_roll_node}"/>
+                <WristLeft id="${wrist_left_node}"/>
+                <WristRight id="${wrist_right_node}"/>
+            </Nodes>
+    </Mechanism>
+</xacro:macro>
 </robot>

Commit message: adding nodes to forearm testbench

File: common/xacro/nodes/forearm_testbench_nodes.xacro (robot description, xacro)
@@ -1,3 +1,4 @@
 <robot xmlns:xacro="http://ros.org/wiki/xacro" name="test_bench_nodes">
+	<xacro:property name="HandSensorNode" value="_arm/forearm_sensors"/>
     <xacro:property name="testbench_node" value="/right_arm/j5" />
     <xacro:property name="IndexNode" value="/right_arm/hand/index" />

File: instance/instances/robots/forearm_testbench_right.xacro (robot description, xacro)
@@ -16,4 +16,5 @@
     <xacro:simple_mechanism name="testbench_actuator" serial_number="${forearm_yaw_serial_number}" node="${testbench_node}" />
     <xacro:hand_mechanism mechanism_name="${prefix}Hand" serial_number="${hand_serial_number}" index_node="${IndexNode}" middle_node="${MiddleNode}" pinky_node="${PinkyNode}" thumb_prox_node="${ThumbProxNode}" thumb_dist_node="${ThumbDistNode}" thumb_roll_node="${ThumbRollNode}" wrist_left_node="${WristLeftNode}" wrist_right_node="${WristRightNode}" />
+    <xacro:hand_sensor_mechanism name="${prefix}HandSensors" serial_number="${hand_serial_number}_midas" node="/${prefix}${HandSensorNode}" />
     </Mechanisms>
     <Devices>
