Commit message: Reduction to single-arm only

File: common/xacro/nodes/valkyrie_arm_sim_nodes.xacro (robot description, xacro)
@@ -1,4 +1,4 @@
 <robot xmlns:xacro="http://www.ros.org/wiki/xacro" name="valkyrie_sim_nodes">
-	<!--<xacro:property name="ShoulderPitchNode" value="/trunk/${prefix}_arm_j1" /> -->
+	<xacro:property name="ShoulderPitchNode" value="/trunk/${prefix}_arm_j1" />
 	<xacro:property name="ShoulderRollNode" value="_arm/j2" />
 	<xacro:property name="ShoulderYawNode" value="_arm/j3" />

File: common/xacro/nodes/valkyrie_nodes.xacro (robot description, xacro)
@@ -6,5 +6,5 @@
 	<xacro:property name="AnkleLeftActuatorNode" value="_leg/ankle/left_actuator" />
 	<xacro:property name="AnkleRightActuatorNode" value="_leg/ankle/right_actuator" />
-	<!--<xacro:property name="ShoulderPitchNode" value="/trunk/${prefix}_arm_j1" /> -->
+	<xacro:property name="ShoulderPitchNode" value="/trunk/${prefix}_arm_j1" />
 	<xacro:property name="ShoulderRollNode" value="_arm/j2" />
 	<xacro:property name="ShoulderYawNode" value="_arm/j3" />

File: common/xacro/nodes/valkyrie_sim_nodes.xacro (robot description, xacro)
@@ -10,5 +10,5 @@
 	<xacro:property name="AnklePitchActuatorNode" value="_leg/ankle/pitch_actuator" />
 	<xacro:property name="AnkleRollActuatorNode" value="_leg/ankle/roll_actuator" />
-	<!--<xacro:property name="ShoulderPitchNode" value="/trunk/${prefix}_arm_j1" /> -->
+	<xacro:property name="ShoulderPitchNode" value="/trunk/${prefix}_arm_j1" />
 	<xacro:property name="ShoulderRollNode" value="_arm/j2" />
 	<xacro:property name="ShoulderYawNode" value="_arm/j3" />

File: instance/instances/robots/xacro/firmware/arm_firmware.xacro (robot description, xacro)
@@ -2,32 +2,4 @@
     <xacro:include filename="$(find val_description)/common/xacro/firmware/valkyrie_firmware.xacro"/>
     <xacro:macro name="arm_firmware"  >
-            <fw id="leftArmJ1">
-                <Node id="/trunk/left_arm_j1" />
-                <PublicProcURLExtension id="${ShoulderPitchPublicProcFirmware}" />
-                <PrivateProcURLExtension id="${ShoulderPitchPrivateProcFirmware}" />
-                <PublicFPGAURLExtension id="${leftShoulderPitchPublicFPGAFirmware}" />
-                <PrivateFPGAURLExtension id="${leftShoulderPitchPrivateFPGAFirmware}" />
-            </fw>
-            <fw id="leftArmJ2">
-                <Node id="/left_arm/j2" />
-                <PublicProcURLExtension id="${ShoulderRollPublicProcFirmware}" />
-                <PrivateProcURLExtension id="${ShoulderRollPrivateProcFirmware}" />
-                <PublicFPGAURLExtension id="${ShoulderRollPublicFPGAFirmware}" />
-                <PrivateFPGAURLExtension id="${ShoulderRollPrivateFPGAFirmware}" />
-            </fw>
-            <fw id="leftArmJ3">
-                <Node id="/left_arm/j3" />
-                <PublicProcURLExtension id="${ShoulderYawPublicProcFirmware}" />
-                <PrivateProcURLExtension id="${ShoulderYawPrivateProcFirmware}" />
-                <PublicFPGAURLExtension id="${ShoulderYawPublicFPGAFirmware}" />
-                <PrivateFPGAURLExtension id="${ShoulderYawPrivateFPGAFirmware}" />
-            </fw>
-            <fw id="leftArmJ4">
-                <Node id="/left_arm/j4" />
-                <PublicProcURLExtension id="${ElbowPitchPublicProcFirmware}" />
-                <PrivateProcURLExtension id="${ElbowPitchPrivateProcFirmware}" />
-                <PublicFPGAURLExtension id="${ElbowPitchPublicFPGAFirmware}" />
-                <PrivateFPGAURLExtension id="${ElbowPitchPrivateFPGAFirmware}" />
-            </fw>
             <fw id="rightArmJ1">
                 <Node id="/trunk/right_arm_j1" />
