Commit message: Updated sim F/T topics.

File: common/xacro/nodes/valkyrie_nodes.xacro (robot description, xacro)
@@ -27,11 +27,11 @@
 	<xacro:property name="Athena1Node" value="/${prefix}_arm/athena1"/>
 	<xacro:property name="Athena2Node" value="/${prefix}_arm/athena2"/>
-	<xacro:property name="pelvis_middle_imu_node" value="/sensors/middlePelvisIMU" />
-	<xacro:property name="pelvis_rear_imu_node" value="/sensors/rearPelvisIMU" />
-	<xacro:property name="torso_left_imu_node" value="/sensors/leftTorsoIMU" />
+	<xacro:property name="pelvis_middle_imu_node" value="/aux/middlePelvisIMU" />
+	<xacro:property name="pelvis_rear_imu_node" value="/aux/rearPelvisIMU" />
+	<xacro:property name="torso_left_imu_node" value="/aux/leftTorsoIMU" />
 	<xacro:property name="left_foot_ATI_node" value="/left_leg/ankle/left_actuator" />
-	<xacro:property name="left_foot_Sim_ATI_node" value="/sensors/leftFootSixAxis" />
+	<xacro:property name="left_foot_Sim_ATI_node" value="/left_leg/ankle/roll_actuator" />
 	<xacro:property name="right_foot_ATI_node" value="/right_leg/ankle/left_actuator" />
-	<xacro:property name="right_foot_Sim_ATI_node" value="/sensors/rightFootSixAxis" />
+	<xacro:property name="right_foot_Sim_ATI_node" value="/right_leg/ankle/roll_actuator" />
 	<xacro:property name="IndexFingerPitch1Node" value="/${prefix}_arm/forearm_sensors/index/pitch_1"/>
 	<xacro:property name="IndexFingerPitch2Node" value="/${prefix}_arm/forearm_sensors/index/pitch_2"/>

Commit message: Moved inclusion of the gazebo plugin out to top level sim xacro so I can create sim URDF's without it.

File: common/xacro/nodes/valkyrie_nodes.xacro (robot description, xacro)
@@ -27,7 +27,7 @@
 	<xacro:property name="Athena1Node" value="/${prefix}_arm/athena1"/>
 	<xacro:property name="Athena2Node" value="/${prefix}_arm/athena2"/>
-	<xacro:property name="pelvis_middle_imu_node" value="/aux/middlePelvisIMU" />
-	<xacro:property name="pelvis_rear_imu_node" value="/aux/rearPelvisIMU" />
-	<xacro:property name="torso_left_imu_node" value="/aux/leftTorsoIMU" />
+	<xacro:property name="pelvis_middle_imu_node" value="/sensors/middlePelvisIMU" />
+	<xacro:property name="pelvis_rear_imu_node" value="/sensors/rearPelvisIMU" />
+	<xacro:property name="torso_left_imu_node" value="/sensors/leftTorsoIMU" />
 	<xacro:property name="left_foot_ATI_node" value="/left_leg/ankle/left_actuator" />
 	<xacro:property name="left_foot_Sim_ATI_node" value="/left_leg/ankle/roll_actuator" />

File: model/robots/common/xacro/sensors/ati_force_torque.xacro (robot description, xacro)
@@ -16,5 +16,5 @@
         <api name="${sensor_api}" />
         <always_on>true</always_on>
-        <update_rate>1000</update_rate>
+        <update_rate>500.0</update_rate>
         <force_torque>
           <frame>sensor</frame>

File: model/robots/common/xacro/sensors/microstrain.xacro (robot description, xacro)
@@ -16,5 +16,5 @@
         <serviceName>${sensorName}/imu_service</serviceName>
         <gaussianNoise>0.0</gaussianNoise>
-        <updateRate>1000.0</updateRate>
+        <updateRate>500.0</updateRate>
       </plugin>
     </gazebo>

File: model/robots/common/xacro/valkyrie_arm_mass_sims_base_sim.xacro (robot description, xacro)
@@ -1,9 +1,3 @@
 <robot xmlns:xacro="http://ros.org/wiki/xacro" name="valkyrie">
-    <gazebo>
-      <plugin filename="libval_gazebo.so" name="SharedMemorySimInterfacePlugin">
-          <robotNamespace>/val</robotNamespace>
-          <updateRateHz>500.0</updateRateHz>
-      </plugin>
-    </gazebo>
     <xacro:make_pelvis />
     <xacro:make_waist waist_root_link="${Pelvis_Link_Name}" />

File: model/robots/common/xacro/valkyrie_base_sim.xacro (robot description, xacro)
@@ -1,9 +1,3 @@
 <robot xmlns:xacro="http://ros.org/wiki/xacro" name="valkyrie">
-    <gazebo>
-      <plugin filename="libval_gazebo.so" name="SharedMemorySimInterfacePlugin">
-      <robotNamespace>/val</robotNamespace>
-      <updateRateHz>500.0</updateRateHz>
-      </plugin>
-    </gazebo>
     <xacro:make_pelvis />
     <xacro:make_waist waist_root_link="${Pelvis_Link_Name}" />

File: model/robots/valkyrie_sim.xacro (robot description, xacro)
@@ -1,3 +1,10 @@
 <robot xmlns:xacro="http://ros.org/wiki/xacro" name="valkyrie">
+    <gazebo>
+      <plugin filename="libval_gazebo.so" name="SharedMemorySimInterfacePlugin">
+          <robotNamespace>/val</robotNamespace>
+          <updateRateHz>500.0</updateRateHz>
+          <writeRateHz>250.0</writeRateHz>
+      </plugin>
+    </gazebo>
     <xacro:property name="mesh_root" value="package://val_description/model/meshes"/>
     <xacro:include filename="$(find val_description)/common/xacro/api/valkyrie_sim_api.xacro"/>
@@ -9,5 +16,4 @@
     <xacro:include filename="$(find val_description)/model/robots/common/xacro/valkyrie_base_sim.xacro"/>
     <xacro:include filename="$(find val_description)/model/robots/common/xacro/gazebo_harness.xacro"/>
-    <!-- Commenting out this next line until the harness makes it into a gazebo_ros_pkgs release -->
     <xacro:add_sim_harness harnessed_link="${TorsoRollLinkName}" />
 </robot>

File: model/robots/valkyrie_sim_arm_mass_sims.xacro (robot description, xacro)
@@ -1,3 +1,10 @@
 <robot xmlns:xacro="http://ros.org/wiki/xacro" name="valkyrie">
+    <gazebo>
+      <plugin filename="libval_gazebo.so" name="SharedMemorySimInterfacePlugin">
+          <robotNamespace>/val</robotNamespace>
+          <updateRateHz>500.0</updateRateHz>
+          <writeRateHz>250.0</writeRateHz>
+      </plugin>
+    </gazebo>
     <xacro:property name="mesh_root" value="package://val_description/model/meshes"/>
     <xacro:include filename="$(find val_description)/common/xacro/api/valkyrie_sim_api.xacro"/>

File: model/robots/valkyrie_sim_pinned.xacro (robot description, xacro)
@@ -1,3 +1,10 @@
 <robot xmlns:xacro="http://ros.org/wiki/xacro" name="valkyrie">
+    <gazebo>
+      <plugin filename="libval_gazebo.so" name="SharedMemorySimInterfacePlugin">
+          <robotNamespace>/val</robotNamespace>
+          <updateRateHz>500.0</updateRateHz>
+          <writeRateHz>250.0</writeRateHz>
+      </plugin>
+    </gazebo>
     <xacro:property name="mesh_root" value="package://val_description/model/meshes"/>
     <xacro:include filename="$(find val_description)/model/robots/common/xacro/generic_models.xacro" />

Commit message: Minor mods to the finger stuff.

File: common/xacro/nodes/valkyrie_nodes.xacro (robot description, xacro)
@@ -47,4 +47,8 @@
 	<xacro:property name="ThumbPitch2Node" value="/${prefix}_arm/forearm_sensors/thumb/pitch_2"/>
 	<xacro:property name="ThumbPitch3Node" value="/${prefix}_arm/forearm_sensors/thumb/pitch_3"/>
+	<xacro:property name="ThumbRollSimNode" value="/remap/${prefix}_hand/thumb/roll"/>
+	<xacro:property name="ThumbPitch1SimNode" value="/remap/${prefix}_hand/thumb/pitch_1"/>
+	<xacro:property name="ThumbPitch2SimNode" value="/remap/${prefix}_hand/thumb/pitch_2"/>
+	<xacro:property name="ThumbPitch3SimNode" value="/remap/${prefix}_hand/thumb/pitch_3"/>
 	<xacro:macro name="all_channels" >
 		<Channels>

File: model/robots/common/xacro/generic_models.xacro (robot description, xacro)
@@ -232,5 +232,5 @@
       </joint>
       <actuator name="${actuatorName}">
-        <node name="${nodeName}"/>
+        <node name="${node1Name}"/>
         <mechanicalReduction>1</mechanicalReduction>
         <api name="${actuatorApi}" />
@@ -242,10 +242,14 @@
     </transmission>
   </xacro:macro>
-  <xacro:macro name="simple_passive_transmission" params="jointName nodeName">
+  <xacro:macro name="simple_passive_transmission" params="jointName nodeName apiName">
     <transmission name="${jointName}PassiveTransmission">
       <type>transmission_interface/SimpleTransmission</type>
       <joint name="${jointName}">
       </joint>
-      <node>${nodeName}</node>
+      <actuator name="${jointName}PassiveActuator">
+        <node name="${nodeName}"/>
+        <mechanicalReduction>1</mechanicalReduction>
+        <api name="${apiName}" />
+      </actuator>
     </transmission>
   </xacro:macro>

File: model/robots/common/xacro/thumb/thumb.xacro (robot description, xacro)
@@ -92,8 +92,8 @@
   </xacro:macro>
   <xacro:macro name="thumb_transmissions_sim" params="prefix">
-    <xacro:simple_position_transmission jointName="${ThumbRollJointName}" actuatorName="${prefix}ThumbRollActuator" nodeName="${ThumbRollNode}" actuatorApi="${ThumbFingerApi}"/>
-    <xacro:finger_transmission joint1Name="${ThumbPitch1JointName}" actuatorName="${prefix}ThumbPitch1Actuator" node1Name="${ThumbPitch1Node}" actuatorApi="${ThumbFingerApi}" joint2Name="${ThumbPitch2JointName}" joint3Name="${ThumbPitch3JointName}" ratio1="${Pulley2Ratio}" ratio2="${Pulley3Ratio}" node2Name="${ThumbPitch2Node}" node3Name="${ThumbPitch3Node}" />
-    <xacro:simple_passive_transmission jointName="${ThumbPitch2JointName}" nodeName="${ThumbPitch2Node}"/>
-    <xacro:simple_passive_transmission jointName="${ThumbPitch3JointName}" nodeName="${ThumbPitch3Node}"/>
+    <xacro:simple_position_transmission jointName="${ThumbRollJointName}" actuatorName="${prefix}ThumbRollActuator" nodeName="${ThumbRollSimNode}" actuatorApi="${SimApi}"/>
+    <xacro:finger_transmission joint1Name="${ThumbPitch1JointName}" actuatorName="${prefix}ThumbPitch1Actuator" node1Name="${ThumbPitch1SimNode}" actuatorApi="${SimApi}" joint2Name="${ThumbPitch2JointName}" joint3Name="${ThumbPitch3JointName}" ratio1="${Pulley2Ratio}" ratio2="${Pulley3Ratio}" node2Name="${ThumbPitch2SimNode}" node3Name="${ThumbPitch3SimNode}" />
+    <xacro:simple_passive_transmission jointName="${ThumbPitch2JointName}" nodeName="${ThumbPitch2SimNode}" apiName="${SimApi}"/>
+    <xacro:simple_passive_transmission jointName="${ThumbPitch3JointName}" nodeName="${ThumbPitch3SimNode}" apiName="${SimApi}"/>
   </xacro:macro>
 </robot>
