Commit message: Reworking some xacro stuff for the sim fingers.

File: common/xacro/nodes/valkyrie_nodes.xacro (robot description, xacro)
@@ -23,6 +23,4 @@
 	<xacro:property name="WaistLeftActuatorNode" value="/trunk/left_actuator" /> <!--pitch-->
 	<xacro:property name="WaistRightActuatorNode" value="/trunk/right_actuator" /> <!--roll-->
-	<xacro:property name="WaistPitchActuatorSimNode" value="/trunk/pitch_actuator" /> <!--pitch-->
-	<xacro:property name="WaistRollActuatorSimNode" value="/trunk/roll_actuator" /> <!--roll-->
 	<xacro:property name="Athena1Node" value="/${prefix}_arm/athena1"/>
 	<xacro:property name="Athena2Node" value="/${prefix}_arm/athena2"/>
@@ -31,7 +29,5 @@
 	<xacro:property name="torso_left_imu_node" value="/sensors/leftTorsoIMU" />
 	<xacro:property name="left_foot_ATI_node" value="/left_leg/ankle/left_actuator" />
-	<xacro:property name="left_foot_Sim_ATI_node" value="/left_leg/ankle/roll_actuator" />
 	<xacro:property name="right_foot_ATI_node" value="/right_leg/ankle/left_actuator" />
-	<xacro:property name="right_foot_Sim_ATI_node" value="/right_leg/ankle/roll_actuator" />
 	<xacro:property name="IndexFingerPitch1Node" value="/${prefix}_arm/forearm_sensors/index/pitch_1"/>
 	<xacro:property name="IndexFingerPitch2Node" value="/${prefix}_arm/forearm_sensors/index/pitch_2"/>
@@ -47,8 +43,4 @@
 	<xacro:property name="ThumbPitch2Node" value="/${prefix}_arm/forearm_sensors/thumb/pitch_2"/>
 	<xacro:property name="ThumbPitch3Node" value="/${prefix}_arm/forearm_sensors/thumb/pitch_3"/>
-	<xacro:property name="ThumbRollSimNode" value="/remap/${prefix}_hand/thumb/roll"/>
-	<xacro:property name="ThumbPitch1SimNode" value="/remap/${prefix}_hand/thumb/pitch_1"/>
-	<xacro:property name="ThumbPitch2SimNode" value="/remap/${prefix}_hand/thumb/pitch_2"/>
-	<xacro:property name="ThumbPitch3SimNode" value="/remap/${prefix}_hand/thumb/pitch_3"/>
 	<xacro:macro name="all_channels" >
 		<Channels>

File: model/robots/common/xacro/arm/arm.xacro (robot description, xacro)
@@ -3,5 +3,4 @@
   <xacro:include filename="$(find val_description)/common/xacro/joint_names/valkyrie_joint_names.xacro"/>
   <xacro:include filename="$(find val_description)/common/xacro/actuator_names/valkyrie_actuator_names.xacro"/>
-  <xacro:include filename="$(find val_description)/common/xacro/nodes/valkyrie_nodes.xacro"/>
   <xacro:include filename="$(find val_description)/model/robots/common/xacro/arm/joint_axes.xacro"/>
   <xacro:include filename="$(find val_description)/model/robots/common/xacro/arm/link_names.xacro"/>
@@ -259,6 +258,6 @@
     <xacro:simple_transmission jointName="${ElbowPitchJointName}" actuatorName="${ElbowPitchActuatorName}" nodeName="${ElbowPitchNode}" actuatorApi="${SimApi}"/>
     <xacro:simple_position_transmission jointName="${ForearmYawActuatorName}" actuatorName="${ForearmYawActuatorName}" nodeName="${ForearmYawNode}" actuatorApi="${SimApi}"/>
-    <xacro:simple_position_transmission jointName="${WristRollJointName}" actuatorName="${WristRollActuatorSimName}" nodeName="${WristRollActuatorSimNode}" actuatorApi="${SimApi}"/>
-    <xacro:simple_position_transmission jointName="${WristPitchJointName}" actuatorName="${WristPitchActuatorSimName}" nodeName="${WristPitchActuatorSimNode}" actuatorApi="${SimApi}"/>
+    <xacro:simple_position_transmission jointName="${WristRollJointName}" actuatorName="${WristRollActuatorSimName}" nodeName="${WristRollActuatorNode}" actuatorApi="${SimApi}"/>
+    <xacro:simple_position_transmission jointName="${WristPitchJointName}" actuatorName="${WristPitchActuatorSimName}" nodeName="${WristPitchActuatorNode}" actuatorApi="${SimApi}"/>
   </xacro:macro>
   <xacro:macro name="arm_transmissions_sim_no_hands" params="prefix">

File: model/robots/common/xacro/leg/leg.xacro (robot description, xacro)
@@ -3,5 +3,4 @@
   <xacro:include filename="$(find val_description)/common/xacro/joint_names/valkyrie_joint_names.xacro"/>
   <xacro:include filename="$(find val_description)/common/xacro/actuator_names/valkyrie_actuator_names.xacro"/>
-  <xacro:include filename="$(find val_description)/common/xacro/nodes/valkyrie_nodes.xacro"/>
   <xacro:include filename="$(find val_description)/model/robots/common/xacro/leg/joint_axes.xacro"/>
   <xacro:include filename="$(find val_description)/model/robots/common/xacro/leg/link_names.xacro"/>
@@ -173,6 +172,6 @@
     <xacro:simple_transmission jointName="${HipPitchJointName}" actuatorName="${HipPitchActuatorName}" nodeName="${HipPitchNode}" actuatorApi="${SimApi}"/>
     <xacro:simple_transmission jointName="${KneePitchJointName}" actuatorName="${KneePitchActuatorName}" nodeName="${KneePitchNode}" actuatorApi="${SimApi}"/>
-    <xacro:simple_transmission jointName="${AnklePitchJointName}" actuatorName="${AnklePitchActuatorSimName}" nodeName="${AnklePitchActuatorSimNode}" actuatorApi="${SimApi}"/>
-    <xacro:simple_transmission jointName="${AnkleRollJointName}" actuatorName="${AnkleRollActuatorSimName}" nodeName="${AnkleRollActuatorSimNode}" actuatorApi="${SimApi}"/>
+    <xacro:simple_transmission jointName="${AnklePitchJointName}" actuatorName="${AnklePitchActuatorSimName}" nodeName="${AnklePitchActuatorNode}" actuatorApi="${SimApi}"/>
+    <xacro:simple_transmission jointName="${AnkleRollJointName}" actuatorName="${AnkleRollActuatorSimName}" nodeName="${AnkleRollActuatorNode}" actuatorApi="${SimApi}"/>
   </xacro:macro>
 </robot>

File: model/robots/common/xacro/thumb/thumb.xacro (robot description, xacro)
@@ -92,8 +92,8 @@
   </xacro:macro>
   <xacro:macro name="thumb_transmissions_sim" params="prefix">
-    <xacro:simple_position_transmission jointName="${ThumbRollJointName}" actuatorName="${prefix}ThumbRollActuator" nodeName="${ThumbRollSimNode}" actuatorApi="${SimApi}"/>
-    <xacro:finger_transmission joint1Name="${ThumbPitch1JointName}" actuatorName="${prefix}ThumbPitch1Actuator" node1Name="${ThumbPitch1SimNode}" actuatorApi="${SimApi}" joint2Name="${ThumbPitch2JointName}" joint3Name="${ThumbPitch3JointName}" ratio1="${Pulley2Ratio}" ratio2="${Pulley3Ratio}" node2Name="${ThumbPitch2SimNode}" node3Name="${ThumbPitch3SimNode}" />
-    <xacro:simple_passive_transmission jointName="${ThumbPitch2JointName}" nodeName="${ThumbPitch2SimNode}" apiName="${SimApi}"/>
-    <xacro:simple_passive_transmission jointName="${ThumbPitch3JointName}" nodeName="${ThumbPitch3SimNode}" apiName="${SimApi}"/>
+    <xacro:simple_position_transmission jointName="${ThumbRollJointName}" actuatorName="${prefix}ThumbRollActuator" nodeName="${ThumbRollNode}" actuatorApi="${SimApi}"/>
+    <xacro:finger_transmission joint1Name="${ThumbPitch1JointName}" actuatorName="${prefix}ThumbPitch1Actuator" node1Name="${ThumbPitch1Node}" actuatorApi="${SimApi}" joint2Name="${ThumbPitch2JointName}" joint3Name="${ThumbPitch3JointName}" ratio1="${Pulley2Ratio}" ratio2="${Pulley3Ratio}" node2Name="${ThumbPitch2Node}" node3Name="${ThumbPitch3Node}" />
+    <xacro:simple_passive_transmission jointName="${ThumbPitch2JointName}" nodeName="${ThumbPitch2Node}" apiName="${SimApi}"/>
+    <xacro:simple_passive_transmission jointName="${ThumbPitch3JointName}" nodeName="${ThumbPitch3Node}" apiName="${SimApi}"/>
   </xacro:macro>
 </robot>

File: model/robots/common/xacro/valkyrie_arm_mass_sims_base_hw.xacro (robot description, xacro)
@@ -1,3 +1,4 @@
 <robot xmlns:xacro="http://ros.org/wiki/xacro" name="valkyrie">
+    <xacro:include filename="$(find val_description)/common/xacro/nodes/valkyrie_nodes.xacro"/>
     <xacro:make_pelvis />
     <xacro:make_waist waist_root_link="${Pelvis_Link_Name}" />

File: model/robots/common/xacro/valkyrie_arm_mass_sims_base_sim.xacro (robot description, xacro)
@@ -1,3 +1,4 @@
 <robot xmlns:xacro="http://ros.org/wiki/xacro" name="valkyrie">
+    <xacro:include filename="$(find val_description)/common/xacro/nodes/valkyrie_sim_nodes.xacro"/>
     <xacro:make_pelvis />
     <xacro:make_waist waist_root_link="${Pelvis_Link_Name}" />
@@ -8,6 +9,6 @@
     <xacro:make_leg prefix="left" reflect="1" leg_root_link="${Pelvis_Link_Name}"/>
     <xacro:v1_pelvis_sensors_usb middle_sensor_node_tag="${pelvis_middle_imu_node}" middle_sensor_api_tag="${ImuSensorSimApi}" middle_sensor_port_tag="${pelvis_middle_imu_port}" rear_sensor_node_tag="${pelvis_rear_imu_node}" rear_sensor_api_tag="${ImuSensorSimApi}" rear_sensor_port_tag="${pelvis_rear_imu_port}"/>
-    <xacro:v1_leg_sensors prefix="left" reflect="1" ATI_serial_number="${sim_ATI_serial}" ATI_node="${left_foot_Sim_ATI_node}"/>
-    <xacro:v1_leg_sensors prefix="right" reflect="-1" ATI_serial_number="${sim_ATI_serial}" ATI_node="${right_foot_Sim_ATI_node}"/>
+    <xacro:v1_leg_sensors prefix="left" reflect="1" ATI_serial_number="${sim_ATI_serial}" ATI_node="${left_foot_ATI_node}"/>
+    <xacro:v1_leg_sensors prefix="right" reflect="-1" ATI_serial_number="${sim_ATI_serial}" ATI_node="${right_foot_ATI_node}"/>
     <xacro:include_multisense_sim />
     <xacro:v1_trunk_sensors_usb sensor_node_tag="${torso_left_imu_node}" sensor_api_tag="${ImuSensorSimApi}" sensor_port_tag="${torso_left_imu_port}"/>

File: model/robots/common/xacro/valkyrie_base_hw.xacro (robot description, xacro)
@@ -1,3 +1,4 @@
 <robot xmlns:xacro="http://ros.org/wiki/xacro" name="valkyrie">
+    <xacro:include filename="$(find val_description)/common/xacro/nodes/valkyrie_nodes.xacro"/>
     <xacro:make_pelvis />
     <xacro:make_waist waist_root_link="${Pelvis_Link_Name}" />

File: model/robots/common/xacro/valkyrie_base_sim.xacro (robot description, xacro)
@@ -1,3 +1,5 @@
 <robot xmlns:xacro="http://ros.org/wiki/xacro" name="valkyrie">
+    <xacro:include filename="$(find val_description)/common/xacro/nodes/valkyrie_sim_nodes.xacro"/>
+    <shm_remap_file package="val_gazebo" relative_file_path="/configurations/valkyrie_sim_shm_remap.yaml"/>
     <xacro:make_pelvis />
     <xacro:make_waist waist_root_link="${Pelvis_Link_Name}" />
@@ -16,6 +18,6 @@
     <xacro:make_leg prefix="left" reflect="1" leg_root_link="${Pelvis_Link_Name}"/>
     <xacro:v1_pelvis_sensors_usb middle_sensor_node_tag="${pelvis_middle_imu_node}" middle_sensor_api_tag="${ImuSensorSimApi}" middle_sensor_port_tag="${pelvis_middle_imu_port}" rear_sensor_node_tag="${pelvis_rear_imu_node}" rear_sensor_api_tag="${ImuSensorSimApi}" rear_sensor_port_tag="${pelvis_rear_imu_port}"/>
-    <xacro:v1_leg_sensors prefix="left" reflect="1" ATI_serial_number="${sim_ATI_serial}" ATI_node="${left_foot_Sim_ATI_node}"/>
-    <xacro:v1_leg_sensors prefix="right" reflect="-1" ATI_serial_number="${sim_ATI_serial}" ATI_node="${right_foot_Sim_ATI_node}"/>
+    <xacro:v1_leg_sensors prefix="left" reflect="1" ATI_serial_number="${sim_ATI_serial}" ATI_node="${left_foot_ATI_node}"/>
+    <xacro:v1_leg_sensors prefix="right" reflect="-1" ATI_serial_number="${sim_ATI_serial}" ATI_node="${right_foot_ATI_node}"/>
     <xacro:include_multisense_sim />
     <xacro:v1_trunk_sensors_usb sensor_node_tag="${torso_left_imu_node}" sensor_api_tag="${ImuSensorSimApi}" sensor_port_tag="${torso_left_imu_port}"/>

File: model/robots/common/xacro/waist/waist.xacro (robot description, xacro)
@@ -2,5 +2,4 @@
   <xacro:include filename="$(find val_description)/common/xacro/joint_names/valkyrie_joint_names.xacro"/>
   <xacro:include filename="$(find val_description)/common/xacro/actuator_names/valkyrie_actuator_names.xacro"/>
-  <xacro:include filename="$(find val_description)/common/xacro/nodes/valkyrie_nodes.xacro"/>
   <xacro:include filename="$(find val_description)/model/robots/common/xacro/waist/joint_axes.xacro"/>
   <xacro:include filename="$(find val_description)/model/robots/common/xacro/waist/joint_axes.xacro"/>
@@ -112,6 +111,6 @@
    <xacro:macro name="waist_transmissions_sim">
     <xacro:simple_transmission jointName="${TorsoYawJointName}" actuatorName="${TorsoYawActuatorName}" nodeName="${TrunkYawNode}" actuatorApi="${SimApi}"/>
-    <xacro:simple_transmission jointName="${TorsoPitchJointName}" actuatorName="${WaistPitchActuatorSimName}" nodeName="${WaistPitchActuatorSimNode}" actuatorApi="${SimApi}"/>
-    <xacro:simple_transmission jointName="${TorsoRollJointName}" actuatorName="${WaistRollActuatorSimName}" nodeName="${WaistRollActuatorSimNode}" actuatorApi="${SimApi}"/>
+    <xacro:simple_transmission jointName="${TorsoPitchJointName}" actuatorName="${WaistPitchActuatorSimName}" nodeName="${WaistPitchActuatorNode}" actuatorApi="${SimApi}"/>
+    <xacro:simple_transmission jointName="${TorsoRollJointName}" actuatorName="${WaistRollActuatorSimName}" nodeName="${WaistRollActuatorNode}" actuatorApi="${SimApi}"/>
    </xacro:macro>
 </robot>

File: model/robots/forearm_left.xacro (robot description, xacro)
@@ -1,4 +1,5 @@
 <robot xmlns:xacro="http://ros.org/wiki/xacro" name="valkyrie">
     <xacro:property name="mesh_root" value="package://val_description/model/meshes"/>
+    <xacro:include filename="$(find val_description)/common/xacro/nodes/valkyrie_nodes.xacro"/>
     <xacro:include filename="$(find val_description)/model/robots/common/xacro/generic_models.xacro" />
     <xacro:include filename="$(find val_description)/model/robots/common/xacro/common_bodies.xacro" />

File: model/robots/forearm_right.xacro (robot description, xacro)
@@ -1,4 +1,5 @@
 <robot xmlns:xacro="http://ros.org/wiki/xacro" name="valkyrie">
     <xacro:property name="mesh_root" value="package://val_description/model/meshes"/>
+    <xacro:include filename="$(find val_description)/common/xacro/nodes/valkyrie_nodes.xacro"/>
     <xacro:include filename="$(find val_description)/model/robots/common/xacro/generic_models.xacro" />
     <xacro:include filename="$(find val_description)/model/robots/common/xacro/common_bodies.xacro" />

File: model/robots/imu_test.xacro (robot description, xacro)
@@ -1,4 +1,5 @@
 <robot xmlns:xacro="http://ros.org/wiki/xacro" name="valkyrie">
     <xacro:property name="mesh_root" value="package://val_description/model/meshes"/>
+    <xacro:include filename="$(find val_description)/common/xacro/nodes/valkyrie_nodes.xacro"/>
     <xacro:include filename="$(find val_description)/model/robots/common/xacro/generic_models.xacro" />
     <xacro:include filename="$(find val_description)/model/robots/common/xacro/common_bodies.xacro" />

Commit message: Removed some unecessary sim nodes from valkyrie_nodes.xacro.

File: common/xacro/nodes/valkyrie_nodes.xacro (robot description, xacro)
@@ -6,6 +6,4 @@
 	<xacro:property name="AnkleLeftActuatorNode" value="/${prefix}_leg/ankle/left_actuator" />
 	<xacro:property name="AnkleRightActuatorNode" value="/${prefix}_leg/ankle/right_actuator" />
-	<xacro:property name="AnklePitchActuatorSimNode" value="/${prefix}_leg/ankle/pitch_actuator" />
-	<xacro:property name="AnkleRollActuatorSimNode" value="/${prefix}_leg/ankle/roll_actuator" />
 	<xacro:property name="ShoulderPitchNode" value="/trunk/${prefix}_arm_j1" />
 	<xacro:property name="ShoulderRollNode" value="/${prefix}_arm/j2" />
@@ -15,6 +13,4 @@
 	<xacro:property name="WristTopActuatorNode" value="/${prefix}_arm/wrist/top_actautor" />
 	<xacro:property name="WristBottomActuatorNode" value="/${prefix}_arm/wrist/bottom_actuator" />
-	<xacro:property name="WristRollActuatorSimNode" value="/${prefix}_arm/wrist/roll_actautor" />
-	<xacro:property name="WristPitchActuatorSimNode" value="/${prefix}_arm/wrist/pitch_actuator" />
 	<xacro:property name="LowerNeckPitchNode" value="/neck/j1" />
 	<xacro:property name="NeckYawNode" value="/neck/j2" />

Commit message: added hands to instance file

File: common/xacro/nodes/valkyrie_nodes.xacro (robot description, xacro)
@@ -15,4 +15,12 @@
 	<xacro:property name="WristLeftActuatorNode" value="/${prefix}_arm/wrist/left_actuator" />
 	<xacro:property name="WristRightActuatorNode" value="/${prefix}_arm/wrist/right_actuator" />
+    	<xacro:property name="IndexNode" value="/${prefix}_arm/hand/index" />
+    	<xacro:property name="MiddleNode" value="/${prefix}_arm/hand/middle" />
+    	<xacro:property name="PinkyNode" value="/${prefix}_arm/hand/pinky" />
+    	<xacro:property name="ThumbProxNode" value="/${prefix}_arm/hand/thumb_proximal" />
+    	<xacro:property name="ThumbDistNode" value="/${prefix}_arm/hand/thumb_distal" />
+    	<xacro:property name="ThumbRollNode" value="/${prefix}_arm/hand/thumb_roll" />
+    	<xacro:property name="WristLeftNode" value="/${prefix}_arm/wrist/left_actuator" />
+    	<xacro:property name="WristRightNode" value="/${prefix}_arm/wrist/right_actuator" />
 	<xacro:property name="LowerNeckPitchNode" value="/neck/j1" />
 	<xacro:property name="NeckYawNode" value="/neck/j2" />

File: common/xacro/serial_numbers/valkyrie_A_serials.xacro (robot description, xacro)
@@ -17,4 +17,5 @@
 	<xacro:property name="leftArmJ4SerialNumber" value="v_f_020" />
 	<xacro:property name="leftArmJ5SerialNumber" value="v_g_016" />
+	<xacro:property name="left_hand_serial_number" value="v_h_005" />
 	<xacro:property name="rightArmJ1SerialNumber" value="v_a_001" />
 	<xacro:property name="rightArmJ2SerialNumber" value="v_b_003" />
@@ -22,4 +23,5 @@
 	<xacro:property name="rightArmJ4SerialNumber" value="v_f_003" />
 	<xacro:property name="rightArmJ5SerialNumber" value="v_g_017" />
+	<xacro:property name="right_hand_serial_number" value="v_h_008" />
 	<xacro:property name="neckJ1SerialNumber" value="v_g_006" />
 	<xacro:property name="neckJ2SerialNumber" value="v_g_007" />

File: instance/instances/robots/xacro/limbs/arm/arm.xacro (robot description, xacro)
@@ -8,5 +8,5 @@
     	<xacro:simple_mechanism name="${ElbowPitchJointName}" serial_number="${j4_serial_number}" node="${ElbowPitchNode}" calibration_angle="${ElbowPitchCalibrationAngle}"/>
     	<xacro:simple_mechanism name="${ForearmYawJointName}" serial_number="${j5_serial_number}" node="${ForearmYawNode}" calibration_angle="${ForearmYawCalibrationAngle}"/>
-        <xacro:forearm mechanism_name="${prefix}Forearm" serial_number="${forearm_serial_number}" athena1_node="${Athena1Node}" athena2_node="${Athena2Node}" />
+    	<xacro:hand_mechanism mechanism_name="${prefix}Hand" serial_number="${forearm_serial_number}" index_node="${IndexNode}" middle_node="${MiddleNode}" pinky_node="${PinkyNode}" thumb_prox_node="${ThumbProxNode}" thumb_dist_node="${ThumbDistNode}" thumb_roll_node="${ThumbRollNode}" wrist_left_node="${WristLeftNode}" wrist_right_node="${WristRightNode}" />
     </xacro:macro>
 </robot>

Commit message: adding forearm serials and mechanisms for the hand sensors

File: common/xacro/nodes/valkyrie_nodes.xacro (robot description, xacro)
@@ -36,4 +36,5 @@
 	<xacro:property name="left_foot_ATI_node" value="/left_leg/ankle/left_actuator" />
 	<xacro:property name="right_foot_ATI_node" value="/right_leg/ankle/left_actuator" />
+	<xacro:property name="HandSensorNode" value="_arm/forearm_sensors"/>
 	<xacro:property name="IndexFingerNode" value="/${prefix}_arm/hand/index"/>
 	<xacro:property name="IndexFingerPitch1Node" value="/${prefix}_arm/forearm_sensors/index"/>

File: common/xacro/serial_numbers/valkyrie_A_serials.xacro (robot description, xacro)
@@ -31,5 +31,5 @@
 	<xacro:property name="waistLeftActuatorSerialNumber" value="v_e_006" />
 	<xacro:property name="leftForearmSerialNumber" value="v_h_005"/>
-    	<xacro:property name="rightForearmSerialNumber" value="v_h_008"/>
+    <xacro:property name="rightForearmSerialNumber" value="v_h_008"/>
 	<xacro:property name="left_foot_ATI_serial" value="FT17218" />
 	<xacro:property name="right_foot_ATI_serial" value="FT14018" />

File: instance/instances/robots/xacro/limbs/arm/arm.xacro (robot description, xacro)
@@ -9,4 +9,5 @@
     	<xacro:simple_mechanism name="${ForearmYawJointName}" serial_number="${j5_serial_number}" node="${ForearmYawNode}" calibration_angle="${ForearmYawCalibrationAngle}"/>
     	<xacro:hand_mechanism mechanism_name="${prefix}Hand" serial_number="${forearm_serial_number}" index_node="${IndexNode}" middle_node="${MiddleNode}" pinky_node="${PinkyNode}" thumb_prox_node="${ThumbProxNode}" thumb_dist_node="${ThumbDistNode}" thumb_roll_node="${ThumbRollNode}" wrist_left_node="${WristLeftNode}" wrist_right_node="${WristRightNode}" />
+        <xacro:hand_sensor_mechanism name="${prefix}HandSensors" serial_number="${forearm_serial_number}_midas" node="/${prefix}${HandSensorNode}" />
     </xacro:macro>
 </robot>

File: instance/instances/robots/xacro/mechanisms/mechanisms.xacro (robot description, xacro)
@@ -54,3 +54,9 @@
     </Mechanism>
 </xacro:macro>
+<xacro:macro name="hand_sensor_mechanism" params="name serial_number node " >
+    <Mechanism id="${name}" type="hand_sensor">
+        <SerialNumber id="${serial_number}" />
+        <Node id="${node}" />
+    </Mechanism>
+</xacro:macro>
 </robot>

Commit message: correcting thumb roll sensor nodes

File: common/xacro/nodes/valkyrie_nodes.xacro (robot description, xacro)
@@ -51,5 +51,5 @@
 	<xacro:property name="ThumbProximalNode" value="_arm/hand/thumb_proximal"/>
 	<xacro:property name="ThumbDistalNode" value="_arm/hand/thumb_distal"/>
-	<xacro:property name="ThumbRollSensNode" value="/${prefix}_arm/forearm_sensors/thumb"/>
+	<xacro:property name="ThumbRollSensNode" value="_arm/forearm_sensors/thumb"/>
 	<xacro:property name="ThumbPitch1Node" value="_arm/forearm_sensors/thumb"/>
 	<xacro:property name="ThumbPitch2Node" value="_arm/forearm_sensors/thumb"/>

File: model/robots/common/xacro/thumb/thumb.xacro (robot description, xacro)
@@ -97,5 +97,5 @@
   </xacro:macro>
   <xacro:macro name="thumb_transmissions_hw" params="prefix reflect">
-    <xacro:simple_position_transmission jointName="${prefix}${ThumbRollJointName}" actuatorName="${prefix}ThumbRollActuator" nodeName="/${prefix}${ThumbRollNode}" actuatorApi="${ThumbFingerRollApi}"/>
+    <xacro:simple_position_transmission jointName="${prefix}${ThumbRollJointName}" actuatorName="${prefix}ThumbRollActuator" nodeName="/${prefix}${ThumbRollSensNode}" actuatorApi="${ThumbFingerRollApi}"/>
     <xacro:simple_forearm_position_transmission jointName="${prefix}${ThumbPitch1JointName}" actuatorName="${prefix}ThumbPitch1Actuator" nodeName="/${prefix}${ThumbPitch1Node}" actuatorApi="${ThumbFingerProximalApi}" reflect="${reflect}"/>
     <xacro:simple_forearm_position_transmission jointName="${prefix}${ThumbPitch2JointName}" actuatorName="${prefix}ThumbPitch2Actuator" nodeName="/${prefix}${ThumbPitch2Node}" actuatorApi="${ThumbFingerMedialApi}" reflect="${reflect}"/>
