Commit message: addning an e

File: common/xacro/nodes/valkyrie_nodes.xacro (robot description, xacro)
@@ -51,5 +51,5 @@
 	<xacro:property name="ThumbProximalNode" value="_arm/hand/thumb_proximal"/>
 	<xacro:property name="ThumbDistalNode" value="_arm/hand/thumb_distal"/>
-	<xacro:property name="ThumbRollSensNode" value="_arm/forearm_sensors/thumb"/>
+	<xacro:property name="ThumbRollSenseNode" value="_arm/forearm_sensors/thumb"/>
 	<xacro:property name="ThumbPitch1Node" value="_arm/forearm_sensors/thumb"/>
 	<xacro:property name="ThumbPitch2Node" value="_arm/forearm_sensors/thumb"/>

File: model/robots/common/xacro/thumb/thumb.xacro (robot description, xacro)
@@ -97,5 +97,5 @@
   </xacro:macro>
   <xacro:macro name="thumb_transmissions_hw" params="prefix reflect">
-    <xacro:simple_position_transmission jointName="${prefix}${ThumbRollJointName}" actuatorName="${prefix}ThumbRollActuator" nodeName="/${prefix}${ThumbRollSensNode}" actuatorApi="${ThumbFingerRollApi}"/>
+    <xacro:simple_position_transmission jointName="${prefix}${ThumbRollJointName}" actuatorName="${prefix}ThumbRollActuator" nodeName="/${prefix}${ThumbRollSenseNode}" actuatorApi="${ThumbFingerRollApi}"/>
     <xacro:simple_forearm_position_transmission jointName="${prefix}${ThumbPitch1JointName}" actuatorName="${prefix}ThumbPitch1Actuator" nodeName="/${prefix}${ThumbPitch1Node}" actuatorApi="${ThumbFingerProximalApi}" reflect="${reflect}"/>
     <xacro:simple_forearm_position_transmission jointName="${prefix}${ThumbPitch2JointName}" actuatorName="${prefix}ThumbPitch2Actuator" nodeName="/${prefix}${ThumbPitch2Node}" actuatorApi="${ThumbFingerMedialApi}" reflect="${reflect}"/>
