Commit message: Still waffling around on the finger transmission xml.

File: common/xacro/nodes/valkyrie_sim_nodes.xacro (robot description, xacro)
@@ -26,5 +26,5 @@
 	<xacro:property name="left_foot_ATI_node" value="/left_leg/ankle/roll_actuator" />
 	<xacro:property name="right_foot_ATI_node" value="/right_leg/ankle/roll_actuator" />
-	<xacro:property name="ThumbRollNode" value="/remap/${prefix}_hand/thumb/roll"/>
+	<xacro:property name="ThumbRollNode" value="/${prefix}_hand/thumb_roll"/>
 	<xacro:property name="ThumbPitch1Node" value="/remap/${prefix}_hand/thumb/pitch_1"/>
 	<xacro:property name="ThumbPitch2Node" value="/remap/${prefix}_hand/thumb/pitch_2"/>

File: model/robots/common/xacro/generic_models.xacro (robot description, xacro)
@@ -225,25 +225,24 @@
     </transmission>
   </xacro:macro>
-  <xacro:macro name="finger_transmission" params="joint1Name actuatorName node1Name actuatorApi joint2Name joint3Name ratio1 ratio2 node2Name node3Name">
-    <transmission name="${joint1Name}Transmission">
-      <type>transmission_interface/SimpleTransmission</type>
-      <joint name="${joint1Name}">
-        <hardwareInterface>PositionJointInterface</hardwareInterface>
+  <xacro:macro name="finger_transmission" params="jointName actuatorName nodeName actuatorApi child1JointName child1Ratio child2JointName child2Ratio">
+    <transmission name="${jointName}Transmission">
+      <type>transmission_interface/SimpleTransmission</type>
+      <joint name="${jointName}">
+        <hardwareInterface>PositionJointInterface</hardwareInterface>
+        <child name="${child1JointName}" ratio="${child1Ratio}"/>
+        <child name="${child2JointName}" ratio="${child2Ratio}"/>
       </joint>
       <actuator name="${actuatorName}">
-        <node name="${node1Name}"/>
+        <node name="${nodeName}"/>
         <mechanicalReduction>1</mechanicalReduction>
         <api name="${actuatorApi}" />
       </actuator>
-      <children>
-        <joint name="${joint2Name}" ratio="${ratio1}" parent="${joint1Name}" childNode="${node2Name}"/>
-        <joint name="${joint3Name}" ratio="${ratio2}" parent="${joint1Name}" childNode="${node3Name}"/>
-      </children>
     </transmission>
   </xacro:macro>
   <xacro:macro name="simple_passive_transmission" params="jointName nodeName apiName">
-    <transmission name="${jointName}PassiveTransmission">
-      <type>transmission_interface/SimpleTransmission</type>
-      <joint name="${jointName}">
+    <transmission name="${jointName}PassiveTransmissionWithParent">
+      <type>transmission_interface/SimpleTransmission</type>
+      <joint name="${jointName}">
+        <hardwareInterface>JointStateInterface</hardwareInterface>
       </joint>
       <actuator name="${jointName}PassiveActuator">

File: model/robots/common/xacro/thumb/thumb.xacro (robot description, xacro)
@@ -93,5 +93,5 @@
   <xacro:macro name="thumb_transmissions_sim" params="prefix">
     <xacro:simple_position_transmission jointName="${ThumbRollJointName}" actuatorName="${prefix}ThumbRollActuator" nodeName="${ThumbRollNode}" actuatorApi="${SimApi}"/>
-    <xacro:finger_transmission joint1Name="${ThumbPitch1JointName}" actuatorName="${prefix}ThumbPitch1Actuator" node1Name="${ThumbPitch1Node}" actuatorApi="${SimApi}" joint2Name="${ThumbPitch2JointName}" joint3Name="${ThumbPitch3JointName}" ratio1="${Pulley2Ratio}" ratio2="${Pulley3Ratio}" node2Name="${ThumbPitch2Node}" node3Name="${ThumbPitch3Node}" />
+    <xacro:finger_transmission jointName="${ThumbPitch1JointName}" actuatorName="${prefix}ThumbPitch1Actuator" nodeName="${ThumbPitch1Node}" actuatorApi="${SimApi}" child1JointName="${ThumbPitch2JointName}" child1Ratio="${Pulley2Ratio}" child2JointName="${ThumbPitch2Node}" child2Ratio="${Pulley3Ratio}"/>
     <xacro:simple_passive_transmission jointName="${ThumbPitch2JointName}" nodeName="${ThumbPitch2Node}" apiName="${SimApi}"/>
     <xacro:simple_passive_transmission jointName="${ThumbPitch3JointName}" nodeName="${ThumbPitch3Node}" apiName="${SimApi}"/>

File: model/robots/common/xacro/valkyrie_base_sim.xacro (robot description, xacro)
@@ -1,5 +1,5 @@
 <robot xmlns:xacro="http://ros.org/wiki/xacro" name="valkyrie">
     <xacro:include filename="$(find val_description)/common/xacro/nodes/valkyrie_sim_nodes.xacro"/>
-    <shm_remap_file package="val_gazebo" relative_file_path="/configurations/valkyrie_sim_shm_remap.yaml"/>
+    <shm_remap_file package="val_gazebo" relative_file_path="/configuration/valkyrie_sim_shm_remap.yaml"/>
     <xacro:make_pelvis />
     <xacro:make_waist waist_root_link="${Pelvis_Link_Name}" />
@@ -29,4 +29,3 @@
     <xacro:neck_transmissions_sim />
     <xacro:thumb_transmissions_sim prefix="left"/>
-    <xacro:thumb_transmissions_sim prefix="right"/>
 </robot>

Commit message: Messing with thumb stuff for sim fingers. Added in friction/damping to hopefully  make them a bit more stable in sim.

File: common/xacro/nodes/valkyrie_sim_nodes.xacro (robot description, xacro)
@@ -27,7 +27,7 @@
 	<xacro:property name="right_foot_ATI_node" value="/right_leg/ankle/roll_actuator" />
 	<xacro:property name="ThumbRollNode" value="/${prefix}_hand/thumb_roll"/>
-	<xacro:property name="ThumbPitch1Node" value="/remap/${prefix}_hand/thumb/pitch_1"/>
-	<xacro:property name="ThumbPitch2Node" value="/remap/${prefix}_hand/thumb/pitch_2"/>
-	<xacro:property name="ThumbPitch3Node" value="/remap/${prefix}_hand/thumb/pitch_3"/>
+	<xacro:property name="ThumbPitch1Node" value="/${prefix}_hand/thumb_pitch_1"/>
+	<xacro:property name="ThumbPitch2Node" value="/${prefix}_hand/thumb_pitch_2"/>
+	<xacro:property name="ThumbPitch3Node" value="/${prefix}_hand/thumb_pitch_3"/>
 	<xacro:macro name="all_channels" >
 		<Channels>

File: model/robots/common/xacro/gains.xacro (robot description, xacro)
@@ -18,3 +18,15 @@
     <xacro:property name="UpperNeckPitchKd" value="0" />
     <xacro:property name="UpperNeckPitchKi" value="0.0" />
+    <xacro:property name="ThumbRollKp" value="5.0" />
+    <xacro:property name="ThumbRollKd" value="0.0" />
+    <xacro:property name="ThumbRollKi" value="0.0" />
+    <xacro:property name="ThumbPitch1Kp" value="5.0" />
+    <xacro:property name="ThumbPitch1Kd" value="0.0" />
+    <xacro:property name="ThumbPitch1Ki" value="0.0" />
+    <xacro:property name="ThumbPitch2Kp" value="5.0" />
+    <xacro:property name="ThumbPitch2Kd" value="0.0" />
+    <xacro:property name="ThumbPitch2Ki" value="0.0" />
+    <xacro:property name="ThumbPitch3Kp" value="5.0" />
+    <xacro:property name="ThumbPitch3Kd" value="0.0" />
+    <xacro:property name="ThumbPitch3Ki" value="0.0" />
 </robot>

File: model/robots/common/xacro/generic_models.xacro (robot description, xacro)
@@ -241,5 +241,5 @@
   </xacro:macro>
   <xacro:macro name="simple_passive_transmission" params="jointName nodeName apiName">
-    <transmission name="${jointName}PassiveTransmissionWithParent">
+    <transmission name="${jointName}PassiveTransmission">
       <type>transmission_interface/SimpleTransmission</type>
       <joint name="${jointName}">

File: model/robots/common/xacro/thumb/thumb.xacro (robot description, xacro)
@@ -8,4 +8,5 @@
   <xacro:include filename="$(find val_description)/model/robots/common/xacro/thumb/mass_parameters.xacro"/>
   <xacro:include filename="$(find val_description)/model/robots/common/xacro/thumb/mechanical_info.xacro"/>
+  <xacro:include filename="$(find val_description)/model/robots/common/xacro/gains.xacro"/>
   <xacro:macro name="make_thumb" params="prefix reflect thumb_root_link">
     <xacro:standard_link name="${ThumbRollLinkName}"
@@ -41,16 +42,17 @@
                     visual_mesh="${mesh_root}/fingers/thumbj4_${prefix}.dae"
                     collision_mesh="${mesh_root}/fingers/thumbj4_${prefix}.dae"/>
-    <xacro:revolute_joint jointName="${ThumbRollJointName}"
+    <xacro:revolute_joint_ex jointName="${ThumbRollJointName}"
                           parent="${ThumbRollParentLinkName}" child="${ThumbRollLinkName}"
                           origin_xyz="${ThumbRollFrameOrigin_X} ${ThumbRollFrameOrigin_Y} ${ThumbRollFrameOrigin_Z}"
                           origin_rpy="${ThumbRollFrameOrientation_Roll} ${ThumbRollFrameOrientation_Pitch} ${ThumbRollFrameOrientation_Yaw}"
-                          axis="${ThumbRollRotationAxis}">
+                          axis="${ThumbRollRotationAxis}" damping="0.5" friction="0.5">
         <limit effort="${ThumbRollTorqueLimit}" lower="${ThumbRollPositionLimit_Lower}" upper="${ThumbRollPositionLimit_Upper}" velocity="${ThumbRollVelocityLimit}"/>
-    </xacro:revolute_joint>
-    <xacro:revolute_joint jointName="${ThumbPitch1JointName}"
+         <controller_gains Kp="${ThumbRollKp}" Kd="${ThumbRollKd}" Ki="${ThumbRollKi}"/>
+    </xacro:revolute_joint_ex>
+    <xacro:revolute_joint_ex jointName="${ThumbPitch1JointName}"
                           parent="${ThumbRollLinkName}" child="${ThumbPitch1LinkName}"
                           origin_xyz="${ThumbPitch1FrameOrigin_X} ${ThumbPitch1FrameOrigin_Y} ${ThumbPitch1FrameOrigin_Z}"
                           origin_rpy="${ThumbPitch1FrameOrientation_Roll} ${ThumbPitch1FrameOrientation_Pitch} ${ThumbPitch1FrameOrientation_Yaw}"
-                          axis="${ThumbPitch1RotationAxis}">
+                          axis="${ThumbPitch1RotationAxis}" damping="0.5" friction="0.5">
         <xacro:if value="${(reflect+1)/2}">
           <limit effort="${ThumbPitch1TorqueLimit}" lower="${-reflect * ThumbPitch1PositionLimit_Upper}" upper="${-reflect * ThumbPitch1PositionLimit_Lower}" velocity="${ThumbPitch1VelocityLimit}"/>
@@ -59,10 +61,11 @@
           <limit effort="${ThumbPitch1TorqueLimit}" lower="${ThumbPitch1PositionLimit_Lower}" upper="${ThumbPitch1PositionLimit_Upper}" velocity="${ThumbPitch1VelocityLimit}"/>
         </xacro:if>
-    </xacro:revolute_joint>
-    <xacro:revolute_joint jointName="${ThumbPitch2JointName}"
+        <controller_gains Kp="${ThumbPitch1Kp}" Kd="${ThumbPitch1Kd}" Ki="${ThumbPitch1Ki}"/>
+    </xacro:revolute_joint_ex>
+    <xacro:revolute_joint_ex jointName="${ThumbPitch2JointName}"
                           parent="${ThumbPitch1LinkName}" child="${ThumbPitch2LinkName}"
                           origin_xyz="${ThumbPitch2FrameOrigin_X} ${ThumbPitch2FrameOrigin_Y} ${ThumbPitch2FrameOrigin_Z}"
                           origin_rpy="${ThumbPitch2FrameOrientation_Roll} ${ThumbPitch2FrameOrientation_Pitch} ${ThumbPitch2FrameOrientation_Yaw}"
-                          axis="${ThumbPitch2RotationAxis}">
+                          axis="${ThumbPitch2RotationAxis}" damping="0.5" friction="0.5">
         <xacro:if value="${(reflect+1)/2}">
           <limit effort="${ThumbPitch2TorqueLimit}" lower="${-reflect * ThumbPitch2PositionLimit_Upper}" upper="${-reflect * ThumbPitch2PositionLimit_Lower}" velocity="${ThumbPitch2VelocityLimit}"/>
@@ -71,10 +74,11 @@
           <limit effort="${ThumbPitch2TorqueLimit}" lower="${ThumbPitch2PositionLimit_Lower}" upper="${ThumbPitch2PositionLimit_Upper}" velocity="${ThumbPitch2VelocityLimit}"/>
         </xacro:if>
-    </xacro:revolute_joint>
-    <xacro:revolute_joint jointName="${ThumbPitch3JointName}"
+        <controller_gains Kp="${ThumbPitch2Kp}" Kd="${ThumbPitch2Kd}" Ki="${ThumbPitch2Ki}"/>
+    </xacro:revolute_joint_ex>
+    <xacro:revolute_joint_ex jointName="${ThumbPitch3JointName}"
                           parent="${ThumbPitch2LinkName}" child="${ThumbPitch3LinkName}"
                           origin_xyz="${ThumbPitch3FrameOrigin_X} ${ThumbPitch3FrameOrigin_Y} ${ThumbPitch3FrameOrigin_Z}"
                           origin_rpy="${ThumbPitch3FrameOrientation_Roll} ${ThumbPitch3FrameOrientation_Pitch} ${ThumbPitch3FrameOrientation_Yaw}"
-                          axis="${ThumbPitch3RotationAxis}">
+                          axis="${ThumbPitch3RotationAxis}" damping="0.5" friction="0.5">
         <xacro:if value="${(reflect+1)/2}">
           <limit effort="${ThumbPitch3TorqueLimit}" lower="${-reflect * ThumbPitch3PositionLimit_Upper}" upper="${-reflect * ThumbPitch3PositionLimit_Lower}" velocity="${ThumbPitch3VelocityLimit}"/>
@@ -83,5 +87,6 @@
           <limit effort="${ThumbPitch3TorqueLimit}" lower="${ThumbPitch3PositionLimit_Lower}" upper="${ThumbPitch3PositionLimit_Upper}" velocity="${ThumbPitch3VelocityLimit}"/>
         </xacro:if>
-    </xacro:revolute_joint>
+        <controller_gains Kp="${ThumbPitch3Kp}" Kd="${ThumbPitch3Kd}" Ki="${ThumbPitch3Ki}"/>
+    </xacro:revolute_joint_ex>
   </xacro:macro>
   <xacro:macro name="thumb_transmissions_hw" params="prefix reflect">
@@ -93,5 +98,5 @@
   <xacro:macro name="thumb_transmissions_sim" params="prefix">
     <xacro:simple_position_transmission jointName="${ThumbRollJointName}" actuatorName="${prefix}ThumbRollActuator" nodeName="${ThumbRollNode}" actuatorApi="${SimApi}"/>
-    <xacro:finger_transmission jointName="${ThumbPitch1JointName}" actuatorName="${prefix}ThumbPitch1Actuator" nodeName="${ThumbPitch1Node}" actuatorApi="${SimApi}" child1JointName="${ThumbPitch2JointName}" child1Ratio="${Pulley2Ratio}" child2JointName="${ThumbPitch2Node}" child2Ratio="${Pulley3Ratio}"/>
+    <xacro:finger_transmission jointName="${ThumbPitch1JointName}" actuatorName="${prefix}ThumbPitch1Actuator" nodeName="${ThumbPitch1Node}" actuatorApi="${SimApi}" child1JointName="${ThumbPitch2JointName}" child1Ratio="${Pulley2Ratio}" child2JointName="${ThumbPitch3JointName}" child2Ratio="${Pulley3Ratio}"/>
     <xacro:simple_passive_transmission jointName="${ThumbPitch2JointName}" nodeName="${ThumbPitch2Node}" apiName="${SimApi}"/>
     <xacro:simple_passive_transmission jointName="${ThumbPitch3JointName}" nodeName="${ThumbPitch3Node}" apiName="${SimApi}"/>

File: model/robots/common/xacro/valkyrie_base_sim.xacro (robot description, xacro)
@@ -1,5 +1,4 @@
 <robot xmlns:xacro="http://ros.org/wiki/xacro" name="valkyrie">
     <xacro:include filename="$(find val_description)/common/xacro/nodes/valkyrie_sim_nodes.xacro"/>
-    <shm_remap_file package="val_gazebo" relative_file_path="/configuration/valkyrie_sim_shm_remap.yaml"/>
     <xacro:make_pelvis />
     <xacro:make_waist waist_root_link="${Pelvis_Link_Name}" />
