Commit message: Added sim transmissions for the rest of the fingers.

File: common/xacro/nodes/valkyrie_sim_nodes.xacro (robot description, xacro)
@@ -1,8 +1,8 @@
 <robot xmlns:xacro="http://ros.org/wiki/xacro" name="valkyrie_sim_nodes">
-	<xacro:property name="HipYawNode" value="/pelvis_neck/pelvis_${prefix}_leg_j1" />
-	<xacro:property name="TrunkYawNode" value="/pelvis_neck/pelvis_waist" /> <!--Yaw-->
-	<xacro:property name="LowerNeckPitchNode" value="/pelvis_neck/neck_j1" />
-	<xacro:property name="NeckYawNode" value="/pelvis_neck/neck_j2" />
-	<xacro:property name="UpperNeckPitchNode" value="/pelvis_neck/neck_j3" />
+	<xacro:property name="HipYawNode" value="/pelvis/${prefix}_leg_j1" />
+	<xacro:property name="TrunkYawNode" value="/pelvis/waist" /> <!--Yaw-->
+	<xacro:property name="LowerNeckPitchNode" value="/neck/j1" />
+	<xacro:property name="NeckYawNode" value="/neck/j2" />
+	<xacro:property name="UpperNeckPitchNode" value="/neck/j3" />
 	<xacro:property name="HipRollNode" value="/${prefix}_leg/j2" />
 	<xacro:property name="HipPitchNode" value="/${prefix}_leg/j3" />
@@ -30,4 +30,13 @@
 	<xacro:property name="ThumbPitch2Node" value="/${prefix}_hand/thumb_pitch_2"/>
 	<xacro:property name="ThumbPitch3Node" value="/${prefix}_hand/thumb_pitch_3"/>
+	<xacro:property name="IndexFingerPitch1Node" value="/${prefix}_hand/index_finger_pitch_1"/>
+	<xacro:property name="IndexFingerPitch2Node" value="/${prefix}_hand/index_finger_pitch_2"/>
+	<xacro:property name="IndexFingerPitch3Node" value="/${prefix}_hand/index_finger_pitch_3"/>
+	<xacro:property name="MiddleFingerPitch1Node" value="/${prefix}_hand/middle_finger_pitch_1"/>
+	<xacro:property name="MiddleFingerPitch2Node" value="/${prefix}_hand/middle_finger_pitch_2"/>
+	<xacro:property name="MiddleFingerPitch3Node" value="/${prefix}_hand/middle_finger_pitch_3"/>
+	<xacro:property name="PinkyPitch1Node" value="/${prefix}_hand/pinky_pitch_1"/>
+	<xacro:property name="PinkyPitch2Node" value="/${prefix}_hand/pinky_pitch_2"/>
+	<xacro:property name="PinkyPitch3Node" value="/${prefix}_hand/pinky_pitch_3"/>
 	<xacro:macro name="all_channels" >
 		<Channels>

File: model/robots/common/xacro/gains.xacro (robot description, xacro)
@@ -30,3 +30,30 @@
     <xacro:property name="ThumbPitch3Kd" value="0.0" />
     <xacro:property name="ThumbPitch3Ki" value="0.0" />
+    <xacro:property name="IndexFingerPitch1Kp" value="5.0" />
+    <xacro:property name="IndexFingerPitch1Kd" value="0.3" />
+    <xacro:property name="IndexFingerPitch1Ki" value="0.0" />
+    <xacro:property name="IndexFingerPitch2Kp" value="5.0" />
+    <xacro:property name="IndexFingerPitch2Kd" value="0.3" />
+    <xacro:property name="IndexFingerPitch2Ki" value="0.0" />
+    <xacro:property name="IndexFingerPitch3Kp" value="5.0" />
+    <xacro:property name="IndexFingerPitch3Kd" value="0.3" />
+    <xacro:property name="IndexFingerPitch3Ki" value="0.0" />
+    <xacro:property name="MiddleFingerPitch1Kp" value="5.0" />
+    <xacro:property name="MiddleFingerPitch1Kd" value="0.3" />
+    <xacro:property name="MiddleFingerPitch1Ki" value="0.0" />
+    <xacro:property name="MiddleFingerPitch2Kp" value="5.0" />
+    <xacro:property name="MiddleFingerPitch2Kd" value="0.3" />
+    <xacro:property name="MiddleFingerPitch2Ki" value="0.0" />
+    <xacro:property name="MiddleFingerPitch3Kp" value="5.0" />
+    <xacro:property name="MiddleFingerPitch3Kd" value="0.3" />
+    <xacro:property name="MiddleFingerPitch3Ki" value="0.0" />
+    <xacro:property name="PinkyPitch1Kp" value="5.0" />
+    <xacro:property name="PinkyPitch1Kd" value="0.3" />
+    <xacro:property name="PinkyPitch1Ki" value="0.0" />
+    <xacro:property name="PinkyPitch2Kp" value="5.0" />
+    <xacro:property name="PinkyPitch2Kd" value="0.3" />
+    <xacro:property name="PinkyPitch2Ki" value="0.0" />
+    <xacro:property name="PinkyPitch3Kp" value="5.0" />
+    <xacro:property name="PinkyPitch3Kd" value="0.3" />
+    <xacro:property name="PinkyPitch3Ki" value="0.0" />
 </robot>

File: model/robots/common/xacro/generic_models.xacro (robot description, xacro)
@@ -225,5 +225,5 @@
     </transmission>
   </xacro:macro>
-  <xacro:macro name="finger_transmission" params="jointName actuatorName nodeName actuatorApi child1JointName child1Ratio child2JointName child2Ratio">
+  <xacro:macro name="simple_transmission_with_child_joints" params="jointName actuatorName nodeName actuatorApi child1JointName child1Ratio child2JointName child2Ratio">
     <transmission name="${jointName}Transmission">
       <type>transmission_interface/SimpleTransmission</type>

File: model/robots/common/xacro/index_finger/index_finger.xacro (robot description, xacro)
@@ -6,4 +6,5 @@
   <xacro:include filename="$(find val_description)/model/robots/common/xacro/index_finger/joint_limits.xacro"/>
   <xacro:include filename="$(find val_description)/model/robots/common/xacro/index_finger/frame_parameters.xacro"/>
+  <xacro:include filename="$(find val_description)/model/robots/common/xacro/index_finger/mechanical_info.xacro"/>
   <xacro:include filename="$(find val_description)/model/robots/common/xacro/index_finger/mass_parameters.xacro"/>
   <xacro:macro name="make_index_finger" params="prefix reflect index_finger_root_link">
@@ -32,9 +33,9 @@
                     visual_mesh="${mesh_root}/fingers/indexj3_${prefix}.dae"
                     collision_mesh="${mesh_root}/fingers/indexj3_${prefix}.dae"/>
-    <xacro:revolute_joint jointName="${IndexFingerPitch1JointName}"
+    <xacro:revolute_joint_ex jointName="${IndexFingerPitch1JointName}"
                           parent="${IndexFingerPitch1ParentLinkName}" child="${IndexFingerPitch1LinkName}"
                           origin_xyz="${IndexFingerPitch1FrameOrigin_X} ${IndexFingerPitch1FrameOrigin_Y} ${IndexFingerPitch1FrameOrigin_Z}"
                           origin_rpy="${IndexFingerPitch1FrameOrientation_Roll} ${IndexFingerPitch1FrameOrientation_Pitch} ${IndexFingerPitch1FrameOrientation_Yaw}"
-                          axis="${IndexFingerPitch1RotationAxis}">
+                          axis="${IndexFingerPitch1RotationAxis}" damping="0.5" friction="0.5">
         <xacro:if value="${(reflect+1)/2}">
           <limit effort="${IndexFingerPitch1TorqueLimit}" lower="${-reflect * IndexFingerPitch1PositionLimit_Upper}" upper="${-reflect * IndexFingerPitch1PositionLimit_Lower}" velocity="${IndexFingerPitch1VelocityLimit}"/>
@@ -43,10 +44,11 @@
           <limit effort="${IndexFingerPitch1TorqueLimit}" lower="${IndexFingerPitch1PositionLimit_Lower}" upper="${IndexFingerPitch1PositionLimit_Upper}" velocity="${IndexFingerPitch1VelocityLimit}"/>
         </xacro:if>
-    </xacro:revolute_joint>
-    <xacro:revolute_joint jointName="${IndexFingerPitch2JointName}"
+        <controller_gains Kp="${IndexFingerPitch1Kp}" Kd="${IndexFingerPitch1Kd}" Ki="${IndexFingerPitch1Ki}"/>
+    </xacro:revolute_joint_ex>
+    <xacro:revolute_joint_ex jointName="${IndexFingerPitch2JointName}"
                           parent="${IndexFingerPitch1LinkName}" child="${IndexFingerPitch2LinkName}"
                           origin_xyz="${IndexFingerPitch2FrameOrigin_X} ${IndexFingerPitch2FrameOrigin_Y} ${IndexFingerPitch2FrameOrigin_Z}"
                           origin_rpy="${IndexFingerPitch2FrameOrientation_Roll} ${IndexFingerPitch2FrameOrientation_Pitch} ${IndexFingerPitch2FrameOrientation_Yaw}"
-                          axis="${IndexFingerPitch2RotationAxis}">
+                          axis="${IndexFingerPitch2RotationAxis}" damping="0.5" friction="0.5">
         <xacro:if value="${(reflect+1)/2}">
           <limit effort="${IndexFingerPitch2TorqueLimit}" lower="${-reflect * IndexFingerPitch2PositionLimit_Upper}" upper="${-reflect * IndexFingerPitch2PositionLimit_Lower}" velocity="${IndexFingerPitch2VelocityLimit}"/>
@@ -55,10 +57,11 @@
           <limit effort="${IndexFingerPitch2TorqueLimit}" lower="${IndexFingerPitch2PositionLimit_Lower}" upper="${IndexFingerPitch2PositionLimit_Upper}" velocity="${IndexFingerPitch2VelocityLimit}"/>
         </xacro:if>
-    </xacro:revolute_joint>
-    <xacro:revolute_joint jointName="${IndexFingerPitch3JointName}"
+        <controller_gains Kp="${IndexFingerPitch1Kp}" Kd="${IndexFingerPitch1Kd}" Ki="${IndexFingerPitch1Ki}"/>
+    </xacro:revolute_joint_ex>
+    <xacro:revolute_joint_ex jointName="${IndexFingerPitch3JointName}"
                           parent="${IndexFingerPitch2LinkName}" child="${IndexFingerPitch3LinkName}"
                           origin_xyz="${IndexFingerPitch3FrameOrigin_X} ${IndexFingerPitch3FrameOrigin_Y} ${IndexFingerPitch3FrameOrigin_Z}"
                           origin_rpy="${IndexFingerPitch3FrameOrientation_Roll} ${IndexFingerPitch3FrameOrientation_Pitch} ${IndexFingerPitch3FrameOrientation_Yaw}"
-                          axis="${IndexFingerPitch3RotationAxis}">
+                          axis="${IndexFingerPitch3RotationAxis}" damping="0.5" friction="0.5">
         <xacro:if value="${(reflect+1)/2}">
           <limit effort="${IndexFingerPitch3TorqueLimit}" lower="${-reflect * IndexFingerPitch3PositionLimit_Upper}" upper="${-reflect * IndexFingerPitch3PositionLimit_Lower}" velocity="${IndexFingerPitch3VelocityLimit}"/>
@@ -67,5 +70,6 @@
           <limit effort="${IndexFingerPitch3TorqueLimit}" lower="${IndexFingerPitch3PositionLimit_Lower}" upper="${IndexFingerPitch3PositionLimit_Upper}" velocity="${IndexFingerPitch3VelocityLimit}"/>
         </xacro:if>
-    </xacro:revolute_joint>
+        <controller_gains Kp="${IndexFingerPitch1Kp}" Kd="${IndexFingerPitch1Kd}" Ki="${IndexFingerPitch1Ki}"/>
+    </xacro:revolute_joint_ex>
   </xacro:macro>
   <xacro:macro name="index_finger_transmissions_hw" params="prefix reflect">
@@ -74,3 +78,8 @@
     <xacro:simple_forearm_position_transmission jointName="${IndexFingerPitch3JointName}" actuatorName="${prefix}IndexPitch3Actuator" nodeName="${IndexFingerPitch3Node}" actuatorApi="${IndexFingerApi}" reflect="${reflect}"/>
   </xacro:macro>
+  <xacro:macro name="index_finger_transmissions_sim" params="prefix">
+    <xacro:simple_transmission_with_child_joints jointName="${IndexFingerPitch1JointName}" actuatorName="${prefix}IndexFingerPitch1Actuator" nodeName="${IndexFingerPitch1Node}" actuatorApi="${SimApi}" child1JointName="${IndexFingerPitch2JointName}" child1Ratio="${Pulley2Ratio}" child2JointName="${IndexFingerPitch3JointName}" child2Ratio="${Pulley3Ratio}"/>
+    <xacro:simple_passive_transmission jointName="${IndexFingerPitch2JointName}" nodeName="${IndexFingerPitch2Node}" apiName="${SimApi}"/>
+    <xacro:simple_passive_transmission jointName="${IndexFingerPitch3JointName}" nodeName="${IndexFingerPitch3Node}" apiName="${SimApi}"/>
+  </xacro:macro>
 </robot>

File: model/robots/common/xacro/middle_finger/middle_finger.xacro (robot description, xacro)
@@ -6,4 +6,5 @@
   <xacro:include filename="$(find val_description)/model/robots/common/xacro/middle_finger/joint_limits.xacro"/>
   <xacro:include filename="$(find val_description)/model/robots/common/xacro/middle_finger/frame_parameters.xacro"/>
+  <xacro:include filename="$(find val_description)/model/robots/common/xacro/middle_finger/mechanical_info.xacro"/>
   <xacro:include filename="$(find val_description)/model/robots/common/xacro/middle_finger/mass_parameters.xacro"/>
   <xacro:macro name="make_middle_finger" params="prefix reflect middle_finger_root_link">
@@ -32,9 +33,9 @@
                     visual_mesh="${mesh_root}/fingers/middlej3_${prefix}.dae"
                     collision_mesh="${mesh_root}/fingers/middlej3_${prefix}.dae"/>
-    <xacro:revolute_joint jointName="${MiddleFingerPitch1JointName}"
+    <xacro:revolute_joint_ex jointName="${MiddleFingerPitch1JointName}"
                           parent="${MiddleFingerPitch1ParentLinkName}" child="${MiddleFingerPitch1LinkName}"
                           origin_xyz="${MiddleFingerPitch1FrameOrigin_X} ${MiddleFingerPitch1FrameOrigin_Y} ${MiddleFingerPitch1FrameOrigin_Z}"
                           origin_rpy="${MiddleFingerPitch1FrameOrientation_Roll} ${MiddleFingerPitch1FrameOrientation_Pitch} ${MiddleFingerPitch1FrameOrientation_Yaw}"
-                          axis="${MiddleFingerPitch1RotationAxis}">
+                          axis="${MiddleFingerPitch1RotationAxis}" damping="0.5" friction="0.5">
         <xacro:if value="${(reflect+1)/2}">
           <limit effort="${MiddleFingerPitch1TorqueLimit}" lower="${-reflect * MiddleFingerPitch1PositionLimit_Upper}" upper="${-reflect * MiddleFingerPitch1PositionLimit_Lower}" velocity="${MiddleFingerPitch1VelocityLimit}"/>
@@ -43,10 +44,11 @@
           <limit effort="${MiddleFingerPitch1TorqueLimit}" lower="${MiddleFingerPitch1PositionLimit_Lower}" upper="${MiddleFingerPitch1PositionLimit_Upper}" velocity="${MiddleFingerPitch1VelocityLimit}"/>
         </xacro:if>
-    </xacro:revolute_joint>
-    <xacro:revolute_joint jointName="${MiddleFingerPitch2JointName}"
+        <controller_gains Kp="${MiddleFingerPitch1Kp}" Kd="${MiddleFingerPitch1Kd}" Ki="${MiddleFingerPitch1Ki}"/>
+    </xacro:revolute_joint_ex>
+    <xacro:revolute_joint_ex jointName="${MiddleFingerPitch2JointName}"
                           parent="${MiddleFingerPitch1LinkName}" child="${MiddleFingerPitch2LinkName}"
                           origin_xyz="${MiddleFingerPitch2FrameOrigin_X} ${MiddleFingerPitch2FrameOrigin_Y} ${MiddleFingerPitch2FrameOrigin_Z}"
                           origin_rpy="${MiddleFingerPitch2FrameOrientation_Roll} ${MiddleFingerPitch2FrameOrientation_Pitch} ${MiddleFingerPitch2FrameOrientation_Yaw}"
-                          axis="${MiddleFingerPitch2RotationAxis}">
+                          axis="${MiddleFingerPitch2RotationAxis}" damping="0.5" friction="0.5">
         <xacro:if value="${(reflect+1)/2}">
           <limit effort="${MiddleFingerPitch2TorqueLimit}" lower="${-reflect * MiddleFingerPitch2PositionLimit_Upper}" upper="${-reflect * MiddleFingerPitch2PositionLimit_Lower}" velocity="${MiddleFingerPitch2VelocityLimit}"/>
@@ -55,10 +57,11 @@
           <limit effort="${MiddleFingerPitch2TorqueLimit}" lower="${MiddleFingerPitch2PositionLimit_Lower}" upper="${MiddleFingerPitch2PositionLimit_Upper}" velocity="${MiddleFingerPitch2VelocityLimit}"/>
         </xacro:if>
-    </xacro:revolute_joint>
-    <xacro:revolute_joint jointName="${MiddleFingerPitch3JointName}"
+        <controller_gains Kp="${MiddleFingerPitch1Kp}" Kd="${MiddleFingerPitch1Kd}" Ki="${MiddleFingerPitch1Ki}"/>
+    </xacro:revolute_joint_ex>
+    <xacro:revolute_joint_ex jointName="${MiddleFingerPitch3JointName}"
                           parent="${MiddleFingerPitch2LinkName}" child="${MiddleFingerPitch3LinkName}"
                           origin_xyz="${MiddleFingerPitch3FrameOrigin_X} ${MiddleFingerPitch3FrameOrigin_Y} ${MiddleFingerPitch3FrameOrigin_Z}"
                           origin_rpy="${MiddleFingerPitch3FrameOrientation_Roll} ${MiddleFingerPitch3FrameOrientation_Pitch} ${MiddleFingerPitch3FrameOrientation_Yaw}"
-                          axis="${MiddleFingerPitch3RotationAxis}">
+                          axis="${MiddleFingerPitch3RotationAxis}" damping="0.5" friction="0.5">
         <xacro:if value="${(reflect+1)/2}">
           <limit effort="${MiddleFingerPitch3TorqueLimit}" lower="${-reflect * MiddleFingerPitch3PositionLimit_Upper}" upper="${-reflect * MiddleFingerPitch3PositionLimit_Lower}" velocity="${MiddleFingerPitch3VelocityLimit}"/>
@@ -67,5 +70,6 @@
           <limit effort="${MiddleFingerPitch3TorqueLimit}" lower="${MiddleFingerPitch3PositionLimit_Lower}" upper="${MiddleFingerPitch3PositionLimit_Upper}" velocity="${MiddleFingerPitch3VelocityLimit}"/>
         </xacro:if>
-    </xacro:revolute_joint>
+        <controller_gains Kp="${MiddleFingerPitch1Kp}" Kd="${MiddleFingerPitch1Kd}" Ki="${MiddleFingerPitch1Ki}"/>
+    </xacro:revolute_joint_ex>
   </xacro:macro>
   <xacro:macro name="middle_finger_transmissions_hw" params="prefix reflect">
@@ -74,3 +78,8 @@
     <xacro:simple_forearm_position_transmission jointName="${MiddleFingerPitch3JointName}" actuatorName="${prefix}MiddlePitch3Actuator" nodeName="${MiddleFingerPitch3Node}" actuatorApi="${MiddleFingerApi}" reflect="${reflect}"/>
   </xacro:macro>
+  <xacro:macro name="middle_finger_transmissions_sim" params="prefix">
+    <xacro:simple_transmission_with_child_joints jointName="${MiddleFingerPitch1JointName}" actuatorName="${prefix}MiddleFingerPitch1Actuator" nodeName="${MiddleFingerPitch1Node}" actuatorApi="${SimApi}" child1JointName="${MiddleFingerPitch2JointName}" child1Ratio="${Pulley2Ratio}" child2JointName="${MiddleFingerPitch3JointName}" child2Ratio="${Pulley3Ratio}"/>
+    <xacro:simple_passive_transmission jointName="${MiddleFingerPitch2JointName}" nodeName="${MiddleFingerPitch2Node}" apiName="${SimApi}"/>
+    <xacro:simple_passive_transmission jointName="${MiddleFingerPitch3JointName}" nodeName="${MiddleFingerPitch3Node}" apiName="${SimApi}"/>
+  </xacro:macro>
 </robot>

File: model/robots/common/xacro/pinky_finger/pinky_finger.xacro (robot description, xacro)
@@ -6,4 +6,5 @@
   <xacro:include filename="$(find val_description)/model/robots/common/xacro/pinky_finger/joint_limits.xacro"/>
   <xacro:include filename="$(find val_description)/model/robots/common/xacro/pinky_finger/frame_parameters.xacro"/>
+  <xacro:include filename="$(find val_description)/model/robots/common/xacro/pinky_finger/mechanical_info.xacro"/>
   <xacro:include filename="$(find val_description)/model/robots/common/xacro/pinky_finger/mass_parameters.xacro"/>
   <xacro:macro name="make_pinky_finger" params="prefix reflect pinky_finger_root_link">
@@ -32,9 +33,9 @@
                     visual_mesh="${mesh_root}/fingers/pinkyj3_${prefix}.dae"
                     collision_mesh="${mesh_root}/fingers/pinkyj3_${prefix}.dae"/>
-    <xacro:revolute_joint jointName="${PinkyPitch1JointName}"
+    <xacro:revolute_joint_ex jointName="${PinkyPitch1JointName}"
                           parent="${PinkyPitch1ParentLinkName}" child="${PinkyPitch1LinkName}"
                           origin_xyz="${PinkyPitch1FrameOrigin_X} ${PinkyPitch1FrameOrigin_Y} ${PinkyPitch1FrameOrigin_Z}"
                           origin_rpy="${PinkyPitch1FrameOrientation_Roll} ${PinkyPitch1FrameOrientation_Pitch} ${PinkyPitch1FrameOrientation_Yaw}"
-                          axis="${PinkyFingerPitch1RotationAxis}">
+                          axis="${PinkyFingerPitch1RotationAxis}" damping="0.5" friction="0.5">
         <xacro:if value="${(reflect+1)/2}">
           <limit effort="${PinkyFingerPitch1TorqueLimit}" lower="${-reflect * PinkyFingerPitch1PositionLimit_Upper}" upper="${-reflect * PinkyFingerPitch1PositionLimit_Lower}" velocity="${PinkyFingerPitch1VelocityLimit}"/>
@@ -43,10 +44,11 @@
           <limit effort="${PinkyFingerPitch1TorqueLimit}" lower="${PinkyFingerPitch1PositionLimit_Lower}" upper="${PinkyFingerPitch1PositionLimit_Upper}" velocity="${PinkyFingerPitch1VelocityLimit}"/>
         </xacro:if>
-    </xacro:revolute_joint>
-    <xacro:revolute_joint jointName="${PinkyPitch2JointName}"
+        <controller_gains Kp="${PinkyPitch1Kp}" Kd="${PinkyPitch1Kd}" Ki="${PinkyPitch1Ki}"/>
+    </xacro:revolute_joint_ex>
+    <xacro:revolute_joint_ex jointName="${PinkyPitch2JointName}"
                           parent="${PinkyPitch1LinkName}" child="${PinkyPitch2LinkName}"
                           origin_xyz="${PinkyPitch2FrameOrigin_X} ${PinkyPitch2FrameOrigin_Y} ${PinkyPitch2FrameOrigin_Z}"
                           origin_rpy="${PinkyPitch2FrameOrientation_Roll} ${PinkyPitch2FrameOrientation_Pitch} ${PinkyPitch2FrameOrientation_Yaw}"
-                          axis="${PinkyFingerPitch2RotationAxis}">
+                          axis="${PinkyFingerPitch2RotationAxis}" damping="0.5" friction="0.5">
         <xacro:if value="${(reflect+1)/2}">
           <limit effort="${PinkyFingerPitch2TorqueLimit}" lower="${-reflect * PinkyFingerPitch2PositionLimit_Upper}" upper="${-reflect * PinkyFingerPitch2PositionLimit_Lower}" velocity="${PinkyFingerPitch2VelocityLimit}"/>
@@ -55,10 +57,11 @@
           <limit effort="${PinkyFingerPitch2TorqueLimit}" lower="${PinkyFingerPitch2PositionLimit_Lower}" upper="${PinkyFingerPitch2PositionLimit_Upper}" velocity="${PinkyFingerPitch2VelocityLimit}"/>
         </xacro:if>
-    </xacro:revolute_joint>
-    <xacro:revolute_joint jointName="${PinkyPitch3JointName}"
+        <controller_gains Kp="${PinkyPitch1Kp}" Kd="${PinkyPitch1Kd}" Ki="${PinkyPitch1Ki}"/>
+    </xacro:revolute_joint_ex>
+    <xacro:revolute_joint_ex jointName="${PinkyPitch3JointName}"
                           parent="${PinkyPitch2LinkName}" child="${PinkyPitch3LinkName}"
                           origin_xyz="${PinkyPitch3FrameOrigin_X} ${PinkyPitch3FrameOrigin_Y} ${PinkyPitch3FrameOrigin_Z}"
                           origin_rpy="${PinkyPitch3FrameOrientation_Roll} ${PinkyPitch3FrameOrientation_Pitch} ${PinkyPitch3FrameOrientation_Yaw}"
-                          axis="${PinkyFingerPitch3RotationAxis}">
+                          axis="${PinkyFingerPitch3RotationAxis}" damping="0.5" friction="0.5">
         <xacro:if value="${(reflect+1)/2}">
           <limit effort="${PinkyFingerPitch3TorqueLimit}" lower="${-reflect * PinkyFingerPitch3PositionLimit_Upper}" upper="${-reflect * PinkyFingerPitch3PositionLimit_Lower}" velocity="${PinkyFingerPitch3VelocityLimit}"/>
@@ -67,5 +70,6 @@
           <limit effort="${PinkyFingerPitch3TorqueLimit}" lower="${PinkyFingerPitch3PositionLimit_Lower}" upper="${PinkyFingerPitch3PositionLimit_Upper}" velocity="${PinkyFingerPitch3VelocityLimit}"/>
         </xacro:if>
-    </xacro:revolute_joint>
+        <controller_gains Kp="${PinkyPitch1Kp}" Kd="${PinkyPitch1Kd}" Ki="${PinkyPitch1Ki}"/>
+    </xacro:revolute_joint_ex>
   </xacro:macro>
   <xacro:macro name="pinky_finger_transmissions_hw" params="prefix reflect">
@@ -74,3 +78,8 @@
     <xacro:simple_forearm_position_transmission jointName="${PinkyPitch3JointName}" actuatorName="${prefix}PinkyPitch3Actuator" nodeName="${PinkyPitch3Node}" actuatorApi="${PinkyApi}" reflect="${reflect}"/>
   </xacro:macro>
+  <xacro:macro name="pinky_transmissions_sim" params="prefix">
+    <xacro:simple_transmission_with_child_joints jointName="${PinkyPitch1JointName}" actuatorName="${prefix}PinkyPitch1Actuator" nodeName="${PinkyPitch1Node}" actuatorApi="${SimApi}" child1JointName="${PinkyPitch2JointName}" child1Ratio="${Pulley2Ratio}" child2JointName="${PinkyPitch3JointName}" child2Ratio="${Pulley3Ratio}"/>
+    <xacro:simple_passive_transmission jointName="${PinkyPitch2JointName}" nodeName="${PinkyPitch2Node}" apiName="${SimApi}"/>
+    <xacro:simple_passive_transmission jointName="${PinkyPitch3JointName}" nodeName="${PinkyPitch3Node}" apiName="${SimApi}"/>
+  </xacro:macro>
 </robot>
