Commit message: Added sim transmissions for the rest of the fingers.

File: model/robots/common/xacro/thumb/thumb.xacro (robot description, xacro)
@@ -98,5 +98,5 @@
   <xacro:macro name="thumb_transmissions_sim" params="prefix">
     <xacro:simple_position_transmission jointName="${ThumbRollJointName}" actuatorName="${prefix}ThumbRollActuator" nodeName="${ThumbRollNode}" actuatorApi="${SimApi}"/>
-    <xacro:finger_transmission jointName="${ThumbPitch1JointName}" actuatorName="${prefix}ThumbPitch1Actuator" nodeName="${ThumbPitch1Node}" actuatorApi="${SimApi}" child1JointName="${ThumbPitch2JointName}" child1Ratio="${Pulley2Ratio}" child2JointName="${ThumbPitch3JointName}" child2Ratio="${Pulley3Ratio}"/>
+    <xacro:simple_transmission_with_child_joints jointName="${ThumbPitch1JointName}" actuatorName="${prefix}ThumbPitch1Actuator" nodeName="${ThumbPitch1Node}" actuatorApi="${SimApi}" child1JointName="${ThumbPitch2JointName}" child1Ratio="${Pulley2Ratio}" child2JointName="${ThumbPitch3JointName}" child2Ratio="${Pulley3Ratio}"/>
     <xacro:simple_passive_transmission jointName="${ThumbPitch2JointName}" nodeName="${ThumbPitch2Node}" apiName="${SimApi}"/>
     <xacro:simple_passive_transmission jointName="${ThumbPitch3JointName}" nodeName="${ThumbPitch3Node}" apiName="${SimApi}"/>

File: model/robots/forearm_sim.xacro (robot description, xacro)
@@ -5,4 +5,5 @@
       </plugin>
     </gazebo>
+    <schedule_topic_creator_file package="val_gazebo" relative_file_path="/configuration/valkyrie_sim_shm_topics.yaml"/>
     <xacro:property name="mesh_root" value="package://val_description/model/meshes"/>
     <xacro:include filename="$(find val_description)/common/xacro/api/valkyrie_sim_api.xacro"/>
@@ -37,8 +38,11 @@
     </link>
     <xacro:make_thumb prefix="left" reflect="1" thumb_root_link="leftPalm"/>
-<!--     <xacro:make_index_finger prefix="left" reflect="1" index_finger_root_link="leftPalm"/>
+    <xacro:make_index_finger prefix="left" reflect="1" index_finger_root_link="leftPalm"/>
     <xacro:make_middle_finger prefix="left" reflect="1" middle_finger_root_link="leftPalm"/>
-    <xacro:make_pinky_finger prefix="left" reflect="1" pinky_finger_root_link="leftPalm"/> -->
+    <xacro:make_pinky_finger prefix="left" reflect="1" pinky_finger_root_link="leftPalm"/>
     <xacro:thumb_transmissions_sim prefix="left"/>
+    <xacro:index_finger_transmissions_sim prefix="left"/>
+    <xacro:middle_finger_transmissions_sim prefix="left"/>
+    <xacro:pinky_transmissions_sim prefix="left"/>
     <xacro:add_sim_harness harnessed_link="leftPalm" />
 </robot>

Commit message: fixing joint smt node names

File: common/xacro/nodes/valkyrie_sim_nodes.xacro (robot description, xacro)
@@ -15,5 +15,5 @@
 	<xacro:property name="ElbowPitchNode" value="_arm/j4" />
 	<xacro:property name="ForearmYawNode" value="_arm/j5" />
-	<xacro:property name="WristRollActuatorNode" value="_arm/wrist/roll_actautor" />
+	<xacro:property name="WristRollActuatorNode" value="_arm/wrist/roll_actuator" />
 	<xacro:property name="WristPitchActuatorNode" value="_arm/wrist/pitch_actuator" />
 	<xacro:property name="WaistPitchActuatorNode" value="/trunk/pitch_actuator" /> <!--pitch-->

File: model/robots/common/xacro/arm/arm.xacro (robot description, xacro)
@@ -246,5 +246,5 @@
   <xacro:macro name="arm_transmissions_no_hands" params="prefix">
     <xacro:simple_transmission jointName="${prefix}${ShoulderPitchJointName}" actuatorName="${prefix}${ShoulderPitchActuatorName}" nodeName="/trunk/${prefix}_arm_j1" actuatorApi="${ShoulderPitchApi}"/>
-    <xacro:simple_transmission jointName="${prefix}${ShoulderRollJointName}" actuatorName="${prefix}${ShoulderRollActuatorName}" nodeName="${prefix}${ShoulderRollNode}" actuatorApi="${ShoulderRollApi}"/>
+    <xacro:simple_transmission jointName="${prefix}${ShoulderRollJointName}" actuatorName="${prefix}${ShoulderRollActuatorName}" nodeName="/${prefix}${ShoulderRollNode}" actuatorApi="${ShoulderRollApi}"/>
     <xacro:simple_transmission jointName="${prefix}${ShoulderYawJointName}" actuatorName="${prefix}${ShoulderYawActuatorName}" nodeName="/${prefix}${ShoulderYawNode}" actuatorApi="${ShoulderYawApi}"/>
     <xacro:simple_transmission jointName="${prefix}${ElbowPitchJointName}" actuatorName="${prefix}${ElbowPitchActuatorName}" nodeName="/${prefix}${ElbowPitchNode}" actuatorApi="${ElbowPitchApi}"/>
@@ -252,14 +252,14 @@
   <xacro:macro name="arm_transmissions_sim" params="prefix">
     <xacro:simple_transmission jointName="${prefix}${ShoulderPitchJointName}" actuatorName="${prefix}${ShoulderPitchActuatorName}" nodeName="/trunk/${prefix}_arm_j1" actuatorApi="${SimApi}"/>
-    <xacro:simple_transmission jointName="${prefix}${ShoulderRollJointName}" actuatorName="${prefix}${ShoulderRollActuatorName}" nodeName="${prefix}${ShoulderRollNode}" actuatorApi="${SimApi}"/>
+    <xacro:simple_transmission jointName="${prefix}${ShoulderRollJointName}" actuatorName="${prefix}${ShoulderRollActuatorName}" nodeName="/${prefix}${ShoulderRollNode}" actuatorApi="${SimApi}"/>
     <xacro:simple_transmission jointName="${prefix}${ShoulderYawJointName}" actuatorName="${prefix}${ShoulderYawActuatorName}" nodeName="/${prefix}${ShoulderYawNode}" actuatorApi="${SimApi}"/>
     <xacro:simple_transmission jointName="${prefix}${ElbowPitchJointName}" actuatorName="${prefix}${ElbowPitchActuatorName}" nodeName="/${prefix}${ElbowPitchNode}" actuatorApi="${SimApi}"/>
     <xacro:simple_position_transmission jointName="${prefix}${ForearmYawActuatorName}" actuatorName="${prefix}${ForearmYawActuatorName}" nodeName="/${prefix}${ForearmYawNode}" actuatorApi="${SimApi}"/>
-    <xacro:simple_position_transmission jointName="${prefix}${WristRollJointName}" actuatorName="${prefix}${WristRollActuatorSimName}" nodeName="${WristRollActuatorNode}" actuatorApi="${SimApi}"/>
-    <xacro:simple_position_transmission jointName="${prefix}${WristPitchJointName}" actuatorName="${prefix}${WristPitchActuatorSimName}" nodeName="${WristPitchActuatorNode}" actuatorApi="${SimApi}"/>
+    <xacro:simple_position_transmission jointName="${prefix}${WristRollJointName}" actuatorName="${prefix}${WristRollActuatorSimName}" nodeName="/${prefix}${WristRollActuatorNode}" actuatorApi="${SimApi}"/>
+    <xacro:simple_position_transmission jointName="${prefix}${WristPitchJointName}" actuatorName="${prefix}${WristPitchActuatorSimName}" nodeName="/${prefix}${WristPitchActuatorNode}" actuatorApi="${SimApi}"/>
   </xacro:macro>
   <xacro:macro name="arm_transmissions_sim_no_hands" params="prefix">
     <xacro:simple_transmission jointName="${prefix}${ShoulderPitchJointName}" actuatorName="${prefix}${ShoulderPitchActuatorName}" nodeName="/trunk/${prefix}_arm_j1" actuatorApi="${SimApi}"/>
-    <xacro:simple_transmission jointName="${prefix}${ShoulderRollJointName}" actuatorName="${prefix}${ShoulderRollActuatorName}" nodeName="${prefix}${ShoulderRollNode}" actuatorApi="${SimApi}"/>
+    <xacro:simple_transmission jointName="${prefix}${ShoulderRollJointName}" actuatorName="${prefix}${ShoulderRollActuatorName}" nodeName="/${prefix}${ShoulderRollNode}" actuatorApi="${SimApi}"/>
     <xacro:simple_transmission jointName="${prefix}${ShoulderYawJointName}" actuatorName="${prefix}${ShoulderYawActuatorName}" nodeName="/${prefix}${ShoulderYawNode}" actuatorApi="${SimApi}"/>
     <xacro:simple_transmission jointName="${prefix}${ElbowPitchJointName}" actuatorName="${prefix}${ElbowPitchActuatorName}" nodeName="/${prefix}${ElbowPitchNode}" actuatorApi="${SimApi}"/>

File: model/robots/common/xacro/leg/leg.xacro (robot description, xacro)
@@ -153,5 +153,5 @@
     <xacro:simple_transmission jointName="${prefix}${HipYawJointName}" actuatorName="${prefix}${HipYawActuatorName}" nodeName="/pelvis/${prefix}_leg_j1" actuatorApi="${HipYawApi}"/>
     <xacro:simple_transmission jointName="${prefix}${HipRollJointName}" actuatorName="${prefix}${HipRollActuatorName}" nodeName="/${prefix}${HipRollNode}" actuatorApi="${HipRollApi}"/>
-    <xacro:simple_transmission jointName="${prefix}${HipRollJointName}" actuatorName="${prefix}${HipPitchActuatorName}" nodeName="/${prefix}${HipPitchNode}" actuatorApi="${HipPitchApi}"/>
+    <xacro:simple_transmission jointName="${prefix}${HipPitchJointName}" actuatorName="${prefix}${HipPitchActuatorName}" nodeName="/${prefix}${HipPitchNode}" actuatorApi="${HipPitchApi}"/>
     <xacro:simple_transmission jointName="${prefix}${KneePitchJointName}" actuatorName="${prefix}${KneePitchActuatorName}" nodeName="/${prefix}${KneePitchNode}" actuatorApi="${KneePitchApi}"/>
     <xacro:pushrod_transmission transmissionName="${prefix}AnkleTransmission" transmissionType="${AnkleTransmissionType}" joint1Name="${prefix}${AnklePitchJointName}" joint2Name="${prefix}${AnkleRollJointName}" joint1Role="pitch" joint2Role="roll" actuator1Name="${prefix}${AnkleRightActuatorName}" actuator2Name="${prefix}${AnkleLeftActuatorName}" actuator1Node="/${prefix}${AnkleRightActuatorNode}" actuator2Node="/${prefix}${AnkleLeftActuatorNode}" actuator1Api="${AnkleRightActuatorApi}" actuator2Api="${AnkleLeftActuatorApi}" actuator1Role="right" actuator2Role="left"/>
@@ -160,5 +160,5 @@
     <xacro:simple_transmission jointName="${prefix}${HipYawJointName}" actuatorName="${prefix}${HipYawActuatorName}" nodeName="/pelvis/${prefix}_leg_j1" actuatorApi="${SimApi}"/>
     <xacro:simple_transmission jointName="${prefix}${HipRollJointName}" actuatorName="${prefix}${HipRollActuatorName}" nodeName="/${prefix}${HipRollNode}" actuatorApi="${SimApi}"/>
-    <xacro:simple_transmission jointName="${prefix}${HipRollJointName}" actuatorName="${prefix}${HipPitchActuatorName}" nodeName="/${prefix}${HipPitchNode}" actuatorApi="${SimApi}"/>
+    <xacro:simple_transmission jointName="${prefix}${HipPitchJointName}" actuatorName="${prefix}${HipPitchActuatorName}" nodeName="/${prefix}${HipPitchNode}" actuatorApi="${SimApi}"/>
     <xacro:simple_transmission jointName="${prefix}${KneePitchJointName}" actuatorName="${prefix}${KneePitchActuatorName}" nodeName="/${prefix}${KneePitchNode}" actuatorApi="${SimApi}"/>
     <xacro:simple_transmission jointName="${prefix}${AnklePitchJointName}" actuatorName="${prefix}${AnklePitchActuatorSimName}" nodeName="/${prefix}${AnklePitchActuatorNode}" actuatorApi="${SimApi}"/>

File: model/robots/common/xacro/thumb/thumb.xacro (robot description, xacro)
@@ -95,5 +95,5 @@
   </xacro:macro>
   <xacro:macro name="thumb_transmissions_hw" params="prefix reflect">
-    <xacro:simple_position_transmission jointName="${prefix}${ThumbRollJointName}" actuatorName="${prefix}ThumbRollActuator" nodeName="${ThumbRollNode}" actuatorApi="${ThumbFingerRollApi}"/>
+    <xacro:simple_position_transmission jointName="${prefix}${ThumbRollJointName}" actuatorName="${prefix}ThumbRollActuator" nodeName="/${prefix}${ThumbRollNode}" actuatorApi="${ThumbFingerRollApi}"/>
     <xacro:simple_forearm_position_transmission jointName="${prefix}${ThumbPitch1JointName}" actuatorName="${prefix}ThumbPitch1Actuator" nodeName="/${prefix}${ThumbPitch1Node}" actuatorApi="${ThumbFingerProximalApi}" reflect="${reflect}"/>
     <xacro:simple_forearm_position_transmission jointName="${prefix}${ThumbPitch2JointName}" actuatorName="${prefix}ThumbPitch2Actuator" nodeName="/${prefix}${ThumbPitch2Node}" actuatorApi="${ThumbFingerMedialApi}" reflect="${reflect}"/>
@@ -101,5 +101,5 @@
   </xacro:macro>
   <xacro:macro name="thumb_transmissions_sim" params="prefix">
-    <xacro:simple_position_transmission jointName="${prefix}${ThumbRollJointName}" actuatorName="${prefix}ThumbRollActuator" nodeName="${ThumbRollNode}" actuatorApi="${SimApi}"/>
+    <xacro:simple_position_transmission jointName="${prefix}${ThumbRollJointName}" actuatorName="${prefix}ThumbRollActuator" nodeName="/${prefix}${ThumbRollNode}" actuatorApi="${SimApi}"/>
     <xacro:simple_transmission_with_two_child_joints jointName="${prefix}${ThumbPitch1JointName}" actuatorName="${prefix}ThumbPitch1Actuator" nodeName="/${prefix}${ThumbPitch1Node}" actuatorApi="${SimApi}" child1JointName="${prefix}${ThumbPitch2JointName}" child1Ratio="${Pulley2Ratio}" child2JointName="${prefix}${ThumbPitch3JointName}" child2Ratio="${Pulley3Ratio}"/>
     <xacro:simple_passive_transmission jointName="${prefix}${ThumbPitch2JointName}" nodeName="/${prefix}${ThumbPitch2Node}" apiName="${SimApi}"/>
