Commit message: adding some extra transmissions make simulation closer to hardware interface wise.

File: common/xacro/nodes/valkyrie_sim_nodes.xacro (robot description, xacro)
@@ -27,13 +27,18 @@
 	<xacro:property name="right_foot_ATI_node" value="/right_leg/ankle/roll_actuator" />
 	<xacro:property name="ThumbRollNode" value="_hand/thumb_roll"/>
+	<xacro:property name="ThumbProximalNode" value="_arm/hand/thumb_proximal"/>
+	<xacro:property name="ThumbDistalNode" value="_arm/hand/thumb_distal"/>
 	<xacro:property name="ThumbPitch1Node" value="_hand/thumb_pitch_1"/>
 	<xacro:property name="ThumbPitch2Node" value="_hand/thumb_pitch_2"/>
 	<xacro:property name="ThumbPitch3Node" value="_hand/thumb_pitch_3"/>
+	<xacro:property name="IndexFingerNode" value="_arm/hand/index"/>
 	<xacro:property name="IndexFingerPitch1Node" value="_hand/index_finger_pitch_1"/>
 	<xacro:property name="IndexFingerPitch2Node" value="_hand/index_finger_pitch_2"/>
 	<xacro:property name="IndexFingerPitch3Node" value="_hand/index_finger_pitch_3"/>
+	<xacro:property name="MiddleFingerNode" value="_arm/hand/middle"/>
 	<xacro:property name="MiddleFingerPitch1Node" value="_hand/middle_finger_pitch_1"/>
 	<xacro:property name="MiddleFingerPitch2Node" value="_hand/middle_finger_pitch_2"/>
 	<xacro:property name="MiddleFingerPitch3Node" value="_hand/middle_finger_pitch_3"/>
+	<xacro:property name="PinkyFingerNode" value="_arm/hand/pinky"/>
 	<xacro:property name="PinkyPitch1Node" value="_hand/pinky_pitch_1"/>
 	<xacro:property name="PinkyPitch2Node" value="_hand/pinky_pitch_2"/>

File: model/robots/common/xacro/generic_models.xacro (robot description, xacro)
@@ -267,5 +267,66 @@
     </transmission>
   </xacro:macro>
-  <xacro:macro name="simple_passive_transmission" params="jointName nodeName apiName">
+  <xacro:macro name="simple_position_transmission_with_three_child_joints" params="jointName actuatorName nodeName actuatorApi child1JointName child1Ratio child2JointName child2Ratio">
+    <transmission name="${jointName}Transmission">
+      <type>transmission_interface/SimpleTransmission</type>
+      <joint name="${jointName}">
+        <hardwareInterface>PositionJointInterface</hardwareInterface>
+        <child name="${child1JointName}" ratio="${child1Ratio}"/>
+        <child name="${child2JointName}" ratio="${child2Ratio}"/>
+      </joint>
+      <actuator name="${actuatorName}">
+        <node name="${nodeName}"/>
+        <mechanicalReduction>1</mechanicalReduction>
+        <api name="${actuatorApi}" />
+      </actuator>
+    </transmission>
+  </xacro:macro>
+  <xacro:macro name="simple_effort_transmission_with_three_child_joints" params="jointName actuatorName nodeName actuatorApi child1JointName child1Ratio child2JointName child2Ratio child3JointName child3Ratio">
+    <transmission name="${jointName}Transmission">
+      <type>transmission_interface/SimpleTransmission</type>
+      <joint name="${jointName}">
+        <hardwareInterface>EffortJointInterface</hardwareInterface>
+        <child name="${child1JointName}" ratio="${child1Ratio}"/>
+        <child name="${child2JointName}" ratio="${child2Ratio}"/>
+        <child name="${child3JointName}" ratio="${child3Ratio}"/>
+      </joint>
+      <actuator name="${actuatorName}">
+        <node name="${nodeName}"/>
+        <mechanicalReduction>1</mechanicalReduction>
+        <api name="${actuatorApi}" />
+      </actuator>
+    </transmission>
+  </xacro:macro>
+  <xacro:macro name="simple_effort_transmission_two_actuator" params="jointName actuatorName nodeName actuatorApi childActuator">
+    <transmission name="${jointName}Transmission">
+      <type>transmission_interface/SimpleTransmission</type>
+      <joint name="${jointName}">
+        <hardwareInterface>EffortJointInterface</hardwareInterface>
+      </joint>
+      <actuator name="${actuatorName}">
+        <node name="${nodeName}"/>
+        <mechanicalReduction>1</mechanicalReduction>
+        <api name="${actuatorApi}" />
+        <child name="${childActuator}" />
+      </actuator>
+    </transmission>
+  </xacro:macro>
+  <xacro:macro name="simple_effort_transmission_two_actuator_three_joint" params="jointName actuatorName nodeName actuatorApi child1JointName child1Ratio child2JointName child2Ratio">
+    <transmission name="${jointName}Transmission">
+      <type>transmission_interface/SimpleTransmission</type>
+      <joint name="${jointName}">
+        <hardwareInterface>EffortJointInterface</hardwareInterface>
+        <child name="${child1JointName}" ratio="${child1Ratio}"/>
+        <child name="${child2JointName}" ratio="${child2Ratio}"/>
+      </joint>
+      <actuator name="${actuatorName}">
+        <node name="${nodeName}"/>
+        <mechanicalReduction>1</mechanicalReduction>
+        <api name="${actuatorApi}" />
+        <child name="${childActuator}" />
+      </actuator>
+    </transmission>
+  </xacro:macro>
+  <xacro:macro name="simple_passive_transmission" params="jointName nodeName apiName reflect">
     <transmission name="${jointName}PassiveTransmission">
       <type>transmission_interface/SimpleTransmission</type>
@@ -275,5 +336,5 @@
       <actuator name="${jointName}PassiveActuator">
         <node name="${nodeName}"/>
-        <mechanicalReduction>1</mechanicalReduction>
+        <mechanicalReduction>${reflect}</mechanicalReduction>
         <api name="${apiName}" />
       </actuator>

File: model/robots/common/xacro/index_finger/index_finger.xacro (robot description, xacro)
@@ -84,7 +84,8 @@
   </xacro:macro>
   <xacro:macro name="index_finger_transmissions_sim" params="prefix">
-    <xacro:simple_transmission_with_two_child_joints jointName="${prefix}${IndexFingerPitch1JointName}" actuatorName="${prefix}IndexFingerPitch1Actuator" nodeName="/${prefix}${IndexFingerPitch1Node}" actuatorApi="${SimApi}" child1JointName="${prefix}${IndexFingerPitch2JointName}" child1Ratio="${Pulley2Ratio}" child2JointName="${prefix}${IndexFingerPitch3JointName}" child2Ratio="${Pulley3Ratio}"/>
-    <xacro:simple_passive_transmission jointName="${prefix}${IndexFingerPitch2JointName}" nodeName="/${prefix}${IndexFingerPitch2Node}" apiName="${SimApi}"/>
-    <xacro:simple_passive_transmission jointName="${prefix}${IndexFingerPitch3JointName}" nodeName="/${prefix}${IndexFingerPitch3Node}" apiName="${SimApi}"/>
+    <xacro:simple_effort_transmission_with_three_child_joints jointName="${prefix}${IndexFingerPitch1ActuatorName}" actuatorName="${prefix}${IndexFingerPitch1ActuatorName}" nodeName="/${prefix}${IndexFingerNode}" actuatorApi="${SimApi}" child1JointName="${prefix}${IndexFingerPitch1JointName}" child1Ratio="${Pulley1Ratio}" child2JointName="${prefix}${IndexFingerPitch2JointName}" child2Ratio="${Pulley2Ratio}" child3JointName="${prefix}${IndexFingerPitch3JointName}" child3Ratio="${Pulley3Ratio}"/>
+    <xacro:simple_passive_transmission jointName="${prefix}${IndexFingerPitch1JointName}" nodeName="/${prefix}${IndexFingerPitch1Node}" apiName="${SimApi}" reflect="1"/>
+    <xacro:simple_passive_transmission jointName="${prefix}${IndexFingerPitch2JointName}" nodeName="/${prefix}${IndexFingerPitch2Node}" apiName="${SimApi}" reflect="1"/>
+    <xacro:simple_passive_transmission jointName="${prefix}${IndexFingerPitch3JointName}" nodeName="/${prefix}${IndexFingerPitch3Node}" apiName="${SimApi}" reflect="1"/>
   </xacro:macro>
 </robot>

File: model/robots/common/xacro/index_finger/mechanical_info.xacro (robot description, xacro)
@@ -1,8 +1,10 @@
 <?xml version="1.0" ?>
 <robot xmlns:xacro="http://www.ros.org/wiki/xacro" name="valkyrie_index_finger_mechanical_info">
+  <!-- Motor Pulley diameter = 0.0152m (approximately)-->
   <!-- Pulley-1 diameter = 0.01707m -->
   <!-- Pulley-2 diameter = 0.0127m -->
   <!-- Pulley-3 diameter = 0.01016 -->
-  <xacro:property name="Pulley2Ratio" value="1.344" />
-  <xacro:property name="Pulley3Ratio" value="1.68" />
+  <xacro:property name="Pulley1Ratio" value="1.123" />
+  <xacro:property name="Pulley2Ratio" value="0.835" />
+  <xacro:property name="Pulley3Ratio" value="0.668" />
 </robot>

File: model/robots/common/xacro/middle_finger/mechanical_info.xacro (robot description, xacro)
@@ -1,8 +1,10 @@
 <?xml version="1.0" ?>
 <robot xmlns:xacro="http://www.ros.org/wiki/xacro" name="valkyrie_middle_finger_mechanical_info">
+  <!-- Motor Pulley diameter = 0.0152m (approximately)-->
   <!-- Pulley-1 diameter = 0.01707m -->
   <!-- Pulley-2 diameter = 0.0127m -->
   <!-- Pulley-3 diameter = 0.01016 -->
-  <xacro:property name="Pulley2Ratio" value="1.344" />
-  <xacro:property name="Pulley3Ratio" value="1.68" />
+  <xacro:property name="Pulley1Ratio" value="1.123" />
+  <xacro:property name="Pulley2Ratio" value="0.835" />
+  <xacro:property name="Pulley3Ratio" value="0.668" />
 </robot>

File: model/robots/common/xacro/middle_finger/middle_finger.xacro (robot description, xacro)
@@ -84,7 +84,8 @@
   </xacro:macro>
   <xacro:macro name="middle_finger_transmissions_sim" params="prefix">
-    <xacro:simple_transmission_with_two_child_joints jointName="${prefix}${MiddleFingerPitch1JointName}" actuatorName="${prefix}MiddleFingerPitch1Actuator" nodeName="/${prefix}${MiddleFingerPitch1Node}" actuatorApi="${SimApi}" child1JointName="${prefix}${MiddleFingerPitch2JointName}" child1Ratio="${Pulley2Ratio}" child2JointName="${prefix}${MiddleFingerPitch3JointName}" child2Ratio="${Pulley3Ratio}"/>
-    <xacro:simple_passive_transmission jointName="${prefix}${MiddleFingerPitch2JointName}" nodeName="/${prefix}${MiddleFingerPitch2Node}" apiName="${SimApi}"/>
-    <xacro:simple_passive_transmission jointName="${prefix}${MiddleFingerPitch3JointName}" nodeName="/${prefix}${MiddleFingerPitch3Node}" apiName="${SimApi}"/>
+    <xacro:simple_effort_transmission_with_three_child_joints jointName="${prefix}${MiddleFingerPitch1ActuatorName}" actuatorName="${prefix}${MiddleFingerPitch1ActuatorName}" nodeName="/${prefix}${MiddleFingerNode}" actuatorApi="${SimApi}" child1JointName="${prefix}${MiddleFingerPitch1JointName}" child1Ratio="${Pulley1Ratio}" child2JointName="${prefix}${MiddleFingerPitch2JointName}" child2Ratio="${Pulley2Ratio}" child3JointName="${prefix}${MiddleFingerPitch3JointName}" child3Ratio="${Pulley3Ratio}"/>
+    <xacro:simple_passive_transmission jointName="${prefix}${MiddleFingerPitch1JointName}" nodeName="/${prefix}${MiddleFingerPitch1Node}" apiName="${SimApi}" reflect="1"/>
+    <xacro:simple_passive_transmission jointName="${prefix}${MiddleFingerPitch2JointName}" nodeName="/${prefix}${MiddleFingerPitch2Node}" apiName="${SimApi}" reflect="1"/>
+    <xacro:simple_passive_transmission jointName="${prefix}${MiddleFingerPitch3JointName}" nodeName="/${prefix}${MiddleFingerPitch3Node}" apiName="${SimApi}" reflect="1"/>
   </xacro:macro>
 </robot>

File: model/robots/common/xacro/pinky_finger/mechanical_info.xacro (robot description, xacro)
@@ -1,8 +1,10 @@
 <?xml version="1.0" ?>
 <robot xmlns:xacro="http://www.ros.org/wiki/xacro" name="valkyrie_pinky_mechanical_info">
+  <!-- Motor Pulley diameter = 0.0152m (approximately)-->
   <!-- Pulley-1 diameter = 0.01707m -->
   <!-- Pulley-2 diameter = 0.0127m -->
   <!-- Pulley-3 diameter = 0.01016 -->
-  <xacro:property name="Pulley2Ratio" value="1.344" />
-  <xacro:property name="Pulley3Ratio" value="1.68" />
+  <xacro:property name="Pulley1Ratio" value="1.123" />
+  <xacro:property name="Pulley2Ratio" value="0.835" />
+  <xacro:property name="Pulley3Ratio" value="0.668" />
 </robot>

File: model/robots/common/xacro/pinky_finger/pinky_finger.xacro (robot description, xacro)
@@ -84,7 +84,8 @@
   </xacro:macro>
   <xacro:macro name="pinky_transmissions_sim" params="prefix">
-    <xacro:simple_transmission_with_two_child_joints jointName="${prefix}${PinkyPitch1JointName}" actuatorName="${prefix}PinkyPitch1Actuator" nodeName="/${prefix}${PinkyPitch1Node}" actuatorApi="${SimApi}" child1JointName="${prefix}${PinkyPitch2JointName}" child1Ratio="${Pulley2Ratio}" child2JointName="${prefix}${PinkyPitch3JointName}" child2Ratio="${Pulley3Ratio}"/>
-    <xacro:simple_passive_transmission jointName="${prefix}${PinkyPitch2JointName}" nodeName="/${prefix}${PinkyPitch2Node}" apiName="${SimApi}"/>
-    <xacro:simple_passive_transmission jointName="${prefix}${PinkyPitch3JointName}" nodeName="/${prefix}${PinkyPitch3Node}" apiName="${SimApi}"/>
+    <xacro:simple_effort_transmission_with_three_child_joints jointName="${prefix}${PinkyPitch1ActuatorName}" actuatorName="${prefix}${PinkyPitch1ActuatorName}" nodeName="/${prefix}${PinkyFingerNode}" actuatorApi="${SimApi}" child1JointName="${prefix}${PinkyPitch1JointName}" child1Ratio="${Pulley1Ratio}" child2JointName="${prefix}${PinkyPitch2JointName}" child2Ratio="${Pulley2Ratio}" child3JointName="${prefix}${PinkyPitch3JointName}" child3Ratio="${Pulley3Ratio}"/>
+    <xacro:simple_passive_transmission jointName="${prefix}${PinkyPitch1JointName}" nodeName="/${prefix}${PinkyPitch1Node}" apiName="${SimApi}" reflect="1"/>
+    <xacro:simple_passive_transmission jointName="${prefix}${PinkyPitch2JointName}" nodeName="/${prefix}${PinkyPitch2Node}" apiName="${SimApi}" reflect="1"/>
+    <xacro:simple_passive_transmission jointName="${prefix}${PinkyPitch3JointName}" nodeName="/${prefix}${PinkyPitch3Node}" apiName="${SimApi}" reflect="1"/>
   </xacro:macro>
 </robot>

File: model/robots/common/xacro/thumb/mechanical_info.xacro (robot description, xacro)
@@ -4,5 +4,6 @@
   <!-- Pulley-2 diameter = 0.0127m -->
   <!-- Pulley-3 diameter = 0.01016 -->
-  <xacro:property name="Pulley2Ratio" value="1.344" />
-  <xacro:property name="Pulley3Ratio" value="1.68" />
+  <xacro:property name="Pulley1Ratio" value="1.123" />
+  <xacro:property name="Pulley2Ratio" value="0.835" />
+  <xacro:property name="Pulley3Ratio" value="0.668" />
 </robot>

File: model/robots/common/xacro/thumb/thumb.xacro (robot description, xacro)
@@ -104,7 +104,8 @@
   <xacro:macro name="thumb_transmissions_sim" params="prefix">
     <xacro:simple_position_transmission jointName="${prefix}${ThumbRollJointName}" actuatorName="${prefix}ThumbRollActuator" nodeName="/${prefix}${ThumbRollNode}" actuatorApi="${SimApi}"/>
-    <xacro:simple_transmission_with_two_child_joints jointName="${prefix}${ThumbPitch1JointName}" actuatorName="${prefix}ThumbPitch1Actuator" nodeName="/${prefix}${ThumbPitch1Node}" actuatorApi="${SimApi}" child1JointName="${prefix}${ThumbPitch2JointName}" child1Ratio="${Pulley2Ratio}" child2JointName="${prefix}${ThumbPitch3JointName}" child2Ratio="${Pulley3Ratio}"/>
-    <xacro:simple_passive_transmission jointName="${prefix}${ThumbPitch2JointName}" nodeName="/${prefix}${ThumbPitch2Node}" apiName="${SimApi}"/>
-    <xacro:simple_passive_transmission jointName="${prefix}${ThumbPitch3JointName}" nodeName="/${prefix}${ThumbPitch3Node}" apiName="${SimApi}"/>
+    <xacro:simple_effort_transmission_with_three_child_joints jointName="${prefix}${ThumbPitch2ActuatorName}" actuatorName="${prefix}${ThumbPitch2ActuatorName}" nodeName="/${prefix}${ThumbDistalNode}" actuatorApi="${SimApi}" child1JointName="${prefix}${ThumbPitch1JointName}" child1Ratio="${Pulley1Ratio}" child2JointName="${prefix}${ThumbPitch2JointName}" child2Ratio="${Pulley2Ratio}" child3JointName="${prefix}${ThumbPitch3JointName}" child3Ratio="${Pulley3Ratio}"/>
+    <xacro:simple_passive_transmission jointName="${prefix}${ThumbPitch1JointName}" nodeName="/${prefix}${ThumbPitch2Node}" apiName="${SimApi}" reflect="1"/>
+    <xacro:simple_passive_transmission jointName="${prefix}${ThumbPitch2JointName}" nodeName="/${prefix}${ThumbPitch2Node}" apiName="${SimApi}" reflect="1"/>
+    <xacro:simple_passive_transmission jointName="${prefix}${ThumbPitch3JointName}" nodeName="/${prefix}${ThumbPitch3Node}" apiName="${SimApi}" reflect="1"/>
   </xacro:macro>
 </robot>

Commit message: updating code to add virtual thumb roll motor

File: common/xacro/nodes/valkyrie_sim_nodes.xacro (robot description, xacro)
@@ -26,7 +26,8 @@
 	<xacro:property name="left_foot_ATI_node" value="/left_leg/ankle/roll_actuator" />
 	<xacro:property name="right_foot_ATI_node" value="/right_leg/ankle/roll_actuator" />
-	<xacro:property name="ThumbRollNode" value="_hand/thumb_roll"/>
+	<xacro:property name="ThumbRollNode" value="_arm/hand/thumb_roll"/>
 	<xacro:property name="ThumbProximalNode" value="_arm/hand/thumb_proximal"/>
 	<xacro:property name="ThumbDistalNode" value="_arm/hand/thumb_distal"/>
+	<xacro:property name="ThumbRollSenseNode" value="_hand/thumb_roll"/>
 	<xacro:property name="ThumbPitch1Node" value="_hand/thumb_pitch_1"/>
 	<xacro:property name="ThumbPitch2Node" value="_hand/thumb_pitch_2"/>

File: model/robots/common/xacro/generic_models.xacro (robot description, xacro)
@@ -252,4 +252,18 @@
     </transmission>
   </xacro:macro>
+  <xacro:macro name="simple_effort_transmission_with_one_child_joint" params="jointName actuatorName nodeName actuatorApi child1JointName child1Ratio">
+    <transmission name="${jointName}Transmission">
+      <type>transmission_interface/SimpleTransmission</type>
+      <joint name="${jointName}">
+        <hardwareInterface>EffortJointInterface</hardwareInterface>
+        <child name="${child1JointName}" ratio="${child1Ratio}"/>
+      </joint>
+      <actuator name="${actuatorName}">
+        <node name="${nodeName}"/>
+        <mechanicalReduction>1</mechanicalReduction>
+        <api name="${actuatorApi}" />
+      </actuator>
+    </transmission>
+  </xacro:macro>
   <xacro:macro name="simple_transmission_with_two_child_joints" params="jointName actuatorName nodeName actuatorApi child1JointName child1Ratio child2JointName child2Ratio">
     <transmission name="${jointName}Transmission">

File: model/robots/common/xacro/thumb/thumb.xacro (robot description, xacro)
@@ -103,6 +103,7 @@
   </xacro:macro>
   <xacro:macro name="thumb_transmissions_sim" params="prefix">
-    <xacro:simple_position_transmission jointName="${prefix}${ThumbRollJointName}" actuatorName="${prefix}ThumbRollActuator" nodeName="/${prefix}${ThumbRollNode}" actuatorApi="${SimApi}"/>
+    <xacro:simple_effort_transmission_with_one_child_joint jointName="${prefix}${ThumbRollActuatorName}" actuatorName="${prefix}${ThumbRollActuatorName}" nodeName="/${prefix}${ThumbRollNode}" actuatorApi="${SimApi}" child1JointName="${prefix}${ThumbRollJointName}" child1Ratio="1"/>
     <xacro:simple_effort_transmission_with_three_child_joints jointName="${prefix}${ThumbPitch2ActuatorName}" actuatorName="${prefix}${ThumbPitch2ActuatorName}" nodeName="/${prefix}${ThumbDistalNode}" actuatorApi="${SimApi}" child1JointName="${prefix}${ThumbPitch1JointName}" child1Ratio="${Pulley1Ratio}" child2JointName="${prefix}${ThumbPitch2JointName}" child2Ratio="${Pulley2Ratio}" child3JointName="${prefix}${ThumbPitch3JointName}" child3Ratio="${Pulley3Ratio}"/>
+    <xacro:simple_passive_transmission jointName="${prefix}${ThumbRollJointName}" nodeName="/${prefix}${ThumbRollSenseNode}" apiName="${SimApi}" reflect="1"/>
     <xacro:simple_passive_transmission jointName="${prefix}${ThumbPitch1JointName}" nodeName="/${prefix}${ThumbPitch2Node}" apiName="${SimApi}" reflect="1"/>
     <xacro:simple_passive_transmission jointName="${prefix}${ThumbPitch2JointName}" nodeName="/${prefix}${ThumbPitch2Node}" apiName="${SimApi}" reflect="1"/>
