Commit message: updating urdf for new forearm description

File: common/xacro/actuator_names/valkyrie_actuator_names.xacro (robot description, xacro)
@@ -24,4 +24,6 @@
 	<xacro:property name="WristBottomActuatorName" value="${prefix}WristBottomActuator"/>
 	<xacro:property name="WristTopActuatorName" value="${prefix}WristTopActuator"/>
+	<xacro:property name="WristRightActuatorName" value="${prefix}WristRightActuator"/>
+	<xacro:property name="WristLeftActuatorName" value="${prefix}WristLeftActuator"/>
 	<xacro:property name="WristPitchActuatorSimName" value="${prefix}WristPitchActuator"/>
 	<xacro:property name="WristRollActuatorSimName" value="${prefix}WristRollActuator"/>

File: common/xacro/api/forearm_api.xacro (robot description, xacro)
@@ -1,9 +1,11 @@
  <robot xmlns:xacro="http://ros.org/wiki/xacro" name="forearm_api">
     <xacro:property name="ForearmYawApi" value="robot_hardware_interface/TurbodriverAPI" />
-    <xacro:property name="ThumbFingerApi" value="midas_finger_interface/MidasFingerAPI" />
     <xacro:property name="IndexFingerApi" value="robot_hardware_interface/TurbodriverAPI"/>
-    <xacro:property name="MiddleFingerApi" value="midas_finger_interface/MidasFingerAPI"/>
-    <xacro:property name="PinkyApi" value="midas_finger_interface/MidasFingerAPI"/>
-    <xacro:property name="Athena1Api" value="athena_forearm_interface/AthenaForearmAPI" />
-    <xacro:property name="Athena2Api" value="athena_finger_interface/AthenaFingerAPI" />
+    <xacro:property name="MiddleFingerApi" value="robot_hardware_interface/TurbodriverAPI"/>
+    <xacro:property name="PinkyFingerApi" value="robot_hardware_interface/TurbodriverAPI"/>
+    <xacro:property name="ThumbRollFingerApi" value="robot_hardware_interface/TurbodriverAPI"/>
+    <xacro:property name="ThumbProximalFingerApi" value="robot_hardware_interface/TurbodriverAPI"/>
+    <xacro:property name="ThumbDistalFingerApi" value="robot_hardware_interface/TurbodriverAPI"/>
+    <xacro:property name="WristRightActuatorApi" value="robot_hardware_interface/TurbodriverAPI_linear_futek"/>
+    <xacro:property name="WristLeftActuatorApi" value="robot_hardware_interface/TurbodriverAPI_linear_futek"/>
 </robot>

File: common/xacro/nodes/valkyrie_nodes.xacro (robot description, xacro)
@@ -13,4 +13,6 @@
 	<xacro:property name="WristTopActuatorNode" value="/${prefix}_arm/wrist/top_actautor" />
 	<xacro:property name="WristBottomActuatorNode" value="/${prefix}_arm/wrist/bottom_actuator" />
+	<xacro:property name="WristLeftActuatorNode" value="/${prefix}_arm/wrist/left_actuator" />
+	<xacro:property name="WristRightActuatorNode" value="/${prefix}_arm/wrist/right_actuator" />
 	<xacro:property name="LowerNeckPitchNode" value="/neck/j1" />
 	<xacro:property name="NeckYawNode" value="/neck/j2" />
@@ -30,11 +32,15 @@
 	<xacro:property name="IndexFingerPitch2Node" value="/${prefix}_arm/forearm_sensors/index/pitch_2"/>
 	<xacro:property name="IndexFingerPitch3Node" value="/${prefix}_arm/forearm_sensors/index/pitch_3"/>
+	<xacro:property name="MiddleFingerNode" value="/${prefix}_arm/hand/middle"/>
 	<xacro:property name="MiddleFingerPitch1Node" value="/${prefix}_arm/forearm_sensors/middle/pitch_1"/>
 	<xacro:property name="MiddleFingerPitch2Node" value="/${prefix}_arm/forearm_sensors/middle/pitch_2"/>
 	<xacro:property name="MiddleFingerPitch3Node" value="/${prefix}_arm/forearm_sensors/middle/pitch_3"/>
+	<xacro:property name="PinkyFingerNode" value="/${prefix}_arm/hand/pinky"/>
 	<xacro:property name="PinkyPitch1Node" value="/${prefix}_arm/forearm_sensors/pinky/pitch_1"/>
 	<xacro:property name="PinkyPitch2Node" value="/${prefix}_arm/forearm_sensors/pinky/pitch_2"/>
 	<xacro:property name="PinkyPitch3Node" value="/${prefix}_arm/forearm_sensors/pinky/pitch_3"/>
-	<xacro:property name="ThumbRollNode" value="/${prefix}_arm/forearm_sensors/thumb/roll"/>
+	<xacro:property name="ThumbRollNode" value="/${prefix}_arm/hand/thumb_roll"/>
+	<xacro:property name="ThumbProximalNode" value="/${prefix}_arm/hand/thumb_proximal"/>
+	<xacro:property name="ThumbDistalNode" value="/${prefix}_arm/hand/thumb_distal"/>
 	<xacro:property name="ThumbPitch1Node" value="/${prefix}_arm/forearm_sensors/thumb/pitch_1"/>
 	<xacro:property name="ThumbPitch2Node" value="/${prefix}_arm/forearm_sensors/thumb/pitch_2"/>

File: model/robots/forearm_left.xacro (robot description, xacro)
@@ -8,6 +8,7 @@
     <!-- Arm include -->
     <xacro:include filename="$(find val_description)/model/robots/common/xacro/arm/arm_includes.xacro"/>
-    <xacro:property name="prefix" value="left"/>
-    <xacro:property name="reflect" value="1"/>
+    <xacro:property name="prefix" value="right"/>
+    <xacro:property name="reflect" value="-1"/>
+    <xacro:property name="WristTransmissionType" value="robot_transmission_interface/WristPushrodTransmission"/>
     <link name="world"/>
     <xacro:make_lower_arm prefix="${prefix}" reflect="${reflect}" lower_arm_root_link="world"/>
@@ -16,10 +17,11 @@
     <xacro:make_middle_finger prefix="${prefix}" reflect="${reflect}" middle_finger_root_link="${prefix}Palm"/>
     <xacro:make_pinky_finger prefix="${prefix}" reflect="${reflect}" pinky_finger_root_link="${prefix}Palm"/>
-    <xacro:simple_position_transmission jointName="${ForearmYawActuatorName}" actuatorName="${ForearmYawActuatorName}" nodeName="${ForearmYawNode}" actuatorApi="${ForearmYawApi}"/>
-    <xacro:index_finger_transmissions_hw prefix="${prefix}" reflect="${reflect}"/>
-    <xacro:middle_finger_transmissions_hw prefix="${prefix}" reflect="${reflect}"/>
-    <xacro:pinky_finger_transmissions_hw prefix="${prefix}" reflect="${reflect}"/>
-    <xacro:thumb_transmissions_hw prefix="${prefix}" reflect="${reflect}"/>
-    <xacro:athena1_transmission prefix="${prefix}" transmissionName="${prefix}ArmAthena1Transmission" actuatorApi="${Athena1Api}" nodeName="${Athena1Node}"/>
-    <xacro:athena2_transmission prefix="${prefix}" transmissionName="${prefix}ArmAthena2Transmission" actuatorApi="${Athena2Api}" nodeName="${Athena2Node}"/>
+    <xacro:simple_transmission jointName="${ForearmYawActuatorName}" actuatorName="${ForearmYawActuatorName}" nodeName="${ForearmYawNode}" actuatorApi="${ForearmYawApi}"/>
+    <xacro:simple_transmission jointName="${IndexFingerPitch1ActuatorName}" actuatorName="${IndexFingerPitch1ActuatorName}" nodeName="${IndexFingerNode}" actuatorApi="${IndexFingerApi}"/>
+    <xacro:simple_transmission jointName="${MiddleFingerPitch1ActuatorName}" actuatorName="${MiddleFingerPitch1ActuatorName}" nodeName="${MiddleFingerNode}" actuatorApi="${MiddleFingerApi}"/>
+    <xacro:simple_transmission jointName="${PinkyPitch1ActuatorName}" actuatorName="${PinkyPitch1ActuatorName}" nodeName="${PinkyFingerNode}" actuatorApi="${PinkyFingerApi}"/>
+    <xacro:simple_transmission jointName="${ThumbRollActuatorName}" actuatorName="${ThumbRollActuatorName}" nodeName="${ThumbRollNode}" actuatorApi="${ThumbRollFingerApi}"/>
+    <xacro:simple_transmission jointName="${ThumbPitch1ActuatorName}" actuatorName="${ThumbPitch1ActuatorName}" nodeName="${ThumbProximalNode}" actuatorApi="${ThumbProximalFingerApi}"/>
+    <xacro:simple_transmission jointName="${ThumbPitch2ActuatorName}" actuatorName="${ThumbPitch2ActuatorName}" nodeName="${ThumbDistalNode}" actuatorApi="${ThumbDistalFingerApi}"/>
+    <xacro:pushrod_transmission transmissionName="${prefix}WristTransmission" transmissionType="${WristTransmissionType}" joint1Name="${WristPitchJointName}" joint2Name="${WristRollJointName}" joint1Role="pitch" joint2Role="roll" actuator1Name="${WristRightActuatorName}" actuator2Name="${WristLeftActuatorName}" actuator1Node="${WristRightActuatorNode}" actuator2Node="${WristLeftActuatorNode}" actuator1Api="${WristRightActuatorApi}" actuator2Api="${WristLeftActuatorApi}" actuator1Role="bottom" actuator2Role="top"/>
 </robot>

File: model/robots/forearm_right.xacro (robot description, xacro)
@@ -10,4 +10,5 @@
     <xacro:property name="prefix" value="right"/>
     <xacro:property name="reflect" value="-1"/>
+    <xacro:property name="WristTransmissionType" value="robot_transmission_interface/WristPushrodTransmission"/>
     <link name="world"/>
     <xacro:make_lower_arm prefix="${prefix}" reflect="${reflect}" lower_arm_root_link="world"/>
@@ -16,5 +17,11 @@
     <xacro:make_middle_finger prefix="${prefix}" reflect="${reflect}" middle_finger_root_link="${prefix}Palm"/>
     <xacro:make_pinky_finger prefix="${prefix}" reflect="${reflect}" pinky_finger_root_link="${prefix}Palm"/>
-    <xacro:simple_position_transmission jointName="${ForearmYawActuatorName}" actuatorName="${ForearmYawActuatorName}" nodeName="${ForearmYawNode}" actuatorApi="${ForearmYawApi}"/>
-    <xacro:simple_position_transmission jointName="${IndexFingerPitch1ActuatorName}" actuatorName="${IndexFingerPitch1ActuatorName}" nodeName="${IndexFingerNode}" actuatorApi="${IndexFingerApi}"/>
+    <xacro:simple_transmission jointName="${ForearmYawActuatorName}" actuatorName="${ForearmYawActuatorName}" nodeName="${ForearmYawNode}" actuatorApi="${ForearmYawApi}"/>
+    <xacro:simple_transmission jointName="${IndexFingerPitch1ActuatorName}" actuatorName="${IndexFingerPitch1ActuatorName}" nodeName="${IndexFingerNode}" actuatorApi="${IndexFingerApi}"/>
+    <xacro:simple_transmission jointName="${MiddleFingerPitch1ActuatorName}" actuatorName="${MiddleFingerPitch1ActuatorName}" nodeName="${MiddleFingerNode}" actuatorApi="${MiddleFingerApi}"/>
+    <xacro:simple_transmission jointName="${PinkyPitch1ActuatorName}" actuatorName="${PinkyPitch1ActuatorName}" nodeName="${PinkyFingerNode}" actuatorApi="${PinkyFingerApi}"/>
+    <xacro:simple_transmission jointName="${ThumbRollActuatorName}" actuatorName="${ThumbRollActuatorName}" nodeName="${ThumbRollNode}" actuatorApi="${ThumbRollFingerApi}"/>
+    <xacro:simple_transmission jointName="${ThumbPitch1ActuatorName}" actuatorName="${ThumbPitch1ActuatorName}" nodeName="${ThumbProximalNode}" actuatorApi="${ThumbProximalFingerApi}"/>
+    <xacro:simple_transmission jointName="${ThumbPitch2ActuatorName}" actuatorName="${ThumbPitch2ActuatorName}" nodeName="${ThumbDistalNode}" actuatorApi="${ThumbDistalFingerApi}"/>
+    <xacro:pushrod_transmission transmissionName="${prefix}WristTransmission" transmissionType="${WristTransmissionType}" joint1Name="${WristPitchJointName}" joint2Name="${WristRollJointName}" joint1Role="pitch" joint2Role="roll" actuator1Name="${WristRightActuatorName}" actuator2Name="${WristLeftActuatorName}" actuator1Node="${WristRightActuatorNode}" actuator2Node="${WristLeftActuatorNode}" actuator1Api="${WristRightActuatorApi}" actuator2Api="${WristLeftActuatorApi}" actuator1Role="bottom" actuator2Role="top"/>
 </robot>

Commit message: updating names for UOE

File: common/xacro/actuator_names/valkyrie_actuator_names.xacro (robot description, xacro)
@@ -28,9 +28,9 @@
 	<xacro:property name="WristPitchActuatorSimName" value="${prefix}WristPitchActuator"/>
 	<xacro:property name="WristRollActuatorSimName" value="${prefix}WristRollActuator"/>
-	<xacro:property name="IndexFingerPitch1ActuatorName" value="${prefix}IndexFingerPitch1"/>
-	<xacro:property name="MiddleFingerPitch1ActuatorName" value="${prefix}MiddleFingerPitch1"/>
-	<xacro:property name="PinkyPitch1ActuatorName" value="${prefix}PinkyPitch1"/>
-	<xacro:property name="ThumbRollActuatorName" value="${prefix}ThumbRoll"/>
-	<xacro:property name="ThumbPitch1ActuatorName" value="${prefix}ThumbPitch1"/>
-	<xacro:property name="ThumbPitch2ActuatorName" value="${prefix}ThumbPitch2"/>
+	<xacro:property name="IndexFingerPitch1ActuatorName" value="${prefix}IndexFingerMotorPitch1"/>
+	<xacro:property name="MiddleFingerPitch1ActuatorName" value="${prefix}MiddleFingerMotorPitch1"/>
+	<xacro:property name="PinkyPitch1ActuatorName" value="${prefix}PinkyMotorPitch1"/>
+	<xacro:property name="ThumbRollActuatorName" value="${prefix}ThumbMotorRoll"/>
+	<xacro:property name="ThumbPitch1ActuatorName" value="${prefix}ThumbMotorPitch1"/>
+	<xacro:property name="ThumbPitch2ActuatorName" value="${prefix}ThumbMotorPitch2"/>
 </robot>

File: common/xacro/joint_names/valkyrie_joint_names.xacro (robot description, xacro)
@@ -20,16 +20,16 @@
 	<xacro:property name="WristRollJointName" value="${prefix}WristRoll"/>
 	<xacro:property name="WristPitchJointName" value="${prefix}WristPitch"/>
-	<xacro:property name="IndexFingerPitch1JointName" value="${prefix}IndexFingerPitch1Sensor"/>
-	<xacro:property name="IndexFingerPitch2JointName" value="${prefix}IndexFingerPitch2Sensor"/>
-	<xacro:property name="IndexFingerPitch3JointName" value="${prefix}IndexFingerPitch3Sensor"/>
-	<xacro:property name="MiddleFingerPitch1JointName" value="${prefix}MiddleFingerPitch1Sensor"/>
-	<xacro:property name="MiddleFingerPitch2JointName" value="${prefix}MiddleFingerPitch2Sensor"/>
-	<xacro:property name="MiddleFingerPitch3JointName" value="${prefix}MiddleFingerPitch3Sensor"/>
-	<xacro:property name="PinkyPitch1JointName" value="${prefix}PinkyPitch1Sensor"/>
-	<xacro:property name="PinkyPitch2JointName" value="${prefix}PinkyPitch2Sensor"/>
-	<xacro:property name="PinkyPitch3JointName" value="${prefix}PinkyPitch3Sensor"/>
-	<xacro:property name="ThumbRollJointName" value="${prefix}ThumbRollSensor"/>
-	<xacro:property name="ThumbPitch1JointName" value="${prefix}ThumbPitch1Sensor"/>
-	<xacro:property name="ThumbPitch2JointName" value="${prefix}ThumbPitch2Sensor"/>
-	<xacro:property name="ThumbPitch3JointName" value="${prefix}ThumbPitch3Sensor"/>
+	<xacro:property name="IndexFingerPitch1JointName" value="${prefix}IndexFingerPitch1"/>
+	<xacro:property name="IndexFingerPitch2JointName" value="${prefix}IndexFingerPitch2"/>
+	<xacro:property name="IndexFingerPitch3JointName" value="${prefix}IndexFingerPitch3"/>
+	<xacro:property name="MiddleFingerPitch1JointName" value="${prefix}MiddleFingerPitch1"/>
+	<xacro:property name="MiddleFingerPitch2JointName" value="${prefix}MiddleFingerPitch2"/>
+	<xacro:property name="MiddleFingerPitch3JointName" value="${prefix}MiddleFingerPitch3"/>
+	<xacro:property name="PinkyPitch1JointName" value="${prefix}PinkyPitch1"/>
+	<xacro:property name="PinkyPitch2JointName" value="${prefix}PinkyPitch2"/>
+	<xacro:property name="PinkyPitch3JointName" value="${prefix}PinkyPitch3"/>
+	<xacro:property name="ThumbRollJointName" value="${prefix}ThumbRoll"/>
+	<xacro:property name="ThumbPitch1JointName" value="${prefix}ThumbPitch1"/>
+	<xacro:property name="ThumbPitch2JointName" value="${prefix}ThumbPitch2"/>
+	<xacro:property name="ThumbPitch3JointName" value="${prefix}ThumbPitch3"/>
 </robot>
