Commit message: starting updates for 16.04

File: common/xacro/actuator_names/valkyrie_actuator_names.xacro (robot description, xacro)
@@ -6,31 +6,31 @@
 	<xacro:property name="WaistPitchActuatorSimName" value="waistPitchActuator"/>
 	<xacro:property name="WaistRollActuatorSimName" value="waistRollActuator"/>
-	<xacro:property name="HipYawActuatorName" value="${prefix}HipYaw"/>
-	<xacro:property name="HipRollActuatorName" value="${prefix}HipRoll"/>
-	<xacro:property name="HipPitchActuatorName" value="${prefix}HipPitch"/>
-	<xacro:property name="KneePitchActuatorName" value="${prefix}KneePitch"/>
-	<xacro:property name="AnkleRightActuatorName" value="${prefix}AnkleRightActuator"/>
-	<xacro:property name="AnkleLeftActuatorName" value="${prefix}AnkleLeftActuator"/>
-	<xacro:property name="AnkleRollActuatorSimName" value="${prefix}AnkleRollActuator"/>
-	<xacro:property name="AnklePitchActuatorSimName" value="${prefix}AnklePitchActuator"/>
+	<xacro:property name="HipYawActuatorName" value="HipYaw"/>
+	<xacro:property name="HipRollActuatorName" value="HipRoll"/>
+	<xacro:property name="HipPitchActuatorName" value="HipPitch"/>
+	<xacro:property name="KneePitchActuatorName" value="KneePitch"/>
+	<xacro:property name="AnkleRightActuatorName" value="AnkleRightActuator"/>
+	<xacro:property name="AnkleLeftActuatorName" value="AnkleLeftActuator"/>
+	<xacro:property name="AnkleRollActuatorSimName" value="AnkleRollActuator"/>
+	<xacro:property name="AnklePitchActuatorSimName" value="AnklePitchActuator"/>
 	<xacro:property name="LowerNeckPitchActuatorName" value="lowerNeckPitch"/>
 	<xacro:property name="NeckYawActuatorName" value="neckYaw"/>
 	<xacro:property name="UpperNeckPitchActuatorName" value="upperNeckPitch"/>
-	<xacro:property name="ShoulderPitchActuatorName" value="${prefix}ShoulderPitch"/>
-	<xacro:property name="ShoulderRollActuatorName" value="${prefix}ShoulderRoll"/>
-	<xacro:property name="ShoulderYawActuatorName" value="${prefix}ShoulderYaw"/>
-	<xacro:property name="ElbowPitchActuatorName" value="${prefix}ElbowPitch"/>
-	<xacro:property name="ForearmYawActuatorName" value="${prefix}ForearmYaw"/>
-	<xacro:property name="WristBottomActuatorName" value="${prefix}WristBottomActuator"/>
-	<xacro:property name="WristTopActuatorName" value="${prefix}WristTopActuator"/>
-	<xacro:property name="WristRightActuatorName" value="${prefix}WristRightActuator"/>
-	<xacro:property name="WristLeftActuatorName" value="${prefix}WristLeftActuator"/>
-	<xacro:property name="WristPitchActuatorSimName" value="${prefix}WristPitchActuator"/>
-	<xacro:property name="WristRollActuatorSimName" value="${prefix}WristRollActuator"/>
-	<xacro:property name="IndexFingerPitch1ActuatorName" value="${prefix}IndexFingerPitch1"/>
-	<xacro:property name="MiddleFingerPitch1ActuatorName" value="${prefix}MiddleFingerPitch1"/>
-	<xacro:property name="PinkyPitch1ActuatorName" value="${prefix}PinkyPitch1"/>
-	<xacro:property name="ThumbRollActuatorName" value="${prefix}ThumbRoll"/>
-	<xacro:property name="ThumbPitch1ActuatorName" value="${prefix}ThumbPitch1"/>
-	<xacro:property name="ThumbPitch2ActuatorName" value="${prefix}ThumbPitch2"/>
+	<xacro:property name="ShoulderPitchActuatorName" value="ShoulderPitch"/>
+	<xacro:property name="ShoulderRollActuatorName" value="ShoulderRoll"/>
+	<xacro:property name="ShoulderYawActuatorName" value="ShoulderYaw"/>
+	<xacro:property name="ElbowPitchActuatorName" value="ElbowPitch"/>
+	<xacro:property name="ForearmYawActuatorName" value="ForearmYaw"/>
+	<xacro:property name="WristBottomActuatorName" value="WristBottomActuator"/>
+	<xacro:property name="WristTopActuatorName" value="WristTopActuator"/>
+	<xacro:property name="WristRightActuatorName" value="WristRightActuator"/>
+	<xacro:property name="WristLeftActuatorName" value="WristLeftActuator"/>
+	<xacro:property name="WristPitchActuatorSimName" value="WristPitchActuator"/>
+	<xacro:property name="WristRollActuatorSimName" value="WristRollActuator"/>
+	<xacro:property name="IndexFingerPitch1ActuatorName" value="IndexFingerPitch1"/>
+	<xacro:property name="MiddleFingerPitch1ActuatorName" value="MiddleFingerPitch1"/>
+	<xacro:property name="PinkyPitch1ActuatorName" value="PinkyPitch1"/>
+	<xacro:property name="ThumbRollActuatorName" value="ThumbRoll"/>
+	<xacro:property name="ThumbPitch1ActuatorName" value="ThumbPitch1"/>
+	<xacro:property name="ThumbPitch2ActuatorName" value="ThumbPitch2"/>
 </robot>

File: common/xacro/api/forearm_api.xacro (robot description, xacro)
@@ -1,3 +1,3 @@
- <robot xmlns:xacro="http://ros.org/wiki/xacro" name="forearm_api">
+ <robot xmlns:xacro="http://www.ros.org/wiki/xacro" name="forearm_api">
     <xacro:property name="ForearmYawApi" value="robot_hardware_interface/TurbodriverAPI" />
     <xacro:property name="IndexFingerApi" value="robot_hardware_interface/TurbodriverAPI"/>

File: common/xacro/api/testbench_api.xacro (robot description, xacro)
@@ -1,3 +1,3 @@
-<robot xmlns:xacro="http://ros.org/wiki/xacro" name="valkyrie_api">
+<robot xmlns:xacro="http://www.ros.org/wiki/xacro" name="valkyrie_api">
     <xacro:property name="testbenchApi" value="robot_hardware_interface/TurbodriverAPI" />
 </robot>

File: common/xacro/api/valkyrie_A_api.xacro (robot description, xacro)
@@ -1,3 +1,3 @@
-<robot xmlns:xacro="http://ros.org/wiki/xacro" name="valkyrie_api">
+<robot xmlns:xacro="http://www.ros.org/wiki/xacro" name="valkyrie_api">
     <xacro:property name="HipYawApi" value="robot_hardware_interface/TurbodriverAPI" />
     <xacro:property name="HipRollApi" value="robot_hardware_interface/TurbodriverAPI" />

File: common/xacro/api/valkyrie_B_api.xacro (robot description, xacro)
@@ -1,3 +1,3 @@
-<robot xmlns:xacro="http://ros.org/wiki/xacro" name="valkyrie_api">
+<robot xmlns:xacro="http://www.ros.org/wiki/xacro" name="valkyrie_api">
     <xacro:property name="HipYawApi" value="robot_hardware_interface/TurbodriverAPI" />
     <xacro:property name="HipRollApi" value="robot_hardware_interface/TurbodriverAPI" />

File: common/xacro/api/valkyrie_C_api.xacro (robot description, xacro)
@@ -1,3 +1,3 @@
-<robot xmlns:xacro="http://ros.org/wiki/xacro" name="valkyrie_api">
+<robot xmlns:xacro="http://www.ros.org/wiki/xacro" name="valkyrie_api">
     <xacro:property name="HipYawApi" value="robot_hardware_interface/TurbodriverAPI" />
     <xacro:property name="HipRollApi" value="robot_hardware_interface/TurbodriverAPI" />

File: common/xacro/api/valkyrie_D_api.xacro (robot description, xacro)
@@ -1,3 +1,3 @@
-<robot xmlns:xacro="http://ros.org/wiki/xacro" name="valkyrie_api">
+<robot xmlns:xacro="http://www.ros.org/wiki/xacro" name="valkyrie_api">
     <xacro:property name="HipYawApi" value="robot_hardware_interface/TurbodriverAPI" />
     <xacro:property name="HipRollApi" value="robot_hardware_interface/TurbodriverAPI" />

File: common/xacro/api/valkyrie_sim_api.xacro (robot description, xacro)
@@ -1,3 +1,3 @@
-<robot xmlns:xacro="http://ros.org/wiki/xacro" name="valkyrie_sim_api">
+<robot xmlns:xacro="http://www.ros.org/wiki/xacro" name="valkyrie_sim_api">
 	<xacro:property name="SimApi" value="robot_hardware_interface/TurbodriverSimAPI" />
     <xacro:property name="ImuSensorSimApi" value="simulated_imu_sensor::SimulatedImuSensor" />

File: common/xacro/dev_ports/valkyrie_A_ports.xacro (robot description, xacro)
@@ -1,3 +1,3 @@
-<robot xmlns:xacro="http://ros.org/wiki/xacro" name="valkyrie_A_ports">
+<robot xmlns:xacro="http://www.ros.org/wiki/xacro" name="valkyrie_A_ports">
 	<xacro:property name="pelvis_middle_imu_port" value="/dev/ttyACM0" />
 	<xacro:property name="pelvis_rear_imu_port" value="/dev/serial/by-id/usb-Lord_Microstrain_Lord_Inertial_Sensor_0000__6233.47095-if00" />

File: common/xacro/dev_ports/valkyrie_B_ports.xacro (robot description, xacro)
@@ -1,3 +1,3 @@
-<robot xmlns:xacro="http://ros.org/wiki/xacro" name="valkyrie_B_ports">
+<robot xmlns:xacro="http://www.ros.org/wiki/xacro" name="valkyrie_B_ports">
 	<xacro:property name="pelvis_middle_imu_port" value="/dev/serial/by-id/usb-Lord_Microstrain_Lord_Inertial_Sensor_0000__6233.47094-if00" />
 	<!-- <xacro:property name="pelvis_rear_imu_port" value="/dev/serial/by-id/usb-FTDI_USB-RS232_Cable_FTY5H9NH-if00-port0" /> -->

File: common/xacro/dev_ports/valkyrie_C_ports.xacro (robot description, xacro)
@@ -1,3 +1,3 @@
-<robot xmlns:xacro="http://ros.org/wiki/xacro" name="valkyrie_C_ports">
+<robot xmlns:xacro="http://www.ros.org/wiki/xacro" name="valkyrie_C_ports">
 	<xacro:property name="pelvis_middle_imu_port" value="UNKNOWN" />
 	<xacro:property name="pelvis_rear_imu_port" value="/dev/serial/by-id/usb-Lord_Microstrain_Lord_Inertial_Sensor_0000__6233.47250-if00" />

File: common/xacro/dev_ports/valkyrie_D_ports.xacro (robot description, xacro)
@@ -1,3 +1,3 @@
-<robot xmlns:xacro="http://ros.org/wiki/xacro" name="valkyrie_D_ports">
+<robot xmlns:xacro="http://www.ros.org/wiki/xacro" name="valkyrie_D_ports">
     <xacro:property name="pelvis_middle_imu_port" value="UNKNOWN" />
     <xacro:property name="pelvis_rear_imu_port" value="/dev/serial/by-id/usb-Lord_Microstrain_Lord_Inertial_Sensor_0000__6233.51067-if00" />

File: common/xacro/dev_ports/valkyrie_gazebo_ports.xacro (robot description, xacro)
@@ -1,3 +1,3 @@
-<robot xmlns:xacro="http://ros.org/wiki/xacro" name="valkyrie_gazebo_ports">
+<robot xmlns:xacro="http://www.ros.org/wiki/xacro" name="valkyrie_gazebo_ports">
 	<xacro:property name="pelvis_middle_imu_port" value="none" />
 	<xacro:property name="pelvis_rear_imu_port" value="none" />

File: common/xacro/dev_ports/valkyrie_imu_test_ports.xacro (robot description, xacro)
@@ -1,3 +1,3 @@
-<robot xmlns:xacro="http://ros.org/wiki/xacro" name="valkyrie_imu_test_ports">
+<robot xmlns:xacro="http://www.ros.org/wiki/xacro" name="valkyrie_imu_test_ports">
 	<xacro:property name="pelvis_middle_imu_port" value="/dev/serial/by-id/usb-FTDI_USB-RS422_Cable_FTVR09ZC-if00-port0" />
 </robot>

File: common/xacro/joint_names/valkyrie_joint_names.xacro (robot description, xacro)
@@ -4,32 +4,32 @@
 	<xacro:property name="TorsoPitchJointName" value="torsoPitch"/>
 	<xacro:property name="TorsoRollJointName" value="torsoRoll"/>
-	<xacro:property name="HipYawJointName" value="${prefix}HipYaw"/>
-	<xacro:property name="HipRollJointName" value="${prefix}HipRoll"/>
-	<xacro:property name="HipPitchJointName" value="${prefix}HipPitch"/>
-	<xacro:property name="KneePitchJointName" value="${prefix}KneePitch"/>
-	<xacro:property name="AnklePitchJointName" value="${prefix}AnklePitch"/>
-	<xacro:property name="AnkleRollJointName" value="${prefix}AnkleRoll"/>
+	<xacro:property name="HipYawJointName" value="HipYaw"/>
+	<xacro:property name="HipRollJointName" value="HipRoll"/>
+	<xacro:property name="HipPitchJointName" value="HipPitch"/>
+	<xacro:property name="KneePitchJointName" value="KneePitch"/>
+	<xacro:property name="AnklePitchJointName" value="AnklePitch"/>
+	<xacro:property name="AnkleRollJointName" value="AnkleRoll"/>
 	<xacro:property name="LowerNeckPitchJointName" value="lowerNeckPitch"/>
 	<xacro:property name="NeckYawJointName" value="neckYaw"/>
 	<xacro:property name="UpperNeckPitchJointName" value="upperNeckPitch"/>
-	<xacro:property name="ShoulderPitchJointName" value="${prefix}ShoulderPitch"/>
-	<xacro:property name="ShoulderRollJointName" value="${prefix}ShoulderRoll"/>
-	<xacro:property name="ShoulderYawJointName" value="${prefix}ShoulderYaw"/>
-	<xacro:property name="ElbowPitchJointName" value="${prefix}ElbowPitch"/>
-	<xacro:property name="ForearmYawJointName" value="${prefix}ForearmYaw"/>
-	<xacro:property name="WristRollJointName" value="${prefix}WristRoll"/>
-	<xacro:property name="WristPitchJointName" value="${prefix}WristPitch"/>
-	<xacro:property name="IndexFingerPitch1JointName" value="${prefix}IndexFingerPitch1"/>
-	<xacro:property name="IndexFingerPitch2JointName" value="${prefix}IndexFingerPitch2"/>
-	<xacro:property name="IndexFingerPitch3JointName" value="${prefix}IndexFingerPitch3"/>
-	<xacro:property name="MiddleFingerPitch1JointName" value="${prefix}MiddleFingerPitch1"/>
-	<xacro:property name="MiddleFingerPitch2JointName" value="${prefix}MiddleFingerPitch2"/>
-	<xacro:property name="MiddleFingerPitch3JointName" value="${prefix}MiddleFingerPitch3"/>
-	<xacro:property name="PinkyPitch1JointName" value="${prefix}PinkyPitch1"/>
-	<xacro:property name="PinkyPitch2JointName" value="${prefix}PinkyPitch2"/>
-	<xacro:property name="PinkyPitch3JointName" value="${prefix}PinkyPitch3"/>
-	<xacro:property name="ThumbRollJointName" value="${prefix}ThumbRoll"/>
-	<xacro:property name="ThumbPitch1JointName" value="${prefix}ThumbPitch1"/>
-	<xacro:property name="ThumbPitch2JointName" value="${prefix}ThumbPitch2"/>
-	<xacro:property name="ThumbPitch3JointName" value="${prefix}ThumbPitch3"/>
+	<xacro:property name="ShoulderPitchJointName" value="ShoulderPitch"/>
+	<xacro:property name="ShoulderRollJointName" value="ShoulderRoll"/>
+	<xacro:property name="ShoulderYawJointName" value="ShoulderYaw"/>
+	<xacro:property name="ElbowPitchJointName" value="ElbowPitch"/>
+	<xacro:property name="ForearmYawJointName" value="ForearmYaw"/>
+	<xacro:property name="WristRollJointName" value="WristRoll"/>
+	<xacro:property name="WristPitchJointName" value="WristPitch"/>
+	<xacro:property name="IndexFingerPitch1JointName" value="IndexFingerPitch1"/>
+	<xacro:property name="IndexFingerPitch2JointName" value="IndexFingerPitch2"/>
+	<xacro:property name="IndexFingerPitch3JointName" value="IndexFingerPitch3"/>
+	<xacro:property name="MiddleFingerPitch1JointName" value="MiddleFingerPitch1"/>
+	<xacro:property name="MiddleFingerPitch2JointName" value="MiddleFingerPitch2"/>
+	<xacro:property name="MiddleFingerPitch3JointName" value="MiddleFingerPitch3"/>
+	<xacro:property name="PinkyPitch1JointName" value="PinkyPitch1"/>
+	<xacro:property name="PinkyPitch2JointName" value="PinkyPitch2"/>
+	<xacro:property name="PinkyPitch3JointName" value="PinkyPitch3"/>
+	<xacro:property name="ThumbRollJointName" value="ThumbRoll"/>
+	<xacro:property name="ThumbPitch1JointName" value="ThumbPitch1"/>
+	<xacro:property name="ThumbPitch2JointName" value="ThumbPitch2"/>
+	<xacro:property name="ThumbPitch3JointName" value="ThumbPitch3"/>
 </robot>

File: common/xacro/nodes/actuator_testbench_nodes.xacro (robot description, xacro)
@@ -1,3 +1,3 @@
-<robot xmlns:xacro="http://ros.org/wiki/xacro" name="test_bench_nodes">
+<robot xmlns:xacro="http://www.ros.org/wiki/xacro" name="test_bench_nodes">
 	<xacro:property name="testbench_node" value="/right_leg/j3" />
 </robot>

File: common/xacro/nodes/forearm_testbench_nodes.xacro (robot description, xacro)
@@ -1,3 +1,3 @@
-<robot xmlns:xacro="http://ros.org/wiki/xacro" name="test_bench_nodes">
+<robot xmlns:xacro="http://www.ros.org/wiki/xacro" name="test_bench_nodes">
     <xacro:property name="testbench_node" value="/right_arm/j5" />
     <xacro:property name="IndexNode" value="/right_arm/hand/index" />

File: common/xacro/nodes/forearm_testbench_nodes_left.xacro (robot description, xacro)
@@ -1,3 +1,3 @@
-<robot xmlns:xacro="http://ros.org/wiki/xacro" name="test_bench_nodes">
+<robot xmlns:xacro="http://www.ros.org/wiki/xacro" name="test_bench_nodes">
 	<xacro:property name="testbench_node" value="/left_arm/j5" />
 	<xacro:property name="Athena1Node" value="/left_arm/athena1" />

File: common/xacro/nodes/forearm_testbench_nodes_right.xacro (robot description, xacro)
@@ -1,3 +1,3 @@
-<robot xmlns:xacro="http://ros.org/wiki/xacro" name="test_bench_nodes">
+<robot xmlns:xacro="http://www.ros.org/wiki/xacro" name="test_bench_nodes">
 	<xacro:property name="testbench_node" value="/right_arm/j5" />
 	<xacro:property name="Athena1Node" value="/right_arm/athena1" />

File: common/xacro/nodes/valkyrie_nodes.xacro (robot description, xacro)
@@ -1,3 +1,3 @@
-<robot xmlns:xacro="http://ros.org/wiki/xacro" name="valkyrie_nodes">
+<robot xmlns:xacro="http://www.ros.org/wiki/xacro" name="valkyrie_nodes">
 	<xacro:property name="HipYawNode" value="/pelvis/${prefix}_leg_j1" />
 	<xacro:property name="HipRollNode" value="/${prefix}_leg/j2" />
@@ -6,13 +6,13 @@
 	<xacro:property name="AnkleLeftActuatorNode" value="/${prefix}_leg/ankle/left_actuator" />
 	<xacro:property name="AnkleRightActuatorNode" value="/${prefix}_leg/ankle/right_actuator" />
-	<xacro:property name="ShoulderPitchNode" value="/trunk/${prefix}_arm_j1" />
-	<xacro:property name="ShoulderRollNode" value="/${prefix}_arm/j2" />
-	<xacro:property name="ShoulderYawNode" value="/${prefix}_arm/j3" />
-	<xacro:property name="ElbowPitchNode" value="/${prefix}_arm/j4" />
-	<xacro:property name="ForearmYawNode" value="/${prefix}_arm/j5" />
-	<xacro:property name="WristTopActuatorNode" value="/${prefix}_arm/wrist/top_actautor" />
-	<xacro:property name="WristBottomActuatorNode" value="/${prefix}_arm/wrist/bottom_actuator" />
-	<xacro:property name="WristLeftActuatorNode" value="/${prefix}_arm/wrist/left_actuator" />
-	<xacro:property name="WristRightActuatorNode" value="/${prefix}_arm/wrist/right_actuator" />
+	<!--<xacro:property name="ShoulderPitchNode" value="/trunk/${prefix}_arm_j1" /> -->
+	<xacro:property name="ShoulderRollNode" value="_arm/j2" />
+	<xacro:property name="ShoulderYawNode" value="_arm/j3" />
+	<xacro:property name="ElbowPitchNode" value="_arm/j4" />
+	<xacro:property name="ForearmYawNode" value="_arm/j5" />
+	<xacro:property name="WristTopActuatorNode" value="_arm/wrist/top_actautor" />
+	<xacro:property name="WristBottomActuatorNode" value="_arm/wrist/bottom_actuator" />
+	<xacro:property name="WristLeftActuatorNode" value="_arm/wrist/left_actuator" />
+	<xacro:property name="WristRightActuatorNode" value="_arm/wrist/right_actuator" />
     	<xacro:property name="IndexNode" value="/${prefix}_arm/hand/index" />
     	<xacro:property name="MiddleNode" value="/${prefix}_arm/hand/middle" />
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