Commit message: added wrist roll and pitch calibrations to hand mechinisms

File: instance/instances/robots/forearm_testbench_right.xacro (robot description, xacro)
@@ -15,5 +15,5 @@
     <Mechanisms>
     <xacro:simple_mechanism name="testbench_actuator" serial_number="${forearm_yaw_serial_number}" node="${testbench_node}" />
-    <xacro:hand_mechanism mechanism_name="${prefix}Hand" serial_number="${hand_serial_number}" index_node="/${prefix}${IndexNode}" middle_node="/${prefix}${MiddleNode}" pinky_node="/${prefix}${PinkyNode}" thumb_prox_node="/${prefix}${ThumbProxNode}" thumb_dist_node="/${prefix}${ThumbDistNode}" thumb_roll_node="/${prefix}${ThumbRollNode}" wrist_left_node="/${prefix}${WristLeftNode}" wrist_right_node="/${prefix}${WristRightNode}" />
+    <xacro:hand_mechanism mechanism_name="${prefix}Hand" serial_number="${hand_serial_number}" index_node="/${prefix}${IndexNode}" middle_node="/${prefix}${MiddleNode}" pinky_node="/${prefix}${PinkyNode}" thumb_prox_node="/${prefix}${ThumbProxNode}" thumb_dist_node="/${prefix}${ThumbDistNode}" thumb_roll_node="/${prefix}${ThumbRollNode}" wrist_left_node="/${prefix}${WristLeftNode}" wrist_right_node="/${prefix}${WristRightNode}" wrist_pitch_calibration_angle="${WristPitchCalibrationAngle}" wrist_roll_calibration_angle="${WristRollCalibrationAngle}" />
     <xacro:hand_sensor_mechanism name="${prefix}HandSensors" serial_number="${hand_serial_number}_midas" node="/${prefix}${HandSensorNode}" />
     </Mechanisms>

File: instance/instances/robots/xacro/limbs/arm/arm.xacro (robot description, xacro)
@@ -8,5 +8,5 @@
     	<xacro:simple_mechanism name="${ElbowPitchJointName}" serial_number="${j4_serial_number}" node="/${prefix}${ElbowPitchNode}" calibration_angle="${ElbowPitchCalibrationAngle}"/>
     	<xacro:simple_mechanism name="${ForearmYawJointName}" serial_number="${j5_serial_number}" node="/${prefix}${ForearmYawNode}" calibration_angle="${ForearmYawCalibrationAngle}"/>
-    	<xacro:hand_mechanism mechanism_name="${prefix}Hand" serial_number="${forearm_serial_number}" index_node="/${prefix}${IndexNode}" middle_node="/${prefix}${MiddleNode}" pinky_node="/${prefix}${PinkyNode}" thumb_prox_node="/${prefix}${ThumbProxNode}" thumb_dist_node="/${prefix}${ThumbDistNode}" thumb_roll_node="/${prefix}${ThumbRollNode}" wrist_left_node="/${prefix}${WristLeftNode}" wrist_right_node="/${prefix}${WristRightNode}" />
+    	<xacro:hand_mechanism mechanism_name="${prefix}Hand" serial_number="${forearm_serial_number}" index_node="/${prefix}${IndexNode}" middle_node="/${prefix}${MiddleNode}" pinky_node="/${prefix}${PinkyNode}" thumb_prox_node="/${prefix}${ThumbProxNode}" thumb_dist_node="/${prefix}${ThumbDistNode}" thumb_roll_node="/${prefix}${ThumbRollNode}" wrist_left_node="/${prefix}${WristLeftNode}" wrist_right_node="/${prefix}${WristRightNode}" wrist_pitch_calibration_angle="${WristPitchCalibrationAngle}" wrist_roll_calibration_angle="${WristRollCalibrationAngle}" />
         <xacro:hand_sensor_mechanism name="${prefix}HandSensors" serial_number="${forearm_serial_number}_midas" node="/${prefix}${HandSensorNode}" />
     </xacro:macro>

File: instance/instances/robots/xacro/mechanisms/mechanisms.xacro (robot description, xacro)
@@ -39,7 +39,9 @@
     </Mechanism>
 </xacro:macro>
-<xacro:macro name="hand_mechanism" params="mechanism_name serial_number index_node middle_node pinky_node thumb_prox_node thumb_dist_node thumb_roll_node wrist_left_node wrist_right_node" >
+<xacro:macro name="hand_mechanism" params="mechanism_name serial_number index_node middle_node pinky_node thumb_prox_node thumb_dist_node thumb_roll_node wrist_left_node wrist_right_node wrist_pitch_calibration_angle wrist_roll_calibration_angle" >
     <Mechanism id="${mechanism_name}" type="hand">
             <SerialNumber id="${serial_number}"/>
+            <WristPitchCalibrationAngle id="${wrist_pitch_calibration_angle}"/>
+            <WristRollCalibrationAngle id="${wrist_roll_calibration_angle}"/>
             <Nodes>
                 <Index id="${index_node}"/>
