Commit message: Reworking a bunch of our xacro files to make it easier to have robots with different kinematics and/or mass properties.

File: model/robots/common/xacro/arm/arm.xacro (robot description, xacro)
@@ -1,12 +1,4 @@
 <?xml version="1.0" ?>
 <robot xmlns:xacro="http://www.ros.org/wiki/xacro" name="arm">
-  <xacro:include filename="$(find val_description)/common/xacro/joint_names/valkyrie_joint_names.xacro"/>
-  <xacro:include filename="$(find val_description)/common/xacro/actuator_names/valkyrie_actuator_names.xacro"/>
-  <xacro:include filename="$(find val_description)/model/robots/common/xacro/arm/joint_axes.xacro"/>
-  <xacro:include filename="$(find val_description)/model/robots/common/xacro/arm/link_names.xacro"/>
-  <xacro:include filename="$(find val_description)/model/robots/common/xacro/arm/joint_limits.xacro"/>
-  <xacro:include filename="$(find val_description)/model/robots/common/xacro/arm/frame_parameters.xacro"/>
-  <xacro:include filename="$(find val_description)/model/robots/common/xacro/arm/mass_parameters.xacro"/>
-  <xacro:include filename="$(find val_description)/model/robots/common/xacro/gains.xacro"/>
   <xacro:macro name="make_upper_arm" params="prefix reflect upper_arm_root_link">
     <xacro:standard_link name="${ShoulderPitchLinkName}"

File: model/robots/common/xacro/common_bodies.xacro (robot description, xacro)
@@ -1,11 +1,6 @@
 <robot xmlns:xacro="http://ros.orgt/wiki/xacro" name="common_bodies">
-    <xacro:include filename="$(find val_description)/model/robots/common/xacro/pelvis/pelvis.xacro" />
-    <xacro:include filename="$(find val_description)/model/robots/common/xacro/waist/waist.xacro" />
-    <xacro:include filename="$(find val_description)/model/robots/common/xacro/head/head.xacro" />
-    <xacro:include filename="$(find val_description)/model/robots/common/xacro/arm/arm.xacro" />
-    <xacro:include filename="$(find val_description)/model/robots/common/xacro/thumb/thumb.xacro" />
-    <xacro:include filename="$(find val_description)/model/robots/common/xacro/leg/leg.xacro" />
     <xacro:include filename="$(find val_description)/model/robots/common/xacro/index_finger/index_finger.xacro" />
     <xacro:include filename="$(find val_description)/model/robots/common/xacro/middle_finger/middle_finger.xacro" />
     <xacro:include filename="$(find val_description)/model/robots/common/xacro/pinky_finger/pinky_finger.xacro" />
+    <xacro:include filename="$(find val_description)/model/robots/common/xacro/thumb/thumb.xacro" />
 </robot>

File: model/robots/common/xacro/head/head.xacro (robot description, xacro)
@@ -1,12 +1,3 @@
 <robot xmlns:xacro="http://www.ros.org/wiki/xacro" name="head">
-  <xacro:include filename="$(find val_description)/common/xacro/joint_names/valkyrie_joint_names.xacro"/>
-  <xacro:include filename="$(find val_description)/common/xacro/actuator_names/valkyrie_actuator_names.xacro"/>
-  <xacro:include filename="$(find val_description)/model/robots/common/xacro/head/joint_axes.xacro"/>
-  <xacro:include filename="$(find val_description)/model/robots/common/xacro/head/link_names.xacro"/>
-  <xacro:include filename="$(find val_description)/model/robots/common/xacro/head/joint_limits.xacro"/>
-  <xacro:include filename="$(find val_description)/model/robots/common/xacro/head/frame_parameters.xacro"/>
-  <xacro:include filename="$(find val_description)/model/robots/common/xacro/head/mass_parameters.xacro"/>
-  <xacro:include filename="$(find val_description)/model/robots/common/xacro/gains.xacro"/>
-  <xacro:property name="NJ3_Link_Radius" value="0.139"/>
   <xacro:macro name="include_head" params="lower_neck_pitch_root_link">
   </xacro:macro>

File: model/robots/common/xacro/leg/leg.xacro (robot description, xacro)
@@ -1,12 +1,4 @@
 <?xml version="1.0" ?>
 <robot xmlns:xacro="http://www.ros.org/wiki/xacro" name="leg">
-  <xacro:include filename="$(find val_description)/common/xacro/joint_names/valkyrie_joint_names.xacro"/>
-  <xacro:include filename="$(find val_description)/common/xacro/actuator_names/valkyrie_actuator_names.xacro"/>
-  <xacro:include filename="$(find val_description)/model/robots/common/xacro/leg/joint_axes.xacro"/>
-  <xacro:include filename="$(find val_description)/model/robots/common/xacro/leg/link_names.xacro"/>
-  <xacro:include filename="$(find val_description)/model/robots/common/xacro/leg/joint_limits.xacro"/>
-  <xacro:include filename="$(find val_description)/model/robots/common/xacro/leg/frame_parameters.xacro"/>
-  <xacro:include filename="$(find val_description)/model/robots/common/xacro/leg/mass_parameters.xacro"/>
-  <xacro:include filename="$(find val_description)/model/robots/common/xacro/sensors/ati_force_torque.xacro"/>
   <xacro:macro name="make_leg_links" params="prefix reflect leg_root_link">
     <xacro:standard_link name="${HipYawLinkName}"

File: model/robots/common/xacro/pelvis/pelvis.xacro (robot description, xacro)
@@ -3,8 +3,8 @@
     <xacro:macro name="make_pelvis">
         <xacro:standard_link name="${Pelvis_Link_Name}"
-                        mass="8.22"
-                        origin_xyz="-0.00532 -0.003512 -0.0036"
-                        ixx="0.11866378" ixy="-0.000143482" ixz="0.003271293"
-                        iyy="0.097963425" iyz="0.002159545" izz="0.083854638"
+                        mass="${PelvisLinkMass}"
+                        origin_xyz="${PelvisLinkComPosition}"
+                        ixx="${PelvisLinkInertia_IXX}" ixy="${PelvisLinkInertia_IXY}" ixz="${PelvisLinkInertia_IXZ}"
+                        iyy="${PelvisLinkInertia_IYY}" iyz="${PelvisLinkInertia_IYZ}" izz="${PelvisLinkInertia_IZZ}"
                         origin_rpy="0 0 0"
                         visual_mesh="${mesh_root}/pelvis/pelvis.dae"

File: model/robots/common/xacro/valkyrie_arm_mass_sims_base_hw.xacro (robot description, xacro)
@@ -1,7 +1,3 @@
 <robot xmlns:xacro="http://ros.org/wiki/xacro" name="valkyrie">
-    <xacro:property name="mesh_root" value="package://val_description/model/meshes"/>
-    <xacro:include filename="$(find val_description)/model/robots/common/xacro/generic_models.xacro" />
-    <xacro:include filename="$(find val_description)/model/robots/common/xacro/common_bodies.xacro" />
-    <xacro:include filename="$(find val_description)/common/xacro/nodes/valkyrie_nodes.xacro"/>
     <xacro:make_pelvis />
     <xacro:make_waist waist_root_link="${Pelvis_Link_Name}" />

File: model/robots/common/xacro/valkyrie_arm_mass_sims_base_sim.xacro (robot description, xacro)
@@ -1,7 +1,3 @@
 <robot xmlns:xacro="http://ros.org/wiki/xacro" name="valkyrie">
-    <xacro:property name="mesh_root" value="package://val_description/model/meshes"/>
-    <xacro:include filename="$(find val_description)/model/robots/common/xacro/generic_models.xacro" />
-    <xacro:include filename="$(find val_description)/model/robots/common/xacro/common_bodies.xacro" />
-    <xacro:include filename="$(find val_description)/common/xacro/nodes/valkyrie_sim_nodes.xacro"/>
     <xacro:make_pelvis />
     <xacro:make_waist waist_root_link="${Pelvis_Link_Name}" />

File: model/robots/common/xacro/valkyrie_base_hw.xacro (robot description, xacro)
@@ -1,7 +1,3 @@
 <robot xmlns:xacro="http://ros.org/wiki/xacro" name="valkyrie">
-    <xacro:property name="mesh_root" value="package://val_description/model/meshes"/>
-    <xacro:include filename="$(find val_description)/model/robots/common/xacro/generic_models.xacro" />
-    <xacro:include filename="$(find val_description)/model/robots/common/xacro/common_bodies.xacro" />
-    <xacro:include filename="$(find val_description)/common/xacro/nodes/valkyrie_nodes.xacro"/>
     <xacro:make_pelvis />
     <xacro:make_waist waist_root_link="${Pelvis_Link_Name}" />

File: model/robots/common/xacro/valkyrie_base_sim.xacro (robot description, xacro)
@@ -1,7 +1,3 @@
 <robot xmlns:xacro="http://ros.org/wiki/xacro" name="valkyrie">
-    <xacro:property name="mesh_root" value="package://val_description/model/meshes"/>
-    <xacro:include filename="$(find val_description)/model/robots/common/xacro/generic_models.xacro" />
-    <xacro:include filename="$(find val_description)/model/robots/common/xacro/common_bodies.xacro" />
-    <xacro:include filename="$(find val_description)/common/xacro/nodes/valkyrie_sim_nodes.xacro"/>
     <xacro:make_pelvis />
     <xacro:make_waist waist_root_link="${Pelvis_Link_Name}" />

File: model/robots/common/xacro/waist/waist.xacro (robot description, xacro)
@@ -1,13 +1,3 @@
 <robot xmlns:xacro="http://www.ros.org/wiki/xacro" name="waist">
-  <xacro:include filename="$(find val_description)/common/xacro/joint_names/valkyrie_joint_names.xacro"/>
-  <xacro:include filename="$(find val_description)/common/xacro/actuator_names/valkyrie_actuator_names.xacro"/>
-  <xacro:include filename="$(find val_description)/model/robots/common/xacro/waist/joint_axes.xacro"/>
-  <xacro:include filename="$(find val_description)/model/robots/common/xacro/waist/joint_axes.xacro"/>
-  <xacro:include filename="$(find val_description)/model/robots/common/xacro/waist/link_names.xacro"/>
-  <xacro:include filename="$(find val_description)/model/robots/common/xacro/waist/joint_limits.xacro"/>
-  <xacro:include filename="$(find val_description)/model/robots/common/xacro/waist/frame_parameters.xacro"/>
-  <xacro:include filename="$(find val_description)/model/robots/common/xacro/waist/mass_parameters.xacro"/>
-  <xacro:include filename="$(find val_description)/model/robots/common/xacro/sensors/microstrain.xacro"/>
-  <xacro:include filename="$(find val_description)/model/robots/common/xacro/sensors/flea.xacro"/>
   <xacro:macro name="make_waist_common" params="waist_root_link">
     <xacro:revolute_joint_ex jointName="${TorsoYawJointName}"

File: model/robots/forearm_left.xacro (robot description, xacro)
@@ -5,4 +5,6 @@
     <xacro:include filename="$(find val_description)/model/robots/common/xacro/common_bodies.xacro" />
     <xacro:include filename="$(find val_description)/common/xacro/api/forearm_api.xacro"/>
+    <!-- Arm include -->
+    <xacro:include filename="$(find val_description)/model/robots/common/xacro/arm/arm_includes.xacro"/>
     <xacro:property name="prefix" value="left"/>
     <xacro:property name="reflect" value="1"/>

File: model/robots/forearm_right.xacro (robot description, xacro)
@@ -5,4 +5,6 @@
     <xacro:include filename="$(find val_description)/model/robots/common/xacro/common_bodies.xacro" />
     <xacro:include filename="$(find val_description)/common/xacro/api/forearm_api.xacro"/>
+    <!-- Arm include -->
+    <xacro:include filename="$(find val_description)/model/robots/common/xacro/arm/arm_includes.xacro"/>
     <xacro:property name="prefix" value="right"/>
     <xacro:property name="reflect" value="-1"/>

File: model/robots/valkyrie_A.xacro (robot description, xacro)
@@ -1,7 +1,21 @@
 <robot xmlns:xacro="http://ros.org/wiki/xacro" name="valkyrie">
+	<xacro:property name="mesh_root" value="package://val_description/model/meshes"/>
+	<xacro:include filename="$(find val_description)/model/robots/common/xacro/generic_models.xacro" />
+    <xacro:include filename="$(find val_description)/common/xacro/nodes/valkyrie_nodes.xacro"/>
     <xacro:include filename="$(find val_description)/model/robots/common/xacro/config/valkyrie_A_transmissions.xacro" />
 	<xacro:include filename="$(find val_description)/common/xacro/serial_numbers/valkyrie_A_serials.xacro"/>
     <xacro:include filename="$(find val_description)/common/xacro/api/valkyrie_A_api.xacro"/>
     <xacro:include filename="$(find val_description)/common/xacro/dev_ports/valkyrie_A_ports.xacro"/>
+    <xacro:include filename="$(find val_description)/model/robots/common/xacro/common_bodies.xacro" />
+    <!-- Pelvis include -->
+    <xacro:include filename="$(find val_description)/model/robots/common/xacro/pelvis/pelvis_includes.xacro"/>
+    <!-- Leg include -->
+    <xacro:include filename="$(find val_description)/model/robots/common/xacro/leg/leg_includes.xacro"/>
+    <!-- Head include -->
+    <xacro:include filename="$(find val_description)/model/robots/common/xacro/head/head_includes.xacro"/>
+    <!-- Arm include -->
+    <xacro:include filename="$(find val_description)/model/robots/common/xacro/arm/arm_includes.xacro"/>
+    <!-- Waist include -->
+    <xacro:include filename="$(find val_description)/model/robots/common/xacro/waist/waist_includes.xacro"/>
     <xacro:include filename="$(find val_description)/model/robots/common/xacro/valkyrie_base_hw.xacro"/>
 </robot>

File: model/robots/valkyrie_A_arm_mass_sims.xacro (robot description, xacro)
@@ -1,7 +1,20 @@
 <robot xmlns:xacro="http://ros.org/wiki/xacro" name="valkyrie">
+	<xacro:property name="mesh_root" value="package://val_description/model/meshes"/>
+    <xacro:include filename="$(find val_description)/model/robots/common/xacro/generic_models.xacro" />
+    <xacro:include filename="$(find val_description)/common/xacro/nodes/valkyrie_nodes.xacro"/>
     <xacro:include filename="$(find val_description)/model/robots/common/xacro/config/valkyrie_A_transmissions.xacro" />
     <xacro:include filename="$(find val_description)/common/xacro/serial_numbers/valkyrie_A_serials.xacro"/>
     <xacro:include filename="$(find val_description)/common/xacro/api/valkyrie_A_api.xacro"/>
     <xacro:include filename="$(find val_description)/common/xacro/dev_ports/valkyrie_A_ports.xacro"/>
+    <!-- Pelvis include -->
+    <xacro:include filename="$(find val_description)/model/robots/common/xacro/pelvis/pelvis_includes.xacro"/>
+    <!-- Leg include -->
+    <xacro:include filename="$(find val_description)/model/robots/common/xacro/leg/leg_includes.xacro"/>
+    <!-- Head include -->
+    <xacro:include filename="$(find val_description)/model/robots/common/xacro/head/head_includes.xacro"/>
+    <!-- Arm include -->
+    <xacro:include filename="$(find val_description)/model/robots/common/xacro/arm/arm_includes.xacro"/>
+    <!-- Waist include -->
+    <xacro:include filename="$(find val_description)/model/robots/common/xacro/waist/waist_includes.xacro"/>
     <xacro:include filename="$(find val_description)/model/robots/common/xacro/valkyrie_arm_mass_sims_base_hw.xacro"/>
 </robot>

File: model/robots/valkyrie_B.xacro (robot description, xacro)
@@ -1,7 +1,21 @@
 <robot xmlns:xacro="http://ros.org/wiki/xacro" name="valkyrie">
+	<xacro:property name="mesh_root" value="package://val_description/model/meshes"/>
+	<xacro:include filename="$(find val_description)/model/robots/common/xacro/generic_models.xacro" />
+    <xacro:include filename="$(find val_description)/common/xacro/nodes/valkyrie_nodes.xacro"/>
     <xacro:include filename="$(find val_description)/model/robots/common/xacro/config/valkyrie_B_transmissions.xacro" />
 	<xacro:include filename="$(find val_description)/common/xacro/serial_numbers/valkyrie_B_serials.xacro"/>
     <xacro:include filename="$(find val_description)/common/xacro/api/valkyrie_B_api.xacro"/>
     <xacro:include filename="$(find val_description)/common/xacro/dev_ports/valkyrie_B_ports.xacro"/>
+    <xacro:include filename="$(find val_description)/model/robots/common/xacro/common_bodies.xacro" />
+    <!-- Pelvis include -->
+    <xacro:include filename="$(find val_description)/model/robots/common/xacro/pelvis/pelvis_includes.xacro"/>
+    <!-- Leg include -->
+    <xacro:include filename="$(find val_description)/model/robots/common/xacro/leg/leg_includes.xacro"/>
+    <!-- Head include -->
+    <xacro:include filename="$(find val_description)/model/robots/common/xacro/head/head_includes.xacro"/>
+    <!-- Arm include -->
+    <xacro:include filename="$(find val_description)/model/robots/common/xacro/arm/arm_includes.xacro"/>
+    <!-- Waist include -->
+    <xacro:include filename="$(find val_description)/model/robots/common/xacro/waist/waist_includes.xacro"/>
     <xacro:include filename="$(find val_description)/model/robots/common/xacro/valkyrie_base_hw.xacro"/>
 </robot>

File: model/robots/valkyrie_B_arm_mass_sims.xacro (robot description, xacro)
@@ -1,7 +1,20 @@
 <robot xmlns:xacro="http://ros.org/wiki/xacro" name="valkyrie">
+	<xacro:property name="mesh_root" value="package://val_description/model/meshes"/>
+    <xacro:include filename="$(find val_description)/model/robots/common/xacro/generic_models.xacro" />
+    <xacro:include filename="$(find val_description)/common/xacro/nodes/valkyrie_nodes.xacro"/>
     <xacro:include filename="$(find val_description)/model/robots/common/xacro/config/valkyrie_B_transmissions.xacro"/>
     <xacro:include filename="$(find val_description)/common/xacro/serial_numbers/valkyrie_B_serials.xacro"/>
     <xacro:include filename="$(find val_description)/common/xacro/api/valkyrie_B_api.xacro"/>
     <xacro:include filename="$(find val_description)/common/xacro/dev_ports/valkyrie_B_ports.xacro"/>
+    <!-- Pelvis include -->
+    <xacro:include filename="$(find val_description)/model/robots/common/xacro/pelvis/pelvis_includes.xacro"/>
+    <!-- Leg include -->
+    <xacro:include filename="$(find val_description)/model/robots/common/xacro/leg/leg_includes.xacro"/>
+    <!-- Head include -->
+    <xacro:include filename="$(find val_description)/model/robots/common/xacro/head/head_includes.xacro"/>
+    <!-- Arm include -->
+    <xacro:include filename="$(find val_description)/model/robots/common/xacro/arm/arm_includes.xacro"/>
+    <!-- Waist include -->
+    <xacro:include filename="$(find val_description)/model/robots/common/xacro/waist/waist_includes.xacro"/>
     <xacro:include filename="$(find val_description)/model/robots/common/xacro/valkyrie_arm_mass_sims_base_hw.xacro"/>
 </robot>

File: model/robots/valkyrie_C.xacro (robot description, xacro)
@@ -1,7 +1,21 @@
 <robot xmlns:xacro="http://ros.org/wiki/xacro" name="valkyrie">
+	<xacro:property name="mesh_root" value="package://val_description/model/meshes"/>
+	<xacro:include filename="$(find val_description)/model/robots/common/xacro/generic_models.xacro" />
+    <xacro:include filename="$(find val_description)/common/xacro/nodes/valkyrie_nodes.xacro"/>
     <xacro:include filename="$(find val_description)/model/robots/common/xacro/config/valkyrie_C_transmissions.xacro" />
     <xacro:include filename="$(find val_description)/common/xacro/serial_numbers/valkyrie_C_serials.xacro"/>
     <xacro:include filename="$(find val_description)/common/xacro/api/valkyrie_C_api.xacro"/>
     <xacro:include filename="$(find val_description)/common/xacro/dev_ports/valkyrie_C_ports.xacro"/>
+    <xacro:include filename="$(find val_description)/model/robots/common/xacro/common_bodies.xacro" />
+    <!-- Pelvis include -->
+    <xacro:include filename="$(find val_description)/model/robots/common/xacro/pelvis/pelvis_includes.xacro"/>
+    <!-- Leg include -->
+    <xacro:include filename="$(find val_description)/model/robots/common/xacro/leg/leg_includes.xacro"/>
+    <!-- Head include -->
+    <xacro:include filename="$(find val_description)/model/robots/common/xacro/head/head_includes.xacro"/>
+    <!-- Arm include -->
+    <xacro:include filename="$(find val_description)/model/robots/common/xacro/arm/arm_includes.xacro"/>
+    <!-- Waist include -->
+    <xacro:include filename="$(find val_description)/model/robots/common/xacro/waist/waist_includes.xacro"/>
     <xacro:include filename="$(find val_description)/model/robots/common/xacro/valkyrie_base_hw.xacro"/>
 </robot>

File: model/robots/valkyrie_C_arm_mass_sims.xacro (robot description, xacro)
@@ -1,7 +1,20 @@
 <robot xmlns:xacro="http://ros.org/wiki/xacro" name="valkyrie">
+	<xacro:property name="mesh_root" value="package://val_description/model/meshes"/>
+    <xacro:include filename="$(find val_description)/model/robots/common/xacro/generic_models.xacro" />
+    <xacro:include filename="$(find val_description)/common/xacro/nodes/valkyrie_nodes.xacro"/>
     <xacro:include filename="$(find val_description)/model/robots/common/xacro/config/valkyrie_C_transmissions.xacro" />
     <xacro:include filename="$(find val_description)/common/xacro/serial_numbers/valkyrie_C_serials.xacro"/>
     <xacro:include filename="$(find val_description)/common/xacro/api/valkyrie_C_api.xacro"/>
     <xacro:include filename="$(find val_description)/common/xacro/dev_ports/valkyrie_C_ports.xacro"/>
+    <!-- Pelvis include -->
+    <xacro:include filename="$(find val_description)/model/robots/common/xacro/pelvis/pelvis_includes.xacro"/>
+    <!-- Leg include -->
+    <xacro:include filename="$(find val_description)/model/robots/common/xacro/leg/leg_includes.xacro"/>
+    <!-- Head include -->
+    <xacro:include filename="$(find val_description)/model/robots/common/xacro/head/head_includes.xacro"/>
+    <!-- Arm include -->
+    <xacro:include filename="$(find val_description)/model/robots/common/xacro/arm/arm_includes.xacro"/>
+    <!-- Waist include -->
+    <xacro:include filename="$(find val_description)/model/robots/common/xacro/waist/waist_includes.xacro"/>
     <xacro:include filename="$(find val_description)/model/robots/common/xacro/valkyrie_arm_mass_sims_base_hw.xacro"/>
 </robot>

File: model/robots/valkyrie_D.xacro (robot description, xacro)
@@ -1,7 +1,21 @@
 <robot xmlns:xacro="http://ros.org/wiki/xacro" name="valkyrie">
+	<xacro:property name="mesh_root" value="package://val_description/model/meshes"/>
+	<xacro:include filename="$(find val_description)/model/robots/common/xacro/generic_models.xacro" />
+    <xacro:include filename="$(find val_description)/common/xacro/nodes/valkyrie_nodes.xacro"/>
     <xacro:include filename="$(find val_description)/model/robots/common/xacro/config/valkyrie_D_transmissions.xacro" />
     <xacro:include filename="$(find val_description)/common/xacro/serial_numbers/valkyrie_D_serials.xacro"/>
     <xacro:include filename="$(find val_description)/common/xacro/api/valkyrie_D_api.xacro"/>
     <xacro:include filename="$(find val_description)/common/xacro/dev_ports/valkyrie_D_ports.xacro"/>
+    <xacro:include filename="$(find val_description)/model/robots/common/xacro/common_bodies.xacro" />
+    <!-- Pelvis include -->
+    <xacro:include filename="$(find val_description)/model/robots/common/xacro/pelvis/pelvis_includes.xacro"/>
+    <!-- Leg include -->
+    <xacro:include filename="$(find val_description)/model/robots/common/xacro/leg/leg_includes.xacro"/>
+    <!-- Head include -->
+    <xacro:include filename="$(find val_description)/model/robots/common/xacro/head/head_includes.xacro"/>
+    <!-- Arm include -->
+    <xacro:include filename="$(find val_description)/model/robots/common/xacro/arm/arm_includes.xacro"/>
+    <!-- Waist include -->
+    <xacro:include filename="$(find val_description)/model/robots/common/xacro/waist/waist_includes.xacro"/>
     <xacro:include filename="$(find val_description)/model/robots/common/xacro/valkyrie_base_hw.xacro"/>
 </robot>
