Commit message: Reworking a bunch of our xacro files to make it easier to have robots with different kinematics and/or mass properties.

File: model/robots/valkyrie_D_arm_mass_sims.xacro (robot description, xacro)
@@ -1,7 +1,20 @@
 <robot xmlns:xacro="http://ros.org/wiki/xacro" name="valkyrie">
+	<xacro:property name="mesh_root" value="package://val_description/model/meshes"/>
+    <xacro:include filename="$(find val_description)/model/robots/common/xacro/generic_models.xacro" />
+    <xacro:include filename="$(find val_description)/common/xacro/nodes/valkyrie_nodes.xacro"/>
     <xacro:include filename="$(find val_description)/model/robots/common/xacro/config/valkyrie_D_transmissions.xacro" />
     <xacro:include filename="$(find val_description)/common/xacro/serial_numbers/valkyrie_D_serials.xacro"/>
     <xacro:include filename="$(find val_description)/common/xacro/api/valkyrie_D_api.xacro"/>
     <xacro:include filename="$(find val_description)/common/xacro/dev_ports/valkyrie_D_ports.xacro"/>
+    <!-- Pelvis include -->
+    <xacro:include filename="$(find val_description)/model/robots/common/xacro/pelvis/pelvis_includes.xacro"/>
+    <!-- Leg include -->
+    <xacro:include filename="$(find val_description)/model/robots/common/xacro/leg/leg_includes.xacro"/>
+    <!-- Head include -->
+    <xacro:include filename="$(find val_description)/model/robots/common/xacro/head/head_includes.xacro"/>
+    <!-- Arm include -->
+    <xacro:include filename="$(find val_description)/model/robots/common/xacro/arm/arm_includes.xacro"/>
+    <!-- Waist include -->
+    <xacro:include filename="$(find val_description)/model/robots/common/xacro/waist/waist_includes.xacro"/>
     <xacro:include filename="$(find val_description)/model/robots/common/xacro/valkyrie_arm_mass_sims_base_hw.xacro"/>
 </robot>
