Commit message: Have new angled j1 kinematics working. Need to fix pretty much all the leg meshes and the torso j1 mesh.

File: model/robots/common/xacro/arm/arm.xacro (robot description, xacro)
@@ -7,6 +7,6 @@
                     ixx="${ShoulderPitchLinkInertia_IXX}" ixy="${ShoulderPitchLinkInertia_IXY}" ixz="${ShoulderPitchLinkInertia_IXZ}"
                     iyy="${ShoulderPitchLinkInertia_IYY}" iyz="${ShoulderPitchLinkInertia_IYZ}" izz="${ShoulderPitchLinkInertia_IZZ}"
-                    visual_mesh="${mesh_root}/arms/aj1_${prefix}.dae"
-                    collision_mesh="${mesh_root}/arms/aj1_${prefix}.dae" />
+                    visual_mesh="${arm_mesh_dir}/aj1_${prefix}.dae"
+                    collision_mesh="${arm_mesh_dir}/aj1_${prefix}.dae" />
     <xacro:standard_link name="${ShoulderRollLinkName}"
                     mass="${ShoulderRollLinkMass}"
@@ -15,6 +15,6 @@
                     iyy="${ShoulderRollLinkInertia_IYY}" iyz="${ShoulderRollLinkInertia_IYZ}" izz="${ShoulderRollLinkInertia_IZZ}"
                     origin_rpy="0 0 0"
-                    visual_mesh="${mesh_root}/arms/aj2_${prefix}.dae"
-                    collision_mesh="${mesh_root}/arms/aj2_${prefix}.dae" />
+                    visual_mesh="${arm_mesh_dir}/aj2_${prefix}.dae"
+                    collision_mesh="${arm_mesh_dir}/aj2_${prefix}.dae" />
     <xacro:standard_link name="${ShoulderYawLinkName}"
                     mass="${ShoulderYawLinkMass}"
@@ -23,6 +23,6 @@
                     iyy="${ShoulderYawLinkInertia_IYY}" iyz="${ShoulderYawLinkInertia_IYZ}" izz="${ShoulderYawLinkInertia_IZZ}"
                     origin_rpy="0 0 0"
-                    visual_mesh="${mesh_root}/arms/aj3_${prefix}.dae"
-                    collision_mesh="${mesh_root}/arms/aj3_${prefix}.dae" />
+                    visual_mesh="${arm_mesh_dir}/aj3_${prefix}.dae"
+                    collision_mesh="${arm_mesh_dir}/aj3_${prefix}.dae" />
     <xacro:standard_link name="${ElbowPitchLinkName}"
                     mass="${ElbowPitchLinkMass}"
@@ -31,6 +31,6 @@
                     iyy="${ElbowPitchLinkInertia_IYY}" iyz="${ElbowPitchLinkInertia_IYZ}" izz="${ElbowPitchLinkInertia_IZZ}"
                     origin_rpy="0 0 0"
-                    visual_mesh="${mesh_root}/arms/aj4_${prefix}.dae"
-                    collision_mesh="${mesh_root}/arms/aj4_${prefix}.dae" />
+                    visual_mesh="${arm_mesh_dir}/aj4_${prefix}.dae"
+                    collision_mesh="${arm_mesh_dir}/aj4_${prefix}.dae" />
     <xacro:revolute_joint_ex jointName="${ShoulderPitchJointName}"
                           parent="${upper_arm_root_link}" child="${ShoulderPitchLinkName}"
@@ -87,6 +87,6 @@
                     iyy="${ForearmYawLinkInertia_IYY}" iyz="${ForearmYawLinkInertia_IYZ}" izz="${ForearmYawLinkInertia_IZZ}"
                     origin_rpy="0 0 0"
-                    visual_mesh="${mesh_root}/arms/aj5_${prefix}.dae"
-                    collision_mesh="${mesh_root}/arms/aj5_${prefix}.dae" />
+                    visual_mesh="${arm_mesh_dir}/aj5_${prefix}.dae"
+                    collision_mesh="${arm_mesh_dir}/aj5_${prefix}.dae" />
     <xacro:standard_link name="${WristRollLinkName}"
                     mass="${WristRollLinkMass}"
@@ -95,6 +95,6 @@
                     iyy="${WristRollLinkInertia_IYY}" iyz="${WristRollLinkInertia_IYZ}" izz="${WristRollLinkInertia_IZZ}"
                     origin_rpy="0 0 0"
-                    visual_mesh="${mesh_root}/arms/aj6_${prefix}.dae"
-                    collision_mesh="${mesh_root}/arms/aj6_${prefix}.dae" />
+                    visual_mesh="${arm_mesh_dir}/aj6_${prefix}.dae"
+                    collision_mesh="${arm_mesh_dir}/aj6_${prefix}.dae" />
     <xacro:standard_link name="${WristPitchLinkName}"
                     mass="${PalmMass}"
@@ -103,6 +103,6 @@
                     iyy="${PalmInertia_IYY}" iyz="${PalmInertia_IYZ}" izz="${PalmInertia_IZZ}"
                     origin_rpy="0 0 0"
-                    visual_mesh="${mesh_root}/arms/palm_${prefix}.dae"
-                    collision_mesh="${mesh_root}/arms/palm_${prefix}.dae"/>
+                    visual_mesh="${arm_mesh_dir}/palm_${prefix}.dae"
+                    collision_mesh="${arm_mesh_dir}/palm_${prefix}.dae"/>
     <xacro:revolute_joint_ex jointName="${ForearmYawJointName}"
                           parent="${lower_arm_root_link}" child="${ForearmLinkName}"
@@ -156,6 +156,6 @@
                     ixx="${ShoulderPitchLinkInertia_IXX}" ixy="${ShoulderPitchLinkInertia_IXY}" ixz="${ShoulderPitchLinkInertia_IXZ}"
                     iyy="${ShoulderPitchLinkInertia_IYY}" iyz="${ShoulderPitchLinkInertia_IYZ}" izz="${ShoulderPitchLinkInertia_IZZ}"
-                    visual_mesh="${mesh_root}/arms/aj1_${prefix}.dae"
-                    collision_mesh="${mesh_root}/arms/aj1_${prefix}.dae" />
+                    visual_mesh="${arm_mesh_dir}/aj1_${prefix}.dae"
+                    collision_mesh="${arm_mesh_dir}/aj1_${prefix}.dae" />
     <xacro:standard_link name="${ShoulderRollLinkName}"
                     mass="${ShoulderRollLinkMass}"
@@ -164,6 +164,6 @@
                     iyy="${ShoulderRollLinkInertia_IYY}" iyz="${ShoulderRollLinkInertia_IYZ}" izz="${ShoulderRollLinkInertia_IZZ}"
                     origin_rpy="0 0 0"
-                    visual_mesh="${mesh_root}/arms/aj2_${prefix}.dae"
-                    collision_mesh="${mesh_root}/arms/aj2_${prefix}.dae" />
+                    visual_mesh="${arm_mesh_dir}/aj2_${prefix}.dae"
+                    collision_mesh="${arm_mesh_dir}/aj2_${prefix}.dae" />
     <xacro:standard_link name="${ShoulderYawLinkName}"
                     mass="${ShoulderYawLinkMass}"
@@ -172,6 +172,6 @@
                     iyy="${ShoulderYawLinkInertia_IYY}" iyz="${ShoulderYawLinkInertia_IYZ}" izz="${ShoulderYawLinkInertia_IZZ}"
                     origin_rpy="0 0 0"
-                    visual_mesh="${mesh_root}/arms/aj3_${prefix}.dae"
-                    collision_mesh="${mesh_root}/arms/aj3_${prefix}.dae" />
+                    visual_mesh="${arm_mesh_dir}/aj3_${prefix}.dae"
+                    collision_mesh="${arm_mesh_dir}/aj3_${prefix}.dae" />
     <xacro:standard_link name="${ElbowPitchLinkName}"
                     mass="${ForearmMassSimLinkMass}"
@@ -180,6 +180,6 @@
                     iyy="${ForearmMassSimInertia_IYY}" iyz="${ForearmMassSimInertia_IYZ}" izz="${ForearmMassSimInertia_IZZ}"
                     origin_rpy="0 0 0"
-                    visual_mesh="${mesh_root}/arms/${prefix}_elbow_mass_sim.dae"
-                    collision_mesh="${mesh_root}/arms/${prefix}_elbow_mass_sim.dae" />
+                    visual_mesh="${arm_mesh_dir}/${prefix}_elbow_mass_sim.dae"
+                    collision_mesh="${arm_mesh_dir}/${prefix}_elbow_mass_sim.dae" />
     <xacro:revolute_joint_ex jointName="${ShoulderPitchJointName}"
                           parent="${arm_root_link}" child="${ShoulderPitchLinkName}"

File: model/robots/common/xacro/head/head.xacro (robot description, xacro)
@@ -9,6 +9,6 @@
                         ixx="${LowerNeckPitchLinkInertia_IXX}" ixy="${LowerNeckPitchLinkInertia_IXY}" ixz="${LowerNeckPitchLinkInertia_IXZ}"
                         iyy="${LowerNeckPitchLinkInertia_IYY}" iyz="${LowerNeckPitchLinkInertia_IYZ}" izz="${LowerNeckPitchLinkInertia_IZZ}"
-                        visual_mesh="${mesh_root}/head/neckj1.dae"
-                        collision_mesh="${mesh_root}/head/neckj1.dae"/>
+                        visual_mesh="${head_mesh_dir}/neckj1.dae"
+                        collision_mesh="${head_mesh_dir}/neckj1.dae"/>
     <xacro:standard_link name="${NeckYawLinkName}"
                         mass="${NeckYawLinkMass}"
@@ -17,6 +17,6 @@
                         ixx="${NeckYawLinkInertia_IXX}" ixy="${NeckYawLinkInertia_IXY}" ixz="${NeckYawLinkInertia_IXZ}"
                         iyy="${NeckYawLinkInertia_IYY}" iyz="${NeckYawLinkInertia_IYZ}" izz="${NeckYawLinkInertia_IZZ}"
-                        visual_mesh="${mesh_root}/head/neckj2.dae"
-                        collision_mesh="${mesh_root}/head/neckj2.dae" />
+                        visual_mesh="${head_mesh_dir}/neckj2.dae"
+                        collision_mesh="${head_mesh_dir}/neckj2.dae" />
     <xacro:standard_link name="${UpperNeckPitchLinkName}"
                        mass="${UpperNeckPitchLinkMass}"
@@ -25,6 +25,6 @@
                        iyy="${UpperNeckPitchLinkInertia_IYY}" iyz="${UpperNeckPitchLinkInertia_IYZ}" izz="${UpperNeckPitchLinkInertia_IZZ}"
                        origin_rpy="0 0 0"
-                       visual_mesh="${mesh_root}/head/head_multisense_no_visor.dae"
-                       collision_mesh="${mesh_root}/head/head_multisense_no_visor.dae"/>
+                       visual_mesh="${head_mesh_dir}/head_multisense_no_visor.dae"
+                       collision_mesh="${head_mesh_dir}/head_multisense_no_visor.dae"/>
     <xacro:revolute_joint_ex jointName="${LowerNeckPitchJointName}"
                           parent="${LowerNeckPitchParentLinkName}" child="${LowerNeckPitchLinkName}"

File: model/robots/common/xacro/index_finger/index_finger.xacro (robot description, xacro)
@@ -15,6 +15,6 @@
                     iyy="${IndexFingerPitch1LinkInertia_IYY}" iyz="${IndexFingerPitch1LinkInertia_IYZ}" izz="${IndexFingerPitch1LinkInertia_IZZ}"
                     origin_rpy="0 0 0"
-                    visual_mesh="${mesh_root}/fingers/indexj1_${prefix}.dae"
-                    collision_mesh="${mesh_root}/fingers/indexj1_${prefix}.dae"/>
+                    visual_mesh="${fingers_mesh_dir}/indexj1_${prefix}.dae"
+                    collision_mesh="${fingers_mesh_dir}/indexj1_${prefix}.dae"/>
     <xacro:standard_link name="${IndexFingerPitch2LinkName}"
                     mass="${IndexFingerPitch2LinkMass}"
@@ -23,6 +23,6 @@
                     iyy="${IndexFingerPitch2LinkInertia_IYY}" iyz="${IndexFingerPitch2LinkInertia_IYZ}" izz="${IndexFingerPitch2LinkInertia_IZZ}"
                     origin_rpy="0 0 0"
-                    visual_mesh="${mesh_root}/fingers/indexj2_${prefix}.dae"
-                    collision_mesh="${mesh_root}/fingers/indexj2_${prefix}.dae"/>
+                    visual_mesh="${fingers_mesh_dir}/indexj2_${prefix}.dae"
+                    collision_mesh="${fingers_mesh_dir}/indexj2_${prefix}.dae"/>
     <xacro:standard_link name="${IndexFingerPitch3LinkName}"
                     mass="${IndexFingerPitch3LinkMass}"
@@ -31,6 +31,6 @@
                     iyy="${IndexFingerPitch3LinkInertia_IYY}" iyz="${IndexFingerPitch3LinkInertia_IYZ}" izz="${IndexFingerPitch3LinkInertia_IZZ}"
                     origin_rpy="0 0 0"
-                    visual_mesh="${mesh_root}/fingers/indexj3_${prefix}.dae"
-                    collision_mesh="${mesh_root}/fingers/indexj3_${prefix}.dae"/>
+                    visual_mesh="${fingers_mesh_dir}/indexj3_${prefix}.dae"
+                    collision_mesh="${fingers_mesh_dir}/indexj3_${prefix}.dae"/>
     <xacro:revolute_joint_ex jointName="${IndexFingerPitch1JointName}"
                           parent="${IndexFingerPitch1ParentLinkName}" child="${IndexFingerPitch1LinkName}"

File: model/robots/common/xacro/leg/leg.xacro (robot description, xacro)
@@ -7,6 +7,6 @@
                     ixx="${HipYawLinkInertia_IXX}" ixy="${HipYawLinkInertia_IXY}" ixz="${HipYawLinkInertia_IXZ}"
                     iyy="${HipYawLinkInertia_IYY}" iyz="${HipYawLinkInertia_IYZ}" izz="${HipYawLinkInertia_IZZ}"
-                    visual_mesh="${mesh_root}/legs/lj1_${prefix}.dae"
-                    collision_mesh="${mesh_root}/legs/lj1_${prefix}.dae"/>
+                    visual_mesh="${leg_mesh_dir}/lj1_${prefix}.dae"
+                    collision_mesh="${leg_mesh_dir}/lj1_${prefix}.dae"/>
     <xacro:standard_link name="${HipRollLinkName}"
                     mass="${HipRollLinkMass}"
@@ -15,6 +15,6 @@
                     iyy="${HipRollLinkInertia_IYY}" iyz="${HipRollLinkInertia_IYZ}" izz="${HipRollLinkInertia_IZZ}"
                     origin_rpy="0 0 0"
-                    visual_mesh="${mesh_root}/legs/lj2_${prefix}.dae"
-                    collision_mesh="${mesh_root}/legs/lj2_${prefix}.dae"/>
+                    visual_mesh="${leg_mesh_dir}/lj2_${prefix}.dae"
+                    collision_mesh="${leg_mesh_dir}/lj2_${prefix}.dae"/>
     <xacro:standard_link name="${HipPitchLinkName}"
                     mass="${HipPitchLinkMass}"
@@ -23,6 +23,6 @@
                     iyy="${HipPitchLinkInertia_IYY}" iyz="${HipPitchLinkInertia_IYZ}" izz="${HipPitchLinkInertia_IZZ}"
                     origin_rpy="0 0 0"
-                    visual_mesh="${mesh_root}/legs/lj3_${prefix}.dae"
-                    collision_mesh="${mesh_root}/legs/lj3_${prefix}.dae"/>
+                    visual_mesh="${leg_mesh_dir}/lj3_${prefix}.dae"
+                    collision_mesh="${leg_mesh_dir}/lj3_${prefix}.dae"/>
     <xacro:standard_link name="${KneePitchLinkName}"
                     mass="${KneePitchLinkMass}"
@@ -31,6 +31,6 @@
                     iyy="${KneePitchLinkInertia_IYY}" iyz="${KneePitchLinkInertia_IYZ}" izz="${KneePitchLinkInertia_IZZ}"
                     origin_rpy="0 0 0"
-                    visual_mesh="${mesh_root}/legs/lj4_${prefix}.dae"
-                    collision_mesh="${mesh_root}/legs/lj4_${prefix}.dae"/>
+                    visual_mesh="${leg_mesh_dir}/lj4_${prefix}.dae"
+                    collision_mesh="${leg_mesh_dir}/lj4_${prefix}.dae"/>
     <xacro:standard_link name="${AnklePitchLinkName}"
                     mass="${AnklePitchLinkMass}"
@@ -39,6 +39,6 @@
                     iyy="${AnklePitchLinkInertia_IYY}" iyz="${AnklePitchLinkInertia_IYZ}" izz="${AnklePitchLinkInertia_IZZ}"
                     origin_rpy="0 0 0"
-                    visual_mesh="${mesh_root}/legs/lj5.dae"
-                    collision_mesh="${mesh_root}/legs/lj5.dae"/>
+                    visual_mesh="${leg_mesh_dir}/lj5.dae"
+                    collision_mesh="${leg_mesh_dir}/lj5.dae"/>
     <xacro:link_box_collision_mesh_visual name="${AnkleRollLinkName}"
                     mass="${FootMass}"
@@ -47,5 +47,5 @@
                     iyy="${FootInertia_IYY}" iyz="${FootInertia_IYZ}" izz="${FootInertia_IZZ}"
                     inertial_rpy="0 0 0"
-                    visual_mesh="${mesh_root}/legs/foot.dae"
+                    visual_mesh="${leg_mesh_dir}/foot.dae"
                     width="0.27"
                     height="0.16"

File: model/robots/common/xacro/middle_finger/middle_finger.xacro (robot description, xacro)
@@ -15,6 +15,6 @@
                     iyy="${MiddleFingerPitch1LinkInertia_IYY}" iyz="${MiddleFingerPitch1LinkInertia_IYZ}" izz="${MiddleFingerPitch1LinkInertia_IZZ}"
                     origin_rpy="0 0 0"
-                    visual_mesh="${mesh_root}/fingers/middlej1_${prefix}.dae"
-                    collision_mesh="${mesh_root}/fingers/middlej1_${prefix}.dae"/>
+                    visual_mesh="${fingers_mesh_dir}/middlej1_${prefix}.dae"
+                    collision_mesh="${fingers_mesh_dir}/middlej1_${prefix}.dae"/>
     <xacro:standard_link name="${MiddleFingerPitch2LinkName}"
                     mass="${MiddleFingerPitch2LinkMass}"
@@ -23,6 +23,6 @@
                     iyy="${MiddleFingerPitch2LinkInertia_IYY}" iyz="${MiddleFingerPitch2LinkInertia_IYZ}" izz="${MiddleFingerPitch2LinkInertia_IZZ}"
                     origin_rpy="0 0 0"
-                    visual_mesh="${mesh_root}/fingers/middlej2_${prefix}.dae"
-                    collision_mesh="${mesh_root}/fingers/middlej2_${prefix}.dae"/>
+                    visual_mesh="${fingers_mesh_dir}/middlej2_${prefix}.dae"
+                    collision_mesh="${fingers_mesh_dir}/middlej2_${prefix}.dae"/>
     <xacro:standard_link name="${MiddleFingerPitch3LinkName}"
                     mass="${MiddleFingerPitch3LinkMass}"
@@ -31,6 +31,6 @@
                     iyy="${MiddleFingerPitch3LinkInertia_IYY}" iyz="${MiddleFingerPitch3LinkInertia_IYZ}" izz="${MiddleFingerPitch3LinkInertia_IZZ}"
                     origin_rpy="0 0 0"
-                    visual_mesh="${mesh_root}/fingers/middlej3_${prefix}.dae"
-                    collision_mesh="${mesh_root}/fingers/middlej3_${prefix}.dae"/>
+                    visual_mesh="${fingers_mesh_dir}/middlej3_${prefix}.dae"
+                    collision_mesh="${fingers_mesh_dir}/middlej3_${prefix}.dae"/>
     <xacro:revolute_joint_ex jointName="${MiddleFingerPitch1JointName}"
                           parent="${MiddleFingerPitch1ParentLinkName}" child="${MiddleFingerPitch1LinkName}"

File: model/robots/common/xacro/pelvis/pelvis.xacro (robot description, xacro)
@@ -8,6 +8,6 @@
                         iyy="${PelvisLinkInertia_IYY}" iyz="${PelvisLinkInertia_IYZ}" izz="${PelvisLinkInertia_IZZ}"
                         origin_rpy="0 0 0"
-                        visual_mesh="${mesh_root}/pelvis/pelvis.dae"
-                        collision_mesh="${mesh_root}/pelvis/pelvis.dae"/>
+                        visual_mesh="${pelvis_mesh_dir}/pelvis.dae"
+                        collision_mesh="${pelvis_mesh_dir}/pelvis.dae"/>
     </xacro:macro>
     <xacro:macro name="v1_pelvis_sensors">

File: model/robots/common/xacro/pinky_finger/pinky_finger.xacro (robot description, xacro)
@@ -15,6 +15,6 @@
                     iyy="${PinkyPitch1LinkInertia_IYY}" iyz="${PinkyPitch1LinkInertia_IYZ}" izz="${PinkyPitch1LinkInertia_IZZ}"
                     origin_rpy="0 0 0"
-                    visual_mesh="${mesh_root}/fingers/pinkyj1_${prefix}.dae"
-                    collision_mesh="${mesh_root}/fingers/pinkyj1_${prefix}.dae"/>
+                    visual_mesh="${fingers_mesh_dir}/pinkyj1_${prefix}.dae"
+                    collision_mesh="${fingers_mesh_dir}/pinkyj1_${prefix}.dae"/>
     <xacro:standard_link name="${PinkyPitch2LinkName}"
                     mass="${PinkyPitch2LinkMass}"
@@ -23,6 +23,6 @@
                     iyy="${PinkyPitch2LinkInertia_IYY}" iyz="${PinkyPitch2LinkInertia_IYZ}" izz="${PinkyPitch2LinkInertia_IZZ}"
                     origin_rpy="0 0 0"
-                    visual_mesh="${mesh_root}/fingers/pinkyj2_${prefix}.dae"
-                    collision_mesh="${mesh_root}/fingers/pinkyj2_${prefix}.dae"/>
+                    visual_mesh="${fingers_mesh_dir}/pinkyj2_${prefix}.dae"
+                    collision_mesh="${fingers_mesh_dir}/pinkyj2_${prefix}.dae"/>
     <xacro:standard_link name="${PinkyPitch3LinkName}"
                     mass="${PinkyPitch3LinkMass}"
@@ -31,6 +31,6 @@
                     iyy="${PinkyPitch3LinkInertia_IYY}" iyz="${PinkyPitch3LinkInertia_IYZ}" izz="${PinkyPitch3LinkInertia_IZZ}"
                     origin_rpy="0 0 0"
-                    visual_mesh="${mesh_root}/fingers/pinkyj3_${prefix}.dae"
-                    collision_mesh="${mesh_root}/fingers/pinkyj3_${prefix}.dae"/>
+                    visual_mesh="${fingers_mesh_dir}/pinkyj3_${prefix}.dae"
+                    collision_mesh="${fingers_mesh_dir}/pinkyj3_${prefix}.dae"/>
     <xacro:revolute_joint_ex jointName="${PinkyPitch1JointName}"
                           parent="${PinkyPitch1ParentLinkName}" child="${PinkyPitch1LinkName}"

File: model/robots/common/xacro/thumb/thumb.xacro (robot description, xacro)
@@ -16,6 +16,6 @@
                     iyy="${ThumbRollLinkInertia_IYY}" iyz="${ThumbRollLinkInertia_IYZ}" izz="${ThumbRollLinkInertia_IZZ}"
                     origin_rpy="0 0 0"
-                    visual_mesh="${mesh_root}/fingers/thumbj1_${prefix}.dae"
-                    collision_mesh="${mesh_root}/fingers/thumbj1_${prefix}.dae"/>
+                    visual_mesh="${fingers_mesh_dir}/thumbj1_${prefix}.dae"
+                    collision_mesh="${fingers_mesh_dir}/thumbj1_${prefix}.dae"/>
     <xacro:standard_link name="${ThumbPitch1LinkName}"
                     mass="${ThumbPitch1LinkMass}"
@@ -24,6 +24,6 @@
                     iyy="${ThumbPitch1LinkInertia_IYY}" iyz="${ThumbPitch1LinkInertia_IYZ}" izz="${ThumbPitch1LinkInertia_IZZ}"
                     origin_rpy="0 0 0"
-                    visual_mesh="${mesh_root}/fingers/thumbj2_${prefix}.dae"
-                    collision_mesh="${mesh_root}/fingers/thumbj2_${prefix}.dae"/>
+                    visual_mesh="${fingers_mesh_dir}/thumbj2_${prefix}.dae"
+                    collision_mesh="${fingers_mesh_dir}/thumbj2_${prefix}.dae"/>
     <xacro:standard_link name="${ThumbPitch2LinkName}"
                     mass="${ThumbPitch2LinkMass}"
@@ -32,6 +32,6 @@
                     iyy="${ThumbPitch2LinkInertia_IYY}" iyz="${ThumbPitch2LinkInertia_IYZ}" izz="${ThumbPitch2LinkInertia_IZZ}"
                     origin_rpy="0 0 0"
-                    visual_mesh="${mesh_root}/fingers/thumbj3_${prefix}.dae"
-                    collision_mesh="${mesh_root}/fingers/thumbj3_${prefix}.dae"/>
+                    visual_mesh="${fingers_mesh_dir}/thumbj3_${prefix}.dae"
+                    collision_mesh="${fingers_mesh_dir}/thumbj3_${prefix}.dae"/>
     <xacro:standard_link name="${ThumbPitch3LinkName}"
                     mass="${ThumbPitch3LinkMass}"
@@ -40,6 +40,6 @@
                     iyy="${ThumbPitch3LinkInertia_IYY}" iyz="${ThumbPitch3LinkInertia_IYZ}" izz="${ThumbPitch3LinkInertia_IZZ}"
                     origin_rpy="0 0 0"
-                    visual_mesh="${mesh_root}/fingers/thumbj4_${prefix}.dae"
-                    collision_mesh="${mesh_root}/fingers/thumbj4_${prefix}.dae"/>
+                    visual_mesh="${fingers_mesh_dir}/thumbj4_${prefix}.dae"
+                    collision_mesh="${fingers_mesh_dir}/thumbj4_${prefix}.dae"/>
     <xacro:revolute_joint_ex jointName="${ThumbRollJointName}"
                           parent="${ThumbRollParentLinkName}" child="${ThumbRollLinkName}"
