Commit message: Have new angled j1 kinematics working. Need to fix pretty much all the leg meshes and the torso j1 mesh.

File: model/robots/common/xacro/waist/waist.xacro (robot description, xacro)
@@ -36,6 +36,6 @@
                     ixx="${TorsoYawLinkInertia_IXX}" ixy="${TorsoYawLinkInertia_IXY}" ixz="${TorsoYawLinkInertia_IXZ}"
                     iyy="${TorsoYawLinkInertia_IYY}" iyz="${TorsoYawLinkInertia_IYZ}" izz="${TorsoYawLinkInertia_IZZ}"
-                    visual_mesh="${mesh_root}/torso/torsoyaw.dae"
-                    collision_mesh="${mesh_root}/torso/torsoyaw.dae" />
+                    visual_mesh="${waist_mesh_dir}/torsoyaw.dae"
+                    collision_mesh="${waist_mesh_dir}/torsoyaw.dae" />
     <xacro:standard_link name="${TorsoPitchLinkName}"
                     mass="${TorsoPitchLinkMass}"
@@ -44,6 +44,6 @@
                     ixx="${TorsoPitchLinkInertia_IXX}" ixy="${TorsoPitchLinkInertia_IXY}" ixz="${TorsoPitchLinkInertia_IXZ}"
                     iyy="${TorsoPitchLinkInertia_IYY}" iyz="${TorsoPitchLinkInertia_IYZ}" izz="${TorsoPitchLinkInertia_IZZ}"
-                    visual_mesh="${mesh_root}/torso/torsopitch.dae"
-                    collision_mesh="${mesh_root}/torso/torsopitch.dae" />
+                    visual_mesh="${waist_mesh_dir}/torsopitch.dae"
+                    collision_mesh="${waist_mesh_dir}/torsopitch.dae" />
     <xacro:standard_link name="${TorsoRollLinkName}"
                     mass="${TorsoRollLinkMass}"
@@ -52,6 +52,6 @@
                     origin_rpy="0 0 0"
                     origin_xyz="${TorsoRollLinkComPosition}"
-                    visual_mesh="${mesh_root}/torso/torso.dae"
-                    collision_mesh="${mesh_root}/torso/torso.dae" />
+                    visual_mesh="${waist_mesh_dir}/torso.dae"
+                    collision_mesh="${waist_mesh_dir}/torso.dae" />
     <xacro:make_waist_common waist_root_link="${waist_root_link}"/>
   </xacro:macro>

File: model/robots/forearm_left.xacro (robot description, xacro)
@@ -1,4 +1,5 @@
 <robot xmlns:xacro="http://ros.org/wiki/xacro" name="valkyrie">
-    <xacro:property name="mesh_root" value="package://val_description/model/meshes"/>
+    <xacro:property name="arm_mesh_dir" value="package://val_description/model/meshes/arms"/>
+    <xacro:property name="fingers_mesh_dir" value="package://val_description/model/meshes/fingers"/>
     <xacro:include filename="$(find val_description)/common/xacro/nodes/valkyrie_nodes.xacro"/>
     <xacro:include filename="$(find val_description)/model/robots/common/xacro/generic_models.xacro" />

File: model/robots/forearm_right.xacro (robot description, xacro)
@@ -1,4 +1,5 @@
 <robot xmlns:xacro="http://ros.org/wiki/xacro" name="valkyrie">
-    <xacro:property name="mesh_root" value="package://val_description/model/meshes"/>
+    <xacro:property name="arm_mesh_dir" value="package://val_description/model/meshes/arms"/>
+    <xacro:property name="fingers_mesh_dir" value="package://val_description/model/meshes/fingers"/>
     <xacro:include filename="$(find val_description)/common/xacro/nodes/valkyrie_nodes.xacro"/>
     <xacro:include filename="$(find val_description)/model/robots/common/xacro/generic_models.xacro" />

File: model/robots/valkyrie_A.xacro (robot description, xacro)
@@ -1,4 +1,9 @@
 <robot xmlns:xacro="http://ros.org/wiki/xacro" name="valkyrie">
-	<xacro:property name="mesh_root" value="package://val_description/model/meshes"/>
+	<xacro:property name="leg_mesh_dir" value="package://val_description/model/meshes/legs"/>
+    <xacro:property name="arm_mesh_dir" value="package://val_description/model/meshes/arms"/>
+    <xacro:property name="waist_mesh_dir" value="package://val_description/model/meshes/torso"/>
+    <xacro:property name="head_mesh_dir" value="package://val_description/model/meshes/head"/>
+    <xacro:property name="pelvis_mesh_dir" value="package://val_description/model/meshes/pelvis"/>
+    <xacro:property name="fingers_mesh_dir" value="package://val_description/model/meshes/fingers"/>
 	<xacro:include filename="$(find val_description)/model/robots/common/xacro/generic_models.xacro" />
     <xacro:include filename="$(find val_description)/common/xacro/nodes/valkyrie_nodes.xacro"/>

File: model/robots/valkyrie_A_arm_mass_sims.xacro (robot description, xacro)
@@ -1,4 +1,9 @@
 <robot xmlns:xacro="http://ros.org/wiki/xacro" name="valkyrie">
-	<xacro:property name="mesh_root" value="package://val_description/model/meshes"/>
+	<xacro:property name="leg_mesh_dir" value="package://val_description/model/meshes/legs"/>
+    <xacro:property name="arm_mesh_dir" value="package://val_description/model/meshes/arms"/>
+    <xacro:property name="waist_mesh_dir" value="package://val_description/model/meshes/torso"/>
+    <xacro:property name="head_mesh_dir" value="package://val_description/model/meshes/head"/>
+    <xacro:property name="pelvis_mesh_dir" value="package://val_description/model/meshes/pelvis"/>
+    <xacro:property name="fingers_mesh_dir" value="package://val_description/model/meshes/fingers"/>
     <xacro:include filename="$(find val_description)/model/robots/common/xacro/generic_models.xacro" />
     <xacro:include filename="$(find val_description)/common/xacro/nodes/valkyrie_nodes.xacro"/>

File: model/robots/valkyrie_B.xacro (robot description, xacro)
@@ -1,4 +1,9 @@
 <robot xmlns:xacro="http://ros.org/wiki/xacro" name="valkyrie">
-	<xacro:property name="mesh_root" value="package://val_description/model/meshes"/>
+	<xacro:property name="leg_mesh_dir" value="package://val_description/model/meshes/legs"/>
+    <xacro:property name="arm_mesh_dir" value="package://val_description/model/meshes/arms"/>
+    <xacro:property name="waist_mesh_dir" value="package://val_description/model/meshes/torso"/>
+    <xacro:property name="head_mesh_dir" value="package://val_description/model/meshes/head"/>
+    <xacro:property name="pelvis_mesh_dir" value="package://val_description/model/meshes/pelvis"/>
+    <xacro:property name="fingers_mesh_dir" value="package://val_description/model/meshes/fingers"/>
 	<xacro:include filename="$(find val_description)/model/robots/common/xacro/generic_models.xacro" />
     <xacro:include filename="$(find val_description)/common/xacro/nodes/valkyrie_nodes.xacro"/>

File: model/robots/valkyrie_B_arm_mass_sims.xacro (robot description, xacro)
@@ -1,4 +1,9 @@
 <robot xmlns:xacro="http://ros.org/wiki/xacro" name="valkyrie">
-	<xacro:property name="mesh_root" value="package://val_description/model/meshes"/>
+	<xacro:property name="leg_mesh_dir" value="package://val_description/model/meshes/legs"/>
+    <xacro:property name="arm_mesh_dir" value="package://val_description/model/meshes/arms"/>
+    <xacro:property name="waist_mesh_dir" value="package://val_description/model/meshes/torso"/>
+    <xacro:property name="head_mesh_dir" value="package://val_description/model/meshes/head"/>
+    <xacro:property name="pelvis_mesh_dir" value="package://val_description/model/meshes/pelvis"/>
+    <xacro:property name="fingers_mesh_dir" value="package://val_description/model/meshes/fingers"/>
     <xacro:include filename="$(find val_description)/model/robots/common/xacro/generic_models.xacro" />
     <xacro:include filename="$(find val_description)/common/xacro/nodes/valkyrie_nodes.xacro"/>

File: model/robots/valkyrie_C.xacro (robot description, xacro)
@@ -1,4 +1,9 @@
 <robot xmlns:xacro="http://ros.org/wiki/xacro" name="valkyrie">
-	<xacro:property name="mesh_root" value="package://val_description/model/meshes"/>
+	<xacro:property name="leg_mesh_dir" value="package://val_description/model/meshes/legs"/>
+    <xacro:property name="arm_mesh_dir" value="package://val_description/model/meshes/arms"/>
+    <xacro:property name="waist_mesh_dir" value="package://val_description/model/meshes/torso"/>
+    <xacro:property name="head_mesh_dir" value="package://val_description/model/meshes/head"/>
+    <xacro:property name="pelvis_mesh_dir" value="package://val_description/model/meshes/pelvis"/>
+    <xacro:property name="fingers_mesh_dir" value="package://val_description/model/meshes/fingers"/>
 	<xacro:include filename="$(find val_description)/model/robots/common/xacro/generic_models.xacro" />
     <xacro:include filename="$(find val_description)/common/xacro/nodes/valkyrie_nodes.xacro"/>

File: model/robots/valkyrie_C_arm_mass_sims.xacro (robot description, xacro)
@@ -1,4 +1,9 @@
 <robot xmlns:xacro="http://ros.org/wiki/xacro" name="valkyrie">
-	<xacro:property name="mesh_root" value="package://val_description/model/meshes"/>
+	<xacro:property name="leg_mesh_dir" value="package://val_description/model/meshes/legs"/>
+    <xacro:property name="arm_mesh_dir" value="package://val_description/model/meshes/arms"/>
+    <xacro:property name="waist_mesh_dir" value="package://val_description/model/meshes/torso"/>
+    <xacro:property name="head_mesh_dir" value="package://val_description/model/meshes/head"/>
+    <xacro:property name="pelvis_mesh_dir" value="package://val_description/model/meshes/pelvis"/>
+    <xacro:property name="fingers_mesh_dir" value="package://val_description/model/meshes/fingers"/>
     <xacro:include filename="$(find val_description)/model/robots/common/xacro/generic_models.xacro" />
     <xacro:include filename="$(find val_description)/common/xacro/nodes/valkyrie_nodes.xacro"/>

File: model/robots/valkyrie_D.xacro (robot description, xacro)
@@ -1,4 +1,9 @@
 <robot xmlns:xacro="http://ros.org/wiki/xacro" name="valkyrie">
-	<xacro:property name="mesh_root" value="package://val_description/model/meshes"/>
+	<xacro:property name="leg_mesh_dir" value="package://val_description/model/meshes/legs"/>
+    <xacro:property name="arm_mesh_dir" value="package://val_description/model/meshes/arms"/>
+    <xacro:property name="waist_mesh_dir" value="package://val_description/model/meshes/torso"/>
+    <xacro:property name="head_mesh_dir" value="package://val_description/model/meshes/head"/>
+    <xacro:property name="pelvis_mesh_dir" value="package://val_description/model/meshes/pelvis"/>
+    <xacro:property name="fingers_mesh_dir" value="package://val_description/model/meshes/fingers"/>
 	<xacro:include filename="$(find val_description)/model/robots/common/xacro/generic_models.xacro" />
     <xacro:include filename="$(find val_description)/common/xacro/nodes/valkyrie_nodes.xacro"/>

File: model/robots/valkyrie_D_arm_mass_sims.xacro (robot description, xacro)
@@ -1,4 +1,9 @@
 <robot xmlns:xacro="http://ros.org/wiki/xacro" name="valkyrie">
-	<xacro:property name="mesh_root" value="package://val_description/model/meshes"/>
+	<xacro:property name="leg_mesh_dir" value="package://val_description/model/meshes/legs"/>
+    <xacro:property name="arm_mesh_dir" value="package://val_description/model/meshes/arms"/>
+    <xacro:property name="waist_mesh_dir" value="package://val_description/model/meshes/torso"/>
+    <xacro:property name="head_mesh_dir" value="package://val_description/model/meshes/head"/>
+    <xacro:property name="pelvis_mesh_dir" value="package://val_description/model/meshes/pelvis"/>
+    <xacro:property name="fingers_mesh_dir" value="package://val_description/model/meshes/fingers"/>
     <xacro:include filename="$(find val_description)/model/robots/common/xacro/generic_models.xacro" />
     <xacro:include filename="$(find val_description)/common/xacro/nodes/valkyrie_nodes.xacro"/>

File: model/robots/valkyrie_sim.xacro (robot description, xacro)
@@ -6,5 +6,10 @@
     </gazebo>
     <schedule_topic_creator_file package="val_gazebo" relative_file_path="/configuration/valkyrie_sim_shm_topics.yaml"/>
-    <xacro:property name="mesh_root" value="package://val_description/model/meshes"/>
+    <xacro:property name="leg_mesh_dir" value="package://val_description/model/meshes/legs"/>
+    <xacro:property name="arm_mesh_dir" value="package://val_description/model/meshes/arms"/>
+    <xacro:property name="waist_mesh_dir" value="package://val_description/model/meshes/torso"/>
+    <xacro:property name="head_mesh_dir" value="package://val_description/model/meshes/head"/>
+    <xacro:property name="pelvis_mesh_dir" value="package://val_description/model/meshes/pelvis"/>
+    <xacro:property name="fingers_mesh_dir" value="package://val_description/model/meshes/fingers"/>
     <xacro:include filename="$(find val_description)/model/robots/common/xacro/generic_models.xacro" />
     <xacro:include filename="$(find val_description)/common/xacro/nodes/valkyrie_sim_nodes.xacro"/>

Commit message: updating gains for finger joints

File: model/robots/common/xacro/arm/arm.xacro (robot description, xacro)
@@ -105,4 +105,5 @@
                     visual_mesh="${arm_mesh_dir}/palm_${prefix}.dae"
                     collision_mesh="${arm_mesh_dir}/palm_${prefix}.dae"/>
+    <xacro:gazebo_hand_contact link_name="${WristPitchLinkName}" />
     <xacro:revolute_joint_ex jointName="${ForearmYawJointName}"
                           parent="${lower_arm_root_link}" child="${ForearmLinkName}"

File: model/robots/common/xacro/arm/arm_includes.xacro (robot description, xacro)
@@ -8,4 +8,5 @@
 	<xacro:include filename="$(find val_description)/common/xacro/actuator_names/valkyrie_actuator_names.xacro"/>
 	<xacro:include filename="$(find val_description)/model/robots/common/xacro/gains.xacro"/>
+	<xacro:include filename="$(find val_description)/model/robots/common/xacro/gazebo_hand_contact.xacro"/>
 	<xacro:include filename="$(find val_description)/model/robots/common/xacro/arm/arm.xacro"/>
 </robot>

File: model/robots/common/xacro/gains.xacro (robot description, xacro)
@@ -31,29 +31,29 @@
     <xacro:property name="ThumbPitch3Ki" value="0.0" />
     <xacro:property name="IndexFingerPitch1Kp" value="5.0" />
-    <xacro:property name="IndexFingerPitch1Kd" value="0.3" />
+    <xacro:property name="IndexFingerPitch1Kd" value="0.0" />
     <xacro:property name="IndexFingerPitch1Ki" value="0.0" />
     <xacro:property name="IndexFingerPitch2Kp" value="5.0" />
-    <xacro:property name="IndexFingerPitch2Kd" value="0.3" />
+    <xacro:property name="IndexFingerPitch2Kd" value="0.0" />
     <xacro:property name="IndexFingerPitch2Ki" value="0.0" />
     <xacro:property name="IndexFingerPitch3Kp" value="5.0" />
-    <xacro:property name="IndexFingerPitch3Kd" value="0.3" />
+    <xacro:property name="IndexFingerPitch3Kd" value="0.0" />
     <xacro:property name="IndexFingerPitch3Ki" value="0.0" />
     <xacro:property name="MiddleFingerPitch1Kp" value="5.0" />
-    <xacro:property name="MiddleFingerPitch1Kd" value="0.3" />
+    <xacro:property name="MiddleFingerPitch1Kd" value="0.0" />
     <xacro:property name="MiddleFingerPitch1Ki" value="0.0" />
     <xacro:property name="MiddleFingerPitch2Kp" value="5.0" />
-    <xacro:property name="MiddleFingerPitch2Kd" value="0.3" />
+    <xacro:property name="MiddleFingerPitch2Kd" value="0.0" />
     <xacro:property name="MiddleFingerPitch2Ki" value="0.0" />
     <xacro:property name="MiddleFingerPitch3Kp" value="5.0" />
-    <xacro:property name="MiddleFingerPitch3Kd" value="0.3" />
+    <xacro:property name="MiddleFingerPitch3Kd" value="0.0" />
     <xacro:property name="MiddleFingerPitch3Ki" value="0.0" />
     <xacro:property name="PinkyPitch1Kp" value="5.0" />
-    <xacro:property name="PinkyPitch1Kd" value="0.3" />
+    <xacro:property name="PinkyPitch1Kd" value="0.0" />
     <xacro:property name="PinkyPitch1Ki" value="0.0" />
     <xacro:property name="PinkyPitch2Kp" value="5.0" />
-    <xacro:property name="PinkyPitch2Kd" value="0.3" />
+    <xacro:property name="PinkyPitch2Kd" value="0.0" />
     <xacro:property name="PinkyPitch2Ki" value="0.0" />
     <xacro:property name="PinkyPitch3Kp" value="5.0" />
-    <xacro:property name="PinkyPitch3Kd" value="0.3" />
+    <xacro:property name="PinkyPitch3Kd" value="0.0" />
     <xacro:property name="PinkyPitch3Ki" value="0.0" />
 </robot>

File: model/robots/common/xacro/index_finger/index_finger.xacro (robot description, xacro)
@@ -8,4 +8,5 @@
   <xacro:include filename="$(find val_description)/model/robots/common/xacro/index_finger/mechanical_info.xacro"/>
   <xacro:include filename="$(find val_description)/model/robots/common/xacro/index_finger/mass_parameters.xacro"/>
+  <xacro:include filename="$(find val_description)/model/robots/common/xacro/gazebo_hand_contact.xacro"/>
   <xacro:macro name="make_index_finger" params="prefix reflect index_finger_root_link">
     <xacro:standard_link name="${IndexFingerPitch1LinkName}"
@@ -17,4 +18,5 @@
                     visual_mesh="${fingers_mesh_dir}/indexj1_${prefix}.dae"
                     collision_mesh="${fingers_mesh_dir}/indexj1_${prefix}.dae"/>
+    <xacro:gazebo_hand_contact link_name="${IndexFingerPitch1LinkName}" />
     <xacro:standard_link name="${IndexFingerPitch2LinkName}"
                     mass="${IndexFingerPitch2LinkMass}"
@@ -25,4 +27,5 @@
                     visual_mesh="${fingers_mesh_dir}/indexj2_${prefix}.dae"
                     collision_mesh="${fingers_mesh_dir}/indexj2_${prefix}.dae"/>
+    <xacro:gazebo_hand_contact link_name="${IndexFingerPitch2LinkName}" />
     <xacro:standard_link name="${IndexFingerPitch3LinkName}"
                     mass="${IndexFingerPitch3LinkMass}"
@@ -33,4 +36,5 @@
                     visual_mesh="${fingers_mesh_dir}/indexj3_${prefix}.dae"
                     collision_mesh="${fingers_mesh_dir}/indexj3_${prefix}.dae"/>
+    <xacro:gazebo_hand_contact link_name="${IndexFingerPitch3LinkName}" />
     <xacro:revolute_joint_ex jointName="${IndexFingerPitch1JointName}"
                           parent="${IndexFingerPitch1ParentLinkName}" child="${IndexFingerPitch1LinkName}"

File: model/robots/common/xacro/middle_finger/middle_finger.xacro (robot description, xacro)
@@ -8,4 +8,5 @@
   <xacro:include filename="$(find val_description)/model/robots/common/xacro/middle_finger/mechanical_info.xacro"/>
   <xacro:include filename="$(find val_description)/model/robots/common/xacro/middle_finger/mass_parameters.xacro"/>
+  <xacro:include filename="$(find val_description)/model/robots/common/xacro/gazebo_hand_contact.xacro"/>
   <xacro:macro name="make_middle_finger" params="prefix reflect middle_finger_root_link">
     <xacro:standard_link name="${MiddleFingerPitch1LinkName}"
@@ -17,4 +18,5 @@
                     visual_mesh="${fingers_mesh_dir}/middlej1_${prefix}.dae"
                     collision_mesh="${fingers_mesh_dir}/middlej1_${prefix}.dae"/>
+    <xacro:gazebo_hand_contact link_name="${MiddleFingerPitch1LinkName}" />
     <xacro:standard_link name="${MiddleFingerPitch2LinkName}"
                     mass="${MiddleFingerPitch2LinkMass}"
@@ -25,4 +27,5 @@
                     visual_mesh="${fingers_mesh_dir}/middlej2_${prefix}.dae"
                     collision_mesh="${fingers_mesh_dir}/middlej2_${prefix}.dae"/>
+    <xacro:gazebo_hand_contact link_name="${MiddleFingerPitch2LinkName}" />
     <xacro:standard_link name="${MiddleFingerPitch3LinkName}"
                     mass="${MiddleFingerPitch3LinkMass}"
@@ -33,4 +36,5 @@
                     visual_mesh="${fingers_mesh_dir}/middlej3_${prefix}.dae"
                     collision_mesh="${fingers_mesh_dir}/middlej3_${prefix}.dae"/>
+    <xacro:gazebo_hand_contact link_name="${MiddleFingerPitch3LinkName}" />
     <xacro:revolute_joint_ex jointName="${MiddleFingerPitch1JointName}"
                           parent="${MiddleFingerPitch1ParentLinkName}" child="${MiddleFingerPitch1LinkName}"

File: model/robots/common/xacro/pinky_finger/pinky_finger.xacro (robot description, xacro)
@@ -8,4 +8,5 @@
   <xacro:include filename="$(find val_description)/model/robots/common/xacro/pinky_finger/mechanical_info.xacro"/>
   <xacro:include filename="$(find val_description)/model/robots/common/xacro/pinky_finger/mass_parameters.xacro"/>
+  <xacro:include filename="$(find val_description)/model/robots/common/xacro/gazebo_hand_contact.xacro"/>
   <xacro:macro name="make_pinky_finger" params="prefix reflect pinky_finger_root_link">
     <xacro:standard_link name="${PinkyPitch1LinkName}"
@@ -17,4 +18,5 @@
                     visual_mesh="${fingers_mesh_dir}/pinkyj1_${prefix}.dae"
                     collision_mesh="${fingers_mesh_dir}/pinkyj1_${prefix}.dae"/>
+    <xacro:gazebo_hand_contact link_name="${PinkyPitch1LinkName}" />
     <xacro:standard_link name="${PinkyPitch2LinkName}"
                     mass="${PinkyPitch2LinkMass}"
@@ -25,4 +27,5 @@
                     visual_mesh="${fingers_mesh_dir}/pinkyj2_${prefix}.dae"
                     collision_mesh="${fingers_mesh_dir}/pinkyj2_${prefix}.dae"/>
+    <xacro:gazebo_hand_contact link_name="${PinkyPitch2LinkName}" />
     <xacro:standard_link name="${PinkyPitch3LinkName}"
                     mass="${PinkyPitch3LinkMass}"
@@ -33,4 +36,5 @@
                     visual_mesh="${fingers_mesh_dir}/pinkyj3_${prefix}.dae"
                     collision_mesh="${fingers_mesh_dir}/pinkyj3_${prefix}.dae"/>
+    <xacro:gazebo_hand_contact link_name="${PinkyPitch3LinkName}" />
     <xacro:revolute_joint_ex jointName="${PinkyPitch1JointName}"
                           parent="${PinkyPitch1ParentLinkName}" child="${PinkyPitch1LinkName}"

File: model/robots/common/xacro/thumb/thumb.xacro (robot description, xacro)
@@ -9,4 +9,5 @@
   <xacro:include filename="$(find val_description)/model/robots/common/xacro/thumb/mechanical_info.xacro"/>
   <xacro:include filename="$(find val_description)/model/robots/common/xacro/gains.xacro"/>
+  <xacro:include filename="$(find val_description)/model/robots/common/xacro/gazebo_hand_contact.xacro"/>
   <xacro:macro name="make_thumb" params="prefix reflect thumb_root_link">
     <xacro:standard_link name="${ThumbRollLinkName}"
@@ -18,4 +19,5 @@
                     visual_mesh="${fingers_mesh_dir}/thumbj1_${prefix}.dae"
                     collision_mesh="${fingers_mesh_dir}/thumbj1_${prefix}.dae"/>
+    <xacro:gazebo_hand_contact link_name="${ThumbRollLinkName}" />
     <xacro:standard_link name="${ThumbPitch1LinkName}"
                     mass="${ThumbPitch1LinkMass}"
@@ -26,4 +28,5 @@
                     visual_mesh="${fingers_mesh_dir}/thumbj2_${prefix}.dae"
                     collision_mesh="${fingers_mesh_dir}/thumbj2_${prefix}.dae"/>
+    <xacro:gazebo_hand_contact link_name="${ThumbPitch1LinkName}" />
     <xacro:standard_link name="${ThumbPitch2LinkName}"
                     mass="${ThumbPitch2LinkMass}"
@@ -34,4 +37,5 @@
                     visual_mesh="${fingers_mesh_dir}/thumbj3_${prefix}.dae"
                     collision_mesh="${fingers_mesh_dir}/thumbj3_${prefix}.dae"/>
+    <xacro:gazebo_hand_contact link_name="${ThumbPitch2LinkName}" />
     <xacro:standard_link name="${ThumbPitch3LinkName}"
                     mass="${ThumbPitch3LinkMass}"
@@ -42,4 +46,5 @@
                     visual_mesh="${fingers_mesh_dir}/thumbj4_${prefix}.dae"
                     collision_mesh="${fingers_mesh_dir}/thumbj4_${prefix}.dae"/>
+    <xacro:gazebo_hand_contact link_name="${ThumbPitch3LinkName}" />
     <xacro:revolute_joint_ex jointName="${ThumbRollJointName}"
                           parent="${ThumbRollParentLinkName}" child="${ThumbRollLinkName}"
