Commit message: creating forearm simulation for testing - Frank Mathiis

File: model/robots/common/xacro/arm/arm.xacro (robot description, xacro)
@@ -265,3 +265,8 @@
     <xacro:simple_transmission jointName="${prefix}${ElbowPitchJointName}" actuatorName="${prefix}${ElbowPitchActuatorName}" nodeName="/${prefix}${ElbowPitchNode}" actuatorApi="${SimApi}"/>
   </xacro:macro>
+  <xacro:macro name="forearm_transmissions_sim" params="prefix">
+    <xacro:simple_transmission jointName="${prefix}${ForearmYawActuatorName}" actuatorName="${prefix}${ForearmYawActuatorName}" nodeName="/${prefix}${ForearmYawNode}" actuatorApi="${SimApi}"/>
+    <xacro:simple_transmission jointName="${prefix}${WristRollJointName}" actuatorName="${prefix}${WristRollActuatorSimName}" nodeName="/${prefix}${WristRollActuatorNode}" actuatorApi="${SimApi}"/>
+    <xacro:simple_transmission jointName="${prefix}${WristPitchJointName}" actuatorName="${prefix}${WristPitchActuatorSimName}" nodeName="/${prefix}${WristPitchActuatorNode}" actuatorApi="${SimApi}"/>
+  </xacro:macro>
 </robot>

Commit message: Generate a reduced URDF model for simulation
Fingers and forearm joints are disabled (set as fixed).
The URDF can be use for full body optimization with less DOFs.

File: model/robots/common/xacro/arm/arm.xacro (robot description, xacro)
@@ -106,5 +106,5 @@
                     collision_mesh="${arm_mesh_dir}/palm_${prefix}.dae"/>
     <xacro:gazebo_hand_contact link_name="${prefix}Palm" />
-    <xacro:revolute_joint_ex jointName="${prefix}${ForearmYawJointName}"
+    <xacro:revolute_joint_ex_reducible jointName="${prefix}${ForearmYawJointName}"
                           parent="${lower_arm_root_link}" child="${prefix}ForearmLink"
                           origin_xyz="${ForearmYawFrameOrigin_X} ${ForearmYawFrameOrigin_Y} ${ForearmYawFrameOrigin_Z}"
@@ -114,6 +114,6 @@
         <limit effort="${ForearmYawTorqueLimit}" lower="${ForearmYawPositionLimit_Lower}" upper="${ForearmYawPositionLimit_Upper}" velocity="${ForearmYawVelocityLimit}"/>
         <controller_gains Kp="${ForearmYawKp}" Kd="${ForearmYawKd}" Ki="${ForearmYawKi}"/>
-    </xacro:revolute_joint_ex>
-    <xacro:revolute_joint_ex jointName="${prefix}${WristRollJointName}"
+    </xacro:revolute_joint_ex_reducible>
+    <xacro:revolute_joint_ex_reducible jointName="${prefix}${WristRollJointName}"
                           parent="${prefix}ForearmLink" child="${prefix}WristRollLink"
                           origin_xyz="${WristRollFrameOrigin_X} ${reflect * 0.2871} ${WristRollFrameOrigin_Z}"
@@ -128,6 +128,6 @@
         </xacro:if>
         <controller_gains Kp="${WristRollKp}" Kd="${WristRollKd}" Ki="${WristRollKi}"/>
-    </xacro:revolute_joint_ex>
-    <xacro:revolute_joint_ex jointName="${prefix}${WristPitchJointName}"
+    </xacro:revolute_joint_ex_reducible>
+    <xacro:revolute_joint_ex_reducible jointName="${prefix}${WristPitchJointName}"
                           parent="${prefix}WristRollLink" child="${prefix}Palm"
                           origin_xyz="${WristPitchFrameOrigin_X} ${WristPitchFrameOrigin_Y} ${WristPitchFrameOrigin_Z}"
@@ -142,5 +142,5 @@
         </xacro:if>
         <controller_gains Kp="${WristPitchKp}" Kd="${WristPitchKd}" Ki="${WristPitchKi}"/>
-    </xacro:revolute_joint_ex>
+    </xacro:revolute_joint_ex_reducible>
   </xacro:macro>
   <xacro:macro name="make_arm" params="prefix reflect arm_root_link">

File: model/robots/common/xacro/generic_models.xacro (robot description, xacro)
@@ -217,4 +217,56 @@
     </gazebo>
   </xacro:macro>
+  <xacro:property name="is_model_reduced" value="false"/>
+  <xacro:macro name="revolute_joint_ex_reducible" params="jointName parent child origin_xyz origin_rpy axis damping friction *limits *controller_gains">
+    <xacro:unless value="${is_model_reduced}">
+      <xacro:revolute_joint_ex
+        jointName="${jointName}"
+        parent="${parent}"
+        child="${child}"
+        origin_xyz="${origin_xyz}"
+        origin_rpy="${origin_rpy}"
+        axis="${axis}"
+        damping="${damping}"
+        friction="${friction}">
+        <xacro:insert_block name="limits" />
+        <xacro:insert_block name="controller_gains" />
+      </xacro:revolute_joint_ex>
+    </xacro:unless>
+    <xacro:if value="${is_model_reduced}">
+      <xacro:fixed_joint
+        jointName="${jointName}"
+        parent="${parent}"
+        child="${child}"
+        origin_xyz="${origin_xyz}"
+        origin_rpy="${origin_rpy}">
+      </xacro:fixed_joint>
+    </xacro:if>
+  </xacro:macro>
+  <xacro:macro name="revolute_joint_ex_mimic_reducible" params="jointName parent child origin_xyz origin_rpy axis damping friction *limits *controller_gains *mimic">
+    <xacro:unless value="${is_model_reduced}">
+      <xacro:revolute_joint_ex_mimic
+        jointName="${jointName}"
+        parent="${parent}"
+        child="${child}"
+        origin_xyz="${origin_xyz}"
+        origin_rpy="${origin_rpy}"
+        axis="${axis}"
+        damping="${damping}"
+        friction="${friction}">
+        <xacro:insert_block name="limits" />
+        <xacro:insert_block name="controller_gains" />
+        <xacro:insert_block name="mimic" />
+      </xacro:revolute_joint_ex_mimic>
+    </xacro:unless>
+    <xacro:if value="${is_model_reduced}">
+      <xacro:fixed_joint
+        jointName="${jointName}"
+        parent="${parent}"
+        child="${child}"
+        origin_xyz="${origin_xyz}"
+        origin_rpy="${origin_rpy}">
+      </xacro:fixed_joint>
+    </xacro:if>
+  </xacro:macro>
   <xacro:macro name="virtual_fixed_frame_offset" params="name parentLink origin_xyz origin_rpy">
     <xacro:virtual_link name="${name}_Frame"

File: model/robots/common/xacro/index_finger/index_finger.xacro (robot description, xacro)
@@ -36,5 +36,5 @@
                     collision_mesh="${fingers_mesh_dir}/indexj3_${prefix}.dae"/>
     <xacro:gazebo_hand_contact link_name="${prefix}IndexFingerPitch3Link" />
-    <xacro:revolute_joint_ex jointName="${prefix}${IndexFingerPitch1JointName}"
+    <xacro:revolute_joint_ex_reducible jointName="${prefix}${IndexFingerPitch1JointName}"
                           parent="${index_finger_root_link}" child="${prefix}IndexFingerPitch1Link"
                           origin_xyz="${IndexFingerPitch1FrameOrigin_X} ${reflect * 0.0976} ${IndexFingerPitch1FrameOrigin_Z}"
@@ -48,6 +48,6 @@
         </xacro:if>
         <controller_gains Kp="${IndexFingerPitch1Kp}" Kd="${IndexFingerPitch1Kd}" Ki="${IndexFingerPitch1Ki}"/>
-    </xacro:revolute_joint_ex>
-    <xacro:revolute_joint_ex_mimic jointName="${prefix}${IndexFingerPitch2JointName}"
+    </xacro:revolute_joint_ex_reducible>
+    <xacro:revolute_joint_ex_mimic_reducible jointName="${prefix}${IndexFingerPitch2JointName}"
                           parent="${prefix}IndexFingerPitch1Link" child="${prefix}IndexFingerPitch2Link"
                           origin_xyz="${IndexFingerPitch2FrameOrigin_X} ${reflect * 0.0381} ${IndexFingerPitch2FrameOrigin_Z}"
@@ -62,6 +62,6 @@
         <controller_gains Kp="${IndexFingerPitch1Kp}" Kd="${IndexFingerPitch1Kd}" Ki="${IndexFingerPitch1Ki}"/>
         <mimic joint="${prefix}${IndexFingerPitch1JointName}" multiplier="${Pulley2Ratio}" offset="0"/>
-    </xacro:revolute_joint_ex_mimic>
-    <xacro:revolute_joint_ex_mimic jointName="${prefix}${IndexFingerPitch3JointName}"
+    </xacro:revolute_joint_ex_mimic_reducible>
+    <xacro:revolute_joint_ex_mimic_reducible jointName="${prefix}${IndexFingerPitch3JointName}"
                           parent="${prefix}IndexFingerPitch2Link" child="${prefix}IndexFingerPitch3Link"
                           origin_xyz="${IndexFingerPitch3FrameOrigin_X} ${reflect * 0.0229} ${IndexFingerPitch3FrameOrigin_Z}"
@@ -76,5 +76,5 @@
         <controller_gains Kp="${IndexFingerPitch1Kp}" Kd="${IndexFingerPitch1Kd}" Ki="${IndexFingerPitch1Ki}"/>
         <mimic joint="${prefix}${IndexFingerPitch1JointName}" multiplier="${Pulley3Ratio}" offset="0"/>
-    </xacro:revolute_joint_ex_mimic>
+    </xacro:revolute_joint_ex_mimic_reducible>
   </xacro:macro>
   <xacro:macro name="index_finger_transmissions_hw" params="prefix reflect">

File: model/robots/common/xacro/middle_finger/middle_finger.xacro (robot description, xacro)
@@ -36,5 +36,5 @@
                     collision_mesh="${fingers_mesh_dir}/middlej3_${prefix}.dae"/>
     <xacro:gazebo_hand_contact link_name="${prefix}MiddleFingerPitch3Link" />
-    <xacro:revolute_joint_ex jointName="${prefix}${MiddleFingerPitch1JointName}"
+    <xacro:revolute_joint_ex_reducible jointName="${prefix}${MiddleFingerPitch1JointName}"
                           parent="${middle_finger_root_link}" child="${prefix}MiddleFingerPitch1Link"
                           origin_xyz="${MiddleFingerPitch1FrameOrigin_X} ${reflect * 0.097} ${MiddleFingerPitch1FrameOrigin_Z}"
@@ -48,6 +48,6 @@
         </xacro:if>
         <controller_gains Kp="${MiddleFingerPitch1Kp}" Kd="${MiddleFingerPitch1Kd}" Ki="${MiddleFingerPitch1Ki}"/>
-    </xacro:revolute_joint_ex>
-    <xacro:revolute_joint_ex_mimic jointName="${prefix}${MiddleFingerPitch2JointName}"
+    </xacro:revolute_joint_ex_reducible>
+    <xacro:revolute_joint_ex_mimic_reducible jointName="${prefix}${MiddleFingerPitch2JointName}"
                           parent="${prefix}MiddleFingerPitch1Link" child="${prefix}MiddleFingerPitch2Link"
                           origin_xyz="${MiddleFingerPitch2FrameOrigin_X} ${reflect * 0.0381} ${MiddleFingerPitch2FrameOrigin_Z}"
@@ -62,6 +62,6 @@
         <controller_gains Kp="${MiddleFingerPitch1Kp}" Kd="${MiddleFingerPitch1Kd}" Ki="${MiddleFingerPitch1Ki}"/>
         <mimic joint="${prefix}${MiddleFingerPitch1JointName}" multiplier="${Pulley2Ratio}" offset="0"/>
-    </xacro:revolute_joint_ex_mimic>
-    <xacro:revolute_joint_ex_mimic jointName="${prefix}${MiddleFingerPitch3JointName}"
+    </xacro:revolute_joint_ex_mimic_reducible>
+    <xacro:revolute_joint_ex_mimic_reducible jointName="${prefix}${MiddleFingerPitch3JointName}"
                           parent="${prefix}MiddleFingerPitch2Link" child="${prefix}MiddleFingerPitch3Link"
                           origin_xyz="${MiddleFingerPitch3FrameOrigin_X} ${reflect * 0.0229} ${MiddleFingerPitch3FrameOrigin_Z}"
@@ -76,5 +76,5 @@
         <controller_gains Kp="${MiddleFingerPitch1Kp}" Kd="${MiddleFingerPitch1Kd}" Ki="${MiddleFingerPitch1Ki}"/>
         <mimic joint="${prefix}${MiddleFingerPitch1JointName}" multiplier="${Pulley3Ratio}" offset="0"/>
-    </xacro:revolute_joint_ex_mimic>
+    </xacro:revolute_joint_ex_mimic_reducible>
   </xacro:macro>
   <xacro:macro name="middle_finger_transmissions_hw" params="prefix reflect">

File: model/robots/common/xacro/pinky_finger/pinky_finger.xacro (robot description, xacro)
@@ -36,5 +36,5 @@
                     collision_mesh="${fingers_mesh_dir}/pinkyj3_${prefix}.dae"/>
     <xacro:gazebo_hand_contact link_name="${prefix}PinkyPitch3Link" />
-    <xacro:revolute_joint_ex jointName="${prefix}${PinkyPitch1JointName}"
+    <xacro:revolute_joint_ex_reducible jointName="${prefix}${PinkyPitch1JointName}"
                           parent="${pinky_finger_root_link}" child="${prefix}PinkyPitch1Link"
                           origin_xyz="${PinkyPitch1FrameOrigin_X} ${reflect * 0.0838} ${PinkyPitch1FrameOrigin_Z}"
@@ -48,6 +48,6 @@
         </xacro:if>
         <controller_gains Kp="${PinkyPitch1Kp}" Kd="${PinkyPitch1Kd}" Ki="${PinkyPitch1Ki}"/>
-    </xacro:revolute_joint_ex>
-    <xacro:revolute_joint_ex_mimic jointName="${prefix}${PinkyPitch2JointName}"
+    </xacro:revolute_joint_ex_reducible>
+    <xacro:revolute_joint_ex_mimic_reducible jointName="${prefix}${PinkyPitch2JointName}"
                           parent="${prefix}PinkyPitch1Link" child="${prefix}PinkyPitch2Link"
                           origin_xyz="${PinkyPitch2FrameOrigin_X} ${reflect * 0.0381} ${PinkyPitch2FrameOrigin_Z}"
@@ -62,6 +62,6 @@
         <controller_gains Kp="${PinkyPitch1Kp}" Kd="${PinkyPitch1Kd}" Ki="${PinkyPitch1Ki}"/>
         <mimic joint="${prefix}${PinkyPitch1JointName}" multiplier="${Pulley2Ratio}" offset="0"/>
-    </xacro:revolute_joint_ex_mimic>
-    <xacro:revolute_joint_ex_mimic jointName="${prefix}${PinkyPitch3JointName}"
+    </xacro:revolute_joint_ex_mimic_reducible>
+    <xacro:revolute_joint_ex_mimic_reducible jointName="${prefix}${PinkyPitch3JointName}"
                           parent="${prefix}PinkyPitch2Link" child="${prefix}PinkyPitch3Link"
                           origin_xyz="${PinkyPitch3FrameOrigin_X} ${reflect * 0.0229} ${PinkyPitch3FrameOrigin_Z}"
@@ -76,5 +76,5 @@
         <controller_gains Kp="${PinkyPitch1Kp}" Kd="${PinkyPitch1Kd}" Ki="${PinkyPitch1Ki}"/>
         <mimic joint="${prefix}${PinkyPitch1JointName}" multiplier="${Pulley3Ratio}" offset="0"/>
-    </xacro:revolute_joint_ex_mimic>
+    </xacro:revolute_joint_ex_mimic_reducible>
   </xacro:macro>
   <xacro:macro name="pinky_finger_transmissions_hw" params="prefix reflect">

File: model/robots/common/xacro/thumb/thumb.xacro (robot description, xacro)
@@ -46,5 +46,5 @@
                     collision_mesh="${fingers_mesh_dir}/thumbj4_${prefix}.dae"/>
     <xacro:gazebo_hand_contact link_name="${prefix}ThumbPitch3Link" />
-    <xacro:revolute_joint_ex jointName="${prefix}${ThumbRollJointName}"
+    <xacro:revolute_joint_ex_reducible jointName="${prefix}${ThumbRollJointName}"
                           parent="${thumb_root_link}" child="${prefix}ThumbRollLink"
                           origin_xyz="${ThumbRollFrameOrigin_X} ${reflect * 0.0351} ${ThumbRollFrameOrigin_Z}"
@@ -53,6 +53,6 @@
         <limit effort="${ThumbRollTorqueLimit}" lower="${ThumbRollPositionLimit_Lower}" upper="${ThumbRollPositionLimit_Upper}" velocity="${ThumbRollVelocityLimit}"/>
          <controller_gains Kp="${ThumbRollKp}" Kd="${ThumbRollKd}" Ki="${ThumbRollKi}"/>
-    </xacro:revolute_joint_ex>
-    <xacro:revolute_joint_ex jointName="${prefix}${ThumbPitch1JointName}"
+    </xacro:revolute_joint_ex_reducible>
+    <xacro:revolute_joint_ex_reducible jointName="${prefix}${ThumbPitch1JointName}"
                           parent="${prefix}ThumbRollLink" child="${prefix}ThumbPitch1Link"
                           origin_xyz="${ThumbPitch1FrameOrigin_X} ${ThumbPitch1FrameOrigin_Y} ${ThumbPitch1FrameOrigin_Z}"
@@ -66,6 +66,6 @@
         </xacro:if>
         <controller_gains Kp="${ThumbPitch1Kp}" Kd="${ThumbPitch1Kd}" Ki="${ThumbPitch1Ki}"/>
-    </xacro:revolute_joint_ex>
-    <xacro:revolute_joint_ex_mimic jointName="${prefix}${ThumbPitch2JointName}"
+    </xacro:revolute_joint_ex_reducible>
+    <xacro:revolute_joint_ex_mimic_reducible jointName="${prefix}${ThumbPitch2JointName}"
                           parent="${prefix}ThumbPitch1Link" child="${prefix}ThumbPitch2Link"
                           origin_xyz="${ThumbPitch2FrameOrigin_X} ${reflect * 0.0066} ${ThumbPitch2FrameOrigin_Z}"
@@ -80,6 +80,6 @@
         <controller_gains Kp="${ThumbPitch2Kp}" Kd="${ThumbPitch2Kd}" Ki="${ThumbPitch2Ki}"/>
         <mimic joint="${prefix}${ThumbPitch1JointName}" multiplier="${Pulley2Ratio}" offset="0"/>
-    </xacro:revolute_joint_ex_mimic>
-    <xacro:revolute_joint_ex_mimic jointName="${prefix}${ThumbPitch3JointName}"
+    </xacro:revolute_joint_ex_mimic_reducible>
+    <xacro:revolute_joint_ex_mimic_reducible jointName="${prefix}${ThumbPitch3JointName}"
                           parent="${prefix}ThumbPitch2Link" child="${prefix}ThumbPitch3Link"
                           origin_xyz="${ThumbPitch3FrameOrigin_X} ${reflect * 0.0049} ${ThumbPitch3FrameOrigin_Z}"
@@ -94,5 +94,5 @@
         <controller_gains Kp="${ThumbPitch3Kp}" Kd="${ThumbPitch3Kd}" Ki="${ThumbPitch3Ki}"/>
         <mimic joint="${prefix}${ThumbPitch1JointName}" multiplier="${Pulley3Ratio}" offset="0"/>
-    </xacro:revolute_joint_ex_mimic>
+    </xacro:revolute_joint_ex_mimic_reducible>
   </xacro:macro>
   <xacro:macro name="thumb_transmissions_hw" params="prefix reflect">

File: model/robots/common/xacro/valkyrie_base_sim.xacro (robot description, xacro)
@@ -23,14 +23,22 @@
     <xacro:leg_transmissions_sim prefix="left"/>
     <xacro:leg_transmissions_sim prefix="right"/>
-    <xacro:arm_transmissions_sim prefix="left"/>
-    <xacro:arm_transmissions_sim prefix="right"/>
+    <xacro:if value="${is_model_reduced}">
+      <xacro:arm_transmissions_sim_no_hands prefix="left"/>
+      <xacro:arm_transmissions_sim_no_hands prefix="right"/>
+    </xacro:if>
+    <xacro:unless value="${is_model_reduced}">
+      <xacro:arm_transmissions_sim prefix="left"/>
+      <xacro:arm_transmissions_sim prefix="right"/>
+    </xacro:unless>
     <xacro:neck_transmissions_sim />
-    <xacro:thumb_transmissions_sim prefix="left"/>
-    <xacro:thumb_transmissions_sim prefix="right"/>
-    <xacro:index_finger_transmissions_sim prefix="left"/>
-    <xacro:index_finger_transmissions_sim prefix="right"/>
-    <xacro:middle_finger_transmissions_sim prefix="left"/>
-    <xacro:middle_finger_transmissions_sim prefix="right"/>
-    <xacro:pinky_transmissions_sim prefix="left"/>
-    <xacro:pinky_transmissions_sim prefix="right"/>
+    <xacro:unless value="${is_model_reduced}">
+      <xacro:thumb_transmissions_sim prefix="left"/>
+      <xacro:thumb_transmissions_sim prefix="right"/>
+      <xacro:index_finger_transmissions_sim prefix="left"/>
+      <xacro:index_finger_transmissions_sim prefix="right"/>
+      <xacro:middle_finger_transmissions_sim prefix="left"/>
+      <xacro:middle_finger_transmissions_sim prefix="right"/>
+      <xacro:pinky_transmissions_sim prefix="left"/>
+      <xacro:pinky_transmissions_sim prefix="right"/>
+    </xacro:unless>
 </robot>

Commit message: Add named virtual frame at the end of arm mass sim model

File: model/robots/common/xacro/arm/arm.xacro (robot description, xacro)
@@ -229,4 +229,8 @@
         <controller_gains Kp="0.0" Kd="0.0" Ki="0.0"/>
     </xacro:revolute_joint_ex>
+    <xacro:massless_virtual_fixed_frame_offset name="${prefix}ArmTip"
+                       parentLink="${prefix}ElbowPitchLink"
+                       origin_xyz="-0.024 ${reflect * 0.400} 0.0"
+                       origin_rpy="${reflect * 1.5708} 0.0 0.0"/>
   </xacro:macro>
   <xacro:macro name="arm_transmissions_hw" params="prefix reflect">

File: model/robots/valkyrie_sim_arm_mass_sims.xacro (robot description, xacro)
@@ -3,6 +3,8 @@
       <plugin filename="libval_gazebo.so" name="SharedMemorySimInterfacePlugin">
           <robotNamespace>/val</robotNamespace>
+          <updateRateHz>500.0</updateRateHz>
       </plugin>
     </gazebo>
+    <schedule_topic_creator_file package="val_gazebo" relative_file_path="/configuration/valkyrie_sim_shm_topics.yaml"/>
     <xacro:property name="leg_mesh_dir" value="model://val_description/model/meshes/legs"/>
     <xacro:property name="arm_mesh_dir" value="model://val_description/model/meshes/arms"/>
@@ -34,3 +36,5 @@
     <xacro:add_self_collide />
     <xacro:add_sim_harness harnessed_link="torso" />
+    <!-- Disable position control joints -->
+    <xacro:property name="is_model_reduced" value="true"/>
 </robot>

Commit message: Add simple sphere collision shape for arm sim contact

File: model/robots/common/xacro/arm/arm.xacro (robot description, xacro)
@@ -229,8 +229,20 @@
         <controller_gains Kp="0.0" Kd="0.0" Ki="0.0"/>
     </xacro:revolute_joint_ex>
-    <xacro:massless_virtual_fixed_frame_offset name="${prefix}ArmTip"
+    <xacro:massless_virtual_fixed_frame_offset_with_collision_sphere name="${prefix}ArmTip"
                        parentLink="${prefix}ElbowPitchLink"
                        origin_xyz="-0.024 ${reflect * 0.400} 0.0"
-                       origin_rpy="${reflect * 1.5708} 0.0 0.0"/>
+                       origin_rpy="${reflect * 1.5708} 0.0 0.0"
+                       radius="0.055"
+                       center_xyz="0.0 0.0 0.049"/>
+    <gazebo reference="${prefix}ArmTip_Frame">
+      <!-- kp and kd for rubber -->
+      <kp>1000000.0</kp>
+      <kd>100.0</kd>
+      <mu1>1.5</mu1>
+      <mu2>1.5</mu2>
+      <fdir1>1 0 0</fdir1>
+      <maxVel>1.0</maxVel>
+      <minDepth>0.00</minDepth>
+    </gazebo>
   </xacro:macro>
   <xacro:macro name="arm_transmissions_hw" params="prefix reflect">

File: model/robots/common/xacro/generic_models.xacro (robot description, xacro)
@@ -110,4 +110,22 @@
                  izz="${(massless_virtual_link_mass*massless_virtual_link_radius*massless_virtual_link_radius)/2}" />
       </inertial>
+    </link>
+  </xacro:macro>
+  <xacro:macro name="massless_virtual_link_with_collision_sphere" params="name origin_xyz origin_rpy radius center_xyz">
+    <link name="${name}">
+      <!-- Virtual Link -->
+      <inertial>
+        <mass value="${massless_virtual_link_mass}" />
+        <origin rpy="${origin_rpy}" xyz="${origin_xyz}"/>
+        <inertia ixx="${(massless_virtual_link_mass*(3*massless_virtual_link_radius*massless_virtual_link_radius + massless_virtual_link_height*massless_virtual_link_height))/12}" ixy="0.0" ixz="0.0"
+                 iyy="${(massless_virtual_link_mass*(3*massless_virtual_link_radius*massless_virtual_link_radius + massless_virtual_link_height*massless_virtual_link_height))/12}" iyz="0.0"
+                 izz="${(massless_virtual_link_mass*massless_virtual_link_radius*massless_virtual_link_radius)/2}" />
+      </inertial>
+      <collision>
+        <geometry>
+          <sphere radius="${radius}"/>
+        </geometry>
+        <origin rpy="0.0 0.0 0.0" xyz="${center_xyz}"/>
+      </collision>
     </link>
   </xacro:macro>
@@ -287,4 +305,15 @@
                        origin_xyz="${origin_xyz}"/>
   </xacro:macro>
+  <xacro:macro name="massless_virtual_fixed_frame_offset_with_collision_sphere" params="name parentLink origin_xyz origin_rpy radius center_xyz">
+    <xacro:massless_virtual_link_with_collision_sphere name="${name}_Frame"
+                    origin_rpy="0 0 0"
+                    origin_xyz="0 0 0"
+                    radius="${radius}"
+                    center_xyz="${center_xyz}"/>
+    <xacro:fixed_joint jointName="${name}_Offset"
+                       parent="${parentLink}" child="${name}_Frame"
+                       origin_rpy="${origin_rpy}"
+                       origin_xyz="${origin_xyz}"/>
+  </xacro:macro>
   <xacro:macro name="simple_transmission" params="jointName actuatorName nodeName actuatorApi">
     <transmission name="${jointName}Transmission">
