Commit message: [val_description] Changed wrist joint limits

File: model/robots/common/xacro/arm/joint_limits.xacro (robot description, xacro)
@@ -13,6 +13,6 @@
   <xacro:property name="ElbowPitchPositionLimit_Lower" value="-2.174" />
   <xacro:property name="ForearmYawPositionLimit_Lower" value="-2.019" />
-  <xacro:property name="WristRollPositionLimit_Lower" value="-0.35" />
-  <xacro:property name="WristPitchPositionLimit_Lower" value="-0.6" />
+  <xacro:property name="WristRollPositionLimit_Lower" value="-0.2" />
+  <xacro:property name="WristPitchPositionLimit_Lower" value="-0.5" />
   <xacro:property name="ShoulderPitchPositionLimit_Upper" value="2.0" />
   <xacro:property name="ShoulderRollPositionLimit_Upper" value="1.266" />
@@ -20,6 +20,6 @@
   <xacro:property name="ElbowPitchPositionLimit_Upper" value="0.12" />
   <xacro:property name="ForearmYawPositionLimit_Upper" value="3.14" />
-  <xacro:property name="WristRollPositionLimit_Upper" value="0.35" />
-  <xacro:property name="WristPitchPositionLimit_Upper" value="0.6" />
+  <xacro:property name="WristRollPositionLimit_Upper" value="0.3" />
+  <xacro:property name="WristPitchPositionLimit_Upper" value="0.5" />
   <xacro:property name="ShoulderPitchVelocityLimit" value="5.89" />
   <xacro:property name="ShoulderRollVelocityLimit" value="5.89" />
