Commit message: Set as fixed joint the hokuyo joint to simplify loading with RBDL

File: model/urdf/multisense_sl.urdf (robot description, URDF)
Before this commit: robot multisense_sl, 12 links, 11 joints
Joints:
- joint hokuyo_joint: type continuous -> fixed

File: model/urdf/multisense_sl_remote.urdf (robot description, URDF)
Before this commit: robot multisense_sl, 12 links, 11 joints
Joints:
- joint hokuyo_joint: type continuous -> fixed

Commit message: Remove head IMU

File: model/urdf/multisense_sl.urdf (robot description, URDF)
Before this commit: robot multisense_sl, 12 links, 11 joints
Links:
- removed link head_imu_link
Joints:
- removed joint head_imu_joint

File: model/urdf/multisense_sl_remote.urdf (robot description, URDF)
Before this commit: robot multisense_sl, 12 links, 11 joints
Links:
- removed link head_imu_link
Joints:
- removed joint head_imu_joint

Commit message: [val_description] Make multisense hokuyo joint continuous

File: model/urdf/multisense_sl.urdf (robot description, URDF)
Before this commit: robot multisense_sl, 11 links, 10 joints
Joints:
- joint hokuyo_joint: type fixed -> continuous

File: model/urdf/multisense_sl_remote.urdf (robot description, URDF)
Before this commit: robot multisense_sl, 11 links, 10 joints
Joints:
- joint hokuyo_joint: type fixed -> continuous
